File: eagle/scart/scartboard.brd (EAGLE design)
At the start: 100 x 80 mm, 12 parts, among them T1 BSS138, T3 BSS138, X1 SCART-F

Commit message: nice so far
Parts:
- added SV1: (no value), con-lstb:MA12-1
- added SV2: (no value), con-lstb:MA03-1
- moved JP1 16.6 mm to (66.0, 27.9), turned to 0 degrees
- moved R2 8.98 mm to (85.1, 19.1), turned to 90 degrees
- moved R4 8.89 mm to (85.1, 22.9), turned to 270 degrees
- moved T1 4.02 mm to (87.6, 17.8)
- moved T3 3.81 mm to (87.6, 24.1)
- moved R1 2.84 mm to (90.2, 17.8)
- moved R3 2.54 mm to (90.2, 24.1)
- moved JP3 1.80 mm to (78.7, 19.1)
Connections:
- removed net XVCC_5V: JP1.6
- removed net XVCC_B2: JP1.4
- net CASIN: now also JP1.1; no longer JP1.5
- net CASMOTOR: now also JP1.5; no longer JP1.1
- net GND: now also JP1.2, SV2.1
- net KBCOL0: now also SV1.1
- net KBCOL1: now also SV1.2
- net KBCOL2: now also SV1.3
- net KBCOL3: now also SV1.4
- net KBCOL4: now also SV1.5
- net KBCOL5: now also SV1.6
- net KBCOL6: now also SV1.7
- net KBCOL7: now also SV1.8
- net KBROW0: now also SV1.9
- net KBROW1: now also SV1.10
- net KBROW2: now also SV1.11
- net KBROW3: now also SV1.12
- net VCC_5V: now also JP1.4; no longer JP1.2
- net VCC_B2: now also JP1.6, SV2.2
Routing:
- net VCC_B2: track 88.8 -> 19.2 mm
- net GND: track 10.2 -> 27.0 mm
- net CASMOTOR: track 12.0 -> 3.59 mm
- net CASOUT: track 12.0 -> 3.59 mm
- net KBROW3: track 0.00 -> 5.61 mm
- net KBROW2: track 0.00 -> 5.61 mm
- net KBROW1: track 0.00 -> 5.61 mm
- net KBROW0: track 0.00 -> 5.61 mm
- net KBCOL4: track 0.00 -> 5.61 mm
- net KBCOL3: track 0.00 -> 5.61 mm
- net KBCOL2: track 0.00 -> 5.61 mm
- net KBCOL1: track 0.00 -> 5.61 mm
- net KBCOL0: track 0.00 -> 5.61 mm
- net KBCOL7: track 0.00 -> 5.61 mm
- net KBCOL6: track 0.00 -> 5.61 mm
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
Commit message: WIP
Parts:
- moved JP1 1.27 mm to (64.8, 27.9)
Routing:
- net CASOUT: track 3.59 -> 2.84 mm
- net CASMOTOR: track 3.59 -> 2.84 mm
- net CASIN: track 8.67 -> 8.15 mm
Changed lines of the file:
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@@
 <element name="R4" library="rcl" package="R0805" value="10K" x="85.09" y="22.86" rot="R270"/>
 <element name="JP3" library="pinhead" package="1X05" value="PS2" x="78.74" y="19.05" rot="R270"/>
-<element name="JP1" library="pinhead" package="2X03" value="" x="66.04" y="27.94"/>
+<element name="JP1" library="pinhead" package="2X03" value="" x="64.77" y="27.94"/>
 <element name="JP2" library="pinhead" package="1X03" value="" x="7.62" y="24.13"/>
 <element name="SV1" library="con-lstb" package="MA12-1" value="" x="45.72" y="29.21">
@@
 <contactref element="JP1" pad="6"/>
 <contactref element="SV2" pad="2"/>
-<wire x1="68.58" y1="29.21" x2="88.646" y2="23.1394" width="0" layer="19" extent="1-1"/>
-<wire x1="26.67" y1="29.21" x2="68.58" y2="29.21" width="0" layer="19" extent="1-1"/>
+<wire x1="67.31" y1="29.21" x2="88.646" y2="23.1394" width="0" layer="19" extent="1-1"/>
+<wire x1="26.67" y1="29.21" x2="67.31" y2="29.21" width="0" layer="19" extent="1-1"/>
 <wire x1="25.4" y1="24.13" x2="22.86" y2="24.13" width="0.4064" layer="1"/>
 <wire x1="25.4" y1="24.13" x2="26.67" y2="25.4" width="0.4064" layer="1"/>
@@
 <contactref element="JP1" pad="1"/>
 <wire x1="60.96" y1="19.05" x2="62.23" y2="20.32" width="0.4064" layer="1"/>
-<wire x1="62.23" y1="20.32" x2="62.23" y2="25.4" width="0.4064" layer="1"/>
-<wire x1="62.23" y1="25.4" x2="63.5" y2="26.67" width="0.4064" layer="1"/>
+<wire x1="62.23" y1="20.32" x2="62.23" y2="26.67" width="0.4064" layer="1"/>
 </signal>
 <signal name="PS2CLK">
@@
 <contactref element="SV9" pad="36"/>
 <contactref element="JP1" pad="5"/>
-<wire x1="66.04" y1="24.13" x2="68.58" y2="26.67" width="0.4064" layer="1"/>
+<wire x1="66.04" y1="24.13" x2="67.31" y2="26.67" width="0.4064" layer="1"/>
 </signal>
 <signal name="CASOUT">
 <contactref element="SV9" pad="34"/>
 <contactref element="JP1" pad="3"/>
-<wire x1="63.5" y1="24.13" x2="66.04" y2="26.67" width="0.4064" layer="1"/>
+<wire x1="63.5" y1="24.13" x2="64.77" y2="26.67" width="0.4064" layer="1"/>
 </signal>
 <signal name="KBROW3">
@@
 <wire x1="84.455" y1="13.97" x2="78.74" y2="13.97" width="0.4064" layer="1"/>
 <contactref element="JP1" pad="4"/>
-<wire x1="78.74" y1="13.97" x2="66.04" y2="29.21" width="0" layer="19" extent="1-1"/>
-<wire x1="7.62" y1="24.13" x2="66.04" y2="29.21" width="0" layer="19" extent="1-1"/>
+<wire x1="78.74" y1="13.97" x2="64.77" y2="29.21" width="0" layer="19" extent="1-1"/>
+<wire x1="7.62" y1="24.13" x2="64.77" y2="29.21" width="0" layer="19" extent="1-1"/>
 <wire x1="5.08" y1="24.13" x2="7.62" y2="24.13" width="0" layer="19" extent="1-1"/>
 </signal>
@@
 <contactref element="JP1" pad="2"/>
 <contactref element="SV2" pad="1"/>
-<wire x1="63.5" y1="29.21" x2="63.5" y2="71.12" width="0" layer="19" extent="16-16"/>
-<wire x1="63.5" y1="21.59" x2="63.5" y2="29.21" width="0" layer="19" extent="16-16"/>
+<wire x1="62.23" y1="29.21" x2="63.5" y2="71.12" width="0" layer="19" extent="16-16"/>
+<wire x1="63.5" y1="21.59" x2="62.23" y2="29.21" width="0" layer="19" extent="16-16"/>
 <wire x1="24.13" y1="29.21" x2="21.59" y2="26.67" width="0.4064" layer="1"/>
 <wire x1="21.59" y1="26.67" x2="21.59" y2="22.86" width="0.4064" layer="1"/>

Commit message: WIP
Parts:
- added Q2, Q3, Q4, Q5: BC548-TO92-E1-REV, bc548:TO92-E1-REV
- added R13, R16, R27, R32: 680, rcl:R0805
- added R14, R24, R29, R5, R6: 2200, rcl:R0805
- added R15, R26, R31: 270, rcl:R0805
- added R20, R28, R33: 4700, rcl:R0805
- added R25, R30, R7: 1000, rcl:R0805
- added SV4: (no value), con-lstb:MA03-2
- added T2, T4, T7, T8: (no value), transistor:TO92-CBE
- moved R1 27.9 mm to (64.8, 6.35), turned to 180 degrees
- moved R3 26.1 mm to (71.1, 6.35), turned to 180 degrees
- moved T1 24.5 mm to (64.8, 8.89), turned to 180 degrees
- moved T3 22.5 mm to (71.1, 8.89), turned to 180 degrees
- moved R2 20.5 mm to (66.0, 11.4), turned to 0 degrees
- moved R4 19.1 mm to (69.8, 11.4), turned to 180 degrees
- moved X1 15.3 mm to (41.9, 43.2)
- moved JP3 13.3 mm to (66.0, 15.2), turned to 180 degrees
- moved JP2 5.08 mm to (12.7, 24.1), turned to 180 degrees
- moved JP1 2.54 mm to (64.8, 30.5)
Connections:
- removed net N$99: SV9.25
- new net B_SPARE: SV4.5, SV9.25
- new net N$1: R13.2, R14.2, T2.E
- new net N$10: R26.2, R27.2, R28.2, T7.E
- new net N$11: R29.2, R30.2, T8.B
- new net N$12: R31.2, R32.2, R33.2, T8.E
- new net N$2: R6.2, R7.2, T4.B
- new net N$3: R5.2, T2.B
- new net N$6: R15.2, R16.2, R20.2, T4.E
- new net N$9: R24.2, R25.2, T7.B
- net B0: now also R30.1
- net B1: now also R29.1
- net BLUE: now also R31.1, R32.1, R33.1
- net B_DEBUG: now also SV4.3
- net B_NMI: now also SV4.1
- net COMP: now also R13.1, R14.1
- net CSYNC: now also R5.1
- net G0: now also R25.1
- net G1: now also R24.1
- net GND: now also JP1.6, SV4.2, SV4.4, SV4.6; no longer JP1.2
- net GREEN: now also R26.1, R27.1, R28.1
- net R0: now also R7.1
- net R1: now also R6.1
- net RED: now also R15.1, R16.1, R20.1
- net VCC_5V: now also JP1.2; no longer JP1.4
- net VCC_B2: now also JP1.4; no longer JP1.6
- net VCC_B3: now also T2.C, T4.C, T7.C, T8.C
Routing:
- net VCC_B2: track 19.2 -> 62.0 mm
- net GND: track 27.0 -> 51.0 mm
- net N$2: track 0.00 -> 9.55 mm
- net N$3: track 0.00 -> 7.94 mm
- net N$9: track 0.00 -> 7.20 mm
- net N$11: track 0.00 -> 6.99 mm
- net B_SPARE: track 0.00 -> 3.81 mm
- net B_NMI: track 0.00 -> 3.81 mm
- net B_DEBUG: track 0.00 -> 3.81 mm
- net R1: track 0.00 -> 2.86 mm
- net R0: track 0.00 -> 2.86 mm
- net G1: track 0.00 -> 2.86 mm
- net G0: track 0.00 -> 2.86 mm
- net CSYNC: track 0.00 -> 2.86 mm
- net B0: track 0.00 -> 2.86 mm
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
Commit message: WIP
Parts:
- removed Q5: BC548-TO92-E1-REV, bc548:TO92-E1-REV
- removed T2, T4, T7, T8: (no value), transistor:TO92-CBE
- added Q1: BC548-TO92-E1-REV, bc548:TO92-E1-REV
- moved Q4 47.9 mm to (43.2, 10.8), turned to 180 degrees
- moved Q2 46.8 mm to (48.3, 10.8), turned to 180 degrees
- moved Q3 40.2 mm to (38.1, 10.8), turned to 180 degrees
- moved R15 12.0 mm to (33.0, 8.89), turned to 180 degrees
- moved R16 8.98 mm to (33.0, 6.35), turned to 180 degrees
- moved R13 8.98 mm to (48.3, 6.35), turned to 180 degrees
- moved R14 7.41 mm to (48.3, 8.89), turned to 180 degrees
- moved R32 7.41 mm to (43.2, 8.89), turned to 180 degrees
- moved R20 6.48 mm to (33.0, 3.81), turned to 180 degrees
- moved R26 4.02 mm to (38.1, 8.89), turned to 180 degrees
- moved R28 4.02 mm to (38.1, 3.81), turned to 180 degrees
- moved R33 4.02 mm to (43.2, 6.35), turned to 180 degrees
- moved R31 1.80 mm to (43.2, 3.81), turned to 180 degrees
- moved R27 1.80 mm to (38.1, 6.35), turned to 180 degrees
Connections:
- net N$1: now also Q2.3; no longer T2.E
- net N$10: now also Q3.3; no longer T7.E
- net N$11: now also Q4.2; no longer T8.B
- net N$12: now also Q4.3; no longer T8.E
- net N$2: now also Q1.2; no longer T4.B
- net N$3: now also Q2.2; no longer T2.B
- net N$6: now also Q1.3; no longer T4.E
- net N$9: now also Q3.2; no longer T7.B
- net VCC_B3: now also Q1.1, Q2.1, Q3.1, Q4.1; no longer T2.C, T4.C, T7.C, T8.C
Routing:
- net VCC_B3: track 0.00 -> 65.3 mm
- net N$10: track 0.00 -> 7.69 mm
- net N$6: track 0.00 -> 7.09 mm
- net N$12: track 0.00 -> 7.01 mm
- net GREEN: track 0.00 -> 5.74 mm
- net BLUE: track 0.00 -> 5.42 mm
- net RED: track 0.00 -> 5.08 mm
- net N$2: track 9.55 -> 4.58 mm
- net N$3: track 7.94 -> 3.20 mm
- net N$1: track 0.00 -> 4.47 mm
- net N$9: track 7.20 -> 4.13 mm
- net COMP: track 0.00 -> 2.54 mm
- net N$11: track 6.99 -> 4.77 mm

Commit message: WIP
Parts:
- added JP4: (no value), pinhead:2X03
- added R10, R11, R8, R9: 1000, rcl:R0805
- moved X1 30.7 mm to (11.4, 47.0), turned to 270 degrees
- moved Q4 26.2 mm to (67.3, 21.0), turned to 270 degrees
- moved Q1 26.2 mm to (57.1, 21.0), turned to 270 degrees
- moved Q3 26.2 mm to (62.2, 21.0), turned to 270 degrees
- moved R30 25.0 mm to (66.0, 25.4)
- moved JP2 25.0 mm to (35.6, 34.3)
- moved R6 25.0 mm to (53.3, 25.4)
- moved JP1 25.0 mm to (87.6, 40.6)
- moved JP3 25.0 mm to (88.9, 25.4)
- moved R1 25.0 mm to (87.6, 16.5)
- moved R2 25.0 mm to (88.9, 21.6)
- moved R24 25.0 mm to (58.4, 25.4)
- moved R25 25.0 mm to (61.0, 25.4)
- moved R29 25.0 mm to (63.5, 25.4)
- moved R3 25.0 mm to (94.0, 16.5)
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Connections:
- removed net AGND: X1.4
- removed net COMPGND: X1.17
- removed net D_GND: X1.18
- removed net VGND: X1.13, X1.5, X1.9
- new net N$4: JP4.5, R10.1
- new net N$5: JP4.3, R11.1
- net ALEFT: now also JP4.4
- net ARIGHT: now also JP4.6
- net AUDLEFT: now also R11.2, SV9.23; no longer SV9.21
- net AUDRIGHT: now also R10.2, SV9.21; no longer SV9.23
- net D_FASTBLANKING: now also R8.1, R9.2
- net GND: now also JP4.1, R9.1, X1.13, X1.17, X1.18, X1.4, X1.5, X1.9
- net VCC_B3: now also R8.2
Routing:
- net GND: track 51.0 -> 244.4 mm
- net COMP: track 2.54 -> 154.3 mm
- net VCC_5V: track 17.3 -> 135.8 mm
- net ALEFT: track 0.00 -> 94.8 mm
- net ARIGHT: track 0.00 -> 80.6 mm
- net BLUE: track 5.42 -> 63.1 mm
- net GREEN: track 5.74 -> 58.2 mm
- net RED: track 5.08 -> 57.4 mm
- net VCC_B2: track 62.0 -> 102.9 mm
- net VCC_B3: track 65.3 -> 101.3 mm
- net D_FASTBLANKING: track 0.00 -> 18.6 mm
- net N$10: track 7.69 -> 17.6 mm
- net N$12: track 7.01 -> 16.2 mm
- net N$5: track 0.00 -> 8.77 mm
- net N$4: track 0.00 -> 8.77 mm
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
Commit message: WIP
Parts:
- Q2: value BC548-TO92-E1-REV -> BC548; device bc548:TO92-E1-REV -> transistor-npn:TO92-EBC
- R8: value 1000 -> 75
- R9: value 1000 -> 750
- moved R14 29.2 mm to (36.8, 15.2)
- moved R31 28.4 mm to (25.4, 20.3), turned to 270 degrees
- moved R32 28.4 mm to (30.5, 20.3), turned to 270 degrees
- moved R33 28.4 mm to (27.9, 20.3), turned to 270 degrees
- moved R9 28.1 mm to (35.6, 30.5)
- moved R8 24.4 mm to (38.1, 30.5), turned to 90 degrees
- moved R13 24.1 mm to (39.4, 15.2)
- moved R28 18.2 mm to (33.0, 22.9)
- moved R27 13.3 mm to (35.6, 22.9)
- moved X1 11.7 mm to (14.0, 35.6), flipped to the bottom
- moved R26 8.52 mm to (38.1, 22.9)
- moved SV8 7.62 mm to (64.8, 71.1)
- moved JP1 7.18 mm to (82.5, 45.7)
- moved Q2 7.10 mm to (64.8, 20.3), flipped to the bottom, turned to 315 degrees
- moved R2 6.35 mm to (82.5, 21.6)
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Connections:
- new net VCC_CORE: SV8.1, SV8.3
- net ALEFT: now also JP4.6; no longer JP4.4
- net ARIGHT: now also JP4.4; no longer JP4.6
- net N$1: now also Q2.E; no longer Q2.3
- net N$3: now also Q2.B; no longer Q2.2
- net VCC_B0: now also SV8.7
- net VCC_B1: now also SV8.11
- net VCC_B3: now also Q2.C; no longer Q2.1
Routing:
- net COMP: track 154.3 -> 77.0 mm
- net GND: track 244.4 -> 311.5 mm
- net BLUE: track 63.1 -> 25.2 mm
- net VCC_B3: track 101.3 -> 65.2 mm
- net ALEFT: track 94.8 -> 67.9 mm
- net N$12: track 16.2 -> 40.0 mm
- net GREEN: track 58.2 -> 34.9 mm
- net N$1: track 8.20 -> 28.7 mm
- net VCC_B2: track 102.9 -> 117.1 mm
- net D_FASTBLANKING: track 18.6 -> 32.4 mm
- net RED: track 57.4 -> 44.3 mm
- net ARIGHT: track 80.6 -> 67.7 mm
- net VCC_5V: track 135.8 -> 147.3 mm
- net N$10: track 17.6 -> 27.3 mm
- net CASMOTOR: track 5.61 -> 9.42 mm
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
Commit message: WIP
Parts:
- added IC1: 25LC080SN, microchip:SO-08
- added JP5: (no value), jumper:JP2
Connections:
- new net N$7: IC1.3, JP5.2
- net GND: now also IC1.4, JP5.3
- net SPI_CLK: now also IC1.6, SV8.8; no longer SV8.6
- net SPI_DI: now also IC1.5, SV8.6; no longer SV8.8
- net SPI_DO: now also IC1.2
- net SPI_SEL0: now also IC1.1
- net VCC_B0: now also IC1.7, IC1.8, JP5.1
Routing:
- net SPI_CLK: track 0.00 -> 65.6 mm
- net SPI_DI: track 0.00 -> 53.5 mm
- net VCC_B0: track 2.54 -> 28.4 mm
- net N$7: track 0.00 -> 18.7 mm
- net GND: track 311.5 -> 330.0 mm
- net SPI_DO: track 0.00 -> 13.4 mm
- net SPI_SEL0: track 0.00 -> 5.74 mm

Commit message: WIP
Parts:
- added C1: (no value), rcl:C0603
- moved JP5 2.54 mm to (27.9, 71.1)
Connections:
- net GND: now also C1.1
- net VCC_B0: now also C1.2
Routing:
- net GND: track 330.0 -> 309.2 mm
- net SPI_CLK: track 65.6 -> 46.1 mm
- net SPI_DI: track 53.5 -> 38.5 mm
- net N$7: track 18.7 -> 13.8 mm
- net VCC_B0: track 28.4 -> 27.6 mm
- net SPI_DO: track 13.4 -> 12.9 mm
Changed lines of the file:
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@@
 <attribute name="OC_FARNELL" value="1137302" x="33.02" y="71.12" size="1.778" layer="27" rot="R180" display="off"/>
 </element>
-<element name="JP5" library="jumper" package="JP2" value="" x="25.4" y="71.12" rot="R90"/>
+<element name="JP5" library="jumper" package="JP2" value="" x="27.94" y="71.12" rot="R90"/>
+<element name="C1" library="rcl" package="C0603" value="" x="38.1" y="68.58" rot="R270"/>
 </elements>
 <signals>
@@
 <contactref element="IC1" pad="6"/>
 <contactref element="SV8" pad="8"/>
-<wire x1="48.26" y1="73.66" x2="48.26" y2="77.47" width="0.254" layer="1"/>
-<wire x1="48.26" y1="77.47" x2="46.99" y2="78.74" width="0.254" layer="1"/>
-<wire x1="46.99" y1="78.74" x2="20.32" y2="78.74" width="0.254" layer="1"/>
-<wire x1="20.32" y1="78.74" x2="17.78" y2="76.2" width="0.254" layer="1"/>
-<wire x1="17.78" y1="76.2" x2="17.78" y2="66.04" width="0.254" layer="1"/>
-<wire x1="17.78" y1="66.04" x2="20.32" y2="63.5" width="0.254" layer="1"/>
-<wire x1="20.32" y1="63.5" x2="30.48" y2="63.5" width="0.254" layer="1"/>
-<wire x1="30.48" y1="63.5" x2="32.385" y2="65.405" width="0.254" layer="1"/>
-<wire x1="32.385" y1="65.405" x2="32.385" y2="68.52" width="0.254" layer="1"/>
+<wire x1="48.26" y1="73.66" x2="48.26" y2="76.2" width="0.254" layer="1"/>
+<wire x1="48.26" y1="76.2" x2="47.625" y2="76.835" width="0.254" layer="1"/>
+<wire x1="47.625" y1="76.835" x2="25.4" y2="76.835" width="0.254" layer="1"/>
+<wire x1="25.4" y1="76.835" x2="24.765" y2="76.2" width="0.254" layer="1"/>
+<wire x1="24.765" y1="76.2" x2="24.765" y2="66.675" width="0.254" layer="1"/>
+<wire x1="24.765" y1="66.675" x2="25.4" y2="66.04" width="0.254" layer="1"/>
+<wire x1="25.4" y1="66.04" x2="31.75" y2="66.04" width="0.254" layer="1"/>
+<wire x1="31.75" y1="66.04" x2="32.385" y2="66.675" width="0.254" layer="1"/>
+<wire x1="32.385" y1="66.675" x2="32.385" y2="68.52" width="0.254" layer="1"/>
+<wire x1="32.385" y1="68.52" x2="32.385" y2="68.58" width="0.254" layer="1"/>
 </signal>
 <signal name="SPI_DI">
 <contactref element="IC1" pad="5"/>
 <contactref element="SV8" pad="6"/>
-<wire x1="45.72" y1="73.66" x2="45.72" y2="76.2" width="0.254" layer="1"/>
-<wire x1="45.72" y1="76.2" x2="44.45" y2="77.47" width="0.254" layer="1"/>
-<wire x1="44.45" y1="77.47" x2="21.59" y2="77.47" width="0.254" layer="1"/>
-<wire x1="21.59" y1="77.47" x2="20.32" y2="76.2" width="0.254" layer="1"/>
-<wire x1="20.32" y1="76.2" x2="20.32" y2="66.04" width="0.254" layer="1"/>
-<wire x1="20.32" y1="66.04" x2="21.59" y2="64.77" width="0.254" layer="1"/>
-<wire x1="21.59" y1="64.77" x2="29.845" y2="64.77" width="0.254" layer="1"/>
-<wire x1="29.845" y1="64.77" x2="31.115" y2="66.04" width="0.254" layer="1"/>
-<wire x1="31.115" y1="68.52" x2="31.115" y2="66.04" width="0.254" layer="1"/>
+<wire x1="45.72" y1="73.66" x2="45.72" y2="75.565" width="0.254" layer="1"/>
+<wire x1="45.72" y1="75.565" x2="45.085" y2="76.2" width="0.254" layer="1"/>
+<wire x1="45.085" y1="76.2" x2="26.035" y2="76.2" width="0.254" layer="1"/>
+<wire x1="26.035" y1="76.2" x2="25.4" y2="75.565" width="0.254" layer="1"/>
+<wire x1="25.4" y1="75.565" x2="25.4" y2="67.31" width="0.254" layer="1"/>
+<wire x1="25.4" y1="67.31" x2="26.035" y2="66.675" width="0.254" layer="1"/>
+<wire x1="26.035" y1="66.675" x2="30.48" y2="66.675" width="0.254" layer="1"/>
+<wire x1="30.48" y1="66.675" x2="31.115" y2="67.31" width="0.254" layer="1"/>
+<wire x1="31.115" y1="67.31" x2="31.115" y2="68.52" width="0.254" layer="1"/>
+<wire x1="31.115" y1="68.58" x2="31.115" y2="68.52" width="0.254" layer="1"/>
 </signal>
 <signal name="SPI_SEL1">
@@
 <contactref element="IC1" pad="2"/>
 <wire x1="33.655" y1="73.72" x2="33.655" y2="75.565" width="0.254" layer="1"/>
-<wire x1="33.655" y1="75.565" x2="34.29" y2="76.2" width="0.254" layer="1"/>
-<wire x1="34.29" y1="76.2" x2="41.91" y2="76.2" width="0.254" layer="1"/>
-<wire x1="41.91" y1="76.2" x2="43.18" y2="74.93" width="0.254" layer="1"/>
+<wire x1="33.655" y1="75.565" x2="42.545" y2="75.565" width="0.254" layer="1"/>
+<wire x1="42.545" y1="75.565" x2="43.18" y2="74.93" width="0.254" layer="1"/>
 <wire x1="43.18" y1="74.93" x2="43.18" y2="73.66" width="0.254" layer="1"/>
 </signal>
@@
 <contactref element="JP5" pad="1"/>
 <wire x1="45.72" y1="68.58" x2="43.18" y2="66.04" width="0.254" layer="1"/>
-<wire x1="43.18" y1="66.04" x2="35.56" y2="66.04" width="0.254" layer="1"/>
+<wire x1="43.18" y1="66.04" x2="38.1" y2="66.04" width="0.254" layer="1"/>
+<wire x1="38.1" y1="66.04" x2="35.56" y2="66.04" width="0.254" layer="1"/>
 <wire x1="35.56" y1="66.04" x2="35.56" y2="67.31" width="0.254" layer="1"/>
 <wire x1="33.655" y1="68.52" x2="34.925" y2="68.52" width="0.254" layer="1"/>
-<wire x1="25.4" y1="68.58" x2="28.575" y2="68.58" width="0.254" layer="1"/>
-<wire x1="28.575" y1="68.58" x2="30.48" y2="70.485" width="0.254" layer="1"/>
 <wire x1="30.48" y1="70.485" x2="33.02" y2="70.485" width="0.254" layer="1"/>
 <wire x1="33.02" y1="70.485" x2="33.655" y2="69.85" width="0.254" layer="1"/>
@@
 <wire x1="34.925" y1="68.52" x2="34.925" y2="67.945" width="0.254" layer="1"/>
 <wire x1="34.925" y1="67.945" x2="35.56" y2="67.31" width="0.254" layer="1"/>
+<contactref element="C1" pad="2"/>
+<wire x1="38.1" y1="67.73" x2="38.1" y2="66.04" width="0.254" layer="1"/>
+<wire x1="30.48" y1="70.485" x2="28.575" y2="68.58" width="0.254" layer="1"/>
+<wire x1="28.575" y1="68.58" x2="27.94" y2="68.58" width="0.254" layer="1"/>
 </signal>
 <signal name="VCC_B1">
@@
 <wire x1="78.74" y1="49.53" x2="77.47" y2="48.26" width="0.254" layer="1"/>
 <wire x1="77.47" y1="48.26" x2="13.97" y2="48.26" width="0.254" layer="1"/>
-<wire x1="78.74" y1="71.12" x2="78.74" y2="52.07" width="0.254" layer="1"/>
+<wire x1="78.74" y1="71.12" x2="78.74" y2="52.07" width="0" layer="19" extent="1-16"/>
 <wire x1="13.97" y1="48.26" x2="13.97" y2="48.895" width="0.254" layer="1"/>
 <contactref element="IC1" pad="4"/>
 <contactref element="JP5" pad="3"/>
-<wire x1="25.4" y1="73.66" x2="27.305" y2="73.66" width="0.254" layer="1"/>
-<wire x1="27.305" y1="73.66" x2="29.21" y2="71.755" width="0.254" layer="1"/>
-<wire x1="29.21" y1="71.755" x2="31.75" y2="71.755" width="0.254" layer="1"/>
 <wire x1="31.75" y1="71.755" x2="33.655" y2="71.755" width="0.254" layer="1"/>
 <wire x1="33.655" y1="71.755" x2="34.29" y2="71.12" width="0.254" layer="1"/>
-<wire x1="34.29" y1="71.12" x2="40.64" y2="71.12" width="0.254" layer="1"/>
+<wire x1="34.29" y1="71.12" x2="39.37" y2="71.12" width="0.254" layer="1"/>
+<wire x1="39.37" y1="71.12" x2="40.64" y2="71.12" width="0.254" layer="1"/>
 <wire x1="31.115" y1="73.72" x2="31.115" y2="72.39" width="0.254" layer="1"/>
 <wire x1="31.115" y1="72.39" x2="31.75" y2="71.755" width="0.254" layer="1"/>
+<contactref element="C1" pad="1"/>
+<wire x1="38.1" y1="69.43" x2="38.1" y2="69.85" width="0.254" layer="1"/>
+<wire x1="38.1" y1="69.85" x2="39.37" y2="71.12" width="0.254" layer="1"/>
+<wire x1="27.94" y1="73.66" x2="28" y2="73.72" width="0.254" layer="1"/>
+<wire x1="28" y1="73.72" x2="31.115" y2="73.72" width="0.254" layer="1"/>
 <wire x1="78.74" y1="71.12" x2="78.74" y2="71.12" width="0" layer="19" extent="1-16"/>
 </signal>
@@
 <contactref element="IC1" pad="3"/>
 <contactref element="JP5" pad="2"/>
-<wire x1="25.4" y1="71.12" x2="23.495" y2="71.12" width="0.254" layer="1"/>
-<wire x1="23.495" y1="71.12" x2="22.225" y2="72.39" width="0.254" layer="1"/>
-<wire x1="22.225" y1="72.39" x2="22.225" y2="74.295" width="0.254" layer="1"/>
-<wire x1="22.225" y1="74.295" x2="24.13" y2="76.2" width="0.254" layer="1"/>
-<wire x1="24.13" y1="76.2" x2="31.75" y2="76.2" width="0.254" layer="1"/>
-<wire x1="31.75" y1="76.2" x2="32.385" y2="75.565" width="0.254" layer="1"/>
+<wire x1="27.94" y1="71.12" x2="26.67" y2="71.12" width="0.254" layer="1"/>
+<wire x1="26.67" y1="71.12" x2="26.035" y2="71.755" width="0.254" layer="1"/>
+<wire x1="26.035" y1="71.755" x2="26.035" y2="74.93" width="0.254" layer="1"/>
+<wire x1="26.035" y1="74.93" x2="26.67" y2="75.565" width="0.254" layer="1"/>
+<wire x1="26.67" y1="75.565" x2="32.385" y2="75.565" width="0.254" layer="1"/>
 <wire x1="32.385" y1="75.565" x2="32.385" y2="73.72" width="0.254" layer="1"/>
 </signal>
