File: eagle/homeboard1/homeboard1.sch (EAGLE design)
At the start: 1 part, among them U1 XC3S400TQ144

Commit message: experiment with VIA_DIY device
Parts:
- added U$1, U$2, U$3, U$4, U$5: VIA_DIY, cpcfpga:VIA_DIY
Connections:
- new net GND: U$5.BOTTOM
- new net N$1: U$5.TOP, U1BGND.GND0, U1BGND.GND1, U1BGND.GND10, U1BGND.GND11, U1BGND.GND12, U1BGND.GND13, U1BGND.GND14, U1BGND.GND15, U1BGND.GND2, U1BGND.GND3, U1BGND.GND4, U1BGND.GND5, U1BGND.GND6, U1BGND.GND7, U1BGND.GND8, U1BGND.GND9
- new net VCC: U1B0AND1.VCCO_TOP0, U1B0AND1.VCCO_TOP1, U1B0AND1.VCCO_TOP2, U1B2AND3.VCCO_RIGHT0, U1B2AND3.VCCO_RIGHT1, U1B2AND3.VCCO_RIGHT2, U1B4AND5.VCCO_BOTTOM0, U1B4AND5.VCCO_BOTTOM1, U1B4AND5.VCCO_BOTTOM2, U1B6AND7.VCCO_LEFT0, U1B6AND7.VCCO_LEFT1, U1B6AND7.VCCO_LEFT2
- new net VCCAUX: U1BVCCAUX.VCCAUX0, U1BVCCAUX.VCCAUX1, U1BVCCAUX.VCCAUX2, U1BVCCAUX.VCCAUX3
Other:
- moved on the sheet: U1BGND
Changed lines of the file:
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@@
 <parts>
 <part name="U1" library="xilinx_spartan3_virtex4_and_5" deviceset="XC3S400TQ144" device=""/>
+<part name="SUPPLY1" library="supply2" deviceset="GND" device=""/>
+<part name="SUPPLY2" library="supply2" deviceset="VCC" device=""/>
+<part name="SUPPLY3" library="supply2" deviceset="VCC" device=""/>
+<part name="SUPPLY4" library="supply2" deviceset="VCC" device=""/>
+<part name="SUPPLY5" library="supply2" deviceset="VCC" device=""/>
+<part name="U$1" library="cpcfpga" deviceset="VIA_DIY" device=""/>
+<part name="U$2" library="cpcfpga" deviceset="VIA_DIY" device=""/>
+<part name="U$3" library="cpcfpga" deviceset="VIA_DIY" device=""/>
+<part name="U$4" library="cpcfpga" deviceset="VIA_DIY" device=""/>
+<part name="U$5" library="cpcfpga" deviceset="VIA_DIY" device=""/>
 </parts>
 <sheets>
@@
 <instance part="U1" gate="B4AND5" x="-114.3" y="20.32" rot="R270"/>
 <instance part="U1" gate="B6AND7" x="-175.26" y="88.9" rot="R180"/>
-<instance part="U1" gate="BGND" x="-233.68" y="91.44"/>
+<instance part="U1" gate="BGND" x="-302.26" y="88.9"/>
 <instance part="U1" gate="BVCCAUX" x="-233.68" y="139.7"/>
 <instance part="U1" gate="BVCCINT" x="-233.68" y="55.88"/>
+<instance part="SUPPLY1" gate="GND" x="-287.02" y="12.7"/>
+<instance part="SUPPLY2" gate="G$1" x="-190.5" y="93.98"/>
+<instance part="SUPPLY3" gate="G$1" x="-114.3" y="177.8"/>
+<instance part="SUPPLY4" gate="G$1" x="-38.1" y="96.52"/>
+<instance part="SUPPLY5" gate="G$1" x="-119.38" y="7.62"/>
+<instance part="U$1" gate="G$1" x="-180.34" y="215.9"/>
+<instance part="U$2" gate="G$1" x="-99.06" y="218.44"/>
+<instance part="U$3" gate="G$1" x="-12.7" y="215.9"/>
+<instance part="U$4" gate="G$1" x="66.04" y="152.4"/>
+<instance part="U$5" gate="G$1" x="-287.02" y="43.18" rot="R270"/>
 </instances>
 <busses>
 </busses>
 <nets>
+<net name="VCC" class="0">
+<segment>
+<pinref part="SUPPLY2" gate="G$1" pin="VCC"/>
+<pinref part="U1" gate="B6AND7" pin="VCCO_LEFT2"/>
+<wire x1="-190.5" y1="91.44" x2="-180.34" y2="91.44" width="0.1524" layer="91"/>
+<pinref part="U1" gate="B6AND7" pin="VCCO_LEFT1"/>
+<wire x1="-180.34" y1="91.44" x2="-180.34" y2="88.9" width="0.1524" layer="91"/>
+<junction x="-180.34" y="91.44"/>
+<pinref part="U1" gate="B6AND7" pin="VCCO_LEFT0"/>
+<wire x1="-180.34" y1="88.9" x2="-180.34" y2="86.36" width="0.1524" layer="91"/>
+<junction x="-180.34" y="88.9"/>
+</segment>
+<segment>
+<pinref part="SUPPLY5" gate="G$1" pin="VCC"/>
+<pinref part="U1" gate="B4AND5" pin="VCCO_BOTTOM2"/>
+<wire x1="-119.38" y1="5.08" x2="-116.84" y2="5.08" width="0.1524" layer="91"/>
+<wire x1="-116.84" y1="5.08" x2="-116.84" y2="15.24" width="0.1524" layer="91"/>
+<pinref part="U1" gate="B4AND5" pin="VCCO_BOTTOM1"/>
+<wire x1="-116.84" y1="15.24" x2="-114.3" y2="15.24" width="0.1524" layer="91"/>
+<junction x="-116.84" y="15.24"/>
+<pinref part="U1" gate="B4AND5" pin="VCCO_BOTTOM0"/>
+<wire x1="-114.3" y1="15.24" x2="-111.76" y2="15.24" width="0.1524" layer="91"/>
+<junction x="-114.3" y="15.24"/>
+</segment>
+<segment>
+<pinref part="U1" gate="B2AND3" pin="VCCO_RIGHT2"/>
+<pinref part="U1" gate="B2AND3" pin="VCCO_RIGHT1"/>
+<wire x1="-48.26" y1="88.9" x2="-48.26" y2="91.44" width="0.1524" layer="91"/>
+<pinref part="U1" gate="B2AND3" pin="VCCO_RIGHT0"/>
+<wire x1="-48.26" y1="91.44" x2="-48.26" y2="93.98" width="0.1524" layer="91"/>
+<junction x="-48.26" y="91.44"/>
+<pinref part="SUPPLY4" gate="G$1" pin="VCC"/>
+<wire x1="-48.26" y1="93.98" x2="-38.1" y2="93.98" width="0.1524" layer="91"/>
+<junction x="-48.26" y="93.98"/>
+</segment>
+<segment>
+<pinref part="SUPPLY3" gate="G$1" pin="VCC"/>
+<pinref part="U1" gate="B0AND1" pin="VCCO_TOP0"/>
+<wire x1="-114.3" y1="175.26" x2="-114.3" y2="167.64" width="0.1524" layer="91"/>
+<pinref part="U1" gate="B0AND1" pin="VCCO_TOP1"/>
+<wire x1="-114.3" y1="167.64" x2="-111.76" y2="167.64" width="0.1524" layer="91"/>
+<junction x="-114.3" y="167.64"/>
+<pinref part="U1" gate="B0AND1" pin="VCCO_TOP2"/>
+<wire x1="-111.76" y1="167.64" x2="-109.22" y2="167.64" width="0.1524" layer="91"/>
+<junction x="-111.76" y="167.64"/>
+</segment>
+</net>
+<net name="VCCAUX" class="0">
+<segment>
+<pinref part="U1" gate="BVCCAUX" pin="VCCAUX0"/>
+<pinref part="U1" gate="BVCCAUX" pin="VCCAUX1"/>
+<wire x1="-228.6" y1="129.54" x2="-228.6" y2="127" width="0.1524" layer="91"/>
+<pinref part="U1" gate="BVCCAUX" pin="VCCAUX2"/>
+<wire x1="-228.6" y1="127" x2="-228.6" y2="124.46" width="0.1524" layer="91"/>
+<junction x="-228.6" y="127"/>
+<pinref part="U1" gate="BVCCAUX" pin="VCCAUX3"/>
+<wire x1="-228.6" y1="124.46" x2="-228.6" y2="121.92" width="0.1524" layer="91"/>
+<junction x="-228.6" y="124.46"/>
+<wire x1="-228.6" y1="121.92" x2="-220.98" y2="121.92" width="0.1524" layer="91"/>
+<junction x="-228.6" y="121.92"/>
+<label x="-220.98" y="121.92" size="1.778" layer="95"/>
+</segment>
+</net>
+<net name="N$1" class="0">
+<segment>
+<pinref part="U1" gate="BGND" pin="GND15"/>
+<pinref part="U1" gate="BGND" pin="GND14"/>
+<wire x1="-297.18" y1="68.58" x2="-297.18" y2="71.12" width="0.1524" layer="91"/>
+<pinref part="U1" gate="BGND" pin="GND13"/>
+<wire x1="-297.18" y1="71.12" x2="-297.18" y2="73.66" width="0.1524" layer="91"/>
+<junction x="-297.18" y="71.12"/>
+<pinref part="U1" gate="BGND" pin="GND12"/>
+<wire x1="-297.18" y1="73.66" x2="-297.18" y2="76.2" width="0.1524" layer="91"/>
+<junction x="-297.18" y="73.66"/>
+<pinref part="U1" gate="BGND" pin="GND11"/>
+<wire x1="-297.18" y1="76.2" x2="-297.18" y2="78.74" width="0.1524" layer="91"/>
+<junction x="-297.18" y="76.2"/>
+<pinref part="U1" gate="BGND" pin="GND10"/>
+<wire x1="-297.18" y1="78.74" x2="-297.18" y2="81.28" width="0.1524" layer="91"/>
+<junction x="-297.18" y="78.74"/>
+<pinref part="U1" gate="BGND" pin="GND9"/>
+<wire x1="-297.18" y1="81.28" x2="-297.18" y2="83.82" width="0.1524" layer="91"/>
+<junction x="-297.18" y="81.28"/>
+<pinref part="U1" gate="BGND" pin="GND8"/>
+<wire x1="-297.18" y1="83.82" x2="-297.18" y2="86.36" width="0.1524" layer="91"/>
+<junction x="-297.18" y="83.82"/>
+<pinref part="U1" gate="BGND" pin="GND7"/>
+<wire x1="-297.18" y1="86.36" x2="-297.18" y2="88.9" width="0.1524" layer="91"/>
+<junction x="-297.18" y="86.36"/>
+<pinref part="U1" gate="BGND" pin="GND6"/>
+<wire x1="-297.18" y1="88.9" x2="-297.18" y2="91.44" width="0.1524" layer="91"/>
+<junction x="-297.18" y="88.9"/>
+<pinref part="U1" gate="BGND" pin="GND5"/>
+<wire x1="-297.18" y1="91.44" x2="-297.18" y2="93.98" width="0.1524" layer="91"/>
+<junction x="-297.18" y="91.44"/>
+<pinref part="U1" gate="BGND" pin="GND4"/>
+<wire x1="-297.18" y1="93.98" x2="-297.18" y2="96.52" width="0.1524" layer="91"/>
+<junction x="-297.18" y="93.98"/>
+<pinref part="U1" gate="BGND" pin="GND3"/>
+<wire x1="-297.18" y1="96.52" x2="-297.18" y2="99.06" width="0.1524" layer="91"/>
+<junction x="-297.18" y="96.52"/>
+<pinref part="U1" gate="BGND" pin="GND2"/>
+<wire x1="-297.18" y1="99.06" x2="-297.18" y2="101.6" width="0.1524" layer="91"/>
+<junction x="-297.18" y="99.06"/>
+<pinref part="U1" gate="BGND" pin="GND1"/>
+<wire x1="-297.18" y1="101.6" x2="-297.18" y2="104.14" width="0.1524" layer="91"/>
+<junction x="-297.18" y="101.6"/>
+<pinref part="U1" gate="BGND" pin="GND0"/>
+<wire x1="-297.18" y1="104.14" x2="-297.18" y2="106.68" width="0.1524" layer="91"/>
+<junction x="-297.18" y="104.14"/>
+<pinref part="U$5" gate="G$1" pin="TOP"/>
+<wire x1="-287.02" y1="60.96" x2="-287.02" y2="68.58" width="0.1524" layer="91"/>
+<wire x1="-287.02" y1="68.58" x2="-297.18" y2="68.58" width="0.1524" layer="91"/>
+<junction x="-297.18" y="68.58"/>
+</segment>
+</net>
+<net name="GND" class="0">
+<segment>
+<pinref part="U$5" gate="G$1" pin="BOTTOM"/>
+<pinref part="SUPPLY1" gate="GND" pin="GND"/>
+<wire x1="-287.02" y1="15.24" x2="-287.02" y2="25.4" width="0.1524" layer="91"/>
+</segment>
+</net>
 </nets>
 </sheet>

Commit message: attempt to imprve via_diy
Parts:
- removed U$1, U$2, U$3, U$4: VIA_DIY, cpcfpga:VIA_DIY
- added U$10, U$11, U$12, U$13, U$14, U$15, U$16, U$17, U$18, U$19, U$20, U$6, U$7, U$8, U$9: VIA_DIY, cpcfpga:VIA_DIY
Connections:
- new net N$10: U$14.T, U1BGND.GND9
- new net N$11: U$15.T, U1BGND.GND10
- new net N$12: U$16.T, U1BGND.GND11
- new net N$13: U$17.T, U1BGND.GND12
- new net N$14: U$18.T, U1BGND.GND13
- new net N$15: U$19.T, U1BGND.GND14
- new net N$16: U$20.T, U1BGND.GND15
- new net N$2: U$6.T, U1BGND.GND1
- new net N$3: U$7.T, U1BGND.GND2
- new net N$4: U$8.T, U1BGND.GND3
- new net N$5: U$9.T, U1BGND.GND4
- new net N$6: U$10.T, U1BGND.GND5
- new net N$7: U$11.T, U1BGND.GND6
- new net N$8: U$12.T, U1BGND.GND7
- new net N$9: U$13.T, U1BGND.GND8
- net GND: now also U$10.B, U$11.B, U$12.B, U$13.B, U$14.B, U$15.B, U$16.B, U$17.B, U$18.B, U$19.B, U$20.B, U$5.B, U$6.B, U$7.B, U$8.B, U$9.B; no longer U$5.BOTTOM
- net N$1: now also U$5.T; no longer U$5.TOP, U1BGND.GND1, U1BGND.GND10, U1BGND.GND11, U1BGND.GND12, U1BGND.GND13, U1BGND.GND14, U1BGND.GND15, U1BGND.GND2, U1BGND.GND3, U1BGND.GND4, U1BGND.GND5, U1BGND.GND6, U1BGND.GND7, U1BGND.GND8, U1BGND.GND9

Commit message: all fpga power and ground done
Parts:
- added U$1, U$2, U$21, U$22, U$23, U$24, U$4: VIA_DIY, cpcfpga:VIA_DIY
Connections:
- new net GND_B: U$10.B, U$11.B, U$12.B, U$13.B, U$14.B, U$15.B, U$16.B, U$17.B, U$18.B, U$19.B, U$20.B, U$5.B, U$6.B, U$7.B, U$8.B, U$9.B
- new net N$17: U$21.B, U$23.B, U$24.B
- new net N$18: U$23.T, U1B0AND1.VCCO_TOP1
- new net N$19: U$21.T, U1B4AND5.VCCO_BOTTOM1
- new net N$20: U$22.B, U$4.B
- new net VCCINT01: U$1.T, U1BVCCINT.VCCINT0, U1BVCCINT.VCCINT1
- new net VCCINT23: U$2.T, U1BVCCINT.VCCINT2, U1BVCCINT.VCCINT3
- new net VCCINT_B: U$1.B, U$2.B
- net GND: now also U$20.T, U1BGND.GND15; no longer U$10.B, U$11.B, U$12.B, U$13.B, U$14.B, U$15.B, U$16.B, U$17.B, U$18.B, U$19.B, U$20.B, U$5.B, U$6.B, U$7.B, U$8.B, U$9.B
- net N$16: now also U$22.T, U1BVCCAUX.VCCAUX0, U1BVCCAUX.VCCAUX1; no longer U$20.T, U1BGND.GND15
- net VCC: now also U$24.T; no longer U1B0AND1.VCCO_TOP1, U1B4AND5.VCCO_BOTTOM1
- net VCCAUX: now also U$4.T; no longer U1BVCCAUX.VCCAUX0, U1BVCCAUX.VCCAUX1
