File: eagle/homeboard1/backup.brd (EAGLE design)
At the start: 100 x 80 mm, 17 parts, among them U1 XC3S400TQ144

Commit message: thinking
Parts:
- removed U$3: VIA_DIY, cpcfpga:VIA_DIY
- added U$10, U$11, U$14, U$15, U$18, U$19, U$6, U$7: VIA_DIY, cpcfpga:VIA_DIY
- moved U$21 28.3 mm to (56.5, 21.0)
- moved U$23 28.2 mm to (56.5, 37.0)
- moved U$24 15.6 mm to (55.0, 28.0)
- moved U$4 9.90 mm to (52.5, 42.0)
- moved U$1 9.22 mm to (59.5, 16.0)
- moved U$9 8.51 mm to (48.5, 20.0)
- moved U$20 8.50 mm to (48.5, 37.5)
- moved U$5 8.50 mm to (48.5, 33.5)
- moved U$8 8.50 mm to (48.5, 23.5)
- moved U$13 7.50 mm to (64.0, 24.0)
- moved U$16 7.50 mm to (64.0, 34.0)
- moved U$17 7.50 mm to (64.0, 37.5)
- moved U$12 7.00 mm to (64.5, 20.0)
- moved U$2 1.00 mm to (59.0, 42.5)
- moved U$22 1.00 mm to (53.0, 15.5)
Connections:
- removed net N$21: U$3.T, U1.P62
- new net N$10: U$14.T, U1.P88
- new net N$11: U$15.T, U1.P94
- new net N$14: U$18.T, U1.P117
- new net N$15: U$19.T, U1.P136
- new net N$3: U$7.T, U1.P22
- new net N$5: U$9.T, U1.P42
- new net N$6: U$10.T, U1.P45
- new net N$7: U$11.T, U1.P64
- net GND: no longer U1.P136
- net GND_B: now also U$10.B, U$11.B, U$14.B, U$15.B, U$18.B, U$19.B, U$6.B, U$7.B
- net N$1: no longer U1.P16
- net N$12: no longer U1.P94
- net N$13: no longer U1.P117
- net N$16: now also U1.P62
- net N$17: now also U$21.B, U$23.B, U$24.B; no longer U$24.T, U1.P133
- net N$18: now also U1.P126; no longer U1.P61
- net N$19: now also U1.P54; no longer U1.P134
- net N$2: now also U$6.T, U1.P16; no longer U$9.T, U1.P42, U1.P45
- net N$20: no longer U$21.B, U$3.B
- net N$4: no longer U1.P22
- net N$8: no longer U1.P64
- net N$9: no longer U1.P88
- net VCC: now also U$24.T; no longer U1.P126, U1.P54
- net VCCAUX: now also U1.P134
- net VCCINT01: now also U1.P61
- net VCCINT23: now also U1.P133
- net VCCINT_B: no longer U$23.B, U$24.B
Routing:
- net GND_B: track 1.56 -> 110.5 mm
- net VCC: track 128.1 -> 85.6 mm
- net N$20: track 0.00 -> 30.9 mm
- net VCCINT_B: track 0.00 -> 28.5 mm
- net N$17: track 0.00 -> 20.1 mm
- net VCCAUX: track 0.00 -> 18.5 mm
- net N$16: track 0.00 -> 18.5 mm
- net VCCINT23: track 0.00 -> 18.0 mm
- net VCCINT01: track 0.00 -> 16.4 mm
- net N$2: track 17.1 -> 2.97 mm
- net GND: track 16.6 -> 3.01 mm
- net N$13: track 15.5 -> 2.95 mm
- net N$8: track 15.5 -> 3.98 mm
- net N$14: track 0.00 -> 9.95 mm
- net N$1: track 12.0 -> 2.95 mm
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