File: eagle/homeboard1/backup.sch (EAGLE design)
At the start: 17 parts, among them U1 XC3S400TQ144

Commit message: thinking
Parts:
- removed U$3: VIA_DIY, cpcfpga:VIA_DIY
- added U$10, U$11, U$14, U$15, U$18, U$19, U$6, U$7: VIA_DIY, cpcfpga:VIA_DIY
Connections:
- removed net N$21: U$3.T, U1BVCCAUX.VCCAUX1
- new net N$10: U$14.T, U1BGND.GND9
- new net N$11: U$15.T, U1BGND.GND10
- new net N$14: U$18.T, U1BGND.GND13
- new net N$15: U$19.T, U1BGND.GND14
- new net N$3: U$7.T, U1BGND.GND2
- new net N$5: U$9.T, U1BGND.GND4
- new net N$6: U$10.T, U1BGND.GND5
- new net N$7: U$11.T, U1BGND.GND6
- net GND: no longer U1BGND.GND14
- net GND_B: now also U$10.B, U$11.B, U$14.B, U$15.B, U$18.B, U$19.B, U$6.B, U$7.B
- net N$1: no longer U1BGND.GND1
- net N$12: no longer U1BGND.GND10
- net N$13: no longer U1BGND.GND13
- net N$16: now also U1BVCCAUX.VCCAUX1
- net N$17: now also U$21.B, U$23.B, U$24.B; no longer U$24.T, U1BVCCINT.VCCINT3
- net N$18: now also U1B0AND1.VCCO_TOP1; no longer U1BVCCINT.VCCINT1
- net N$19: now also U1B4AND5.VCCO_BOTTOM1; no longer U1BVCCAUX.VCCAUX3
- net N$2: now also U$6.T, U1BGND.GND1; no longer U$9.T, U1BGND.GND4, U1BGND.GND5
- net N$20: no longer U$21.B, U$3.B
- net N$4: no longer U1BGND.GND2
- net N$8: no longer U1BGND.GND6
- net N$9: no longer U1BGND.GND9
- net VCC: now also U$24.T; no longer U1B0AND1.VCCO_TOP1, U1B4AND5.VCCO_BOTTOM1
- net VCCAUX: now also U1BVCCAUX.VCCAUX3
- net VCCINT01: now also U1BVCCINT.VCCINT1
- net VCCINT23: now also U1BVCCINT.VCCINT3
- net VCCINT_B: no longer U$23.B, U$24.B
