File: eagle/drutest/drutest2.brd (EAGLE design)
At the start: 100 x 80 mm, 53 parts, among them IC1 XCF02S, Q5 BC848SMD, Q6 BC848SMD, Q7 BC848SMD, Q8 BC848SMD, T1 BSS138, T2 BC848, T3 BSS138, U1 XC3S400TQ144, X1 1503_04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

Commit message: vcc wide everywhere
Parts:
- added U$3: 2.5V, cpcfpga:SOT223
- added U$4: 1.2V, cpcfpga:SOT223
- added U$5: EXPHDR, cpcfpga:EXPHDR
- moved X3 60.6 mm to (91.0, 34.5)
- moved U$2 9.01 mm to (52.0, 8.00)
- moved JP2 8.50 mm to (18.5, 37.0)
- moved X2 8.50 mm to (11.5, 32.5)
- moved U$1 0.50 mm to (33.8, 36.8)
Connections:
- net GND: now also U$3.1, U$4.1
- net VCC: now also U$3.3, U$4.3
- net VCCAUX: now also U$3.4
- net VCCINT: now also U$4.4
Routing:
- net GND: track 243.1 -> 278.8 mm
- net VCC: track 134.5 -> 164.6 mm, vias 8 -> 11
- net N$40: track 0.00 -> 27.6 mm, vias 0 -> 3
- net VCCAUX: track 48.3 -> 73.2 mm, vias 0 -> 1
- net VCCINT: track 49.4 -> 67.2 mm, vias 2 -> 3
- net N$66: track 7.96 -> 0.00 mm
- net N$15: track 19.5 -> 20.7 mm
- net PROM_INITB: track 12.4 -> 11.4 mm
- net N$9: track 13.0 -> 13.5 mm
- net N$8: track 12.0 -> 12.5 mm
- net N$7: track 9.98 -> 10.5 mm
- net N$6: track 8.98 -> 9.48 mm
- net N$5: track 7.98 -> 8.48 mm
- net N$4: track 6.98 -> 7.48 mm
- net N$3: track 5.98 -> 6.48 mm
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
Commit message: headache
Parts:
- removed JP1: (no value), pinhead:2X20
- added JP3: (no value), pinhead:2X03
- moved X2 74.0 mm to (85.0, 41.0), turned to 90 degrees
- moved JP2 59.5 mm to (78.0, 36.5), turned to 90 degrees
- moved U$2 44.8 mm to (96.5, 3.00)
- moved X3 43.9 mm to (69.0, 72.5), turned to 90 degrees
- moved R2 28.0 mm to (31.0, 42.6)
- moved R1 28.0 mm to (14.5, 42.7)
- moved U$1 28.0 mm to (5.79, 37.8)
- moved U$3 28.0 mm to (5.50, 43.5)
- moved U$4 28.0 mm to (5.50, 33.5)
- moved U1 28.0 mm to (22.7, 37.8)
- moved IC1 28.0 mm to (20.5, 34.1)
- moved R3 28.0 mm to (31.0, 44.7)
- moved U$5 26.5 mm to (22.0, 37.5)
Connections:
- removed net N$30: JP1.1, U1.P108
- removed net N$31: JP1.39, U1.P73
- removed net N$32: JP1.40, U1.P74
- removed net N$33: JP1.37, U1.P76
- removed net N$34: JP1.38, U1.P77
- removed net N$37: JP1.35, U1.P78
- removed net N$41: JP1.36, U1.P79
- removed net N$44: JP1.33, U1.P80
- removed net N$45: JP1.34, U1.P82
- removed net N$46: JP1.31, U1.P83
- removed net N$47: JP1.32, U1.P84
- removed net N$48: JP1.29, U1.P85
- removed net N$49: JP1.30, U1.P86
- removed net N$50: JP1.27, U1.P87
- removed net N$51: JP1.28, U1.P89
- removed net N$52: JP1.25, U1.P90
- new net N$68: JP3.3
- new net N$69: JP3.5
- new net N$70: JP3.6
- new net N$72: JP3.4
- net TCK: now also JP3.1
- net TMS: now also JP3.2
Routing:
- net N$32: track 34.1 -> 0.00 mm
- net N$34: track 33.1 -> 0.00 mm
- net N$41: track 32.5 -> 0.00 mm
- net N$31: track 31.3 -> 0.00 mm
- net N$45: track 31.1 -> 0.00 mm
- net N$33: track 30.7 -> 0.00 mm
- net N$37: track 29.7 -> 0.00 mm
- net N$47: track 29.2 -> 0.00 mm
- net N$44: track 28.5 -> 0.00 mm
- net N$49: track 27.8 -> 0.00 mm
- net N$51: track 27.0 -> 0.00 mm
- net N$46: track 26.9 -> 0.00 mm
- net N$48: track 25.4 -> 0.00 mm
- net N$50: track 24.2 -> 0.00 mm
- net N$52: track 23.0 -> 0.00 mm
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