File: eagle/drutest/drutest2.sch (EAGLE design)
At the start: 53 parts, among them IC1 XCF02S, Q5 BC848SMD, Q6 BC848SMD, Q7 BC848SMD, Q8 BC848SMD, T1 BSS138, T2 BC848, T3 BSS138, U1 XC3S400TQ144, X1 1503_04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

Commit message: vcc wide everywhere
Parts:
- added U$3: 2.5V, cpcfpga:NX1117
- added U$4: 1.2V, cpcfpga:NX1117
- added U$5: EXPHDR, cpcfpga:EXPHDR
Connections:
- net GND: now also U$3.GND, U$4.GND
- net VCC: now also U$3.VCC, U$4.VCC
- net VCCAUX: now also U$3.VOUT1
- net VCCINT: now also U$4.VOUT1
Changed lines of the file:
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@@
 <part name="C4" library="resistor" deviceset="C-EU" device="C0603"/>
 <part name="U$2" library="cpcfpga" deviceset="TXO_7C" device=""/>
+<part name="U$3" library="cpcfpga" deviceset="NX1117" device="" value="2.5V"/>
+<part name="U$4" library="cpcfpga" deviceset="NX1117" device="" value="1.2V"/>
+<part name="SUPPLY3" library="supply2" deviceset="GND" device=""/>
+<part name="U$5" library="cpcfpga" deviceset="EXPHDR" device=""/>
 </parts>
 <sheets>
@@
 <instance part="C4" gate="G$1" x="200.66" y="-223.52" rot="R90"/>
 <instance part="U$2" gate="G$1" x="68.58" y="-66.04"/>
+<instance part="U$3" gate="G$1" x="-195.58" y="58.42"/>
+<instance part="U$4" gate="G$1" x="-195.58" y="35.56"/>
+<instance part="SUPPLY3" gate="GND" x="-203.2" y="20.32"/>
+<instance part="U$5" gate="G$1" x="91.44" y="109.22"/>
+<instance part="U$5" gate="G$2" x="91.44" y="-99.06"/>
 </instances>
 <busses>
@@
 <label x="48.26" y="-71.12" size="1.778" layer="95"/>
 </segment>
+<segment>
+<pinref part="U$4" gate="G$1" pin="GND"/>
+<pinref part="U$3" gate="G$1" pin="GND"/>
+<wire x1="-203.2" y1="30.48" x2="-203.2" y2="53.34" width="0.1524" layer="91"/>
+<wire x1="-203.2" y1="30.48" x2="-203.2" y2="22.86" width="0.1524" layer="91"/>
+<junction x="-203.2" y="30.48"/>
+<pinref part="SUPPLY3" gate="GND" pin="GND"/>
+</segment>
 </net>
 <net name="VCC" class="0">
@@
 <label x="48.26" y="-60.96" size="1.778" layer="95"/>
 </segment>
+<segment>
+<pinref part="U$4" gate="G$1" pin="VCC"/>
+<wire x1="-203.2" y1="38.1" x2="-205.74" y2="38.1" width="0.1524" layer="91"/>
+<wire x1="-205.74" y1="38.1" x2="-205.74" y2="60.96" width="0.1524" layer="91"/>
+<pinref part="U$3" gate="G$1" pin="VCC"/>
+<wire x1="-205.74" y1="60.96" x2="-203.2" y2="60.96" width="0.1524" layer="91"/>
+<wire x1="-205.74" y1="60.96" x2="-205.74" y2="73.66" width="0.1524" layer="91"/>
+<junction x="-205.74" y="60.96"/>
+<wire x1="-205.74" y1="73.66" x2="-198.12" y2="73.66" width="0.1524" layer="91"/>
+<label x="-198.12" y="73.66" size="1.778" layer="95"/>
+</segment>
 </net>
 <net name="TCK" class="0">
@@
 <label x="-127" y="2.54" size="1.778" layer="95"/>
 </segment>
+<segment>
+<pinref part="U$4" gate="G$1" pin="VOUT1"/>
+<wire x1="-172.72" y1="38.1" x2="-167.64" y2="38.1" width="0.1524" layer="91"/>
+<label x="-167.64" y="38.1" size="1.778" layer="95"/>
+</segment>
 </net>
 <net name="VCCAUX" class="0">
@@
 <label x="-142.24" y="-73.66" size="1.778" layer="95"/>
 </segment>
-</net>
+<segment>
+<pinref part="U$3" gate="G$1" pin="VOUT1"/>
+<wire x1="-172.72" y1="60.96" x2="-167.64" y2="60.96" width="0.1524" layer="91"/>
+<label x="-167.64" y="60.96" size="1.778" layer="95"/>
+</segment>
+</net>

Commit message: headache
Parts:
- removed JP1: (no value), pinhead:PINHD-2X20
- added JP3: (no value), pinhead:PINHD-2X3
Connections:
- removed net N$30: JP1.1, U1B2.IO_L01N_2VRP_2
- removed net N$31: JP1.39, U1B3.IO_L01P_3VRN_3
- removed net N$32: JP1.40, U1B3.IO_L01N_3VRP_3
- removed net N$33: JP1.37, U1B3.IO
- removed net N$34: JP1.38, U1B3.IO_L20P_3
- removed net N$37: JP1.35, U1B3.IO_L20N_3
- removed net N$41: JP1.36, U1B3.IO_L21P_3
- removed net N$44: JP1.33, U1B3.IO_L21N_3
- removed net N$45: JP1.34, U1B3.IO_L22P_3
- removed net N$46: JP1.31, U1B3.IO_L22N_3
- removed net N$47: JP1.32, U1B3.IO_L23P_3VREF_3
- removed net N$48: JP1.29, U1B3.IO_L23N_3
- removed net N$49: JP1.30, U1B3.IO_L24P_3
- removed net N$50: JP1.27, U1B3.IO_L24N_3
- removed net N$51: JP1.28, U1B3.IO_L40P_3
- removed net N$52: JP1.25, U1B3.IO_L40N_3VREF_3
- new net N$68: JP3.3
- new net N$69: JP3.5
- new net N$70: JP3.6
- new net N$72: JP3.4
- net TCK: now also JP3.1
- net TMS: now also JP3.2
Other:
- moved on the sheet: JP2, X2
