File: eagle/drutest/durtest-ripup.brd (EAGLE design)
At the start: 100 x 80 mm, 56 parts, among them IC1 XCF02S, Q5 BC848SMD, Q6 BC848SMD, Q7 BC848SMD, Q8 BC848SMD, T1 BSS138, T2 BC848, T3 BSS138, U1 XC3S400TQ144, X1 1503_04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

Commit message: more fiddling
Parts:
- added R35, R36, R37, R38, R39, R40, R41, R42, R43, R44, R45, R46: (no value), resistor:M0805
- added X4, X5: (no value), con-subd:F09HP
- R4, R5, R6, R7: value 10K -> 1000
- moved R5 98.7 mm to (14.5, 46.5), flipped to the bottom, turned to 90 degrees
- moved R4 93.3 mm to (17.5, 42.5), flipped to the bottom, turned to 90 degrees
- moved R7 91.4 mm to (14.5, 34.0), flipped to the bottom, turned to 270 degrees
- moved R6 91.0 mm to (17.5, 38.0), flipped to the bottom, turned to 90 degrees
- moved T1 75.5 mm to (14.5, 42.5), flipped to the bottom, turned to 90 degrees
- moved X3 71.8 mm to (5.00, 40.0)
- moved T3 70.1 mm to (14.5, 38.0), flipped to the bottom, turned to 90 degrees
- moved U$4 68.6 mm to (73.0, 21.5)
- moved U$3 67.0 mm to (72.5, 41.5)
- moved R1 54.7 mm to (66.5, 59.7)
- moved U$5 50.9 mm to (72.5, 31.0)
- moved R3 40.8 mm to (68.5, 28.7)
- moved R2 39.1 mm to (69.0, 33.6)
- moved JP3 35.4 mm to (65.0, 74.5)
- moved IC1 25.5 mm to (46.0, 34.6)
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Connections:
- new net N$30: R35.1, X5.7
- new net N$31: R36.1, X5.6
- new net N$32: R37.1, X5.4
- new net N$33: R38.1, X5.3
- new net N$34: R39.1, X5.2
- new net N$37: R46.1, X5.1
- new net N$41: R40.2, X4.1
- new net N$44: R41.2, X4.2
- new net N$45: R42.2, X4.3
- new net N$46: R43.2, X4.4
- new net N$47: R44.2, X4.6
- new net N$48: R45.2, X4.7
- net GND: now also X4.8, X4.G1, X5.8, X5.G1
- net VCC: now also R35.2, R36.2, R37.2, R38.2, R39.2, R40.1, R41.1, R42.1, R43.1, R44.1, R45.1, R46.2
Routing:
- net GND: track 267.1 -> 109.2 mm, vias 15 -> 0
- net VCC: track 163.8 -> 44.3 mm, vias 11 -> 0
- net VCCAUX: track 73.7 -> 0.00 mm, vias 1 -> 0
- net VCCINT: track 67.2 -> 0.00 mm, vias 3 -> 0
- net N$40: track 29.1 -> 0.00 mm, vias 3 -> 0
- net PROM_DO: track 21.2 -> 0.00 mm, vias 1 -> 0
- net TMS: track 20.8 -> 0.00 mm
- net N$35: track 16.4 -> 0.00 mm, vias 1 -> 0
- net VCC_B2: track 0.00 -> 14.5 mm, vias 0 -> 2
- net N$39: track 11.7 -> 0.00 mm, vias 1 -> 0
- net PROM_INITB: track 11.4 -> 0.00 mm, vias 1 -> 0
- net N$38: track 11.4 -> 0.00 mm, vias 1 -> 0
- net CLK_5V: track 0.00 -> 11.3 mm
- net TCK: track 10.9 -> 0.00 mm
- net N$45: track 0.00 -> 10.1 mm
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
Commit message: hmmm
Parts:
- removed JP2: (no value), pinhead:2X08
- removed U$3: 2.5V, cpcfpga:SOT223
- removed U$4: 1.2V, cpcfpga:SOT223
- removed U$5: EXPHDR, cpcfpga:EXPHDR
- added C1, C5: (no value), resistor:C0603
- added IC2: 25LC080SN, microchip:SO-08
- added JP1: (no value), jumper:JP1
- added R47: 4K7, rcl:R0805
- added R48, R49: (no value), resistor:M0805
- added REG1.2: 1.2V, cpcfpga:SOT223
- added REG2.5: 2.5V, cpcfpga:SOT223
- moved R26 123.2 mm to (46.0, 67.0), flipped to the bottom, turned to 180 degrees
- moved C4 121.9 mm to (25.5, 65.8), flipped to the bottom, turned to 90 degrees
- moved C3 121.8 mm to (29.5, 65.8), flipped to the bottom, turned to 90 degrees
- moved R27 119.4 mm to (46.0, 64.8), flipped to the bottom, turned to 180 degrees
- moved R31 119.3 mm to (39.0, 67.5), flipped to the bottom
- moved R32 116.2 mm to (39.0, 65.2), flipped to the bottom
- moved R28 112.6 mm to (46.0, 62.5), flipped to the bottom, turned to 180 degrees
- moved R23 112.0 mm to (29.5, 55.5), flipped to the bottom, turned to 90 degrees
- moved R13 111.8 mm to (62.5, 65.5), flipped to the bottom, turned to 180 degrees
- moved R34 111.5 mm to (25.5, 55.5), flipped to the bottom, turned to 90 degrees
- moved R14 111.1 mm to (62.5, 63.0), flipped to the bottom, turned to 180 degrees
- moved R25 110.9 mm to (43.0, 59.5), flipped to the bottom, turned to 90 degrees
- moved R33 107.3 mm to (39.0, 63.0), flipped to the bottom
- moved R29 105.0 mm to (34.5, 59.5), flipped to the bottom, turned to 90 degrees
- moved R11 104.3 mm to (94.4, 1.25)
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Connections:
- removed net AOUTLEFT: JP2.13, R23.1, X2.3
- removed net AOUTRIGHT: JP2.15, R34.1, X2.1
- removed net AUDLEFT: C3.2
- removed net AUDRIGHT: C4.2
- removed net BLUE: JP2.11, X2.7
- removed net COMPOUT: JP2.1, X2.19
- removed net D_MODESWITCH: JP2.9, X2.8
- removed net GREEN: JP2.7, X2.11
- removed net N$66: U$2.OUT, U1.P55
- removed net RED: JP2.5, X2.15
- removed net VCC_B2: R22.1, R4.2, R6.2, T1.3, T2.3, T3.3
- new net FPGA_AUDIO_LEFT: R23.1
- new net FPGA_AUDIO_RIGHT: R34.1
- new net N$49: IC2.3, JP1.2, R47.1
- new net N$50: U$2.OUT, U1.P52
- new net N$51: C1.2, R23.2, R48.1
- new net N$52: C3.1, R48.2
- new net SPI_CLK: IC2.6, U1.P46
- new net SPI_DI: IC2.5, U1.P44
- new net SPI_DO: IC2.2, U1.P40
- new net SPI_SEL0: IC2.1, U1.P41
- net D_FASTBLANKING: no longer JP2.3, X2.16
- net GND: now also C1.1, C5.1, IC2.4, JP1.1, REG1.2.1, REG2.5.1; no longer U$3.1, U$4.1
- net N$64: now also C4.1, R49.2; no longer C3.1, R23.2
- net N$65: now also C5.2, R49.1; no longer C4.1
- net SCART_BLANKING: now also X2.16; no longer JP2.4
- net SCART_BLUE: now also X2.7; no longer JP2.12
- net SCART_COMP: now also X2.19; no longer JP2.2
- net SCART_GREEN: now also X2.11; no longer JP2.8
- net SCART_LEFT: now also C3.2, X2.3; no longer JP2.14
- net SCART_MODE: now also X2.8; no longer JP2.10
- net SCART_RED: now also X2.15; no longer JP2.6
- net SCART_RIGHT: now also C4.2, X2.1; no longer JP2.16
- net VCC: now also IC2.7, IC2.8, R22.1, R4.2, R47.2, R6.2, REG1.2.3, REG2.5.3, T1.3, T2.3, T3.3; no longer U$3.3, U$4.3
- net VCCAUX: now also REG2.5.4; no longer U$3.4
- net VCCINT: now also REG1.2.4; no longer U$4.4
Routing:
- net VCC: track 44.3 -> 181.5 mm, vias 0 -> 7
- net VCC_5V: track 0.00 -> 25.7 mm, vias 0 -> 2
- net AOUTRIGHT: track 25.0 -> 0.00 mm
- net GND: track 109.2 -> 133.5 mm, vias 0 -> 3
- net AOUTLEFT: track 23.7 -> 0.00 mm
- net VCCAUX: track 0.00 -> 20.6 mm
- net SPI_DI: track 0.00 -> 20.2 mm, vias 0 -> 1
- net SPI_CLK: track 0.00 -> 19.6 mm, vias 0 -> 1
- net D_MODESWITCH: track 17.6 -> 0.00 mm
- net BLUE: track 17.2 -> 0.00 mm
- net VCCINT: track 0.00 -> 16.5 mm
- net GREEN: track 15.9 -> 0.00 mm
- net VCC_B2: track 14.5 -> 0.00 mm, vias 2 -> 0
- net SPI_SEL0: track 0.00 -> 12.2 mm, vias 0 -> 1
- net SPI_DO: track 0.00 -> 12.2 mm, vias 0 -> 1
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
Commit message: hmmm
Parts:
- moved X2 51.0 mm to (7.00, 37.5), turned to 270 degrees
- moved R13 50.0 mm to (13.5, 55.5), turned to 90 degrees
- moved C4 48.8 mm to (13.2, 18.5), turned to 0 degrees
- moved R15 47.5 mm to (12.0, 49.0), turned to 270 degrees
- moved R14 47.1 mm to (16.0, 55.5), turned to 90 degrees
- moved C3 46.2 mm to (13.2, 22.5), turned to 0 degrees
- moved R31 44.9 mm to (11.5, 32.0), turned to 270 degrees
- moved R20 44.6 mm to (14.2, 49.0), turned to 270 degrees
- moved R49 44.3 mm to (17.0, 18.5), turned to 0 degrees
- moved R26 44.0 mm to (12.0, 39.0), turned to 90 degrees
- moved Q5 43.2 mm to (19.5, 55.5), turned to 90 degrees
- moved R32 41.8 mm to (13.8, 32.0), turned to 270 degrees
- moved R16 41.7 mm to (16.5, 49.0), turned to 270 degrees
- moved R48 41.4 mm to (17.0, 22.5), turned to 0 degrees
- moved R27 40.9 mm to (14.2, 39.0), turned to 90 degrees
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
Commit message: scart socket
Parts:
- added R50: 2k2, resistor:M0805
- moved REG2.5 31.8 mm to (54.5, 63.5)
- moved IC2 30.2 mm to (44.0, 8.50)
- moved JP3 27.5 mm to (58.0, 53.0)
- moved JP1 27.3 mm to (44.5, 2.25)
- moved R47 26.6 mm to (39.0, 2.50)
- moved R29 8.38 mm to (27.5, 25.0)
- moved R9 8.38 mm to (27.5, 42.0)
- moved R24 8.31 mm to (27.5, 36.0)
- moved R25 8.31 mm to (27.5, 33.8)
- moved R10 8.25 mm to (27.5, 44.2)
- moved R30 8.25 mm to (27.5, 27.2)
- moved R15 8.00 mm to (19.8, 47.0), turned to 90 degrees
- moved R16 8.00 mm to (24.2, 47.0), turned to 90 degrees
- moved R20 8.00 mm to (22.0, 47.0), turned to 90 degrees
- moved C1 8.00 mm to (28.2, 22.0)
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Connections:
- net B0: now also U1.P40
- net B1: now also U1.P41
- net CSYNC: now also U1.P137
- net FPGA_AUDIO_LEFT: now also U1.P47
- net FPGA_AUDIO_RIGHT: now also U1.P50
- net G0: now also U1.P44
- net G1: now also U1.P46
- net R0: now also U1.P140
- net R1: now also U1.P141
- net SCART_BLANKING: now also R50.1
- net SPI_CLK: no longer U1.P46
- net SPI_DI: no longer U1.P44
- net SPI_DO: no longer U1.P40
- net SPI_SEL0: no longer U1.P41
- net VCCAUX: now also R50.2
Routing:
- net SCART_BLANKING: track 1.87 -> 36.9 mm
- net GND: track 133.5 -> 162.3 mm, vias 3 -> 9
- net SCART_BLUE: track 0.00 -> 22.9 mm
- net SCART_RED: track 0.00 -> 22.3 mm
- net SPI_DI: track 20.2 -> 0.00 mm, vias 1 -> 0
- net SPI_CLK: track 19.6 -> 0.00 mm, vias 1 -> 0
- net SCART_LEFT: track 0.00 -> 18.1 mm
- net SCART_RIGHT: track 0.00 -> 18.0 mm
- net SCART_GREEN: track 4.50 -> 22.3 mm
- net VCCAUX: track 20.6 -> 38.1 mm
- net R0: track 0.00 -> 16.2 mm, vias 0 -> 1
- net G1: track 0.00 -> 15.5 mm, vias 0 -> 1
- net R1: track 0.00 -> 15.4 mm, vias 0 -> 1
- net FPGA_AUDIO_RIGHT: track 0.00 -> 14.7 mm, vias 0 -> 1
- net CSYNC: track 0.00 -> 13.2 mm, vias 0 -> 1
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