File: eagle/drutest/durtest-ripup.sch (EAGLE design)
At the start: 56 parts, among them IC1 XCF02S, Q5 BC848SMD, Q6 BC848SMD, Q7 BC848SMD, Q8 BC848SMD, T1 BSS138, T2 BC848, T3 BSS138, U1 XC3S400TQ144, X1 1503_04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

Commit message: more fiddling
Parts:
- added R35, R36, R37, R38, R39, R40, R41, R42, R43, R44, R45, R46: (no value), resistor:R-EU_M0805
- added X4, X5: (no value), con-subd:F09HPS
- R4, R5, R6, R7: value 10K -> 1000
Connections:
- new net N$30: R35.1, X5-7.F
- new net N$31: R36.1, X5-6.F
- new net N$32: R37.1, X5-4.F
- new net N$33: R38.1, X5-3.F
- new net N$34: R39.1, X5-2.F
- new net N$37: R46.1, X5-1.F
- new net N$41: R40.2, X4-1.F
- new net N$44: R41.2, X4-2.F
- new net N$45: R42.2, X4-3.F
- new net N$46: R43.2, X4-4.F
- new net N$47: R44.2, X4-6.F
- new net N$48: R45.2, X4-7.F
- net GND: now also X4-8.F, X4-G.G1, X5-8.F, X5-G.G1
- net VCC: now also R35.2, R36.2, R37.2, R38.2, R39.2, R40.1, R41.1, R42.1, R43.1, R44.1, R45.1, R46.2
Other:
- moved on the sheet: U$2, U1B0, U1B1, U1B2, U1B3, U1B4, U1B5

Commit message: hmmm
Parts:
- removed JP2: (no value), pinhead:PINHD-2X8
- removed U$5: EXPHDR, cpcfpga:EXPHDR
- added C1, C5: (no value), resistor:C-EUC0603
- added IC2: 25LC080SN, microchip:25LC080SN
- added JP1: (no value), jumper:JP1Q
- added R47: 4K7, rcl:R-EU_R0805
- added R48, R49: (no value), resistor:R-EU_M0805
- renumbered U$3 to REG2.5, U$4 to REG1.2
Connections:
- removed net AOUTLEFT: JP2.13, R23.1, X2.3
- removed net AOUTRIGHT: JP2.15, R34.1, X2.1
- removed net AUDLEFT: C3.2
- removed net AUDRIGHT: C4.2
- removed net BLUE: JP2.11, X2.7
- removed net COMPOUT: JP2.1, X2.19
- removed net D_MODESWITCH: JP2.9, X2.8
- removed net GREEN: JP2.7, X2.11
- removed net N$66: U$2.OUT, U1B4.IO_L32P_4GCLK0
- removed net RED: JP2.5, X2.15
- removed net VCC_B2: R22.1, R4.2, R6.2, T1.G, T2.C, T3.G
- new net FPGA_AUDIO_LEFT: R23.1
- new net FPGA_AUDIO_RIGHT: R34.1
- new net N$49: IC2.!WP, JP1.2, R47.1
- new net N$50: U$2.OUT, U1B5.IO_L32P_5GCLK2
- new net N$51: C1.2, R23.2, R48.1
- new net N$52: C3.1, R48.2
- new net SPI_CLK: IC2.SCK, U1B5.IO_L28P_5D7
- new net SPI_DI: IC2.SI, U1B5.IOVREF_5
- new net SPI_DO: IC2.SO, U1B5.IO_L01P_5CS_B
- new net SPI_SEL0: IC2.!CS, U1B5.IO_L01N_5RDWR_B
- net D_FASTBLANKING: no longer JP2.3, X2.16
- net GND: now also C1.1, C5.1, IC2.GND, JP1.1
- net N$64: now also C4.1, R49.2; no longer C3.1, R23.2
- net N$65: now also C5.2, R49.1; no longer C4.1
- net SCART_BLANKING: now also X2.16; no longer JP2.4
- net SCART_BLUE: now also X2.7; no longer JP2.12
- net SCART_COMP: now also X2.19; no longer JP2.2
- net SCART_GREEN: now also X2.11; no longer JP2.8
- net SCART_LEFT: now also C3.2, X2.3; no longer JP2.14
- net SCART_MODE: now also X2.8; no longer JP2.10
- net SCART_RED: now also X2.15; no longer JP2.6
- net SCART_RIGHT: now also C4.2, X2.1; no longer JP2.16
- net VCC: now also IC2.!HOLD, IC2.VCC, R22.1, R4.2, R47.2, R6.2, T1.G, T2.C, T3.G
Other:
- moved on the sheet: C4, R23, R34, U$2

Commit message: scart socket
Parts:
- added R50: 2k2, resistor:R-EU_M0805
Connections:
- net B0: now also U1B5.IO_L01P_5CS_B
- net B1: now also U1B5.IO_L01N_5RDWR_B
- net CSYNC: now also U1B0.IO_L27N_0
- net FPGA_AUDIO_LEFT: now also U1B5.IO_L28N_5D6
- net FPGA_AUDIO_RIGHT: now also U1B5.IO_L31P_5D5
- net G0: now also U1B5.IOVREF_5
- net G1: now also U1B5.IO_L28P_5D7
- net R0: now also U1B0.IO_L01P_0VRN_0
- net R1: now also U1B0.IO_L01N_0VRP_0
- net SCART_BLANKING: now also R50.1
- net SPI_CLK: no longer U1B5.IO_L28P_5D7
- net SPI_DI: no longer U1B5.IOVREF_5
- net SPI_DO: no longer U1B5.IO_L01P_5CS_B
- net SPI_SEL0: no longer U1B5.IO_L01N_5RDWR_B
- net VCCAUX: now also R50.2
Other:
- moved on the sheet: C1, C3, C4, C5, IC2, JP1, R23, R34, R47, R48, R49
