File: eagle/drutest/durtest4.brd (EAGLE design)
At the start: 100 x 80 mm, 76 parts, among them IC1 XCF02S, IC2 25LC080SN, Q5 BC848SMD, Q6 BC848SMD, Q7 BC848SMD, Q8 BC848SMD, T1 BSS138, T2 BC848, T3 BSS138, U1 XC3S400TQ144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

Commit message: sleepy
Parts:
- added R51: 2k2, resistor:M0805
- added SJ2: (no value), jumper:SJ_2
- moved IC1 15.3 mm to (51.9, 14.5), turned to 0 degrees
- moved X4 4.00 mm to (89.0, 64.5), turned to 270 degrees
- moved REG1.2 2.00 mm to (39.0, 35.5)
- moved R50 1.00 mm to (25.5, 20.0)
Connections:
- new net N$66: R51.2, SJ2.2
- net SCART_MODE: now also R51.1
- net VCC: now also SJ2.1
- net VCCAUX: now also SJ2.3
Routing:
- net SCART_MODE: track 0.00 -> 22.6 mm, vias 0 -> 2
- net GND: track 233.8 -> 254.1 mm
- net PROM_INITB: track 0.00 -> 12.4 mm, vias 0 -> 1
- net N$35: track 0.00 -> 9.50 mm, vias 0 -> 1
- net PROM_DO: track 0.00 -> 8.24 mm, vias 0 -> 1
- net N$38: track 0.00 -> 7.45 mm, vias 0 -> 1
- net N$66: track 0.00 -> 3.55 mm
- net VCCAUX: track 38.1 -> 41.5 mm
- net VCC: track 227.1 -> 230.4 mm
- net SCART_BLANKING: track 37.6 -> 39.6 mm

Commit message: mah
Parts:
- added R52: 4K7, resistor:M0805
- added RESET_SW: (no value), jumper:JP1
- moved IC2 45.7 mm to (65.0, 24.5)
- moved R34 1.41 mm to (31.0, 15.0), turned to 270 degrees
- moved R23 0.50 mm to (32.0, 18.5)
- moved U$2 0.50 mm to (41.1, 15.9)
Connections:
- new net RESET: R52.2, RESET_SW.1, U1.P51
- net GND: now also RESET_SW.2
- net VCC: now also R52.1
Routing:
- net GND: track 254.1 -> 267.7 mm, vias 10 -> 12
- net VCC: track 230.4 -> 243.9 mm, vias 8 -> 9
- net RESET: track 0.00 -> 12.4 mm
- net TMS: track 0.00 -> 8.49 mm
- net N$36: track 0.00 -> 8.30 mm
- net TCK: track 0.00 -> 7.43 mm
- net N$40: track 0.00 -> 6.37 mm
- net PROM_INITB: track 12.4 -> 11.4 mm

Commit message: mah
Parts:
- moved REG2.5 30.3 mm to (44.5, 31.0), turned to 270 degrees
- moved REG1.2 1.80 mm to (40.0, 37.0), turned to 90 degrees
Routing:
- net VCCAUX: track 41.5 -> 66.2 mm, vias 0 -> 4
- net VCCINT: track 16.5 -> 40.7 mm, vias 0 -> 4

Commit message: regulators etc
Parts:
- moved REG1.2 0.50 mm to (40.0, 36.5)
- moved REG2.5 0.25 mm to (44.5, 31.2)
Connections:
- new net VCCAUX_R: REG2.5.2, U1.P120, U1.P62
- net VCCAUX: no longer U1.P120, U1.P62
Routing:
- net GND: track 267.5 -> 352.3 mm, vias 12 -> 21
- net VCCAUX_R: track 0.00 -> 24.2 mm, vias 0 -> 2
- net VCCAUX: track 66.2 -> 44.6 mm, vias 4 -> 2
- net VCC: track 243.9 -> 254.3 mm, vias 9 -> 11
- net VCCINT: track 40.7 -> 43.4 mm
- net SCART_BLUE: track 23.4 -> 25.1 mm
- net SCART_RED: track 22.8 -> 23.4 mm

Commit message: mah
Parts:
- moved JP3 26.7 mm to (63.0, 33.0), turned to 0 degrees
Routing:
- net N$42: track 0.00 -> 54.8 mm, vias 0 -> 1
- net N$40: track 6.37 -> 57.5 mm, vias 0 -> 1
- net R0: track 16.2 -> 17.7 mm
- net CSYNC: track 13.2 -> 14.3 mm
- net R1: track 15.4 -> 16.3 mm
- net GND: track 352.3 -> 352.0 mm, vias 21 -> 19

Commit message: se power
Parts:
- moved IC2 23.8 mm to (61.0, 48.0), flipped to the top, turned to 90 degrees
Routing:
- net VCC: track 254.3 -> 258.8 mm
- net R0: track 17.7 -> 18.3 mm
Changed lines of the file:
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@@
 <element name="R45" library="resistor" package="M0805" value="" x="92" y="43" rot="R180"/>
 <element name="R46" library="resistor" package="M0805" value="" x="97.5" y="24"/>
-<element name="IC2" library="microchip" package="SO-08" value="25LC080SN" x="65" y="24.5" rot="MR180">
-<attribute name="OC_NEWARK" value="96K4092" x="56" y="12" size="1.778" layer="28" rot="MR180" display="off"/>
-<attribute name="MPN" value="25LC080/SN" x="56" y="12" size="1.778" layer="28" rot="MR180" display="off"/>
-<attribute name="MF" value="MICROCHIP" x="56" y="12" size="1.778" layer="28" rot="MR180" display="off"/>
-<attribute name="OC_FARNELL" value="1137302" x="56" y="12" size="1.778" layer="28" rot="MR180" display="off"/>
+<element name="IC2" library="microchip" package="SO-08" value="25LC080SN" x="61" y="48" rot="R90">
+<attribute name="OC_NEWARK" value="96K4092" x="48.5" y="39" size="1.778" layer="27" rot="R90" display="off"/>
+<attribute name="MPN" value="25LC080/SN" x="48.5" y="39" size="1.778" layer="27" rot="R90" display="off"/>
+<attribute name="MF" value="MICROCHIP" x="48.5" y="39" size="1.778" layer="27" rot="R90" display="off"/>
+<attribute name="OC_FARNELL" value="1137302" x="48.5" y="39" size="1.778" layer="27" rot="R90" display="off"/>
 </element>
 <element name="R47" library="rcl" package="R0805" value="4K7" x="74.5" y="76" rot="MR180"/>
@@
 <wire x1="48.475" y1="23.13" x2="48.475" y2="23.975" width="0.2" layer="1"/>
 <wire x1="48.475" y1="23.975" x2="49" y2="24.5" width="0.2" layer="1"/>
-<wire x1="49" y1="24.5" x2="49" y2="25" width="0.2" layer="1"/>
-<wire x1="49" y1="25" x2="49.25" y2="25.25" width="0.2" layer="1"/>
-<via x="49.25" y="25.25" extent="1-16" drill="0.6" shape="square"/>
-<wire x1="49.25" y1="25.25" x2="50.5" y2="26.5" width="0.2" layer="16"/>
+<wire x1="49" y1="24.5" x2="49" y2="25.5" width="0.2" layer="1"/>
+<via x="49" y="25.5" extent="1-16" drill="0.6" shape="square"/>
+<wire x1="49" y1="25.5" x2="50.5" y2="26.5" width="0.2" layer="16"/>
 <wire x1="50.5" y1="26.5" x2="51.25" y2="26.5" width="0.2" layer="16"/>
 <wire x1="90.27" y1="63.1284" x2="89" y2="77.0222" width="0" layer="19" extent="1-1"/>
 <wire x1="67.73" y1="76.25" x2="89" y2="77.0222" width="0" layer="19" extent="1-1"/>
 <wire x1="55.7" y1="64.25" x2="67.73" y2="76.25" width="0" layer="19" extent="1-1"/>
-<wire x1="48.475" y1="44.53" x2="55.7" y2="64.25" width="0" layer="19" extent="1-1"/>
+<wire x1="63.6" y1="49.905" x2="55.7" y2="64.25" width="0" layer="19" extent="1-1"/>
+<wire x1="51.25" y1="43" x2="63.6" y2="49.905" width="0" layer="19" extent="1-16"/>
 <wire x1="46.975" y1="23.13" x2="47" y2="23" width="0" layer="19" extent="1-1"/>
 <wire x1="7.5" y1="19.665" x2="7.5" y2="19.5" width="0" layer="19" extent="1-1"/>
 <wire x1="4.93" y1="44.5" x2="5" y2="46.5" width="0" layer="19" extent="1-1"/>
-<wire x1="66.905" y1="27.1" x2="52.925" y2="29.08" width="0" layer="19" extent="1-16"/>
-<wire x1="69.25" y1="12.9" x2="66.905" y2="27.1" width="0" layer="19" extent="16-16"/>
+<wire x1="69.25" y1="12.9" x2="52" y2="14.2164" width="0" layer="19" extent="16-16"/>
 <wire x1="85.55" y1="12.5" x2="73.05" y2="9.5" width="0" layer="19" extent="1-1"/>
 <wire x1="86.5" y1="19.9778" x2="85.55" y2="12.5" width="0" layer="19" extent="1-1"/>
@@
 <wire x1="35" y1="26.75" x2="36.475" y2="26.75" width="0.8" layer="1"/>
 <wire x1="36.475" y1="26.75" x2="42" y2="26.75" width="0.8" layer="1"/>
-<wire x1="42" y1="26.75" x2="48.5" y2="26.75" width="0.8" layer="1"/>
-<wire x1="48.5" y1="26.75" x2="49.5" y2="26.75" width="0.8" layer="1"/>
+<wire x1="42" y1="26.75" x2="48.25" y2="26.75" width="0.8" layer="1"/>
+<wire x1="48.25" y1="26.75" x2="49.5" y2="26.75" width="0.8" layer="1"/>
 <wire x1="49.5" y1="26.75" x2="49.5" y2="34" width="0.8" layer="1"/>
 <wire x1="49.5" y1="34" x2="49.5" y2="41" width="0.8" layer="1"/>
@@
 <contactref element="IC2" pad="7"/>
 <contactref element="R47" pad="2"/>
-<wire x1="64.365" y1="21.9" x2="63.095" y2="21.9" width="0.2" layer="16"/>
+<wire x1="58.4" y1="47.365" x2="58.4" y2="46.095" width="0.2" layer="1"/>
 <via x="74.25" y="65.75" extent="1-16" drill="0.6" shape="square"/>
 <via x="72.75" y="65.25" extent="1-16" drill="0.6" shape="square"/>
@@
 <wire x1="21.476" y1="15.5" x2="19.5" y2="15.5" width="0.2" layer="1"/>
 <wire x1="47.975" y1="23.13" x2="48" y2="23.13" width="0.2" layer="1"/>
-<wire x1="48" y1="23.13" x2="48" y2="24.5" width="0.2" layer="1"/>
-<wire x1="48" y1="24.5" x2="48.5" y2="25" width="0.2" layer="1"/>
-<wire x1="48.5" y1="25" x2="48.5" y2="26.75" width="0.2" layer="1"/>
 <wire x1="46.0196" y1="14.2164" x2="46.6696" y2="14.2164" width="0.4" layer="16"/>
 <wire x1="46.6696" y1="14.2164" x2="47.3196" y2="14.2164" width="0.4" layer="16"/>
@@
 <via x="47.5" y="27.5" extent="1-16" drill="0.6" shape="square"/>
 <wire x1="47.5" y1="27.5" x2="47.5" y2="27" width="0.8" layer="1"/>
-<wire x1="47.5" y1="27" x2="48.5" y2="26.75" width="0.8" layer="1"/>
 <wire x1="36.901" y1="38.811" x2="36.901" y2="39.599" width="0.8" layer="16"/>
 <wire x1="36.901" y1="39.599" x2="36" y2="40.25" width="0.8" layer="16"/>
@@
 <wire x1="47.975" y1="44.53" x2="48" y2="44.53" width="0.2" layer="1"/>
 <wire x1="48" y1="44.53" x2="48" y2="40.5" width="0.2" layer="1"/>
+<wire x1="53.25" y1="23" x2="51.5" y2="24.75" width="0.8" layer="1"/>
+<wire x1="48" y1="23.13" x2="48" y2="24.5" width="0.2" layer="1"/>
+<wire x1="48" y1="24.5" x2="48.25" y2="24.75" width="0.2" layer="1"/>
+<wire x1="48.25" y1="24.75" x2="48.25" y2="26.75" width="0.2" layer="1"/>
+<wire x1="51.5" y1="25" x2="51.5" y2="25.75" width="0.8" layer="1"/>
+<wire x1="51.5" y1="25.75" x2="51.25" y2="26" width="0.8" layer="1"/>
+<wire x1="51.25" y1="26" x2="50.25" y2="26" width="0.8" layer="1"/>
+<wire x1="50.25" y1="26" x2="49.5" y2="26.75" width="0.8" layer="1"/>
 <wire x1="74.25" y1="65.75" x2="75.45" y2="76" width="0" layer="19" extent="16-16"/>
 <wire x1="72.75" y1="65.25" x2="74.25" y2="65.75" width="0" layer="19" extent="1-1"/>
-<wire x1="92.95" y1="43" x2="74.25" y2="65.75" width="0" layer="19" extent="1-1"/>
-<wire x1="98.45" y1="32.5" x2="97.45" y2="38.5" width="0" layer="19" extent="1-1"/>
-<wire x1="91.45" y1="7.5" x2="98.45" y2="24" width="0" layer="19" extent="1-16"/>
-<wire x1="89.9" y1="4" x2="91.45" y2="7.5" width="0" layer="19" extent="1-16"/>
-<wire x1="61.984" y1="6.0094" x2="89.9" y2="4" width="0" layer="19" extent="1-16"/>
-<wire x1="60" y1="11.05" x2="60.0094" y2="11.0094" width="0" layer="19" extent="16-16"/>
-<wire x1="63.095" y1="21.9" x2="61.984" y2="11.0094" width="0" layer="19" extent="16-16"/>
-<wire x1="52.925" y1="26.08" x2="63.095" y2="21.9" width="0" layer="19" extent="1-16"/>
+<wire x1="58.4" y1="47.365" x2="72.75" y2="65.25" width="0" layer="19" extent="1-1"/>
+<wire x1="52.925" y1="41.58" x2="58.4" y2="46.095" width="0" layer="19" extent="1-1"/>
+<wire x1="51.5" y1="24.75" x2="51.5" y2="25" width="0" layer="19" extent="1-1"/>
+<wire x1="47.5" y1="27" x2="48.25" y2="26.75" width="0" layer="19" extent="1-1"/>
+<wire x1="59.5" y1="11.5" x2="47.3196" y2="14.2164" width="0" layer="19" extent="16-16"/>
+<wire x1="60.0094" y1="11.0094" x2="60" y2="11.05" width="0" layer="19" extent="16-16"/>
+<wire x1="89.9" y1="4" x2="61.984" y2="6.0094" width="0" layer="19" extent="1-16"/>
+<wire x1="91.45" y1="7.5" x2="89.9" y2="4" width="0" layer="19" extent="1-16"/>
+<wire x1="98.45" y1="24" x2="91.45" y2="7.5" width="0" layer="19" extent="1-16"/>
+<wire x1="97.45" y1="38.5" x2="98.45" y2="32.5" width="0" layer="19" extent="1-1"/>
 </signal>
 <signal name="TCK">
@@
 <wire x1="47.3196" y1="24.3196" x2="47.5" y2="24.5" width="0.2" layer="16"/>
 <wire x1="47.5" y1="24.5" x2="50.5" y2="24.5" width="0.2" layer="16"/>
-<wire x1="50.5" y1="24.5" x2="50.5" y2="25" width="0.2" layer="16"/>
-<via x="50.5" y="25" extent="1-16" drill="0.6" shape="square"/>
+<wire x1="50.5" y1="24.5" x2="50.25" y2="24.75" width="0.2" layer="16"/>
+<via x="50.25" y="24.75" extent="1-16" drill="0.6" shape="square"/>
 <wire x1="51" y1="23.155" x2="50.975" y2="23.13" width="0.2" layer="1"/>
-<wire x1="50.5" y1="25" x2="50.5" y2="24.5" width="0.2" layer="1"/>
-<wire x1="50.5" y1="24.5" x2="51" y2="24" width="0.2" layer="1"/>
+<wire x1="50.25" y1="24.75" x2="51" y2="24" width="0.2" layer="1"/>
 <wire x1="51" y1="24" x2="51" y2="23" width="0.2" layer="1"/>
 <wire x1="51" y1="23" x2="50.975" y2="23.13" width="0" layer="19" extent="1-1"/>
@@
 <wire x1="36" y1="46" x2="36" y2="46.5" width="0.2" layer="1"/>
 <wire x1="30.5" y1="46.5" x2="31.5" y2="47.5" width="0.2" layer="16"/>
-<wire x1="31.5" y1="47.5" x2="35" y2="47.5" width="0.2" layer="16"/>
-<wire x1="35" y1="47.5" x2="36" y2="46.5" width="0.2" layer="16"/>
+<wire x1="31.5" y1="47.5" x2="36" y2="47.5" width="0.2" layer="16"/>
+<wire x1="36" y1="47.5" x2="36" y2="46.5" width="0.2" layer="16"/>
 </signal>
 <signal name="G1">
@@
 <contactref element="JP1" pad="2"/>
 <wire x1="70.27" y1="76.25" x2="73.55" y2="76" width="0" layer="19" extent="16-16"/>
-<wire x1="65.635" y1="27.1" x2="70.27" y2="76.25" width="0" layer="19" extent="16-16"/>
+<wire x1="63.6" y1="48.635" x2="70.27" y2="76.25" width="0" layer="19" extent="1-1"/>
 </signal>
 <signal name="N$50">

Commit message: ne power
Routing:
- net VCC: track 258.8 -> 266.1 mm
Changed lines of the file:
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@@
 <wire x1="49.5" y1="26.75" x2="49.5" y2="34" width="0.8" layer="1"/>
 <wire x1="49.5" y1="34" x2="49.5" y2="41" width="0.8" layer="1"/>
-<wire x1="49.5" y1="41" x2="48.5" y2="41" width="0.8" layer="1"/>
+<wire x1="49.5" y1="41" x2="49.25" y2="41" width="0.8" layer="1"/>
+<wire x1="49.25" y1="41" x2="48.5" y2="41" width="0.8" layer="1"/>
 <wire x1="48.5" y1="41" x2="48" y2="40.5" width="0.8" layer="1"/>
 <wire x1="48" y1="40.5" x2="46.5" y2="39" width="0.8" layer="1"/>
@@
 <wire x1="72.75" y1="65.25" x2="74.25" y2="65.75" width="0" layer="19" extent="1-1"/>
 <wire x1="58.4" y1="47.365" x2="72.75" y2="65.25" width="0" layer="19" extent="1-1"/>
-<wire x1="52.925" y1="41.58" x2="58.4" y2="46.095" width="0" layer="19" extent="1-1"/>
+<wire x1="49.25" y1="41" x2="52.925" y2="41.58" width="0" layer="19" extent="1-16"/>
 <wire x1="51.5" y1="24.75" x2="51.5" y2="25" width="0" layer="19" extent="1-1"/>
 <wire x1="47.5" y1="27" x2="48.25" y2="26.75" width="0" layer="19" extent="1-1"/>
@@
 <wire x1="98.45" y1="24" x2="91.45" y2="7.5" width="0" layer="19" extent="1-16"/>
 <wire x1="97.45" y1="38.5" x2="98.45" y2="32.5" width="0" layer="19" extent="1-1"/>
+<wire x1="58.4" y1="46.095" x2="54.345" y2="46.095" width="0" layer="19" extent="1-16"/>
+<wire x1="54.345" y1="46.095" x2="49.25" y2="41" width="0.8" layer="1"/>
 </signal>
 <signal name="TCK">

Commit message: ne gnd
Parts:
- moved IC2 27.3 mm to (67.5, 21.5), flipped to the bottom
Routing:
- net GND: track 352.2 -> 360.4 mm
Changed lines of the file:
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@@
 <element name="R45" library="resistor" package="M0805" value="" x="92" y="43" rot="R180"/>
 <element name="R46" library="resistor" package="M0805" value="" x="97.5" y="24"/>
-<element name="IC2" library="microchip" package="SO-08" value="25LC080SN" x="61" y="48" rot="R90">
-<attribute name="OC_NEWARK" value="96K4092" x="48.5" y="39" size="1.778" layer="27" rot="R90" display="off"/>
-<attribute name="MPN" value="25LC080/SN" x="48.5" y="39" size="1.778" layer="27" rot="R90" display="off"/>
-<attribute name="MF" value="MICROCHIP" x="48.5" y="39" size="1.778" layer="27" rot="R90" display="off"/>
-<attribute name="OC_FARNELL" value="1137302" x="48.5" y="39" size="1.778" layer="27" rot="R90" display="off"/>
+<element name="IC2" library="microchip" package="SO-08" value="25LC080SN" x="67.5" y="21.5" rot="MR90">
+<attribute name="OC_NEWARK" value="96K4092" x="80" y="12.5" size="1.778" layer="28" rot="MR90" display="off"/>
+<attribute name="MPN" value="25LC080/SN" x="80" y="12.5" size="1.778" layer="28" rot="MR90" display="off"/>
+<attribute name="MF" value="MICROCHIP" x="80" y="12.5" size="1.778" layer="28" rot="MR90" display="off"/>
+<attribute name="OC_FARNELL" value="1137302" x="80" y="12.5" size="1.778" layer="28" rot="MR90" display="off"/>
 </element>
 <element name="R47" library="rcl" package="R0805" value="4K7" x="74.5" y="76" rot="MR180"/>
@@
 <wire x1="67.73" y1="76.25" x2="89" y2="77.0222" width="0" layer="19" extent="1-1"/>
 <wire x1="55.7" y1="64.25" x2="67.73" y2="76.25" width="0" layer="19" extent="1-1"/>
-<wire x1="63.6" y1="49.905" x2="55.7" y2="64.25" width="0" layer="19" extent="1-1"/>
-<wire x1="51.25" y1="43" x2="63.6" y2="49.905" width="0" layer="19" extent="1-16"/>
+<wire x1="64.9" y1="23.405" x2="55.7" y2="64.25" width="0" layer="19" extent="1-1"/>
 <wire x1="46.975" y1="23.13" x2="47" y2="23" width="0" layer="19" extent="1-1"/>
 <wire x1="7.5" y1="19.665" x2="7.5" y2="19.5" width="0" layer="19" extent="1-1"/>
@@
 <wire x1="95.05" y1="3.5" x2="95.55" y2="7" width="0" layer="19" extent="1-1"/>
 <wire x1="85.23" y1="33.8716" x2="86.5" y2="19.9778" width="0" layer="19" extent="1-1"/>
+<wire x1="51.25" y1="26.25" x2="46.975" y2="23.13" width="0" layer="19" extent="1-16"/>
+<wire x1="52.5" y1="46" x2="55.5" y2="49.905" width="0" layer="19" extent="1-16"/>
+<wire x1="53.25" y1="45" x2="51.25" y2="43" width="0.8" layer="16"/>
+<wire x1="64.9" y1="23.405" x2="61.905" y2="23.405" width="0" layer="19" extent="1-16"/>
+<wire x1="61.905" y1="23.405" x2="58.5" y2="20" width="0" layer="19" extent="1-16"/>
+<wire x1="58.5" y1="20" x2="58.5" y2="22" width="0" layer="19" extent="1-16"/>
+<wire x1="58.5" y1="22" x2="53.5" y2="24" width="0" layer="19" extent="1-16"/>
+<wire x1="53.5" y1="24" x2="52.25" y2="24" width="0.8" layer="16"/>
+<wire x1="52.25" y1="24" x2="51.5" y2="24.75" width="0.8" layer="16"/>
+<wire x1="51.25" y1="26.5" x2="51.25" y2="26.25" width="0" layer="19" extent="1-16"/>
+<wire x1="51.5" y1="24.75" x2="51.25" y2="26.5" width="0.8" layer="16"/>
+<wire x1="53.25" y1="45" x2="53.25" y2="45.25" width="0.8" layer="16"/>
+<wire x1="53.25" y1="45.25" x2="52.5" y2="46" width="0.8" layer="16"/>
 </signal>
 <signal name="VCC">
@@
 <contactref element="IC2" pad="7"/>
 <contactref element="R47" pad="2"/>
-<wire x1="58.4" y1="47.365" x2="58.4" y2="46.095" width="0.2" layer="1"/>
+<wire x1="70.1" y1="20.865" x2="70.1" y2="19.595" width="0.2" layer="16"/>
 <via x="74.25" y="65.75" extent="1-16" drill="0.6" shape="square"/>
 <via x="72.75" y="65.25" extent="1-16" drill="0.6" shape="square"/>
@@
 <wire x1="48" y1="24.5" x2="48.25" y2="24.75" width="0.2" layer="1"/>
 <wire x1="48.25" y1="24.75" x2="48.25" y2="26.75" width="0.2" layer="1"/>
-<wire x1="51.5" y1="25" x2="51.5" y2="25.75" width="0.8" layer="1"/>
+<wire x1="51.5" y1="24.75" x2="51.5" y2="25.75" width="0.8" layer="1"/>
 <wire x1="51.5" y1="25.75" x2="51.25" y2="26" width="0.8" layer="1"/>
 <wire x1="51.25" y1="26" x2="50.25" y2="26" width="0.8" layer="1"/>
@@
 <wire x1="74.25" y1="65.75" x2="75.45" y2="76" width="0" layer="19" extent="16-16"/>
 <wire x1="72.75" y1="65.25" x2="74.25" y2="65.75" width="0" layer="19" extent="1-1"/>
-<wire x1="58.4" y1="47.365" x2="72.75" y2="65.25" width="0" layer="19" extent="1-1"/>
+<wire x1="70.1" y1="20.865" x2="72.75" y2="65.25" width="0" layer="19" extent="1-1"/>
 <wire x1="49.25" y1="41" x2="52.925" y2="41.58" width="0" layer="19" extent="1-16"/>
-<wire x1="51.5" y1="24.75" x2="51.5" y2="25" width="0" layer="19" extent="1-1"/>
 <wire x1="47.5" y1="27" x2="48.25" y2="26.75" width="0" layer="19" extent="1-1"/>
 <wire x1="59.5" y1="11.5" x2="47.3196" y2="14.2164" width="0" layer="19" extent="16-16"/>
@@
 <wire x1="98.45" y1="24" x2="91.45" y2="7.5" width="0" layer="19" extent="1-16"/>
 <wire x1="97.45" y1="38.5" x2="98.45" y2="32.5" width="0" layer="19" extent="1-1"/>
-<wire x1="58.4" y1="46.095" x2="54.345" y2="46.095" width="0" layer="19" extent="1-16"/>
+<wire x1="70.1" y1="19.595" x2="54.345" y2="46.095" width="0" layer="19" extent="1-16"/>
 <wire x1="54.345" y1="46.095" x2="49.25" y2="41" width="0.8" layer="1"/>
 </signal>
@@
 <contactref element="JP1" pad="2"/>
 <wire x1="70.27" y1="76.25" x2="73.55" y2="76" width="0" layer="19" extent="16-16"/>
-<wire x1="63.6" y1="48.635" x2="70.27" y2="76.25" width="0" layer="19" extent="1-1"/>
+<wire x1="64.9" y1="22.135" x2="70.27" y2="76.25" width="0" layer="19" extent="1-1"/>
 </signal>
 <signal name="N$50">
