File: eagle/drutest/durtest4.sch (EAGLE design)
At the start: 76 parts, among them IC1 XCF02S, IC2 25LC080SN, Q5 BC848SMD, Q6 BC848SMD, Q7 BC848SMD, Q8 BC848SMD, T1 BSS138, T2 BC848, T3 BSS138, U1 XC3S400TQ144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

Commit message: sleepy
Parts:
- added R51: 2k2, resistor:R-EU_M0805
- added SJ2: (no value), jumper:SJ2W
Connections:
- new net N$66: R51.2, SJ2.2
- net SCART_MODE: now also R51.1
- net VCC: now also SJ2.1
- net VCCAUX: now also SJ2.3
Changed lines of the file:
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@@
 <part name="SUPPLY7" library="supply2" deviceset="GND" device=""/>
 <part name="R50" library="resistor" deviceset="R-EU_" device="M0805" value="2k2"/>
+<part name="R51" library="resistor" deviceset="R-EU_" device="M0805" value="2k2"/>
+<part name="SJ2" library="jumper" deviceset="SJ2W" device=""/>
 </parts>
 <sheets>
@@
 <instance part="SUPPLY7" gate="GND" x="96.52" y="-142.24"/>
 <instance part="R50" gate="G$1" x="259.08" y="-50.8" rot="MR0"/>
+<instance part="R51" gate="G$1" x="259.08" y="-60.96" rot="MR0"/>
+<instance part="SJ2" gate="G$1" x="246.38" y="-60.96" rot="R180"/>
 </instances>
 <busses>
@@
 <wire x1="-96.52" y1="-127" x2="-88.9" y2="-127" width="0.1524" layer="91"/>
 </segment>
+<segment>
+<wire x1="246.38" y1="-66.04" x2="246.38" y2="-71.12" width="0.1524" layer="91"/>
+<wire x1="246.38" y1="-71.12" x2="241.3" y2="-71.12" width="0.1524" layer="91"/>
+<label x="241.3" y="-71.12" size="1.778" layer="95"/>
+<pinref part="SJ2" gate="G$1" pin="1"/>
+</segment>
 </net>
 <net name="TCK" class="0">
@@
 <segment>
 <pinref part="R50" gate="G$1" pin="2"/>
-<wire x1="254" y1="-50.8" x2="241.3" y2="-50.8" width="0.1524" layer="91"/>
+<wire x1="254" y1="-50.8" x2="246.38" y2="-50.8" width="0.1524" layer="91"/>
 <label x="251.46" y="-50.8" size="1.778" layer="95" rot="MR0"/>
+<wire x1="246.38" y1="-50.8" x2="241.3" y2="-50.8" width="0.1524" layer="91"/>
+<wire x1="246.38" y1="-55.88" x2="246.38" y2="-50.8" width="0.1524" layer="91"/>
+<junction x="246.38" y="-50.8"/>
+<pinref part="SJ2" gate="G$1" pin="3"/>
 </segment>
 </net>
@@
 <wire x1="299.72" y1="2.54" x2="299.72" y2="10.16" width="0.1524" layer="91"/>
 <wire x1="299.72" y1="10.16" x2="332.74" y2="10.16" width="0.1524" layer="91"/>
+</segment>
+<segment>
+<wire x1="299.72" y1="-60.96" x2="264.16" y2="-60.96" width="0.1524" layer="91"/>
+<label x="299.72" y="-60.96" size="1.778" layer="95" rot="MR0"/>
+<pinref part="R51" gate="G$1" pin="1"/>
 </segment>
 </net>
@@
 </segment>
 </net>
+<net name="N$66" class="0">
+<segment>
+<pinref part="R51" gate="G$1" pin="2"/>
+<wire x1="254" y1="-60.96" x2="251.46" y2="-60.96" width="0.1524" layer="91"/>
+<pinref part="SJ2" gate="G$1" pin="2"/>
+</segment>
+</net>

Commit message: mah
Parts:
- added R52: 4K7, resistor:R-EU_M0805
- added RESET_SW: (no value), jumper:JP1Q
Connections:
- new net RESET: R52.2, RESET_SW.1, U1B5.IO_L31N_5D4
- net GND: now also RESET_SW.2
- net VCC: now also R52.1
Changed lines of the file:
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@@
 <part name="R51" library="resistor" deviceset="R-EU_" device="M0805" value="2k2"/>
 <part name="SJ2" library="jumper" deviceset="SJ2W" device=""/>
+<part name="RESET_SW" library="jumper" deviceset="JP1Q" device=""/>
+<part name="R52" library="resistor" deviceset="R-EU_" device="M0805" value="4K7"/>
 </parts>
 <sheets>
@@
 <instance part="R51" gate="G$1" x="259.08" y="-60.96" rot="MR0"/>
 <instance part="SJ2" gate="G$1" x="246.38" y="-60.96" rot="R180"/>
+<instance part="RESET_SW" gate="A" x="81.28" y="-76.2" rot="R90"/>
+<instance part="R52" gate="G$1" x="81.28" y="-83.82"/>
 </instances>
 <busses>
@@
 <pinref part="SUPPLY7" gate="GND" pin="GND"/>
 </segment>
+<segment>
+<pinref part="RESET_SW" gate="A" pin="2"/>
+<wire x1="73.66" y1="-76.2" x2="66.04" y2="-76.2" width="0.1524" layer="91"/>
+<label x="66.04" y="-76.2" size="1.778" layer="95"/>
+</segment>
 </net>
 <net name="VCC" class="0">
@@
 <pinref part="SJ2" gate="G$1" pin="1"/>
 </segment>
+<segment>
+<pinref part="R52" gate="G$1" pin="1"/>
+<wire x1="66.04" y1="-83.82" x2="76.2" y2="-83.82" width="0.1524" layer="91"/>
+<label x="66.04" y="-83.82" size="1.778" layer="95"/>
+</segment>
 </net>
 <net name="TCK" class="0">
@@
 <net name="N$50" class="0">
 <segment>
+<pinref part="U$2" gate="G$1" pin="OUT"/>
+<wire x1="162.56" y1="-68.58" x2="162.56" y2="-88.9" width="0.1524" layer="91"/>
 <pinref part="U1" gate="B5" pin="IO_L32P_5GCLK2"/>
 <wire x1="132.08" y1="-40.64" x2="132.08" y2="-68.58" width="0.1524" layer="91"/>
-<pinref part="U$2" gate="G$1" pin="OUT"/>
 <wire x1="132.08" y1="-68.58" x2="162.56" y2="-68.58" width="0.1524" layer="91"/>
-<wire x1="162.56" y1="-68.58" x2="162.56" y2="-88.9" width="0.1524" layer="91"/>
 </segment>
 </net>
@@
 </segment>
 </net>
+<net name="RESET" class="0">
+<segment>
+<pinref part="R52" gate="G$1" pin="2"/>
+<pinref part="RESET_SW" gate="A" pin="1"/>
+<wire x1="86.36" y1="-83.82" x2="88.9" y2="-83.82" width="0.1524" layer="91"/>
+<wire x1="88.9" y1="-83.82" x2="88.9" y2="-76.2" width="0.1524" layer="91"/>
+<pinref part="U1" gate="B5" pin="IO_L31N_5D4"/>
+<wire x1="88.9" y1="-76.2" x2="137.16" y2="-76.2" width="0.1524" layer="91"/>
+<wire x1="137.16" y1="-76.2" x2="137.16" y2="-40.64" width="0.1524" layer="91"/>
+<junction x="88.9" y="-76.2"/>
+<label x="93.98" y="-76.2" size="1.778" layer="95"/>
+</segment>
+</net>

Commit message: regulators etc
Connections:
- new net VCCAUX_R: REG2.5.VOUT2, U1BVCCAUX.VCCAUX1, U1BVCCAUX.VCCAUX2
- net VCCAUX: no longer U1BVCCAUX.VCCAUX1, U1BVCCAUX.VCCAUX2
Changed lines of the file:
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@@
 <net name="VCCAUX" class="0">
 <segment>
+<pinref part="U1" gate="BVCCAUX" pin="VCCAUX3"/>
+<wire x1="-154.94" y1="-73.66" x2="-152.4" y2="-73.66" width="0.1524" layer="91"/>
+<label x="-142.24" y="-73.66" size="1.778" layer="95"/>
 <pinref part="U1" gate="BVCCAUX" pin="VCCAUX0"/>
-<pinref part="U1" gate="BVCCAUX" pin="VCCAUX1"/>
-<wire x1="-154.94" y1="-66.04" x2="-154.94" y2="-68.58" width="0.1524" layer="91"/>
-<pinref part="U1" gate="BVCCAUX" pin="VCCAUX2"/>
-<wire x1="-154.94" y1="-68.58" x2="-154.94" y2="-71.12" width="0.1524" layer="91"/>
-<junction x="-154.94" y="-68.58"/>
-<pinref part="U1" gate="BVCCAUX" pin="VCCAUX3"/>
-<wire x1="-154.94" y1="-71.12" x2="-154.94" y2="-73.66" width="0.1524" layer="91"/>
-<junction x="-154.94" y="-71.12"/>
-<wire x1="-154.94" y1="-73.66" x2="-142.24" y2="-73.66" width="0.1524" layer="91"/>
-<junction x="-154.94" y="-73.66"/>
-<label x="-142.24" y="-73.66" size="1.778" layer="95"/>
+<wire x1="-152.4" y1="-73.66" x2="-142.24" y2="-73.66" width="0.1524" layer="91"/>
+<wire x1="-154.94" y1="-66.04" x2="-152.4" y2="-66.04" width="0.1524" layer="91"/>
+<wire x1="-152.4" y1="-66.04" x2="-152.4" y2="-73.66" width="0.1524" layer="91"/>
+<junction x="-152.4" y="-73.66"/>
 </segment>
 <segment>
@@
 </segment>
 </net>
+<net name="VCCAUX_R" class="0">
+<segment>
+<pinref part="REG2.5" gate="G$1" pin="VOUT2"/>
+<wire x1="-172.72" y1="53.34" x2="-167.64" y2="53.34" width="0.1524" layer="91"/>
+<label x="-167.64" y="53.34" size="1.778" layer="95"/>
+</segment>
+<segment>
+<pinref part="U1" gate="BVCCAUX" pin="VCCAUX1"/>
+<wire x1="-154.94" y1="-68.58" x2="-144.78" y2="-68.58" width="0.1524" layer="91"/>
+<wire x1="-144.78" y1="-68.58" x2="-144.78" y2="-71.12" width="0.1524" layer="91"/>
+<wire x1="-144.78" y1="-71.12" x2="-144.78" y2="-78.74" width="0.1524" layer="91"/>
+<wire x1="-144.78" y1="-78.74" x2="-142.24" y2="-78.74" width="0.1524" layer="91"/>
+<pinref part="U1" gate="BVCCAUX" pin="VCCAUX2"/>
+<wire x1="-154.94" y1="-71.12" x2="-144.78" y2="-71.12" width="0.1524" layer="91"/>
+<junction x="-144.78" y="-71.12"/>
+<label x="-142.24" y="-78.74" size="1.778" layer="95"/>
+</segment>
+</net>
