File: eagle/homeboard/homeboard2.sch (EAGLE design)
At the start: 81 parts, among them IC1 XCF02S, IC2 25LC080SN, Q5 BC848SMD, Q6 BC848SMD, Q7 BC848SMD, Q8 BC848SMD, T1 BSS138, T2 BC848, T3 BSS138, U1 XC3S400TQ144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

Commit message: mah
Connections:
- new net N$67: U1B6.IO_L23N_6
- new net N$73: U1B7.IO_L23P_7
- net N$1: now also U$1.A4, U1B2.IO_L01N_2VRP_2; no longer U$1.A3, U1B7.IO_L01P_7VRN_7
- net N$10: now also U$1.A17, U1B2.IO_L23P_2; no longer U$1.DQ5, U1B7.IO_L23P_7
- net N$11: now also U$1.WE, U1B2.IO_L24N_2; no longer U$1.DQ6, U1B7.IO_L23N_7
- net N$12: now also U$1.A13, U1B2.IO_L24P_2; no longer U$1.DQ7, U1B7.IO_L24P_7
- net N$13: now also U$1.A8, U1B2.IO_L40N_2; no longer U$1.A10, U1B7.IO_L24N_7
- net N$14: now also U$1.A9, U1B2.IO_L40P_2VREF_2; no longer U$1.OE, U1B7.IO_L40P_7
- net N$15: now also U1B3.IO_L40N_3VREF_3; no longer U1B7.IO_L40N_7VREF_7
- net N$16: now also U$1.A3, U1B3.IO_L01P_3VRN_3; no longer U$1.A9, U1B6.IO_L40P_6VREF_6
- net N$17: now also U$1.A2, U1B3.IO_L01N_3VRP_3; no longer U$1.A8, U1B6.IO_L40N_6
- net N$18: now also U$1.A1, U1B3.IO; no longer U$1.A13, U1B6.IO_L24P_6
- net N$19: now also U$1.A0, U1B3.IO_L20P_3; no longer U$1.WE, U1B6.IO_L24N_6VREF_6
- net N$2: now also U$1.A5, U1B2.IO_L01P_2VRN_2; no longer U$1.A2, U1B7.IO_L01N_7VRP_7
- net N$20: now also U$1.DQ0, U1B3.IO_L20N_3; no longer U$1.A17, U1B6.IO_L23P_6
- net N$21: now also U$1.DQ1, U1B3.IO_L21P_3; no longer U$1.A15, U1B6.IO_L23N_6
- net N$22: now also U$1.DQ2, U1B3.IO_L21N_3; no longer U$1.A18, U1B6.IO_L22P_6
- net N$23: now also U$1.DQ3, U1B3.IO_L22P_3; no longer U$1.A16, U1B6.IO_L22N_6
- net N$24: now also U$1.DQ4, U1B3.IO_L22N_3; no longer U$1.A14, U1B6.IO_L21P_6
- net N$25: now also U$1.DQ5, U1B3.IO_L23P_3VREF_3; no longer U$1.A12, U1B6.IO_L21N_6
- net N$26: now also U$1.DQ6, U1B3.IO_L23N_3; no longer U$1.A7, U1B6.IO_L20P_6
- net N$27: now also U$1.DQ7, U1B3.IO_L24P_3; no longer U$1.A6, U1B6.IO_L20N_6
- net N$28: now also U$1.A10, U1B3.IO_L24N_3; no longer U$1.A5, U1B6.IO_L01P_6VRN_6
- net N$29: now also U$1.OE, U1B3.IO_L40P_3; no longer U$1.A4, U1B6.IO_L01N_6VRP_6
- net N$3: now also U$1.A6, U1B2.IO_L20N_2; no longer U$1.A1, U1B7.IOVREF_7
- net N$4: now also U$1.A7, U1B2.IO_L20P_2; no longer U$1.A0, U1B7.IO_L20P_7
- net N$5: now also U$1.A12, U1B2.IO_L21N_2; no longer U$1.DQ0, U1B7.IO_L20N_7
- net N$6: now also U$1.A14, U1B2.IO_L21P_2; no longer U$1.DQ1, U1B7.IO_L21P_7
- net N$7: now also U$1.A16, U1B2.IO_L22N_2; no longer U$1.DQ2, U1B7.IO_L21N_7
- net N$8: now also U$1.A18, U1B2.IO_L22P_2; no longer U$1.DQ3, U1B7.IO_L22P_7
- net N$9: now also U$1.A15, U1B2.IO_L23N_2VREF_2; no longer U$1.DQ4, U1B7.IO_L22N_7
Other:
- moved on the sheet: JP3, U1B2, U1B3
