File: eagle/homeboard/homeboard4.brd (EAGLE design)
At the start: 100 x 80 mm, 81 parts, among them IC1 XCF02S, IC2 25LC080SN, Q5 BC848SMD, Q6 BC848SMD, Q7 BC848SMD, Q8 BC848SMD, T1 BSS138, T2 BC848, T3 BSS138, U1 XC3S400TQ144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

Commit message: stuff
Parts:
- moved IC2 48.5 mm to (6.35, 35.6)
- moved U$2 2.30 mm to (33.9, 26.6), turned to 0 degrees
- moved R29 1.77 mm to (42.5, 20.8), turned to 270 degrees
- moved R25 1.41 mm to (38.5, 19.8), turned to 180 degrees
Connections:
- new net X6: U1.P51
- new net X7: U1.P50
- new net X8: U1.P47
- new net X9: U1.P46
- net B0: now also U1.P68; no longer U1.P57
- net B1: now also U1.P63; no longer U1.P56
- net CLK16: now also U1.P56; no longer U1.P52
- net CSYNC: now also U1.P53; no longer U1.P46
- net FPGA_AUDIO_LEFT: now also U1.P69; no longer U1.P59
- net FPGA_AUDIO_RIGHT: now also U1.P70; no longer U1.P60
- net G0: now also U1.P60; no longer U1.P55
- net G1: now also U1.P59; no longer U1.P51
- net MISO: no longer U1.P63
- net MOSI: no longer U1.P69
- net R0: now also U1.P57; no longer U1.P50
- net R1: now also U1.P55; no longer U1.P47
- net RESET: now also U1.P52; no longer U1.P53
- net SCLK: no longer U1.P70
- net SPI_SEL0: no longer U1.P68
Routing:
- net GND: track 326.6 -> 263.2 mm, vias 23 -> 20
- net RESET: track 46.1 -> 0.00 mm, vias 1 -> 0
- net MISO: track 29.4 -> 0.00 mm, vias 1 -> 0
- net SPI_SEL0: track 26.2 -> 0.00 mm, vias 1 -> 0
- net CSYNC: track 22.7 -> 46.1 mm, vias 0 -> 1
- net R1: track 18.9 -> 0.00 mm
- net MOSI: track 15.3 -> 0.00 mm, vias 1 -> 0
- net SCLK: track 13.8 -> 0.00 mm, vias 1 -> 0
- net VCC: track 274.7 -> 262.3 mm, vias 8 -> 7
- net R0: track 17.9 -> 25.8 mm
- net N$49: track 6.06 -> 0.00 mm
- net B0: track 23.3 -> 19.3 mm
- net B1: track 22.2 -> 18.6 mm
- net FPGA_AUDIO_RIGHT: track 31.1 -> 28.7 mm
- net CLK16: track 9.00 -> 11.1 mm
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