File: eagle/homeboard/homeboard4.sch (EAGLE design)
At the start: 81 parts, among them IC1 XCF02S, IC2 25LC080SN, Q5 BC848SMD, Q6 BC848SMD, Q7 BC848SMD, Q8 BC848SMD, T1 BSS138, T2 BC848, T3 BSS138, U1 XC3S400TQ144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

Commit message: stuff
Connections:
- new net X6: U1B5.IO_L31N_5D4
- new net X7: U1B5.IO_L31P_5D5
- new net X8: U1B5.IO_L28N_5D6
- new net X9: U1B5.IO_L28P_5D7
- net B0: now also U1B4.IO_L01P_4VRN_4; no longer U1B4.IO_L31P_4DOUTBUSY
- net B1: now also U1B4.IO_L27P_4D1; no longer U1B4.IO_L32N_4GCLK1
- net CLK16: now also U1B4.IO_L32N_4GCLK1; no longer U1B5.IO_L32P_5GCLK2
- net CSYNC: now also U1B5.IO_L32N_5GCLK3; no longer U1B5.IO_L28P_5D7
- net FPGA_AUDIO_LEFT: now also U1B4.IO_L01N_4VRP_4; no longer U1B4.IO_L30P_4D3
- net FPGA_AUDIO_RIGHT: now also U1B4.IOVREF_4; no longer U1B4.IO_L30N_4D2
- net G0: now also U1B4.IO_L30N_4D2; no longer U1B4.IO_L32P_4GCLK0
- net G1: now also U1B4.IO_L30P_4D3; no longer U1B5.IO_L31N_5D4
- net MISO: no longer U1B4.IO_L27P_4D1
- net MOSI: no longer U1B4.IO_L01N_4VRP_4
- net R0: now also U1B4.IO_L31P_4DOUTBUSY; no longer U1B5.IO_L31P_5D5
- net R1: now also U1B4.IO_L32P_4GCLK0; no longer U1B5.IO_L28N_5D6
- net RESET: now also U1B5.IO_L32P_5GCLK2; no longer U1B5.IO_L32N_5GCLK3
- net SCLK: no longer U1B4.IOVREF_4
- net SPI_SEL0: no longer U1B4.IO_L01P_4VRN_4
