File: eagle/homeboard/homeboard5.brd (EAGLE design)
At the start: 100 x 80 mm, 81 parts, among them IC1 XCF02S, IC2 25LC080SN, Q5 BC848SMD, Q6 BC848SMD, Q7 BC848SMD, Q8 BC848SMD, T1 BSS138, T2 BC848, T3 BSS138, U1 XC3S400TQ144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

Commit message: rework
Parts:
- removed R47: 4K7, rcl:R0805
- removed WR_PROT: (no value), jumper:JP1
- moved IC2 17.0 mm to (13.1, 23.6), flipped to the top
- moved U$2 0.35 mm to (22.1, 25.9), turned to 180 degrees
Connections:
- net SPI_SEL0 renamed FL_SEL
- removed net N$49: IC2.3, R47.1, WR_PROT.2
- new net FL_DI: IC2.5
- new net FL_DO: IC2.2
- new net FL_HOLD: IC2.7
- new net FL_SCLK: IC2.6
- new net FL_WP: IC2.3
- net GND: no longer WR_PROT.1
- net MISO: no longer IC2.2
- net MOSI: no longer IC2.5
- net SCLK: no longer IC2.6
- net VCC: no longer IC2.7, R47.2
Routing:
- net RESET: track 0.00 -> 18.7 mm
- net CLK16: track 10.0 -> 23.7 mm
- net VCC: track 236.3 -> 235.0 mm
- net VCCAUX: track 25.5 -> 24.3 mm
- net G1: track 22.1 -> 22.7 mm

Commit message: rework
Parts:
- removed R51: 2k2, resistor:M0805
- removed SJ2: (no value), jumper:SJ_2
- moved JP3 79.2 mm to (40.0, 76.0)
- moved R52 74.6 mm to (13.0, 31.5)
- moved RESET_SW 61.5 mm to (20.5, 34.5)
- moved IC1 26.2 mm to (64.1, 16.2), flipped to the top, turned to 90 degrees
- moved IC2 3.54 mm to (9.65, 24.1)
- moved U$1 3.00 mm to (57.2, 47.7)
- moved U$2 2.75 mm to (24.9, 25.9), turned to 270 degrees
Connections:
- removed net N$66: R51.2, SJ2.2
- net CLK16: now also U1.P55; no longer U1.P53
- net CSYNC: now also U1.P53; no longer U1.P55
- net SCART_MODE: no longer R51.1
- net VCC: no longer SJ2.1
- net VCCAUX: no longer SJ2.3
Routing:
- net GND: track 234.6 -> 269.1 mm, vias 19 -> 20
- net CSYNC: track 30.4 -> 0.00 mm
- net CLK16: track 23.7 -> 0.00 mm
- net PROM_INITB: track 24.5 -> 39.4 mm, vias 1 -> 2
- net VCC: track 235.0 -> 220.9 mm
- net N$35: track 10.3 -> 24.0 mm, vias 1 -> 0
- net N$40: track 22.1 -> 30.2 mm
- net TCK: track 22.7 -> 29.1 mm
- net N$38: track 16.2 -> 22.1 mm, vias 1 -> 0
- net TMS: track 23.7 -> 28.6 mm
- net TDI: track 24.8 -> 28.1 mm
- net N$9: track 16.9 -> 13.9 mm
- net N$8: track 15.4 -> 12.4 mm
- net N$7: track 14.4 -> 11.4 mm
- net N$6: track 12.9 -> 9.92 mm
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
Commit message: rework
Parts:
- moved R50 43.8 mm to (39.2, 20.8), turned to 90 degrees
- moved R52 12.4 mm to (3.50, 39.5)
- moved RESET_SW 11.1 mm to (14.0, 43.5)
- moved U$2 8.14 mm to (17.1, 23.4), turned to 0 degrees
- moved IC2 4.01 mm to (9.90, 28.1), turned to 0 degrees
- moved R24 1.25 mm to (34.0, 20.8)
- moved R25 1.25 mm to (36.2, 20.8)
Connections:
- removed net X7: U1.P50
- removed net X8: U1.P47
- removed net X9: U1.P46
- removed net XG1: U1.P44
- removed net XR0: U1.P41
- removed net XR1: U1.P40
- net CLK16: now also U1.P53; no longer U1.P55
- net CSYNC: now also U1.P55; no longer U1.P53
- net FL_DI: now also U1.P40
- net FL_DO: now also U1.P47
- net FL_HOLD: now also U1.P44
- net FL_SCLK: now also U1.P41
- net FL_SEL: now also U1.P46
- net FL_WP: now also U1.P50
- net VCCAUX: no longer R50.2
- net VCCAUX_R: now also R50.2
Routing:
- net VCC: track 220.9 -> 284.3 mm, vias 6 -> 7
- net FL_SEL: track 0.00 -> 37.6 mm
- net FL_WP: track 0.00 -> 37.2 mm
- net FL_DO: track 0.00 -> 37.1 mm
- net FL_HOLD: track 0.00 -> 34.9 mm
- net FL_SCLK: track 0.00 -> 31.3 mm
- net CSYNC: track 0.00 -> 31.2 mm
- net CLK16: track 0.00 -> 30.9 mm
- net FL_DI: track 0.00 -> 28.6 mm
- net SCART_BLANKING: track 0.00 -> 27.6 mm
- net GND: track 269.1 -> 293.1 mm, vias 20 -> 22
- net RESET: track 18.7 -> 0.00 mm
- net VCCAUX_R: track 24.2 -> 42.2 mm
- net N$36: track 26.5 -> 38.8 mm
- net PROM_DO: track 20.6 -> 28.3 mm
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
Commit message: pre-shift down
Parts:
- moved RESET_SW 29.1 mm to (6.00, 15.5), turned to 180 degrees
- moved R52 24.0 mm to (2.50, 15.5), turned to 90 degrees
- moved IC2 5.52 mm to (4.40, 27.6)
- moved U$2 4.47 mm to (13.1, 21.4)
- moved REG1.2 3.61 mm to (35.5, 47.0)
- moved REG2.5 3.61 mm to (40.0, 41.8)
- moved U$1 3.61 mm to (55.2, 44.7)
- moved U1 3.61 mm to (37.7, 44.3)
Routing:
- net GND: track 293.1 -> 367.1 mm, vias 22 -> 23
- net RESET: track 0.00 -> 46.9 mm, vias 0 -> 1
- net N$36: track 38.8 -> 17.3 mm
- net VCC: track 284.3 -> 300.6 mm, vias 7 -> 8
- net TDI: track 28.1 -> 13.2 mm
- net TMS: track 28.6 -> 14.3 mm
- net TCK: track 29.1 -> 15.3 mm
- net N$40: track 30.2 -> 16.4 mm
- net N$35: track 21.1 -> 27.7 mm
- net VCCAUX_R: track 42.2 -> 37.4 mm
- net CSYNC: track 31.2 -> 26.6 mm
- net G0: track 20.2 -> 15.7 mm
- net G1: track 22.2 -> 18.0 mm
- net R1: track 25.8 -> 21.7 mm
- net R0: track 23.6 -> 19.9 mm
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
Commit message: post-shift down
Parts:
- moved REG1.2 3.00 mm to (35.5, 44.0)
- moved REG2.5 3.00 mm to (40.0, 38.8)
- moved U$1 3.00 mm to (55.2, 41.7)
- moved U1 3.00 mm to (37.7, 41.3)
Routing:
- net VCC: track 300.6 -> 304.9 mm
- net RESET: track 46.9 -> 43.9 mm
- net FL_SEL: track 39.0 -> 36.0 mm
- net FL_HOLD: track 36.0 -> 33.0 mm
- net R1: track 21.7 -> 18.7 mm
- net FL_SCLK: track 32.3 -> 29.3 mm
- net FL_DO: track 38.0 -> 35.0 mm
- net FL_DI: track 29.7 -> 26.7 mm
- net CSYNC: track 26.6 -> 23.6 mm
- net CLK16: track 31.6 -> 28.6 mm
- net G1: track 18.0 -> 15.0 mm
- net R0: track 19.9 -> 16.9 mm
- net N$35: track 27.7 -> 24.7 mm
- net G0: track 15.7 -> 12.7 mm
- net FPGA_AUDIO_RIGHT: track 16.0 -> 13.0 mm
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
Commit message: rework
Parts:
- moved IC1 2.50 mm to (64.1, 18.7)
- moved R52 2.00 mm to (2.50, 17.5), turned to 270 degrees
- moved U$2 1.12 mm to (13.6, 22.4)
Routing:
- net VCC: track 304.9 -> 298.4 mm
- net GND: track 364.1 -> 360.1 mm
- net PROM_INITB: track 40.1 -> 37.6 mm
- net TMS: track 14.3 -> 11.8 mm
- net TDI: track 13.2 -> 10.7 mm
- net TCK: track 15.3 -> 12.8 mm
- net PROM_DO: track 24.0 -> 21.5 mm
- net N$40: track 16.4 -> 13.9 mm
- net N$38: track 24.1 -> 21.6 mm
- net N$36: track 14.3 -> 11.8 mm
- net N$35: track 24.7 -> 22.2 mm
- net RESET: track 43.9 -> 45.7 mm
- net N$65: track 7.46 -> 8.29 mm

Commit message: mah
Parts:
- moved X4 86.6 mm to (80.0, 17.5), turned to 270 degrees
- moved X5 82.4 mm to (86.0, 33.5), turned to 270 degrees
- moved JP3 49.0 mm to (84.0, 54.5), turned to 270 degrees
- moved R1 11.0 mm to (19.7, 61.2)
- moved R2 11.0 mm to (37.1, 61.7)
- moved R3 11.0 mm to (34.2, 61.7)
- moved U$3 10.5 mm to (61.0, 66.0), turned to 315 degrees
- moved RESET_SW 2.75 mm to (6.00, 18.2), turned to 270 degrees
- moved R52 0.90 mm to (2.00, 18.2)
- moved C1 0.25 mm to (49.5, 17.0)
- moved C3 0.25 mm to (47.2, 12.2)
- moved C4 0.25 mm to (52.0, 11.8)
- moved C5 0.25 mm to (53.0, 17.0)
- moved IC1 0.25 mm to (64.1, 18.5)
- moved IC2 0.25 mm to (4.40, 27.4)
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Routing:
- net VCC: track 298.4 -> 380.6 mm
- net RESET: track 45.7 -> 42.9 mm
- net R1: track 18.7 -> 16.5 mm
- net CSYNC: track 23.6 -> 21.3 mm
- net PROM_INITB: track 37.6 -> 39.7 mm
- net G1: track 15.0 -> 12.9 mm
- net CLK16: track 28.5 -> 26.8 mm
- net N$38: track 21.6 -> 23.3 mm
- net R0: track 16.9 -> 15.2 mm
- net FL_WP: track 35.2 -> 34.1 mm
- net GND: track 360.1 -> 361.1 mm
- net FPGA_AUDIO_RIGHT: track 13.0 -> 13.9 mm
- net FL_SEL: track 36.0 -> 35.1 mm
- net FL_DO: track 35.0 -> 34.2 mm
- net B0: track 9.55 -> 8.85 mm
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
Commit message: mah
Routing:
- net VCC: track 380.6 -> 386.6 mm
Changed lines of the file:
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@@
 <wire x1="10" y1="19.25" x2="9.5" y2="19.25" width="0.254" layer="1"/>
 <wire x1="9.5" y1="19.25" x2="8.5" y2="20.25" width="0.254" layer="1"/>
-<wire x1="55.5" y1="51.17" x2="55.5" y2="54.25" width="0.254" layer="1"/>
+<wire x1="55.5" y1="51.17" x2="55.5" y2="52.5" width="0.254" layer="1"/>
+<wire x1="55.5" y1="52.5" x2="55.5" y2="54.25" width="0.254" layer="1"/>
 <wire x1="55.5" y1="54.25" x2="52.5" y2="57.25" width="0.254" layer="1"/>
 <wire x1="8.5" y1="20.25" x2="11.5" y2="23.25" width="0.254" layer="1"/>
@@
 <wire x1="1" y1="20.25" x2="1" y2="20.2" width="0.254" layer="1"/>
 <wire x1="1" y1="20.2" x2="2" y2="19.2" width="0.254" layer="1"/>
+<wire x1="49.845" y1="53.345" x2="54.655" y2="53.345" width="0.254" layer="1"/>
+<wire x1="54.655" y1="53.345" x2="55.5" y2="52.5" width="0.254" layer="1"/>
 <wire x1="90.9" y1="64.5" x2="92.45" y2="68" width="0" layer="19" extent="1-16"/>
 <wire x1="73.984" y1="67.5094" x2="90.9" y2="64.5" width="0" layer="19" extent="1-16"/>
 <wire x1="72" y1="72.55" x2="72.0094" y2="72.5094" width="0" layer="19" extent="16-16"/>
-<wire x1="21.5" y1="57.25" x2="72" y2="66" width="0" layer="19" extent="1-1"/>
-<wire x1="49.845" y1="53.345" x2="52.5" y2="57.25" width="0" layer="19" extent="1-1"/>
-<wire x1="45.5" y1="33.33" x2="45.75" y2="33.25" width="0" layer="19" extent="1-1"/>
-<wire x1="71.5" y1="46.5" x2="21.5" y2="57.25" width="0" layer="19" extent="1-1"/>
 <wire x1="97.45" y1="47" x2="90.9" y2="64.5" width="0" layer="19" extent="1-1"/>
 <wire x1="98.45" y1="32.5" x2="97.45" y2="38.5" width="0" layer="19" extent="1-1"/>
+<wire x1="71.5" y1="46.5" x2="72" y2="66" width="0" layer="19" extent="1-1"/>
+<wire x1="55.5" y1="51.17" x2="71.5" y2="46.5" width="0" layer="19" extent="1-1"/>
+<wire x1="45.5" y1="33.33" x2="45.75" y2="33.25" width="0" layer="19" extent="1-1"/>
 </signal>
 <signal name="TCK">
