File: eagle/homeboard/homeboard7.sch (EAGLE design)
At the start: 77 parts, among them IC1 XCF02S, IC2 25LC080SN, IC3 ATMEGA32U2-TQFP, Q5 BC848SMD, Q6 BC848SMD, Q7 BC848SMD, Q8 BC848SMD, T1 BSS138, T2 BC848, T3 BSS138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

Commit message: need to stop changing my mind
Connections:
- removed net X6: U1B5.IO_L31N_5D4
- new net XX: U1B4.IO_L31P_4DOUTBUSY
- net CLK16: now also U1B4.IO_L32P_4GCLK0; no longer U1B5.IO_L32N_5GCLK3
- net CSYNC: now also U1B5.IO_L31N_5D4; no longer U1B4.IO_L32P_4GCLK0
- net FL_SEL: now also U1B5.IO_L28P_5D7; no longer U1B5.IO_L31P_5D5
- net FL_WP: now also U1B5.IO_L31P_5D5; no longer U1B5.IO_L28P_5D7
- net R0: now also U1B5.IO_L32N_5GCLK3; no longer U1B4.IO_L31P_4DOUTBUSY
- net R1: now also U1B5.IO_L32P_5GCLK2; no longer U1B4.IO_L32N_4GCLK1
- net RESET: now also U1B4.IO_L32N_4GCLK1; no longer U1B5.IO_L32P_5GCLK2
Changed lines of the file:
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@@
 </segment>
 <segment>
-<pinref part="U1" gate="B4" pin="IO_L32N_4GCLK1"/>
-<wire x1="185.42" y1="-76.2" x2="160.02" y2="-76.2" width="0.1524" layer="91"/>
-<wire x1="160.02" y1="-76.2" x2="160.02" y2="-40.64" width="0.1524" layer="91"/>
-<label x="185.42" y="-76.2" size="1.778" layer="95"/>
+<wire x1="106.68" y1="-71.12" x2="132.08" y2="-71.12" width="0.1524" layer="91"/>
+<label x="106.68" y="-71.12" size="1.778" layer="95"/>
+<pinref part="U1" gate="B5" pin="IO_L32P_5GCLK2"/>
+<wire x1="132.08" y1="-40.64" x2="132.08" y2="-71.12" width="0.1524" layer="91"/>
 </segment>
 </net>
@@
 </segment>
 <segment>
-<pinref part="U1" gate="B4" pin="IO_L31P_4DOUTBUSY"/>
-<wire x1="185.42" y1="-73.66" x2="177.8" y2="-73.66" width="0.1524" layer="91"/>
-<wire x1="177.8" y1="-73.66" x2="177.8" y2="-40.64" width="0.1524" layer="91"/>
-<label x="185.42" y="-73.66" size="1.778" layer="95"/>
+<pinref part="U1" gate="B5" pin="IO_L32N_5GCLK3"/>
+<wire x1="129.54" y1="-40.64" x2="129.54" y2="-73.66" width="0.1524" layer="91"/>
+<wire x1="106.68" y1="-73.66" x2="129.54" y2="-73.66" width="0.1524" layer="91"/>
+<label x="106.68" y="-73.66" size="1.778" layer="95"/>
 </segment>
 </net>
@@
 </segment>
 <segment>
-<wire x1="185.42" y1="-78.74" x2="162.56" y2="-78.74" width="0.1524" layer="91"/>
-<wire x1="162.56" y1="-78.74" x2="162.56" y2="-40.64" width="0.1524" layer="91"/>
-<pinref part="U1" gate="B4" pin="IO_L32P_4GCLK0"/>
-<label x="185.42" y="-78.74" size="1.778" layer="95"/>
+<pinref part="U1" gate="B5" pin="IO_L31N_5D4"/>
+<wire x1="137.16" y1="-40.64" x2="137.16" y2="-68.58" width="0.1524" layer="91"/>
+<wire x1="137.16" y1="-68.58" x2="106.68" y2="-68.58" width="0.1524" layer="91"/>
+<label x="106.68" y="-68.58" size="1.778" layer="95"/>
 </segment>
 </net>
@@
 </segment>
 <segment>
-<pinref part="U1" gate="B5" pin="IO_L31P_5D5"/>
-<wire x1="106.68" y1="-66.04" x2="134.62" y2="-66.04" width="0.1524" layer="91"/>
-<wire x1="134.62" y1="-66.04" x2="134.62" y2="-40.64" width="0.1524" layer="91"/>
-<label x="106.68" y="-66.04" size="1.778" layer="95"/>
+<pinref part="U1" gate="B5" pin="IO_L28P_5D7"/>
+<wire x1="106.68" y1="-60.96" x2="139.7" y2="-60.96" width="0.1524" layer="91"/>
+<wire x1="139.7" y1="-60.96" x2="139.7" y2="-40.64" width="0.1524" layer="91"/>
+<label x="106.68" y="-60.96" size="1.778" layer="95"/>
 </segment>
 </net>
@@
 </segment>
 <segment>
-<wire x1="106.68" y1="-71.12" x2="132.08" y2="-71.12" width="0.1524" layer="91"/>
-<label x="106.68" y="-71.12" size="1.778" layer="95"/>
-<pinref part="U1" gate="B5" pin="IO_L32P_5GCLK2"/>
-<wire x1="132.08" y1="-40.64" x2="132.08" y2="-71.12" width="0.1524" layer="91"/>
+<pinref part="U1" gate="B4" pin="IO_L32N_4GCLK1"/>
+<wire x1="185.42" y1="-76.2" x2="160.02" y2="-76.2" width="0.1524" layer="91"/>
+<wire x1="160.02" y1="-76.2" x2="160.02" y2="-40.64" width="0.1524" layer="91"/>
+<label x="185.42" y="-76.2" size="1.778" layer="95"/>
 </segment>
 </net>
@@
 </segment>
 <segment>
-<pinref part="U1" gate="B5" pin="IO_L32N_5GCLK3"/>
-<wire x1="129.54" y1="-40.64" x2="129.54" y2="-73.66" width="0.1524" layer="91"/>
-<wire x1="106.68" y1="-73.66" x2="129.54" y2="-73.66" width="0.1524" layer="91"/>
-<label x="106.68" y="-73.66" size="1.778" layer="95"/>
+<wire x1="185.42" y1="-78.74" x2="162.56" y2="-78.74" width="0.1524" layer="91"/>
+<wire x1="162.56" y1="-78.74" x2="162.56" y2="-40.64" width="0.1524" layer="91"/>
+<pinref part="U1" gate="B4" pin="IO_L32P_4GCLK0"/>
+<label x="185.42" y="-78.74" size="1.778" layer="95"/>
 </segment>
 </net>
@@
 </segment>
 </net>
-<net name="X6" class="0">
-<segment>
-<pinref part="U1" gate="B5" pin="IO_L31N_5D4"/>
-<wire x1="137.16" y1="-40.64" x2="137.16" y2="-68.58" width="0.1524" layer="91"/>
-<wire x1="137.16" y1="-68.58" x2="106.68" y2="-68.58" width="0.1524" layer="91"/>
-<label x="106.68" y="-68.58" size="1.778" layer="95"/>
-</segment>
-</net>
 <net name="FL_HOLD" class="0">
 <segment>
@@
 </segment>
 <segment>
-<pinref part="U1" gate="B5" pin="IO_L28P_5D7"/>
-<wire x1="106.68" y1="-60.96" x2="139.7" y2="-60.96" width="0.1524" layer="91"/>
-<wire x1="139.7" y1="-60.96" x2="139.7" y2="-40.64" width="0.1524" layer="91"/>
-<label x="106.68" y="-60.96" size="1.778" layer="95"/>
+<pinref part="U1" gate="B5" pin="IO_L31P_5D5"/>
+<wire x1="106.68" y1="-66.04" x2="134.62" y2="-66.04" width="0.1524" layer="91"/>
+<wire x1="134.62" y1="-66.04" x2="134.62" y2="-40.64" width="0.1524" layer="91"/>
+<label x="106.68" y="-66.04" size="1.778" layer="95"/>
 </segment>
 </net>
@@
 </segment>
 </net>
+<net name="XX" class="0">
+<segment>
+<pinref part="U1" gate="B4" pin="IO_L31P_4DOUTBUSY"/>
+<wire x1="185.42" y1="-73.66" x2="177.8" y2="-73.66" width="0.1524" layer="91"/>
+<wire x1="177.8" y1="-73.66" x2="177.8" y2="-40.64" width="0.1524" layer="91"/>
+<label x="185.42" y="-73.66" size="1.778" layer="95"/>
+</segment>
+</net>
