File: eagle/homeboard/homeboard8.brd (EAGLE design)
At the start: 100 x 80 mm, 77 parts, among them IC1 XCF02S, IC2 25LC080SN, IC3 ATMEGA32U2-TQFP, Q5 BC848SMD, Q6 BC848SMD, Q7 BC848SMD, Q8 BC848SMD, T1 BSS138, T2 BC848, T3 BSS138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

Commit message: need to stop changing my mind
Parts:
- moved JP3 44.3 mm to (60.5, 17.0), turned to 0 degrees
- moved IC2 26.1 mm to (4.40, 27.4), turned to 0 degrees
- moved IC3 16.6 mm to (61.0, 58.0)
- moved REG1.2 13.0 mm to (35.5, 43.8)
- moved REG2.5 13.0 mm to (40.0, 38.5)
- moved U$1 13.0 mm to (55.2, 41.4)
- moved U1 13.0 mm to (37.7, 41.1)
- moved R1 9.00 mm to (19.7, 61.2)
- moved R2 9.00 mm to (37.1, 61.7)
- moved R3 9.00 mm to (34.2, 61.7)
- moved IC1 5.10 mm to (63.1, 23.5)
Connections:
- net FL_SEL: now also U1.P46; no longer U1.P50
- net FL_WP: now also U1.P50; no longer U1.P46
Routing:
- net VCC: track 335.3 -> 379.9 mm, vias 7 -> 8
- net GND: track 338.5 -> 368.3 mm, vias 22 -> 23
- net PROM_INITB: track 52.7 -> 23.8 mm
- net FL_WP: track 7.85 -> 34.1 mm
- net FL_DO: track 9.75 -> 34.2 mm
- net FL_SEL: track 12.3 -> 35.1 mm
- net N$35: track 35.1 -> 12.9 mm
- net N$38: track 36.3 -> 16.7 mm
- net FL_HOLD: track 12.8 -> 32.4 mm
- net FL_SCLK: track 9.94 -> 29.3 mm
- net FL_DI: track 8.03 -> 26.7 mm
- net PROM_DO: track 33.8 -> 19.4 mm
- net R1: track 29.5 -> 16.5 mm
- net R0: track 28.2 -> 15.2 mm
- net FPGA_AUDIO_RIGHT: track 26.9 -> 13.9 mm
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
Commit message: rework
Parts:
- moved JP3 1.50 mm to (60.5, 18.5), turned to 90 degrees
Routing:
- net TCK: track 18.7 -> 25.6 mm
- net TMS: track 18.4 -> 24.8 mm
- net GND: track 368.3 -> 371.0 mm, vias 23 -> 24
- net FPGA_AUDIO_LEFT: track 11.3 -> 9.43 mm
- net FPGA_AUDIO_RIGHT: track 13.9 -> 12.4 mm
Changed lines of the file:
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@@
 <element name="REG2.5" library="cpcfpga" package="SOT223" value="2.5V" x="40" y="38.5" rot="MR270"/>
 <element name="REG1.2" library="cpcfpga" package="SOT223" value="1.2V" x="35.5" y="43.75" rot="MR90"/>
-<element name="JP3" library="pinhead" package="2X03" value="" x="60.5" y="17"/>
+<element name="JP3" library="pinhead" package="2X03" value="" x="60.5" y="18.5" rot="R90"/>
 <element name="X4" library="con-subd" package="F09HP" value="" x="80" y="17.5" rot="R270">
 <attribute name="OC_NEWARK" value="unknown" x="80" y="17.5" size="1.778" layer="27" rot="R270" display="off"/>
@@
 <wire x1="65" y1="22.25" x2="65" y2="14" width="0.254" layer="1"/>
 <wire x1="65" y1="14" x2="55.5" y2="14" width="0.254" layer="1"/>
-<wire x1="55.5" y1="14" x2="55.5" y2="10.75" width="0.254" layer="1"/>
 <wire x1="55.5" y1="10.75" x2="50.25" y2="10.75" width="0.254" layer="1"/>
 <wire x1="50.25" y1="10.75" x2="50" y2="10.75" width="0.254" layer="1"/>
@@
 <wire x1="63" y1="21.25" x2="67.25" y2="21.25" width="0.254" layer="16"/>
 <wire x1="67.25" y1="21.25" x2="67.5" y2="21" width="0.254" layer="16"/>
+<wire x1="55.5" y1="10.75" x2="55.5" y2="11" width="0.254" layer="1"/>
+<wire x1="55.5" y1="11" x2="55" y2="11.5" width="0.254" layer="1"/>
+<via x="55" y="11.5" extent="1-16" drill="0.6" shape="square"/>
+<wire x1="55" y1="11.5" x2="57" y2="11.5" width="0.254" layer="16"/>
+<wire x1="55.5" y1="14" x2="55.5" y2="11" width="0.254" layer="1"/>
 <wire x1="96.05" y1="71" x2="95.55" y2="76" width="0" layer="19" extent="1-1"/>
 <wire x1="96.55" y1="67.5" x2="96.05" y2="71" width="0" layer="19" extent="1-1"/>
@@
 <wire x1="38" y1="31.75" x2="38" y2="33.75" width="0.254" layer="1"/>
 <wire x1="36.5" y1="21.85" x2="28.75" y2="21.85" width="0.254" layer="16"/>
-<wire x1="44" y1="21.85" x2="44" y2="23.75" width="0.254" layer="16"/>
+<wire x1="44" y1="21.85" x2="44" y2="22.75" width="0.254" layer="16"/>
 <via x="44" y="23.75" extent="1-16" drill="0.6" shape="square"/>
 <wire x1="44" y1="23.75" x2="44" y2="27.75" width="0.254" layer="1"/>
@@
 <wire x1="62.087409375" y1="29.337409375" x2="62" y2="29.25" width="0.254" layer="1"/>
 <wire x1="62" y1="29.25" x2="62" y2="22.75" width="0.254" layer="1"/>
-<wire x1="62" y1="22.75" x2="54" y2="22.75" width="0.254" layer="1"/>
-<wire x1="44" y1="23.75" x2="52.75" y2="23.75" width="0.254" layer="16"/>
-<wire x1="53.75" y1="22.75" x2="54" y2="22.75" width="0.254" layer="16"/>
-<via x="54" y="22.75" extent="1-16" drill="0.6" shape="square"/>
+<wire x1="62" y1="22.75" x2="53" y2="22.75" width="0.254" layer="1"/>
+<wire x1="44" y1="23.75" x2="44" y2="22.75" width="0.254" layer="16"/>
+<via x="53" y="22.75" extent="1-16" drill="0.6" shape="square"/>
 <wire x1="2.491446875" y1="29.9609125" x2="1.7109125" y2="29.9609125" width="0.254" layer="1"/>
 <wire x1="1.7109125" y1="29.9609125" x2="1" y2="29.25" width="0.254" layer="1"/>
@@
 <wire x1="49.845" y1="53.345" x2="54.655" y2="53.345" width="0.254" layer="1"/>
 <wire x1="54.655" y1="53.345" x2="55.5" y2="52.5" width="0.254" layer="1"/>
-<wire x1="53.75" y1="22.75" x2="52.75" y2="23.75" width="0.254" layer="16"/>
+<wire x1="53" y1="22.75" x2="44" y2="22.75" width="0.254" layer="16"/>
 <wire x1="90.9" y1="64.5" x2="92.45" y2="68" width="0" layer="19" extent="1-16"/>
 <wire x1="73.984" y1="67.5094" x2="90.9" y2="64.5" width="0" layer="19" extent="1-16"/>
@@
 <wire x1="60.337409375" y1="26.087409375" x2="60.5" y2="26.25" width="0.254" layer="1"/>
 <via x="60.5" y="26.75" extent="1-16" drill="0.6" shape="square"/>
-<wire x1="60.5" y1="26.75" x2="60.5" y2="24" width="0.254" layer="16"/>
+<wire x1="60.5" y1="26.75" x2="60.5" y2="26.25" width="0.254" layer="16"/>
 <wire x1="60.5" y1="26.25" x2="60.5" y2="26.75" width="0.254" layer="1"/>
 <wire x1="56.943396875" y1="26.087409375" x2="60.75" y2="26.087409375" width="0.254" layer="1"/>
@@
 <wire x1="60.5" y1="26.25" x2="60.587409375" y2="26.25" width="0.254" layer="1"/>
 <wire x1="60.587409375" y1="26.25" x2="60.75" y2="26.087409375" width="0.254" layer="1"/>
+<wire x1="60.5" y1="26.25" x2="60.25" y2="26" width="0.254" layer="16"/>
+<wire x1="60.25" y1="26" x2="55.5" y2="26" width="0.254" layer="16"/>
+<wire x1="55.5" y1="26" x2="55.25" y2="25.75" width="0.254" layer="16"/>
+<wire x1="55.25" y1="25.75" x2="55.25" y2="22" width="0.254" layer="16"/>
 <wire x1="61" y1="37" x2="37.0824" y2="62.6999" width="0" layer="19" extent="1-16"/>
-<wire x1="57.96" y1="15.73" x2="60.5" y2="24" width="0" layer="19" extent="16-16"/>
+<wire x1="61.77" y1="15.96" x2="55.25" y2="22" width="0" layer="19" extent="16-16"/>
 </signal>
 <signal name="TMS">
@@
 <wire x1="59" y1="28.5" x2="59.5" y2="28" width="0.254" layer="1"/>
 <via x="59.5" y="28" extent="1-16" drill="0.6" shape="square"/>
-<wire x1="59.5" y1="28" x2="59.5" y2="24" width="0.254" layer="16"/>
+<wire x1="59.5" y1="28" x2="59" y2="27.5" width="0.254" layer="16"/>
 <wire x1="60.5" y1="28.5" x2="59" y2="28.5" width="0.254" layer="1"/>
+<wire x1="59" y1="27.5" x2="59" y2="27" width="0.254" layer="16"/>
+<wire x1="59" y1="27" x2="58.75" y2="26.75" width="0.254" layer="16"/>
+<wire x1="58.75" y1="26.75" x2="54.75" y2="26.75" width="0.254" layer="16"/>
+<wire x1="54.75" y1="26.75" x2="54.5" y2="26.5" width="0.254" layer="16"/>
+<wire x1="54.5" y1="26.5" x2="54.5" y2="22" width="0.254" layer="16"/>
 <wire x1="60.5" y1="37" x2="34.1805" y2="62.6881" width="0" layer="19" extent="1-16"/>
-<wire x1="57.96" y1="18.27" x2="59.5" y2="24" width="0" layer="19" extent="16-16"/>
+<wire x1="59.23" y1="15.96" x2="54.5" y2="22" width="0" layer="19" extent="16-16"/>
 </signal>
 <signal name="TDI">
@@
 <wire x1="39.475" y1="26.975" x2="38.75" y2="26" width="0.254" layer="1"/>
 <via x="38.75" y="26" extent="1-16" drill="0.6" shape="square"/>
-<wire x1="38.75" y1="26" x2="54.5" y2="26" width="0.254" layer="16"/>
-<via x="54.5" y="26" extent="1-16" drill="0.6" shape="square"/>
-<wire x1="54.5" y1="26" x2="54.5" y2="25.25" width="0.254" layer="1"/>
-<wire x1="54.5" y1="25.25" x2="55" y2="24.75" width="0.254" layer="1"/>
-<wire x1="55" y1="24.75" x2="56.9059875" y2="24.75" width="0.254" layer="1"/>
+<wire x1="38.75" y1="26" x2="53.5" y2="26" width="0.254" layer="16"/>
+<via x="53.5" y="26" extent="1-16" drill="0.6" shape="square"/>
+<wire x1="53.5" y1="26" x2="53.5" y2="24.75" width="0.254" layer="1"/>
+<wire x1="53.5" y1="24.75" x2="56.9059875" y2="24.75" width="0.254" layer="1"/>
 <wire x1="56.9059875" y1="24.75" x2="56.943396875" y2="24.787409375" width="0.254" layer="1"/>
 </signal>
@@
 <contactref element="U1" pad="P71"/>
 <contactref element="IC1" pad="10"/>
-<wire x1="56.943396875" y1="23.487409375" x2="55.012590625" y2="23.487409375" width="0.254" layer="1"/>
-<wire x1="55.012590625" y1="23.487409375" x2="53" y2="25.5" width="0.254" layer="1"/>
-<wire x1="53" y1="25.5" x2="53" y2="26.5" width="0.254" layer="1"/>
-<wire x1="53" y1="26.5" x2="46" y2="26.5" width="0.254" layer="1"/>
 <wire x1="46" y1="26.5" x2="46" y2="30.355" width="0.254" layer="1"/>
 <wire x1="46" y1="30.355" x2="45.975" y2="30.38" width="0.254" layer="1"/>
+<wire x1="56.943396875" y1="23.487409375" x2="54.012590625" y2="23.487409375" width="0.254" layer="1"/>
+<wire x1="54.012590625" y1="23.487409375" x2="54" y2="23.5" width="0.254" layer="1"/>
+<wire x1="54" y1="23.5" x2="54" y2="24" width="0.254" layer="1"/>
+<wire x1="54" y1="24" x2="48.5" y2="24" width="0.254" layer="1"/>
+<wire x1="46" y1="26.5" x2="48.5" y2="24" width="0.254" layer="1"/>
 </signal>
 <signal name="N$40">
@@
 <contactref element="R23" pad="1"/>
 <contactref element="U1" pad="P69"/>
-<wire x1="44.975" y1="30.38" x2="44.975" y2="25.275" width="0.254" layer="1"/>
-<wire x1="44.975" y1="25.275" x2="45.5" y2="24.75" width="0.254" layer="1"/>
-<wire x1="45.5" y1="24.75" x2="48" y2="24.75" width="0.254" layer="1"/>
-<wire x1="48" y1="24.75" x2="48" y2="22.2" width="0.254" layer="1"/>
-<wire x1="48" y1="22.2" x2="47.75" y2="21.95" width="0.254" layer="1"/>
+<wire x1="44.975" y1="30.38" x2="44.975" y2="25.525" width="0.254" layer="1"/>
+<wire x1="44.975" y1="25.525" x2="47.5" y2="23" width="0.254" layer="1"/>
+<wire x1="47.5" y1="23" x2="47.5" y2="22" width="0.254" layer="1"/>
+<wire x1="47.5" y1="22" x2="47.75" y2="21.95" width="0" layer="19" extent="1-1"/>
 </signal>
 <signal name="FPGA_AUDIO_RIGHT">
 <contactref element="R34" pad="1"/>
 <contactref element="U1" pad="P70"/>
-<wire x1="45.475" y1="30.38" x2="45.475" y2="25.775" width="0.254" layer="1"/>
-<wire x1="45.475" y1="25.775" x2="45.5" y2="25.75" width="0.254" layer="1"/>
-<wire x1="45.5" y1="25.75" x2="51" y2="25.75" width="0.254" layer="1"/>
-<wire x1="51" y1="25.75" x2="51" y2="21.95" width="0.254" layer="1"/>
+<wire x1="45.475" y1="30.38" x2="45.475" y2="26.025" width="0.254" layer="1"/>
+<wire x1="45.475" y1="26.025" x2="48" y2="23.5" width="0.254" layer="1"/>
+<wire x1="48" y1="23.5" x2="50.95" y2="23.5" width="0.254" layer="1"/>
+<wire x1="50.95" y1="23.5" x2="51" y2="21.95" width="0.254" layer="1"/>
 </signal>
 <signal name="RESET">

Commit message: rework
Parts:
- moved IC1 0.50 mm to (62.6, 23.5)
- moved R34 0.50 mm to (50.5, 21.0)
- moved U$1 0.50 mm to (54.8, 41.4)
Routing:
- net N$36: track 13.5 -> 16.4 mm, vias 0 -> 1
- net VCC: track 379.5 -> 381.1 mm, vias 8 -> 9
- net GND: track 371.0 -> 370.3 mm, vias 24 -> 27
- net PROM_INITB: track 24.1 -> 23.6 mm
- net PROM_DO: track 19.4 -> 18.9 mm
- net N$9: track 13.9 -> 13.4 mm
- net N$8: track 12.4 -> 11.9 mm
- net N$7: track 11.4 -> 10.9 mm
- net N$6: track 9.92 -> 9.42 mm
- net N$5: track 8.92 -> 8.42 mm
- net N$4: track 7.92 -> 7.42 mm
- net N$38: track 16.4 -> 15.9 mm
- net N$35: track 12.9 -> 12.4 mm
- net N$3: track 6.92 -> 6.42 mm
- net N$29: track 19.7 -> 19.2 mm
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
Commit message: rework
Parts:
- moved IC3 1.41 mm to (60.0, 59.0), turned to 270 degrees
- moved IC1 0.50 mm to (63.1, 23.5)
- moved IC2 0.50 mm to (4.90, 27.4)
- moved U$2 0.50 mm to (14.1, 22.6)
- turned JP3 to 270 degrees
Connections:
- removed net N$36: IC1.17, R1.2
- removed net N$68: JP3.3
- removed net N$69: JP3.5
- removed net N$70: JP3.6
- removed net N$72: JP3.4
- removed net TDI: IC1.4
- removed net TDO: U1.P109
- new net SPI_MISO: IC3.17
- new net SPI_MOSI: IC3.16
- new net SPI_SCLK: IC3.15
- new net SPI_SEL: IC3.14
- new net TDI_FPGA: IC3.20, R1.2
- new net TDO_EXP: IC3.12, JP3.1
- new net TDO_FPGA: IC1.4, U1.P109
- new net TDO_PROM: IC1.17, IC3.21, JP3.2
- net GND: now also JP3.6
- net TCK: now also IC3.18, JP3.3; no longer JP3.1
- net TMS: now also IC3.19, JP3.5; no longer JP3.2
- net VCC: now also JP3.4
Routing:
- net TDO_PROM: track 0.00 -> 19.0 mm, vias 0 -> 1
- net TDO_EXP: track 0.00 -> 17.7 mm, vias 0 -> 1
- net N$36: track 16.4 -> 0.00 mm, vias 1 -> 0
- net TDI: track 12.6 -> 0.00 mm
- net TDO_FPGA: track 0.00 -> 12.1 mm
- net TMS: track 24.8 -> 33.3 mm
- net TCK: track 25.6 -> 31.5 mm
- net VCC: track 381.1 -> 386.6 mm
- net GND: track 370.3 -> 372.1 mm
- net PROM_INITB: track 23.6 -> 24.1 mm
- net PROM_DO: track 18.9 -> 19.4 mm
- net N$40: track 15.8 -> 15.3 mm
- net N$38: track 15.9 -> 16.4 mm
- net N$35: track 12.4 -> 12.9 mm
- net FL_WP: track 34.1 -> 33.6 mm
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
Commit message: rework
Parts:
- moved RESET_SW 1.80 mm to (7.00, 16.8), turned to 180 degrees
- moved R52 1.27 mm to (3.25, 18.5), turned to 0 degrees
- moved U$2 0.56 mm to (14.4, 22.1), turned to 90 degrees
Routing:
- net VCC: track 386.6 -> 378.7 mm
- net CLK16: track 26.3 -> 28.4 mm
- net RESET: track 42.6 -> 41.6 mm
- net GND: track 372.1 -> 372.8 mm
Changed lines of the file:
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@@
 <element name="C3" library="resistor" package="C0603" value="" x="47.25" y="12.25" rot="MR180"/>
 <element name="C4" library="resistor" package="C0603" value="" x="52" y="11.75" rot="MR270"/>
-<element name="U$2" library="cpcfpga" package="OSC_7C" value="TXO_7C" x="14.125" y="22.625"/>
+<element name="U$2" library="cpcfpga" package="OSC_7C" value="TXO_7C" x="14.375" y="22.125" rot="R90"/>
 <element name="REG2.5" library="cpcfpga" package="SOT223" value="2.5V" x="40" y="38.5" rot="MR270"/>
 <element name="REG1.2" library="cpcfpga" package="SOT223" value="1.2V" x="35.5" y="43.75" rot="MR90"/>
@@
 <element name="R49" library="resistor" package="M0805" value="" x="53" y="14.5" rot="MR0"/>
 <element name="R50" library="resistor" package="M0805" value="2k2" x="39.25" y="21" rot="R90"/>
-<element name="RESET_SW" library="jumper" package="JP1" value="" x="6" y="18.25" rot="R270"/>
-<element name="R52" library="resistor" package="M0805" value="4K7" x="2" y="18.25" rot="R270"/>
+<element name="RESET_SW" library="jumper" package="JP1" value="" x="7" y="16.75" rot="R180"/>
+<element name="R52" library="resistor" package="M0805" value="4K7" x="3.25" y="18.5"/>
 <element name="IC3" library="adafruit" package="TQFP32-08" value="ATMEGA32U2-TQFP" x="60" y="59" rot="R270"/>
 </elements>
@@
 <wire x1="55.5" y1="10.75" x2="50.25" y2="10.75" width="0.254" layer="1"/>
 <wire x1="50.25" y1="10.75" x2="50" y2="10.75" width="0.254" layer="1"/>
-<wire x1="13" y1="3.75" x2="14" y2="2.75" width="0.254" layer="1"/>
-<wire x1="7.27" y1="14.25" x2="7.27" y2="18.25" width="0.254" layer="1"/>
-<wire x1="13" y1="3.75" x2="13" y2="14.25" width="0.254" layer="1"/>
-<wire x1="13" y1="14.25" x2="13" y2="18.25" width="0.254" layer="1"/>
+<wire x1="14" y1="14.25" x2="14" y2="2.75" width="0.254" layer="1"/>
+<wire x1="14" y1="14.25" x2="14" y2="16.75" width="0.254" layer="1"/>
 <wire x1="6.801446875" y1="24.7609125" x2="6.801446875" y2="22.051446875" width="0.254" layer="1"/>
 <wire x1="6.801446875" y1="22.051446875" x2="6" y2="21.25" width="0.254" layer="1"/>
-<wire x1="6" y1="21.25" x2="4" y2="21.25" width="0.254" layer="1"/>
-<via x="4" y="21.25" extent="1-16" drill="0.6" shape="square"/>
-<wire x1="4" y1="21.25" x2="3" y2="21.25" width="0.254" layer="16"/>
-<wire x1="3" y1="21.25" x2="2.5" y2="4.25" width="0.254" layer="16"/>
+<wire x1="6" y1="21.25" x2="4.5" y2="21.25" width="0.254" layer="1"/>
+<via x="4.5" y="21.25" extent="1-16" drill="0.6" shape="square"/>
+<wire x1="4.5" y1="21.25" x2="3.25" y2="21.25" width="0.254" layer="16"/>
+<wire x1="3.25" y1="21.25" x2="3.25" y2="4.25" width="0.254" layer="16"/>
 <wire x1="57" y1="30.25" x2="54.5" y2="30.25" width="0.254" layer="1"/>
 <wire x1="54.5" y1="30.25" x2="50" y2="30.25" width="0.254" layer="1"/>
@@
 <wire x1="58" y1="30.25" x2="57.5" y2="30.25" width="0.254" layer="1"/>
 <wire x1="57.5" y1="30.25" x2="57.25" y2="30.5" width="0.254" layer="1"/>
-<wire x1="7.27" y1="14.25" x2="13" y2="14.25" width="0.254" layer="1"/>
-<wire x1="2.5" y1="4.25" x2="11" y2="4.25" width="0.254" layer="16"/>
+<wire x1="7.25" y1="14.25" x2="14" y2="14.25" width="0.254" layer="1"/>
+<wire x1="3.25" y1="4.25" x2="11" y2="4.25" width="0.254" layer="16"/>
 <wire x1="11" y1="4.25" x2="12" y2="3.25" width="0.254" layer="16"/>
 <wire x1="12" y1="3.25" x2="13.37" y2="3.25" width="0.254" layer="16"/>
 <wire x1="13.37" y1="3.25" x2="13.95" y2="2.67" width="0.254" layer="16"/>
-<wire x1="13" y1="18.25" x2="15.5" y2="20.25" width="0.254" layer="1"/>
-<wire x1="15.5" y1="20.25" x2="15.5" y2="21.42" width="0.254" layer="1"/>
-<wire x1="15.5" y1="21.42" x2="15.395" y2="21.525" width="0.254" layer="1"/>
 <wire x1="61.75" y1="23.25" x2="61.75" y2="23.5" width="0.254" layer="16"/>
 <wire x1="61.75" y1="23.5" x2="64.5" y2="23.5" width="0.254" layer="16"/>
@@
 <wire x1="58" y1="30.25" x2="64.5" y2="30.25" width="0.254" layer="16"/>
 <wire x1="64.5" y1="30.25" x2="64.5" y2="23.5" width="0.254" layer="16"/>
+<wire x1="14" y1="16.75" x2="14.75" y2="17.5" width="0.254" layer="1"/>
+<wire x1="14.75" y1="17.5" x2="17" y2="17.5" width="0.254" layer="1"/>
+<wire x1="15.475" y1="23.395" x2="17" y2="21.87" width="0.254" layer="1"/>
+<wire x1="17" y1="21.87" x2="17" y2="17.5" width="0.254" layer="1"/>
 <wire x1="96.05" y1="71" x2="95.55" y2="76" width="0" layer="19" extent="1-1"/>
 <wire x1="96.55" y1="67.5" x2="96.05" y2="71" width="0" layer="19" extent="1-1"/>
@@
 <wire x1="46.335" y1="7.75" x2="46.5" y2="7.75" width="0" layer="19" extent="1-1"/>
 <wire x1="98.3" y1="2.25" x2="81.27" y2="16.1284" width="0" layer="19" extent="1-1"/>
+<wire x1="7.25" y1="14.25" x2="7" y2="14.5" width="0.254" layer="1"/>
+<wire x1="7" y1="14.5" x2="7" y2="15.48" width="0.254" layer="1"/>
 </signal>
 <signal name="VCC">
@@
 <wire x1="1.5" y1="29.25" x2="1.5" y2="20.25" width="0.254" layer="1"/>
 <wire x1="1.5" y1="20.25" x2="9" y2="20.25" width="0.254" layer="1"/>
-<wire x1="20.75" y1="21.85" x2="17.6" y2="21.85" width="0.254" layer="16"/>
-<wire x1="17.6" y1="21.85" x2="17.5" y2="21.75" width="0.254" layer="16"/>
-<wire x1="17.5" y1="21.75" x2="17.5" y2="17.75" width="0.254" layer="16"/>
-<wire x1="17.5" y1="17.75" x2="10" y2="17.75" width="0.254" layer="16"/>
-<wire x1="10" y1="17.75" x2="10.5" y2="19.25" width="0.254" layer="16"/>
-<via x="10.5" y="19.25" extent="1-16" drill="0.6" shape="square"/>
-<wire x1="10.5" y1="19.25" x2="10" y2="19.25" width="0.254" layer="1"/>
+<wire x1="17" y1="19.25" x2="12" y2="19.25" width="0.254" layer="16"/>
+<via x="12" y="19.25" extent="1-16" drill="0.6" shape="square"/>
+<wire x1="12" y1="19.25" x2="11.25" y2="19.25" width="0.254" layer="1"/>
+<wire x1="11.25" y1="19.25" x2="10" y2="19.25" width="0.254" layer="1"/>
 <wire x1="10" y1="19.25" x2="9" y2="20.25" width="0.254" layer="1"/>
 <wire x1="55" y1="51.17" x2="55.5" y2="52.5" width="0.254" layer="1"/>
 <wire x1="55.5" y1="52.5" x2="55.5" y2="54.25" width="0.254" layer="1"/>
 <wire x1="55.5" y1="54.25" x2="52.5" y2="57.25" width="0.254" layer="1"/>
-<wire x1="9" y1="20.25" x2="12" y2="23.25" width="0.254" layer="1"/>
-<wire x1="12" y1="23.25" x2="12.83" y2="23.25" width="0.254" layer="1"/>
-<wire x1="12.83" y1="23.25" x2="12.855" y2="23.725" width="0.254" layer="1"/>
 <wire x1="52.5" y1="57.25" x2="21.5" y2="57.25" width="0.254" layer="1"/>
 <wire x1="21.5" y1="57.25" x2="12.5" y2="48.25" width="0.254" layer="1"/>
@@
 <wire x1="26.5" y1="29.75" x2="27.5" y2="30.75" width="0.254" layer="1"/>
 <wire x1="1.5" y1="20.25" x2="1.5" y2="20.2" width="0.254" layer="1"/>
-<wire x1="1.5" y1="20.2" x2="2" y2="19.2" width="0.254" layer="1"/>
 <wire x1="49.845" y1="53.345" x2="54.655" y2="53.345" width="0.254" layer="1"/>
 <wire x1="54.655" y1="53.345" x2="55.5" y2="52.5" width="0.254" layer="1"/>
@@
 <wire x1="61.77" y1="18.5" x2="63.5" y2="18.5" width="0.254" layer="1"/>
 <wire x1="63.5" y1="18.5" x2="63.5" y2="22.25" width="0.254" layer="1"/>
+<wire x1="17" y1="19.25" x2="18.5" y2="20.75" width="0.254" layer="16"/>
+<wire x1="18.5" y1="20.75" x2="18.5" y2="22" width="0.254" layer="16"/>
+<wire x1="18.5" y1="22" x2="20.5" y2="22" width="0.254" layer="16"/>
+<wire x1="13.275" y1="20.855" x2="11.855" y2="20.855" width="0.254" layer="1"/>
+<wire x1="11.855" y1="20.855" x2="11.5" y2="20.5" width="0.254" layer="1"/>
+<wire x1="11.5" y1="20.5" x2="11.5" y2="19.5" width="0.254" layer="1"/>
+<wire x1="11.25" y1="19.25" x2="11.5" y2="19.5" width="0.254" layer="1"/>
 <wire x1="90.9" y1="64.5" x2="92.45" y2="68" width="0" layer="19" extent="1-16"/>
 <wire x1="73.984" y1="67.5094" x2="90.9" y2="64.5" width="0" layer="19" extent="1-16"/>
@@
 <wire x1="55.5" y1="52.5" x2="71.5" y2="46.5" width="0" layer="19" extent="1-1"/>
 <wire x1="45.5" y1="33.33" x2="45.75" y2="33.25" width="0" layer="19" extent="1-1"/>
+<wire x1="2.3" y1="18.5" x2="1.5" y2="20.2" width="0" layer="19" extent="1-1"/>
 </signal>
 <signal name="TCK">
@@
 <via x="9" y="23.75" extent="1-16" drill="0.6" shape="square"/>
 <wire x1="9" y1="25.75" x2="9" y2="23.75" width="0.254" layer="1"/>
-<wire x1="9" y1="23.75" x2="9" y2="23.25" width="0.254" layer="16"/>
-<wire x1="9" y1="23.25" x2="5" y2="19.25" width="0.254" layer="16"/>
-<wire x1="4.5" y1="18.48" x2="5" y2="19.25" width="0.254" layer="16"/>
-<wire x1="4.5" y1="18.48" x2="4.73" y2="18.25" width="0.254" layer="16"/>
-<wire x1="2" y1="17.3" x2="3.78" y2="17.3" width="0.254" layer="1"/>
-<wire x1="3.78" y1="17.3" x2="4.73" y2="18.25" width="0.254" layer="1"/>
+<wire x1="9" y1="23.75" x2="9" y2="20.02" width="0.254" layer="16"/>
+<wire x1="4.2" y1="18.5" x2="6.5" y2="18.5" width="0.254" layer="1"/>
+<wire x1="6.5" y1="18.5" x2="7" y2="18" width="0.254" layer="1"/>
+<wire x1="9" y1="20.02" x2="7" y2="18.02" width="0.254" layer="16"/>
+<wire x1="7" y1="18" x2="7" y2="18.02" width="0" layer="19" extent="1-1"/>
 </signal>
 <signal name="VCCAUX_R">
@@
 <wire x1="36.975" y1="30.38" x2="36.975" y2="28.725" width="0.254" layer="1"/>
 <wire x1="36.975" y1="28.725" x2="33.5" y2="25.25" width="0.254" layer="1"/>
-<wire x1="33.5" y1="25.25" x2="16" y2="25.25" width="0.254" layer="1"/>
-<wire x1="16" y1="25.25" x2="15.5" y2="24.75" width="0.254" layer="1"/>
-<wire x1="15.5" y1="24.75" x2="15.5" y2="23.25" width="0.254" layer="1"/>
-<wire x1="15.5" y1="23.25" x2="15.395" y2="23.725" width="0" layer="19" extent="1-1"/>
+<wire x1="33.5" y1="25.25" x2="13.75" y2="25.25" width="0.254" layer="1"/>
+<wire x1="13.75" y1="25.25" x2="13.5" y2="25" width="0.254" layer="1"/>
+<wire x1="13.5" y1="25" x2="13.5" y2="23.62" width="0.254" layer="1"/>
+<wire x1="13.5" y1="23.62" x2="13.275" y2="23.395" width="0.254" layer="1"/>
 </signal>
 <signal name="XXR1">
