File: eagle/homeboard/homeboard8.brd (EAGLE design)
At the start: 100 x 80 mm, 77 parts, among them IC1 XCF02S, IC2 25LC080SN, IC3 ATMEGA32U2-TQFP, Q5 BC848SMD, Q6 BC848SMD, Q7 BC848SMD, Q8 BC848SMD, T1 BSS138, T2 BC848, T3 BSS138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

Commit message: rework
Parts:
- moved IC3 8.60 mm to (55.0, 66.0), turned to 0 degrees
- moved C1 2.00 mm to (47.5, 17.0)
- moved C3 2.00 mm to (45.2, 12.2)
- moved C4 2.00 mm to (50.0, 11.8)
- moved C5 2.00 mm to (51.0, 17.0)
- moved IC1 2.00 mm to (61.1, 23.5)
- moved JP3 2.00 mm to (58.5, 18.5)
- moved Q5 2.00 mm to (18.8, 20.8)
- moved Q6 2.00 mm to (26.8, 20.8)
- moved Q7 2.00 mm to (42.0, 20.8)
- moved Q8 2.00 mm to (34.5, 20.8)
- moved R1 2.00 mm to (17.7, 61.2)
- moved R10 2.00 mm to (27.8, 21.0)
- moved R13 2.00 mm to (16.8, 12.8)
- moved R14 2.00 mm to (16.8, 15.0)
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Connections:
- net TDO_EXP: now also IC3.21; no longer IC3.12
- net TDO_PROM: now also IC3.22; no longer IC3.21
Routing:
- net VCC: track 378.7 -> 372.4 mm
- net CLK16: track 28.4 -> 25.0 mm
- net GND: track 372.8 -> 375.3 mm, vias 27 -> 28
- net FL_WP: track 33.6 -> 31.6 mm
- net FL_SEL: track 34.6 -> 32.6 mm
- net FL_SCLK: track 28.8 -> 26.8 mm
- net FL_HOLD: track 31.9 -> 29.9 mm
- net FL_DO: track 33.7 -> 31.7 mm
- net FL_DI: track 26.2 -> 24.2 mm
- net RESET: track 41.6 -> 42.4 mm
