File: eagle/homeboard/homeboard8.sch (EAGLE design)
At the start: 77 parts, among them IC1 XCF02S, IC2 25LC080SN, IC3 ATMEGA32U2-TQFP, Q5 BC848SMD, Q6 BC848SMD, Q7 BC848SMD, Q8 BC848SMD, T1 BSS138, T2 BC848, T3 BSS138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

Commit message: need to stop changing my mind
Connections:
- net FL_SEL: now also U1B5.IO_L28P_5D7; no longer U1B5.IO_L31P_5D5
- net FL_WP: now also U1B5.IO_L31P_5D5; no longer U1B5.IO_L28P_5D7
Changed lines of the file:
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@@
 </segment>
 <segment>
-<pinref part="U1" gate="B5" pin="IO_L31P_5D5"/>
-<wire x1="106.68" y1="-66.04" x2="134.62" y2="-66.04" width="0.1524" layer="91"/>
-<wire x1="134.62" y1="-66.04" x2="134.62" y2="-40.64" width="0.1524" layer="91"/>
-<label x="106.68" y="-66.04" size="1.778" layer="95"/>
+<pinref part="U1" gate="B5" pin="IO_L28P_5D7"/>
+<wire x1="106.68" y1="-60.96" x2="139.7" y2="-60.96" width="0.1524" layer="91"/>
+<wire x1="139.7" y1="-60.96" x2="139.7" y2="-40.64" width="0.1524" layer="91"/>
+<label x="106.68" y="-60.96" size="1.778" layer="95"/>
 </segment>
 </net>
@@
 </segment>
 <segment>
-<pinref part="U1" gate="B5" pin="IO_L28P_5D7"/>
-<wire x1="106.68" y1="-60.96" x2="139.7" y2="-60.96" width="0.1524" layer="91"/>
-<wire x1="139.7" y1="-60.96" x2="139.7" y2="-40.64" width="0.1524" layer="91"/>
-<label x="106.68" y="-60.96" size="1.778" layer="95"/>
-</segment>
-</net>
+<pinref part="U1" gate="B5" pin="IO_L31P_5D5"/>
+<wire x1="106.68" y1="-66.04" x2="134.62" y2="-66.04" width="0.1524" layer="91"/>
+<wire x1="134.62" y1="-66.04" x2="134.62" y2="-40.64" width="0.1524" layer="91"/>
+<label x="106.68" y="-66.04" size="1.778" layer="95"/>
+</segment>
+</net>

Commit message: rework
Connections:
- removed net N$36: IC1.TDO, R1.2
- removed net N$68: JP3.3
- removed net N$69: JP3.5
- removed net N$70: JP3.6
- removed net N$72: JP3.4
- removed net TDI: IC1.TDI
- removed net TDO: U1BVCCAUX.TDO
- new net SPI_MISO: IC3.PB3(PDO/MISO/PCINT3)
- new net SPI_MOSI: IC3.PB2(PDI/MOSI/PCINT2)
- new net SPI_SCLK: IC3.PB1(SCK/PCINT1)
- new net SPI_SEL: IC3.PB0(SS/PCINT0)
- new net TDI_FPGA: IC3.PB6(PCINT6), R1.2
- new net TDO_EXP: IC3.PD6(INT6/AIN5/RTS), JP3.1
- new net TDO_FPGA: IC1.TDI, U1BVCCAUX.TDO
- new net TDO_PROM: IC1.TDO, IC3.PB7(OC0A/OC1C/PCINT7), JP3.2
- net GND: now also JP3.6
- net TCK: now also IC3.PB4(T1/PCINT4), JP3.3; no longer JP3.1
- net TMS: now also IC3.PB5(PCINT5), JP3.5; no longer JP3.2
- net VCC: now also JP3.4
Other:
- moved on the sheet: IC3, JP3

Commit message: rework
Connections:
- net TDO_EXP: now also IC3.PB7(OC0A/OC1C/PCINT7); no longer IC3.PD6(INT6/AIN5/RTS)
- net TDO_PROM: now also IC3.PC7(ICP1/INT4/CLKO); no longer IC3.PB7(OC0A/OC1C/PCINT7)
Changed lines of the file:
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@@
 </segment>
 <segment>
-<wire x1="-203.2" y1="-63.5" x2="-215.9" y2="-63.5" width="0.1524" layer="91"/>
-<label x="-203.2" y="-63.5" size="1.778" layer="95"/>
-<pinref part="IC3" gate="G$1" pin="PB7(OC0A/OC1C/PCINT7)"/>
+<label x="-203.2" y="-78.74" size="1.778" layer="95"/>
+<pinref part="IC3" gate="G$1" pin="PC7(ICP1/INT4/CLKO)"/>
+<wire x1="-203.2" y1="-78.74" x2="-215.9" y2="-78.74" width="0.1524" layer="91"/>
 </segment>
 </net>
@@
 </segment>
 <segment>
-<pinref part="IC3" gate="G$1" pin="PD6(INT6/AIN5/RTS)"/>
-<wire x1="-203.2" y1="-35.56" x2="-215.9" y2="-35.56" width="0.1524" layer="91"/>
-<label x="-203.2" y="-35.56" size="1.778" layer="95"/>
+<wire x1="-203.2" y1="-63.5" x2="-215.9" y2="-63.5" width="0.1524" layer="91"/>
+<label x="-203.2" y="-63.5" size="1.778" layer="95"/>
+<pinref part="IC3" gate="G$1" pin="PB7(OC0A/OC1C/PCINT7)"/>
 </segment>
 </net>
