File: eagle/homeboard/homeboard9.brd (EAGLE design)
At the start: 100 x 80 mm, 79 parts, among them IC1 XCF02S, IC2 25LC080SN, IC3 ATMEGA32U2-TQFP, Q5 BC848SMD, Q6 BC848SMD, Q7 BC848SMD, Q8 BC848SMD, T1 BSS138, T2 BC848, T3 BSS138, U1 XC3S400TQ144, X1 1503_04, X2 SCART-F

Commit message: rework
Parts:
- moved U$1 0.33 mm to (52.8, 41.8)
- moved U1 0.17 mm to (35.7, 41.2)
Routing:
- net VCC: track 364.4 -> 183.2 mm, vias 7 -> 5
- net GND: track 440.4 -> 388.5 mm, vias 33 -> 31
- net VCCINT: track 43.3 -> 5.61 mm, vias 7 -> 0
- net VCCAUX_R: track 34.2 -> 10.2 mm, vias 3 -> 0
- net VCCAUX: track 26.4 -> 2.90 mm, vias 3 -> 0
- net B1: track 8.85 -> 0.74 mm
- net N$29: track 19.2 -> 16.4 mm
- net N$28: track 17.7 -> 15.8 mm
- net N$27: track 16.2 -> 14.6 mm
- net N$26: track 15.2 -> 13.6 mm
- net N$25: track 14.2 -> 12.6 mm
- net N$24: track 13.2 -> 11.6 mm
- net N$23: track 12.2 -> 10.6 mm
- net N$22: track 10.2 -> 9.20 mm
- net N$21: track 9.23 -> 8.20 mm
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
Commit message: rework
Parts:
- added C10, C11, C12, C13, C14, C15, C16, C17, C18, C19, C20, C21, C22, C23, C24, C25, C6, C7, C8, C9: 100nF, rcl:C0603
Connections:
- net GND: now also C10.2, C11.2, C12.2, C13.2, C14.2, C15.2, C16.2, C17.2, C18.2, C19.2, C20.2, C21.2, C22.2, C23.2, C24.2, C25.2, C6.2, C7.2, C8.2, C9.2
- net VCC: now also C10.1, C11.1, C12.1, C13.1, C14.1, C15.1, C16.1, C17.1, C6.1, C7.1, C8.1, C9.1
- net VCCAUX: now also C18.1, C19.1, C20.1, C21.1, REG2.5.2
- net VCCAUX_R: no longer REG2.5.2
- net VCCINT: now also C22.1, C23.1, C24.1, C25.1, REG1.2.2
Routing:
- net VCC: track 183.2 -> 210.7 mm, vias 5 -> 15
- net GND: track 388.5 -> 364.9 mm, vias 31 -> 29
- net VCCINT: track 5.61 -> 13.0 mm, vias 0 -> 1
- net VCCAUX: track 2.90 -> 9.10 mm
- net N$42: track 0.00 -> 5.06 mm
- net N$40: track 15.3 -> 19.9 mm

Commit message: rework
Parts:
- moved C25 42.2 mm to (37.2, 34.0), turned to 90 degrees
- moved C21 41.9 mm to (32.5, 34.2), turned to 90 degrees
- moved C24 41.8 mm to (35.0, 34.0), turned to 90 degrees
- moved C20 40.2 mm to (38.0, 39.5)
- moved C14 1.60 mm to (30.2, 35.5)
Routing:
- net VCCINT: track 13.0 -> 27.6 mm, vias 1 -> 2
- net GND: track 364.9 -> 377.9 mm
- net VCC: track 210.7 -> 223.0 mm
- net VCCAUX: track 9.10 -> 18.2 mm, vias 0 -> 1
- net VCCAUX_R: track 10.2 -> 17.2 mm

Commit message: rework
Parts:
- moved C18 49.4 mm to (39.0, 35.5), turned to 90 degrees
- moved C20 19.6 mm to (18.5, 41.0), turned to 90 degrees
- moved C24 0.56 mm to (34.5, 34.2)
- moved C25 0.56 mm to (36.8, 34.2)
- moved C14 0.25 mm to (30.0, 35.5)
- moved C16 0.25 mm to (27.8, 34.5)
- moved C17 0.25 mm to (43.5, 35.0)
- moved C21 0.25 mm to (32.2, 34.2)
- moved C8 0.25 mm to (41.2, 35.2)
Connections:
- net VCCAUX: now also U1.P120, U1.P62
- net VCCAUX_R: no longer U1.P120, U1.P62
Routing:
- net VCCAUX: track 18.2 -> 33.2 mm, vias 1 -> 2
- net VCCAUX_R: track 17.2 -> 4.90 mm
- net B1: track 0.74 -> 9.02 mm
- net GND: track 377.9 -> 384.6 mm, vias 29 -> 30
- net VCCINT: track 27.6 -> 33.3 mm

Commit message: rework
Parts:
- moved C15 7.11 mm to (33.8, 37.0)
Routing:
- net VCCINT: track 33.3 -> 37.3 mm
- net VCC: track 223.0 -> 221.8 mm, vias 15 -> 16
- net GND: track 384.6 -> 385.5 mm
Changed lines of the file:
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@@
 <element name="C13" library="rcl" package="C0603" value="100nF" x="43" y="46.25" rot="MR270"/>
 <element name="C14" library="rcl" package="C0603" value="100nF" x="30" y="35.5" rot="MR90"/>
-<element name="C15" library="rcl" package="C0603" value="100nF" x="35" y="44" rot="MR0"/>
+<element name="C15" library="rcl" package="C0603" value="100nF" x="33.75" y="37" rot="MR0"/>
 <element name="C16" library="rcl" package="C0603" value="100nF" x="27.75" y="34.5" rot="MR90"/>
 <element name="C17" library="rcl" package="C0603" value="100nF" x="43.5" y="35" rot="MR90"/>
@@
 <contactref element="C25" pad="2"/>
 <contactref element="C22" pad="2"/>
-<wire x1="30" y1="36.35" x2="30.15" y2="36.5" width="0.254" layer="16"/>
 <wire x1="30.15" y1="36.5" x2="28" y2="36.5" width="0.254" layer="16"/>
 <wire x1="28" y1="36.5" x2="27.75" y2="35.35" width="0.254" layer="16"/>
-<wire x1="32.25" y1="35.1" x2="32.5" y2="36.5" width="0.254" layer="16"/>
-<wire x1="32.5" y1="36.5" x2="32.35" y2="36.35" width="0.254" layer="16"/>
-<wire x1="32.35" y1="36.35" x2="30" y2="36.35" width="0.254" layer="16"/>
 <wire x1="36.75" y1="35.1" x2="34.5" y2="35.1" width="0.254" layer="16"/>
 <wire x1="34.5" y1="35.1" x2="32.25" y2="35.1" width="0.254" layer="16"/>
@@
 <via x="40.5" y="37.5" extent="1-16" drill="0.6" shape="square"/>
 <wire x1="40.5" y1="37.5" x2="40.5" y2="36.35" width="0.254" layer="16"/>
+<wire x1="32.9" y1="37" x2="32.9" y2="35.75" width="0.254" layer="16"/>
+<wire x1="32.9" y1="35.75" x2="32.25" y2="35.1" width="0.254" layer="16"/>
+<wire x1="32.25" y1="35.1" x2="32.25" y2="35.25" width="0.254" layer="16"/>
+<wire x1="32.25" y1="35.25" x2="31" y2="36.5" width="0.254" layer="16"/>
+<wire x1="31" y1="36.5" x2="30.15" y2="36.5" width="0.254" layer="16"/>
+<wire x1="30.15" y1="36.5" x2="30" y2="36.35" width="0.254" layer="16"/>
 <wire x1="96.05" y1="71" x2="95.55" y2="76" width="0" layer="19" extent="1-1"/>
 <wire x1="96.55" y1="67.5" x2="96.05" y2="71" width="0" layer="19" extent="1-1"/>
@@
 <wire x1="46.42" y1="43" x2="46.42" y2="40" width="0" layer="19" extent="1-1"/>
 <wire x1="43" y1="45.4" x2="43" y2="45.5" width="0" layer="19" extent="16-16"/>
-<wire x1="34.15" y1="44" x2="32.65" y2="46.65" width="0" layer="19" extent="16-16"/>
 <wire x1="26.75" y1="32.25" x2="27.15" y2="35.35" width="0" layer="19" extent="16-16"/>
 <wire x1="41.97" y1="51.95" x2="44.5" y2="46.5" width="0" layer="19" extent="1-1"/>
@@
 <wire x1="29.6" y1="33.65" x2="27.75" y2="33.65" width="0.254" layer="16"/>
 <wire x1="35.475" y1="33.475" x2="35.5" y2="33.5" width="0.254" layer="1"/>
-<wire x1="35.5" y1="33.5" x2="35.5" y2="39.5" width="0.254" layer="1"/>
+<via x="36" y="36.5" extent="1-16" drill="0.6" shape="square"/>
+<wire x1="35.5" y1="33.5" x2="35.5" y2="36" width="0.254" layer="1"/>
+<wire x1="35.5" y1="36" x2="36" y2="36.5" width="0.254" layer="1"/>
+<wire x1="34.6" y1="37" x2="35.5" y2="37" width="0.254" layer="16"/>
+<wire x1="35.5" y1="37" x2="36" y2="36.5" width="0.254" layer="16"/>
 <wire x1="90.9" y1="64.5" x2="92.45" y2="68" width="0" layer="19" extent="1-16"/>
 <wire x1="73.984" y1="67.5094" x2="90.9" y2="64.5" width="0" layer="19" extent="1-16"/>
@@
 <wire x1="30.5" y1="48.35" x2="31" y2="48.5" width="0" layer="19" extent="16-16"/>
 <wire x1="28" y1="49" x2="29.97" y2="49.78" width="0" layer="19" extent="1-16"/>
-<wire x1="35.85" y1="44" x2="31.5" y2="48.5" width="0" layer="19" extent="16-16"/>
-<wire x1="35.5" y1="39.5" x2="35.85" y2="44" width="0" layer="19" extent="1-16"/>
-<wire x1="29.97" y1="30.55" x2="35.47" y2="30.55" width="0" layer="19" extent="1-1"/>
+<wire x1="28" y1="41.5" x2="28" y2="48.35" width="0" layer="19" extent="16-16"/>
+<wire x1="30" y1="34.65" x2="27.5" y2="41" width="0" layer="19" extent="16-16"/>
+<wire x1="34.6" y1="37" x2="30" y2="34.65" width="0" layer="19" extent="16-16"/>
 <wire x1="41" y1="33.5" x2="35.5" y2="33.5" width="0" layer="19" extent="1-16"/>
 <wire x1="18.5" y1="22" x2="18.75" y2="21.85" width="0" layer="19" extent="16-16"/>
-<wire x1="27.5" y1="41" x2="30" y2="34.65" width="0" layer="19" extent="16-16"/>
 <wire x1="20.15" y1="58" x2="25.02" y2="49" width="0" layer="19" extent="1-1"/>
 <wire x1="20.15" y1="63" x2="20.15" y2="58" width="0" layer="19" extent="1-1"/>
@@
 <wire x1="32.47" y1="51.95" x2="30" y2="76.35" width="0" layer="19" extent="1-16"/>
 <wire x1="38.47" y1="51.95" x2="32.47" y2="51.95" width="0" layer="19" extent="1-1"/>
-<wire x1="33" y1="37.5" x2="32.47" y2="51.95" width="0" layer="19" extent="1-1"/>
+<wire x1="37" y1="37.5" x2="32.47" y2="51.95" width="0" layer="19" extent="1-16"/>
 <wire x1="14.25" y1="37" x2="33" y2="37.5" width="0" layer="19" extent="1-1"/>
+<wire x1="33" y1="37.5" x2="37" y2="37.5" width="0.254" layer="1"/>
 </signal>
 <signal name="VCCAUX">
@@
 <wire x1="32.47" y1="30.55" x2="32.5" y2="30.58" width="0.254" layer="1"/>
 <wire x1="32.5" y1="30.58" x2="32.5" y2="37.5" width="0.254" layer="1"/>
-<wire x1="31.97" y1="51.95" x2="15" y2="76.35" width="0" layer="19" extent="1-16"/>
-<wire x1="38.97" y1="51.95" x2="31.97" y2="51.95" width="0" layer="19" extent="1-1"/>
-<wire x1="39.5" y1="43" x2="38.97" y2="51.95" width="0" layer="19" extent="1-1"/>
-<wire x1="39.5" y1="33" x2="39.5" y2="30.58" width="0" layer="19" extent="1-16"/>
-<wire x1="32.5" y1="37.5" x2="39" y2="34.65" width="0" layer="19" extent="1-16"/>
-<wire x1="32.5" y1="32" x2="32.5" y2="30.58" width="0" layer="19" extent="1-1"/>
-<wire x1="18.5" y1="40.15" x2="32.5" y2="37.5" width="0" layer="19" extent="1-16"/>
-<wire x1="14.5" y1="44.75" x2="18.5" y2="40.15" width="0" layer="19" extent="1-16"/>
-<wire x1="11.5" y1="45" x2="11.599" y2="44.75" width="0" layer="19" extent="1-1"/>
 <wire x1="39" y1="34.65" x2="38.5" y2="34.15" width="0.254" layer="16"/>
 <wire x1="38.5" y1="34.15" x2="38.5" y2="33.25" width="0.254" layer="16"/>
@@
 <wire x1="38.5" y1="33.25" x2="39" y2="33" width="0.254" layer="1"/>
 <wire x1="39" y1="33" x2="39.5" y2="33" width="0.254" layer="1"/>
+<wire x1="31.97" y1="51.95" x2="15" y2="76.35" width="0" layer="19" extent="1-16"/>
+<wire x1="38.97" y1="51.95" x2="31.97" y2="51.95" width="0" layer="19" extent="1-1"/>
+<wire x1="39.5" y1="43" x2="38.97" y2="51.95" width="0" layer="19" extent="1-1"/>
+<wire x1="32.5" y1="32" x2="38.5" y2="33.25" width="0" layer="19" extent="1-16"/>
+<wire x1="32.5" y1="30.58" x2="32.5" y2="32" width="0" layer="19" extent="1-1"/>
+<wire x1="18.5" y1="40.15" x2="32.5" y2="37.5" width="0" layer="19" extent="1-16"/>
+<wire x1="14.5" y1="44.75" x2="18.5" y2="40.15" width="0" layer="19" extent="1-16"/>
+<wire x1="11.5" y1="45" x2="11.599" y2="44.75" width="0" layer="19" extent="1-1"/>
 </signal>
 <signal name="D_FASTBLANKING">

Commit message: rework
Parts:
- moved C19 32.7 mm to (32.2, 47.8)
- moved C22 27.6 mm to (34.5, 48.2)
- moved C23 27.3 mm to (36.8, 48.2)
- moved C7 23.0 mm to (41.2, 47.0), flipped to the bottom, turned to 270 degrees
- moved C20 21.4 mm to (39.0, 47.2), turned to 270 degrees
- moved R2 19.1 mm to (53.1, 55.2)
- moved R3 16.2 mm to (47.2, 55.7)
- moved R1 12.5 mm to (25.8, 57.2), flipped to the bottom
- moved C13 0.90 mm to (43.5, 47.0)
- moved C12 0.71 mm to (30.0, 47.0)
- moved C9 0.25 mm to (27.8, 47.5)
Routing:
- net VCCAUX: track 33.2 -> 48.8 mm, vias 2 -> 4
- net VCCINT: track 37.3 -> 48.8 mm, vias 2 -> 4
- net GND: track 385.5 -> 391.1 mm, vias 30 -> 32
- net VCC: track 221.8 -> 227.0 mm
