File: eagle/homeboard/homeboard11.brd (EAGLE design)
At the start: 100 x 80 mm, 113 parts, among them IC1 XCF02S, IC2 25LC080SN, IC3 ATMEGA32U2-TQFP, Q5 BC848SMD, Q6 BC848SMD, Q7 BC848SMD, Q8 BC848SMD, T1 BSS138, T2 BC848, T3 BSS138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

Commit message: got both rams for now...
Parts:
- added C34: 100nF, rcl:C0603
- added U$6: AS6C4008, cpcfpga:TSOP32
Connections:
- removed net XXR0: U1.P140
- removed net XXR1: U1.P141
- new net N$71: U$6.P2, U1.P2
- new net N$72: U$6.P3, U1.P4
- new net N$74: U$6.P5, U1.P6
- new net N$75: U$6.P6, U1.P7
- new net N$76: U$6.P7, U1.P8
- new net N$77: U$6.P9, U1.P10
- new net N$78: U$6.P10, U1.P11
- new net N$79: U$6.P11, U1.P12
- new net N$80: U$6.P12, U1.P13
- new net N$81: U$6.P13, U1.P14
- new net N$82: U$6.P14, U1.P15
- new net N$83: U$6.P15, U1.P17
- new net N$84: U$6.P16, U1.P18
- new net N$85: U$6.P17, U1.P20
- new net N$86: U$6.P18, U1.P21
- new net N$87: U$6.P19, U1.P23
- new net N$88: U$6.P20, U1.P24
- new net N$89: U$6.P21, U1.P25
- new net N$90: U$6.P22, U1.P26
- new net N$91: U$6.P23, U1.P27
- new net N$92: U$6.P25, U1.P28
- new net N$93: U$6.P26, U1.P30
- new net N$94: U$6.P27, U1.P31
- new net N$95: U$6.P28, U1.P32
- new net N$96: U$6.P29, U1.P33
- new net N$97: U$6.P31, U1.P35
- new net N$98: U$6.P32, U1.P36
- net GND: now also C34.2, U$6.P24, U$6.P30
- net N$67: now also U$6.P1, U1.P1; no longer U1.P26
- net N$73: now also U$6.P4, U1.P5; no longer U1.P12
- net PS2CLK: now also U1.P141; no longer U1.P2
- net PS2DAT: now also U1.P140; no longer U1.P1
- net VCC: now also C34.1, U$6.P8
Routing:
- net N$84: track 0.00 -> 19.6 mm
- net N$83: track 0.00 -> 18.6 mm
- net N$85: track 0.00 -> 18.5 mm
- net N$86: track 0.00 -> 17.5 mm
- net N$82: track 0.00 -> 17.1 mm
- net N$81: track 0.00 -> 16.1 mm
- net N$87: track 0.00 -> 16.0 mm
- net N$80: track 0.00 -> 15.1 mm
- net N$88: track 0.00 -> 15.0 mm
- net N$79: track 0.00 -> 14.1 mm
- net N$89: track 0.00 -> 14.0 mm
- net N$78: track 0.00 -> 13.1 mm
- net N$90: track 0.00 -> 13.0 mm
- net N$77: track 0.00 -> 12.1 mm
- net N$91: track 0.00 -> 12.0 mm
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
Commit message: got both rams for now...
Parts:
- moved IC3 5.70 mm to (59.0, 59.5)
- moved C10 1.00 mm to (42.0, 40.8)
- moved C11 1.00 mm to (27.8, 41.0)
- moved C12 1.00 mm to (29.0, 47.0)
- moved C13 1.00 mm to (42.5, 47.0)
- moved C14 1.00 mm to (29.0, 35.5)
- moved C15 1.00 mm to (32.8, 37.0)
- moved C16 1.00 mm to (26.8, 34.5)
- moved C17 1.00 mm to (42.5, 35.0)
- moved C18 1.00 mm to (38.0, 35.5)
- moved C19 1.00 mm to (31.2, 47.8)
- moved C20 1.00 mm to (38.0, 47.2)
- moved C21 1.00 mm to (31.2, 34.2)
- moved C22 1.00 mm to (33.5, 48.2)
- moved C23 1.00 mm to (35.8, 48.2)
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Routing:
- net GND: track 592.1 -> 594.7 mm
- net R0: track 15.4 -> 13.8 mm
- net G0: track 12.7 -> 11.1 mm
- net CSYNC: track 21.3 -> 19.7 mm
- net N$29: track 16.4 -> 17.9 mm
- net CLK16: track 25.0 -> 23.6 mm
- net VCCAUX: track 98.4 -> 97.0 mm
- net R1: track 16.7 -> 15.4 mm
- net PROM_INITB: track 24.3 -> 25.3 mm
- net N$5: track 7.99 -> 8.99 mm
- net VCCINT: track 84.6 -> 83.6 mm
- net RESET: track 42.4 -> 41.4 mm
- net PROM_DO: track 19.5 -> 20.5 mm
- net N$9: track 13.0 -> 14.0 mm
- net N$8: track 11.5 -> 12.5 mm
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
Commit message: more than enough for one day...
Parts:
- moved R1 1.75 mm to (24.0, 53.7), turned to 180 degrees
- moved R4 1.50 mm to (18.5, 62.8)
- moved R47 1.50 mm to (15.2, 63.0)
- moved R5 1.50 mm to (14.5, 66.2)
- moved R51 1.50 mm to (22.0, 66.2)
- moved R6 1.50 mm to (24.5, 62.8)
- moved R7 1.50 mm to (28.5, 66.2)
- moved T1 1.50 mm to (18.5, 65.8)
- moved T3 1.50 mm to (24.5, 65.8)
Connections:
- removed net PE1: X3.SH1
- removed net PE3: X3.SH3
- net GND: now also X3.SH1, X3.SH3
Routing:
- net GND: track 594.7 -> 605.3 mm
- net CLK_5V: track 9.74 -> 8.24 mm
- net DATA_5V: track 13.3 -> 11.8 mm
- net VCC: track 409.5 -> 410.4 mm
- net VCC5: track 89.1 -> 88.2 mm
