File: eagle/homeboard/homeboard11.sch (EAGLE design)
At the start: 113 parts, among them IC1 XCF02S, IC2 25LC080SN, IC3 ATMEGA32U2-TQFP, Q5 BC848SMD, Q6 BC848SMD, Q7 BC848SMD, Q8 BC848SMD, T1 BSS138, T2 BC848, T3 BSS138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

Commit message: got both rams for now...
Parts:
- added C34: 100nF, rcl:C-EUC0603
- added U$6: AS6C4008, cpcfpga:AS6C4008
Connections:
- removed net XXR0: U1B0.IO_L01P_0VRN_0
- removed net XXR1: U1B0.IO_L01N_0VRP_0
- new net N$71: U$6.A9, U1B7.IO_L01N_7VRP_7
- new net N$72: U$6.A8, U1B7.IOVREF_7
- new net N$74: U$6.WE, U1B7.IO_L20N_7
- new net N$75: U$6.A17, U1B7.IO_L21P_7
- new net N$76: U$6.A15, U1B7.IO_L21N_7
- new net N$77: U$6.A18, U1B7.IO_L22P_7
- new net N$78: U$6.A16, U1B7.IO_L22N_7
- new net N$79: U$6.A14, U1B7.IO_L23P_7
- new net N$80: U$6.A12, U1B7.IO_L23N_7
- new net N$81: U$6.A7, U1B7.IO_L24P_7
- new net N$82: U$6.A6, U1B7.IO_L24N_7
- new net N$83: U$6.A5, U1B7.IO_L40P_7
- new net N$84: U$6.A4, U1B7.IO_L40N_7VREF_7
- new net N$85: U$6.A3, U1B6.IO_L40P_6VREF_6
- new net N$86: U$6.A2, U1B6.IO_L40N_6
- new net N$87: U$6.A1, U1B6.IO_L24P_6
- new net N$88: U$6.A0, U1B6.IO_L24N_6VREF_6
- new net N$89: U$6.DQ0, U1B6.IO_L23P_6
- new net N$90: U$6.DQ1, U1B6.IO_L23N_6
- new net N$91: U$6.DQ2, U1B6.IO_L22P_6
- new net N$92: U$6.DQ3, U1B6.IO_L22N_6
- new net N$93: U$6.DQ4, U1B6.IO_L21P_6
- new net N$94: U$6.DQ5, U1B6.IO_L21N_6
- new net N$95: U$6.DQ6, U1B6.IO_L20P_6
- new net N$96: U$6.DQ7, U1B6.IO_L20N_6
- new net N$97: U$6.A10, U1B6.IO_L01P_6VRN_6
- new net N$98: U$6.OE, U1B6.IO_L01N_6VRP_6
- net GND: now also C34.2, U$6.CE, U$6.VSS
- net N$67: now also U$6.A11, U1B7.IO_L01P_7VRN_7; no longer U1B6.IO_L23N_6
- net N$73: now also U$6.A13, U1B7.IO_L20P_7; no longer U1B7.IO_L23P_7
- net PS2CLK: now also U1B0.IO_L01N_0VRP_0; no longer U1B7.IO_L01N_7VRP_7
- net PS2DAT: now also U1B0.IO_L01P_0VRN_0; no longer U1B7.IO_L01P_7VRN_7
- net VCC: now also C34.1, U$6.VCC
Other:
- moved on the sheet: R35, R36, R37, R38, R39, R40, R41, R42, R43, R44, R45, R46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

Commit message: more than enough for one day...
Connections:
- net GND: now also X3.PE1, X3.PE3
Changed lines of the file:
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@@
 <segment>
 <pinref part="X3" gate="G$1" pin="PE2"/>
-<wire x1="279.4" y1="-236.22" x2="309.88" y2="-236.22" width="0.1524" layer="91"/>
+<wire x1="279.4" y1="-236.22" x2="292.1" y2="-236.22" width="0.1524" layer="91"/>
 <label x="309.88" y="-236.22" size="1.778" layer="95"/>
+<pinref part="X3" gate="G$1" pin="PE1"/>
+<wire x1="292.1" y1="-236.22" x2="309.88" y2="-236.22" width="0.1524" layer="91"/>
+<wire x1="292.1" y1="-231.14" x2="292.1" y2="-236.22" width="0.1524" layer="91"/>
+<junction x="292.1" y="-236.22"/>
+<pinref part="X3" gate="G$1" pin="PE3"/>
+<wire x1="266.7" y1="-231.14" x2="266.7" y2="-236.22" width="0.1524" layer="91"/>
+<wire x1="266.7" y1="-236.22" x2="279.4" y2="-236.22" width="0.1524" layer="91"/>
+<junction x="279.4" y="-236.22"/>
 </segment>
 <segment>
