File: eagle/homeboard/homeboard14.brd (EAGLE design)
At the start: 100 x 80 mm, 121 parts, among them IC1 XCF02S, IC2 25LC080SN, IC3 ATMEGA32U2-TQFP, Q5 BC848SMD, Q6 BC848SMD, Q7 BC848SMD, Q8 BC848SMD, T1 BSS138, T2 BC848, T3 BSS138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

Commit message: mah
Parts:
- moved X6 24.0 mm to (91.5, 77.0), turned to 270 degrees
- moved R8 3.88 mm to (32.0, 21.8), turned to 270 degrees
- moved R9 1.41 mm to (34.5, 21.8), turned to 270 degrees
- moved R10 1.12 mm to (37.2, 21.8), turned to 270 degrees
- moved SV1 1.00 mm to (27.0, 25.5)
Connections:
- removed net N$104: SV1.7, U1.P50
- removed net N$106: SV1.8, U1.P52
- new net N$1111: SV1.7, U1.P47
- new net N$1112: SV1.8, U1.P51
- new net N$1113: SV1.9, U1.P53
- net CSYNC: now also U1.P50; no longer U1.P47
- net G1: now also U1.P57; no longer U1.P56
- net GND: now also SV1.2; no longer SV1.1
- net R0: now also U1.P55; no longer U1.P53
- net R1: now also U1.P52; no longer U1.P51
- net VCC: now also SV1.1; no longer SV1.2
- net X: no longer SV1.9, U1.P55
- net XXX: now also U1.P56; no longer U1.P57
Routing:
- net N$38: track 13.3 -> 29.3 mm
- net PROM_INITB: track 24.5 -> 8.73 mm, vias 3 -> 0
- net N$35: track 11.4 -> 25.5 mm
- net PROM_DO: track 16.9 -> 29.5 mm
- net VCCAUX: track 111.5 -> 101.1 mm, vias 7 -> 6
- net GND: track 698.7 -> 688.6 mm, vias 35 -> 34
- net G0: track 0.00 -> 8.81 mm
- net B1: track 0.00 -> 6.06 mm
- net N$1111: track 0.00 -> 5.70 mm
- net N$104: track 5.49 -> 0.00 mm
- net X: track 5.23 -> 0.00 mm
- net N$1113: track 0.00 -> 5.18 mm
- net N$63: track 5.05 -> 0.00 mm, vias 1 -> 0
- net N$1112: track 0.00 -> 4.99 mm
- net N$106: track 4.85 -> 0.00 mm
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
Commit message: mah
Parts:
- moved R8 4.61 mm to (27.5, 20.8), turned to 0 degrees
- moved R9 1.60 mm to (33.2, 20.8), turned to 0 degrees
- moved R10 1.03 mm to (37.5, 20.8), turned to 180 degrees
- moved SV1 1.00 mm to (27.0, 24.5)
Routing:
- net VCC: track 332.3 -> 359.5 mm
- net N$99: track 12.6 -> 0.00 mm
- net G1: track 12.3 -> 0.00 mm
- net N$100: track 10.1 -> 0.00 mm
- net G0: track 8.81 -> 0.00 mm
- net PROM_INITB: track 8.73 -> 0.00 mm
- net N$101: track 8.67 -> 0.00 mm
- net CSYNC: track 8.21 -> 0.00 mm
- net R0: track 8.08 -> 0.00 mm
- net N$53: track 0.00 -> 7.46 mm, vias 0 -> 1
- net N$102: track 6.87 -> 0.00 mm
- net B1: track 6.06 -> 0.00 mm
- net N$1111: track 5.70 -> 0.00 mm
- net N$63: track 0.00 -> 4.23 mm, vias 0 -> 1
- net R1: track 7.63 -> 11.8 mm
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
Commit message: mah
Connections:
- net B0: now also U1.P63; no longer U1.P68
- net B1: now also U1.P60; no longer U1.P63
- net FPGA_AUDIO_LEFT: now also U1.P68; no longer U1.P69
- net FPGA_AUDIO_RIGHT: now also U1.P69; no longer U1.P70
- net G0: now also U1.P59; no longer U1.P60
- net X: now also U1.P70; no longer U1.P59
Routing:
- net PROM_INITB: track 0.00 -> 41.4 mm, vias 0 -> 2
- net FPGA_AUDIO_RIGHT: track 0.00 -> 25.7 mm
- net FPGA_AUDIO_LEFT: track 0.00 -> 24.3 mm
- net B0: track 0.00 -> 23.3 mm
- net B1: track 0.00 -> 18.5 mm
- net G0: track 0.00 -> 17.8 mm
- net CSYNC: track 0.00 -> 14.8 mm
- net N$99: track 0.00 -> 13.1 mm
- net VCCAUX: track 101.1 -> 113.0 mm, vias 6 -> 7
- net G1: track 0.00 -> 11.5 mm
- net N$100: track 0.00 -> 11.1 mm
- net R0: track 0.00 -> 11.1 mm
- net N$101: track 0.00 -> 10.1 mm
- net N$102: track 0.00 -> 8.59 mm
- net N$1111: track 0.00 -> 6.28 mm
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
Commit message: mah
Routing:
- net VCC: vias 21 -> 19
- net GND: vias 34 -> 33
Changed lines of the file:
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@@
 <wire x1="75.5" y1="30.25" x2="76.5" y2="30.25" width="0.254" layer="16"/>
 <wire x1="76.5" y1="30.25" x2="76.5" y2="23.25" width="0.254" layer="16"/>
-<via x="12" y="1.25" extent="1-16" drill="0.6" shape="square"/>
 <contactref element="REG2.5" pad="1"/>
 <contactref element="U$4" pad="1"/>
@@
 <wire x1="58.335" y1="7.5" x2="58.5" y2="7.5" width="0" layer="19" extent="1-1"/>
 <wire x1="26.75" y1="32" x2="27.15" y2="35.1" width="0" layer="19" extent="16-16"/>
-<wire x1="12" y1="1.25" x2="15.5" y2="4" width="0" layer="19" extent="16-16"/>
 <wire x1="62.15" y1="17.5" x2="67.5" y2="13.25" width="0" layer="19" extent="1-16"/>
 <wire x1="58.1" y1="17.5" x2="62.15" y2="17.5" width="0" layer="19" extent="16-16"/>
@@
 <wire x1="75.393396875" y1="28.437409375" x2="75.393396875" y2="29.087409375" width="0.254" layer="1"/>
 <wire x1="75.393396875" y1="28.437409375" x2="75.393396875" y2="27.787409375" width="0.254" layer="1"/>
-<via x="87" y="24.5" extent="1-16" drill="0.6" shape="square"/>
 <via x="65" y="22.5" extent="1-16" drill="0.6" shape="square"/>
-<via x="14" y="1.5" extent="1-16" drill="0.6" shape="square"/>
 <wire x1="65" y1="22.5" x2="51.5" y2="22.5" width="0.254" layer="16"/>
 <wire x1="75.393396875" y1="27.787409375" x2="76.962590625" y2="27.787409375" width="0.254" layer="1"/>
@@
 <wire x1="91.4" y1="7" x2="92.95" y2="10.5" width="0" layer="19" extent="1-16"/>
 <wire x1="15.5" y1="62.5" x2="18.6" y2="53.5" width="0" layer="19" extent="1-1"/>
-<wire x1="87" y1="24.5" x2="77" y2="22.75" width="0" layer="19" extent="1-1"/>
-<wire x1="87.15" y1="31.5" x2="87" y2="24.5" width="0" layer="19" extent="1-1"/>
-<wire x1="86.65" y1="35.5" x2="87.15" y2="31.5" width="0" layer="19" extent="1-1"/>
-<wire x1="86.65" y1="40.5" x2="86.65" y2="35.5" width="0" layer="19" extent="1-1"/>
+<wire x1="80.355" y1="39.975" x2="75.5" y2="30.4" width="0" layer="19" extent="1-1"/>
+<wire x1="86.65" y1="40.5" x2="80.355" y2="39.975" width="0" layer="19" extent="1-1"/>
 <wire x1="86.65" y1="45.5" x2="86.65" y2="40.5" width="0" layer="19" extent="1-1"/>
+<wire x1="86.65" y1="35.5" x2="86.65" y2="40.5" width="0" layer="19" extent="1-1"/>
+<wire x1="87.15" y1="31.5" x2="86.65" y2="35.5" width="0" layer="19" extent="1-1"/>
 <wire x1="92.95" y1="40" x2="86.65" y2="40.5" width="0" layer="19" extent="1-1"/>
 <wire x1="98.45" y1="32.5" x2="97.45" y2="38.5" width="0" layer="19" extent="1-1"/>
-<wire x1="80.355" y1="39.975" x2="86.65" y2="40.5" width="0" layer="19" extent="1-1"/>
 <wire x1="37.57" y1="64.27" x2="35.97" y2="51.7" width="0" layer="19" extent="1-1"/>
-<wire x1="14" y1="1.5" x2="16" y2="22.5" width="0" layer="19" extent="16-16"/>
 </signal>
 <signal name="TCK">

Commit message: mah
Routing:
- net SCART_RED: track 0.00 -> 14.2 mm
- net SCART_BLUE: track 0.00 -> 14.2 mm
- net SCART_GREEN: track 0.00 -> 14.1 mm
- net GND: track 689.6 -> 702.8 mm
- net SCART_COMP: track 0.00 -> 12.4 mm
- net SCART_RIGHT: track 0.00 -> 10.3 mm
- net SCART_LEFT: track 0.00 -> 9.64 mm
- net N$58: track 0.00 -> 6.90 mm
- net N$56: track 0.00 -> 6.90 mm
- net N$54: track 0.00 -> 6.90 mm
- net N$51: track 0.00 -> 6.60 mm, vias 0 -> 1
- net N$59: track 0.00 -> 6.40 mm
- net N$65: track 0.00 -> 6.14 mm, vias 0 -> 1
- net N$57: track 0.00 -> 5.32 mm, vias 0 -> 1
- net PROM_DO: track 32.0 -> 35.7 mm
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
Commit message: work time
Parts:
- moved X1 85.8 mm to (68.5, 77.2), turned to 0 degrees
- moved X6 34.1 mm to (57.5, 74.5)
- moved X5 31.3 mm to (96.5, 64.0), turned to 270 degrees
- moved U$3 16.3 mm to (81.5, 57.0)
Connections:
- removed net N$102: SV1.6, U1.P46
- removed net N$1111: SV1.7, U1.P47
- removed net N$1112: SV1.8, U1.P51
- new net N$104: SV1.6, U1.P47
- new net QQQ: SV1.8, U1.P52
- new net QQQQ: SV1.7, U1.P50
- net CSYNC: now also U1.P46; no longer U1.P50
- net R1: now also U1.P51; no longer U1.P52
Routing:
- net N$102: track 8.59 -> 0.00 mm
- net N$104: track 0.00 -> 8.21 mm
- net QQQQ: track 0.00 -> 6.90 mm
- net N$1111: track 6.28 -> 0.00 mm
- net QQQ: track 0.00 -> 6.26 mm
- net N$1112: track 6.06 -> 0.00 mm
- net PROM_DO: track 35.7 -> 30.2 mm
- net CSYNC: track 14.8 -> 13.1 mm
- net N$99: track 13.1 -> 12.0 mm
- net N$100: track 11.1 -> 9.95 mm
- net R1: track 11.8 -> 10.8 mm
- net N$101: track 10.1 -> 9.23 mm
