File: eagle/homeboard/homeboard15.brd (EAGLE design)
At the start: 100 x 80 mm, 121 parts, among them IC1 XCF02S, IC2 25LC080SN, IC3 ATMEGA32U2-TQFP, Q5 BC848SMD, Q6 BC848SMD, Q7 BC848SMD, Q8 BC848SMD, T1 BSS138, T2 BC848, T3 BSS138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

Commit message: moved and ripped up... again
Parts:
- moved X1 38.9 mm to (107.2, 74.0), turned to 270 degrees
- moved X5 18.3 mm to (79.0, 69.5), turned to 0 degrees
- moved U$5 11.5 mm to (8.50, 38.0), flipped to the bottom, turned to 90 degrees
- moved C36 10.6 mm to (6.00, 20.0), turned to 180 degrees
- moved C33 6.50 mm to (6.25, 27.0)
- moved C35 6.50 mm to (6.00, 29.0)
- moved REG1.2 6.50 mm to (8.50, 41.8)
- moved REG2.5 6.50 mm to (8.50, 49.5)
- moved U$4 6.50 mm to (8.50, 34.0)
- moved IC3 6.32 mm to (91.5, 59.8)
- moved SV1 3.04 mm to (24.0, 25.0)
- moved U$3 3.00 mm to (81.5, 54.0)
- moved C1 2.00 mm to (55.2, 17.5)
- moved C3 2.00 mm to (57.2, 12.0)
- moved C4 2.00 mm to (60.5, 12.0)
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Routing:
- net FPGA_AUDIO_RIGHT: track 25.7 -> 0.00 mm
- net GND: track 702.8 -> 677.9 mm, vias 33 -> 32
- net FPGA_AUDIO_LEFT: track 24.3 -> 0.00 mm
- net B0: track 23.3 -> 0.00 mm
- net B1: track 18.5 -> 0.00 mm
- net G0: track 17.8 -> 0.00 mm
- net CSYNC: track 13.1 -> 0.64 mm
- net G1: track 11.5 -> 0.00 mm
- net R0: track 11.1 -> 0.03 mm
- net N$99: track 12.0 -> 1.33 mm
- net VCCAUX: track 113.0 -> 102.6 mm, vias 7 -> 6
- net R1: track 10.8 -> 0.71 mm
- net N$100: track 9.95 -> 0.00 mm
- net N$101: track 9.23 -> 0.00 mm
- net N$104: track 8.21 -> 0.00 mm
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
Commit message: mah
Parts:
- removed X8: DC21MMX, powersupply:DC-21MM
- added J1: (no value), con-jack:DCJ0303
- added X7: DC21MMX, powersupply:DC-21MM
Connections:
- new net 1: X7.1
- net GND: now also J1.3, X7.3; no longer X8.1, X8.3
- net VCC5: now also J1.1, X7.2; no longer X8.2
Routing:
- net VCC: track 363.2 -> 389.0 mm, vias 20 -> 22
- net GND: track 677.9 -> 653.0 mm, vias 32 -> 33
- net VCCAUX: track 102.6 -> 89.2 mm
- net VCC5: track 110.3 -> 98.1 mm
- net VCCINT: track 80.8 -> 82.1 mm

Commit message: mah
Routing:
- net GND: track 653.0 -> 664.9 mm, vias 33 -> 35
- net VCC: track 389.0 -> 398.4 mm
- net VCCAUX: track 89.2 -> 95.8 mm
- net VCCINT: track 82.1 -> 81.1 mm
Changed lines of the file:
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@@
 <contactref element="U$6" pad="P30"/>
 <wire x1="21.25" y1="31" x2="21.25" y2="30.25" width="0.254" layer="1"/>
-<wire x1="18.25" y1="30.5" x2="17.75" y2="30" width="0.254" layer="1"/>
-<wire x1="17.75" y1="30" x2="15.25" y2="30" width="0.254" layer="1"/>
-<wire x1="21.25" y1="30.25" x2="21" y2="30" width="0.254" layer="1"/>
-<wire x1="21" y1="30" x2="17.75" y2="30" width="0.254" layer="1"/>
 <contactref element="C34" pad="2"/>
 <wire x1="16.9" y1="53.5" x2="15.75" y2="53.5" width="0.254" layer="1"/>
@@
 <wire x1="25" y1="33" x2="26" y2="32" width="0.6" layer="16"/>
 <wire x1="26" y1="32" x2="26.75" y2="32" width="0.6" layer="16"/>
+<via x="21.25" y="30.25" extent="1-16" drill="0.6" shape="square"/>
+<wire x1="21.25" y1="30.25" x2="21.25" y2="30" width="0.254" layer="16"/>
+<wire x1="21.25" y1="30" x2="18.25" y2="30" width="0.254" layer="16"/>
+<via x="18.25" y="30.5" extent="1-16" drill="0.6" shape="square"/>
+<wire x1="18.25" y1="30.5" x2="18.25" y2="30" width="0.254" layer="16"/>
+<wire x1="18.25" y1="30" x2="15.25" y2="30" width="0.254" layer="16"/>
+<wire x1="15.25" y1="30" x2="15.25" y2="25.14" width="0.254" layer="16"/>
+<wire x1="15.25" y1="25.14" x2="15.11" y2="25" width="0.254" layer="16"/>
+<wire x1="26" y1="30" x2="21.5" y2="30" width="0.254" layer="16"/>
+<wire x1="21.5" y1="30" x2="21.25" y2="30.25" width="0.254" layer="16"/>
+<wire x1="26" y1="30" x2="26" y2="30.5" width="0.254" layer="16"/>
+<wire x1="26" y1="30.5" x2="26.5" y2="31" width="0.254" layer="16"/>
+<wire x1="26.75" y1="30.25" x2="26.75" y2="30.75" width="0.254" layer="16"/>
+<wire x1="26.75" y1="30.75" x2="26.5" y2="31" width="0.254" layer="16"/>
 <wire x1="80.3716" y1="70.77" x2="97" y2="76.3" width="0" layer="19" extent="1-1"/>
 <wire x1="71.4890875" y1="62.801446875" x2="80.3716" y2="70.77" width="0" layer="19" extent="1-1"/>
@@
 <wire x1="41.97" y1="51.7" x2="42" y2="51.75" width="0" layer="19" extent="1-1"/>
 <wire x1="29.47" y1="51.7" x2="29.5" y2="51.75" width="0" layer="19" extent="1-1"/>
-<wire x1="21.25" y1="31" x2="25" y2="33" width="0" layer="19" extent="1-16"/>
-<wire x1="15.11" y1="25" x2="15.25" y2="30" width="0" layer="19" extent="1-1"/>
 <wire x1="56.335" y1="7.5" x2="56.5" y2="7.5" width="0" layer="19" extent="1-1"/>
 <wire x1="8.4" y1="29" x2="8.65" y2="27" width="0" layer="19" extent="1-16"/>
@@
 <via x="13.75" y="31.5" extent="1-16" drill="0.6" shape="square"/>
 <wire x1="13.75" y1="31.5" x2="13.75" y2="32.25" width="0.6" layer="1"/>
-<wire x1="13.75" y1="32.25" x2="12" y2="34" width="0.6" layer="1"/>
+<wire x1="13.75" y1="32.25" x2="12.57" y2="33.43" width="0.6" layer="1"/>
+<wire x1="12.57" y1="25" x2="12.57" y2="33.43" width="0.6" layer="1"/>
+<wire x1="12.57" y1="33.43" x2="12" y2="34" width="0.6" layer="1"/>
+<wire x1="12" y1="34" x2="11.5" y2="34" width="0.6" layer="1"/>
+<wire x1="11.5" y1="34" x2="11.5" y2="33.5" width="0.6" layer="1"/>
 <wire x1="88.7" y1="64.0426" x2="89.5" y2="64.0426" width="0" layer="19" extent="1-1"/>
 <wire x1="87.2074" y1="60.15" x2="88.7" y2="64.0426" width="0" layer="19" extent="1-1"/>
 <wire x1="75.5" y1="52.25" x2="87.2074" y2="60.15" width="0" layer="19" extent="1-1"/>
-<wire x1="11.599" y1="34" x2="12" y2="34" width="0" layer="19" extent="1-1"/>
-<wire x1="12.57" y1="25" x2="14" y2="31.25" width="0" layer="19" extent="16-16"/>
+<wire x1="11.599" y1="34" x2="11.5" y2="34" width="0" layer="19" extent="1-1"/>
 <wire x1="16" y1="22.5" x2="12.57" y2="25" width="0" layer="19" extent="16-16"/>
 <wire x1="66.2890875" y1="58.991446875" x2="67" y2="52.25" width="0" layer="19" extent="1-1"/>
@@
 <wire x1="37" y1="44.25" x2="38" y2="45.25" width="0.6" layer="1"/>
 <wire x1="38" y1="45.25" x2="38" y2="50.25" width="0.6" layer="1"/>
-<via x="13.5" y="42.25" extent="1-16" drill="0.6" shape="square"/>
 <wire x1="26.5" y1="39.25" x2="26.5" y2="38.25" width="0.6" layer="16"/>
 <wire x1="26.5" y1="38.25" x2="31" y2="38.25" width="0.6" layer="16"/>
 <wire x1="31" y1="38.25" x2="33.5" y2="40.75" width="0.6" layer="16"/>
 <wire x1="33.5" y1="40.75" x2="37" y2="40.75" width="0.6" layer="16"/>
-<wire x1="11" y1="42.349" x2="11.599" y2="41.75" width="0.6" layer="1"/>
 <wire x1="26.5" y1="39.25" x2="16" y2="39.25" width="0.6" layer="16"/>
 <wire x1="16" y1="39.25" x2="14" y2="40.5" width="0.6" layer="16"/>
-<wire x1="14" y1="40.5" x2="13.5" y2="40.5" width="0.6" layer="16"/>
-<wire x1="13.5" y1="40.5" x2="14.75" y2="39.25" width="0" layer="19" extent="1-16"/>
-<wire x1="14.5" y1="39.25" x2="15.25" y2="39.25" width="0" layer="19" extent="1-16"/>
-<wire x1="14.75" y1="39.25" x2="14.5" y2="39.25" width="0" layer="19" extent="1-16"/>
-<wire x1="13.5" y1="42.25" x2="11.25" y2="42.25" width="0.6" layer="1"/>
-<wire x1="11.25" y1="42.25" x2="11" y2="42.5" width="0.6" layer="1"/>
-<wire x1="11" y1="42.349" x2="11" y2="42.5" width="0.6" layer="1"/>
+<via x="14" y="40.5" extent="1-16" drill="0.6" shape="square"/>
+<wire x1="14" y1="40.5" x2="13" y2="40.5" width="0.6" layer="1"/>
+<wire x1="13" y1="40.5" x2="11.5" y2="42" width="0.6" layer="1"/>
 <wire x1="38.5" y1="51.75" x2="38.47" y2="51.7" width="0" layer="19" extent="1-1"/>
-<wire x1="13.5" y1="42.25" x2="14.5" y2="39.25" width="0" layer="19" extent="16-16"/>
+<wire x1="11.599" y1="41.75" x2="11.5" y2="42" width="0" layer="19" extent="1-1"/>
 </signal>
 <signal name="VCCAUX">
@@
 <wire x1="32.5" y1="37.75" x2="33.5" y2="38.75" width="0.254" layer="1"/>
 <wire x1="33.5" y1="38.75" x2="39.5" y2="38.75" width="0.254" layer="1"/>
-<via x="13.5" y="50" extent="1-16" drill="0.6" shape="square"/>
 <wire x1="26.5" y1="42.25" x2="26.5" y2="43.75" width="0.6" layer="16"/>
 <wire x1="26.5" y1="43.75" x2="31.5" y2="43.75" width="0.6" layer="16"/>
@@
 <wire x1="39" y1="47.85" x2="39" y2="49.25" width="0.254" layer="16"/>
 <wire x1="11" y1="48.75" x2="11.5" y2="49.25" width="0.6" layer="1"/>
-<wire x1="26.5" y1="42.25" x2="15" y2="42.25" width="0.6" layer="16"/>
+<wire x1="26.5" y1="42.25" x2="14.25" y2="42.25" width="0.6" layer="16"/>
 <wire x1="11.5" y1="49.25" x2="12" y2="49.25" width="0.6" layer="1"/>
 <wire x1="12" y1="49.25" x2="12" y2="49" width="0.6" layer="1"/>
 <wire x1="12" y1="49" x2="11.599" y2="49" width="0.6" layer="1"/>
 <wire x1="11.599" y1="49" x2="11.599" y2="49.5" width="0.6" layer="1"/>
-<wire x1="13.5" y1="50" x2="12.099" y2="50" width="0.6" layer="1"/>
-<wire x1="12.099" y1="50" x2="11.599" y2="49.5" width="0.6" layer="1"/>
 <wire x1="32" y1="31.25" x2="32" y2="31.75" width="0.254" layer="16"/>
 <wire x1="20.3" y1="19.75" x2="20.3" y2="20.7" width="0.254" layer="1"/>
 <wire x1="20.3" y1="20.7" x2="20.5" y2="22.5" width="0.254" layer="1"/>
 <wire x1="20.5" y1="22.5" x2="19.5" y2="22.5" width="0.254" layer="1"/>
-<wire x1="15" y1="42.25" x2="12" y2="49" width="0" layer="19" extent="1-16"/>
+<wire x1="14.25" y1="42.25" x2="14" y2="42.5" width="0.6" layer="16"/>
+<wire x1="14" y1="42.5" x2="14" y2="47.5" width="0.6" layer="16"/>
+<wire x1="14" y1="47.5" x2="13.5" y2="48" width="0.6" layer="16"/>
+<via x="13.5" y="48" extent="1-16" drill="0.6" shape="square"/>
+<wire x1="13.5" y1="48" x2="13" y2="48" width="0.6" layer="1"/>
+<wire x1="13" y1="48" x2="12" y2="49" width="0.6" layer="1"/>
 <wire x1="20.5" y1="22.5" x2="32.47" y2="30.3" width="0" layer="19" extent="1-1"/>
 </signal>

Commit message: mah
Connections:
- removed net N$1113: SV1.9, U1.P53
- removed net QQQ: SV1.8, U1.P52
- new net AASA: SV1.8, U1.P51
- new net SAA: SV1.9, U1.P52
- net R0: now also U1.P56; no longer U1.P55
- net R1: now also U1.P53; no longer U1.P51
- net XXX: now also U1.P55; no longer U1.P56
Routing:
- net CSYNC: track 0.64 -> 17.1 mm
- net N$99: track 1.33 -> 16.2 mm
- net N$100: track 0.00 -> 14.1 mm
- net R1: track 0.71 -> 13.9 mm
- net N$101: track 0.00 -> 12.5 mm
- net N$104: track 0.00 -> 11.2 mm
- net R0: track 0.03 -> 10.00 mm
- net QQQQ: track 0.00 -> 9.69 mm, vias 0 -> 1
- net AASA: track 0.00 -> 7.62 mm
- net SAA: track 0.00 -> 5.91 mm
- net XXX: track 0.00 -> 5.49 mm
- net GND: track 664.9 -> 666.1 mm
Changed lines of the file:
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@@
 <wire x1="26.75" y1="32" x2="26.75" y2="30.25" width="0.6" layer="16"/>
 <contactref element="U$6" pad="P24"/>
-<wire x1="18.25" y1="31" x2="18.25" y2="30.5" width="0.254" layer="1"/>
+<wire x1="18.25" y1="31" x2="18.25" y2="30" width="0.254" layer="1"/>
 <via x="51" y="57.75" extent="1-16" drill="0.6" shape="square"/>
 <contactref element="U$6" pad="P30"/>
-<wire x1="21.25" y1="31" x2="21.25" y2="30.25" width="0.254" layer="1"/>
+<wire x1="21.25" y1="31" x2="21.25" y2="30" width="0.254" layer="1"/>
 <contactref element="C34" pad="2"/>
 <wire x1="16.9" y1="53.5" x2="15.75" y2="53.5" width="0.254" layer="1"/>
@@
 <wire x1="25" y1="33" x2="26" y2="32" width="0.6" layer="16"/>
 <wire x1="26" y1="32" x2="26.75" y2="32" width="0.6" layer="16"/>
-<via x="21.25" y="30.25" extent="1-16" drill="0.6" shape="square"/>
-<wire x1="21.25" y1="30.25" x2="21.25" y2="30" width="0.254" layer="16"/>
-<wire x1="21.25" y1="30" x2="18.25" y2="30" width="0.254" layer="16"/>
-<via x="18.25" y="30.5" extent="1-16" drill="0.6" shape="square"/>
-<wire x1="18.25" y1="30.5" x2="18.25" y2="30" width="0.254" layer="16"/>
-<wire x1="18.25" y1="30" x2="15.25" y2="30" width="0.254" layer="16"/>
-<wire x1="15.25" y1="30" x2="15.25" y2="25.14" width="0.254" layer="16"/>
+<via x="21.25" y="30" extent="1-16" drill="0.6" shape="square"/>
+<wire x1="21.25" y1="30" x2="21.25" y2="29.5" width="0.254" layer="16"/>
+<wire x1="21.25" y1="29.5" x2="18.25" y2="29.5" width="0.254" layer="16"/>
+<via x="18.25" y="30" extent="1-16" drill="0.6" shape="square"/>
+<wire x1="18.25" y1="30" x2="18.25" y2="29.5" width="0.254" layer="16"/>
+<wire x1="18.25" y1="29.5" x2="15.25" y2="29.5" width="0.254" layer="16"/>
+<wire x1="15.25" y1="29.5" x2="15.25" y2="25.14" width="0.254" layer="16"/>
 <wire x1="15.25" y1="25.14" x2="15.11" y2="25" width="0.254" layer="16"/>
-<wire x1="26" y1="30" x2="21.5" y2="30" width="0.254" layer="16"/>
-<wire x1="21.5" y1="30" x2="21.25" y2="30.25" width="0.254" layer="16"/>
-<wire x1="26" y1="30" x2="26" y2="30.5" width="0.254" layer="16"/>
+<wire x1="26" y1="29.5" x2="21.5" y2="29.5" width="0.254" layer="16"/>
+<wire x1="21.5" y1="29.5" x2="21.25" y2="30" width="0.254" layer="16"/>
+<wire x1="26" y1="29.5" x2="26" y2="30.5" width="0.254" layer="16"/>
 <wire x1="26" y1="30.5" x2="26.5" y2="31" width="0.254" layer="16"/>
 <wire x1="26.75" y1="30.25" x2="26.75" y2="30.75" width="0.254" layer="16"/>
@@
 <signal name="R1">
 <contactref element="R9" pad="1"/>
-<contactref element="U1" pad="P51"/>
 <wire x1="30" y1="21" x2="30.5" y2="20.5" width="0.254" layer="1"/>
-<wire x1="30" y1="21" x2="33.97" y2="30.3" width="0" layer="19" extent="1-1"/>
+<contactref element="U1" pad="P53"/>
+<wire x1="34.97" y1="30.3" x2="34.97" y2="26.97" width="0.254" layer="1"/>
+<wire x1="34.97" y1="26.97" x2="34.25" y2="26.25" width="0.254" layer="1"/>
+<wire x1="34.25" y1="26.25" x2="34.25" y2="23.25" width="0.254" layer="1"/>
+<wire x1="34.25" y1="23.25" x2="33.5" y2="22.5" width="0.254" layer="1"/>
+<wire x1="33.5" y1="22.5" x2="30.5" y2="22.5" width="0.254" layer="1"/>
+<wire x1="30.5" y1="22.5" x2="30.5" y2="20.95" width="0.254" layer="1"/>
+<wire x1="30.5" y1="20.95" x2="30.3" y2="20.75" width="0.254" layer="1"/>
 <wire x1="30.3" y1="20.75" x2="30.5" y2="20.5" width="0" layer="19" extent="1-1"/>
 </signal>
 <signal name="R0">
 <contactref element="R10" pad="1"/>
-<contactref element="U1" pad="P55"/>
-<wire x1="35.97" y1="30.3" x2="36" y2="30.3" width="0.254" layer="1"/>
-<wire x1="36.45" y1="20.75" x2="35.97" y2="30.3" width="0" layer="19" extent="1-1"/>
+<contactref element="U1" pad="P56"/>
+<wire x1="36.47" y1="30.3" x2="36.47" y2="26.53" width="0.254" layer="1"/>
+<wire x1="36.47" y1="26.53" x2="37" y2="26" width="0.254" layer="1"/>
+<wire x1="37" y1="26" x2="37" y2="21.3" width="0.254" layer="1"/>
+<wire x1="37" y1="21.3" x2="36.45" y2="20.75" width="0.254" layer="1"/>
 </signal>
 <signal name="G1">
@@
 <contactref element="U1" pad="P46"/>
 <wire x1="25" y1="21.2" x2="24.55" y2="20.75" width="0.254" layer="1"/>
-<wire x1="25" y1="21.2" x2="31.47" y2="30.3" width="0" layer="19" extent="1-1"/>
+<wire x1="31.47" y1="30.3" x2="31.5" y2="30.3" width="0.254" layer="1"/>
+<wire x1="24" y1="27.5" x2="24" y2="21" width="0.254" layer="1"/>
+<wire x1="24" y1="21" x2="24.55" y2="21" width="0.254" layer="1"/>
+<wire x1="24.55" y1="21" x2="24.55" y2="20.75" width="0.254" layer="1"/>
+<wire x1="24" y1="27.5" x2="30" y2="27.5" width="0.254" layer="1"/>
+<wire x1="30" y1="27.5" x2="31.5" y2="29" width="0.254" layer="1"/>
+<wire x1="31.5" y1="29" x2="31.5" y2="30" width="0.254" layer="1"/>
+<wire x1="31.5" y1="30" x2="31.47" y2="30.3" width="0" layer="19" extent="1-1"/>
 </signal>
 <signal name="CASIN">
@@
 <contactref element="U1" pad="P40"/>
 <contactref element="SV1" pad="3"/>
-<wire x1="28.47" y1="30.3" x2="28.47" y2="28.97" width="0.254" layer="1"/>
-<wire x1="17.65" y1="25" x2="28.47" y2="28.97" width="0" layer="19" extent="1-1"/>
+<wire x1="28.47" y1="30.3" x2="28.5" y2="30.3" width="0.254" layer="1"/>
+<wire x1="28.5" y1="30.3" x2="28.5" y2="29" width="0.254" layer="1"/>
+<wire x1="28.5" y1="29" x2="17.65" y2="29" width="0.254" layer="1"/>
+<wire x1="17.65" y1="29" x2="17.65" y2="25" width="0.254" layer="1"/>
 </signal>
 <signal name="N$100">
 <contactref element="U1" pad="P41"/>
 <contactref element="SV1" pad="4"/>
-<wire x1="20.19" y1="25" x2="28.97" y2="30.3" width="0" layer="19" extent="1-1"/>
+<wire x1="28.97" y1="30.3" x2="29" y2="30.3" width="0.254" layer="1"/>
+<wire x1="29" y1="30.3" x2="29" y2="28.5" width="0.254" layer="1"/>
+<wire x1="29" y1="28.5" x2="20.19" y2="28.5" width="0.254" layer="1"/>
+<wire x1="20.19" y1="28.5" x2="20.19" y2="25" width="0.254" layer="1"/>
 </signal>
 <signal name="N$101">
 <contactref element="U1" pad="P44"/>
 <contactref element="SV1" pad="5"/>
-<wire x1="22.73" y1="25" x2="30.47" y2="30.3" width="0" layer="19" extent="1-1"/>
+<wire x1="30.47" y1="30.3" x2="30.5" y2="30.3" width="0.254" layer="1"/>
+<wire x1="22.73" y1="28" x2="22.73" y2="25" width="0.254" layer="1"/>
+<wire x1="30.5" y1="30.3" x2="30.5" y2="29" width="0.254" layer="1"/>
+<wire x1="30.5" y1="29" x2="29.5" y2="28" width="0.254" layer="1"/>
+<wire x1="29.5" y1="28" x2="22.75" y2="28" width="0.254" layer="1"/>
+<wire x1="22.73" y1="28" x2="22.75" y2="28" width="0" layer="19" extent="1-1"/>
 </signal>
 <signal name="X">
@@
 <signal name="XXX">
 <contactref element="SV1" pad="10"/>
-<contactref element="U1" pad="P56"/>
-<wire x1="35.43" y1="25" x2="36.47" y2="30.3" width="0" layer="19" extent="1-1"/>
-</signal>
-<signal name="N$1113">
-<contactref element="U1" pad="P53"/>
-<contactref element="SV1" pad="9"/>
-<wire x1="32.89" y1="25" x2="34.97" y2="30.3" width="0" layer="19" extent="1-1"/>
+<contactref element="U1" pad="P55"/>
+<wire x1="35.97" y1="30.3" x2="35.97" y2="25.47" width="0.254" layer="1"/>
+<wire x1="35.97" y1="25.47" x2="35.5" y2="25" width="0.254" layer="1"/>
+<wire x1="35.5" y1="25" x2="35.43" y2="25" width="0" layer="19" extent="1-1"/>
 </signal>
 <signal name="N$104">
 <contactref element="SV1" pad="6"/>
 <contactref element="U1" pad="P47"/>
-<wire x1="25.27" y1="25" x2="31.97" y2="30.3" width="0" layer="19" extent="1-1"/>
+<wire x1="31.97" y1="30.3" x2="32" y2="30.3" width="0.254" layer="1"/>
+<wire x1="25.27" y1="27" x2="25.27" y2="25" width="0.254" layer="1"/>
+<wire x1="25.27" y1="27" x2="30.5" y2="27" width="0.254" layer="1"/>
+<wire x1="30.5" y1="27" x2="32" y2="28.5" width="0.254" layer="1"/>
+<wire x1="32" y1="28.5" x2="32" y2="30.27" width="0.254" layer="1"/>
+<wire x1="32" y1="30.27" x2="31.97" y2="30.3" width="0.254" layer="1"/>
 </signal>
 <signal name="QQQQ">
 <contactref element="U1" pad="P50"/>
 <contactref element="SV1" pad="7"/>
-<wire x1="27.81" y1="25" x2="33.47" y2="30.3" width="0" layer="19" extent="1-1"/>
-</signal>
-<signal name="QQQ">
-<contactref element="U1" pad="P52"/>
-<contactref element="SV1" pad="8"/>
-<wire x1="30.35" y1="25" x2="34.47" y2="30.3" width="0" layer="19" extent="1-1"/>
+<wire x1="33.47" y1="30.3" x2="33.47" y2="28.97" width="0.254" layer="1"/>
+<wire x1="33.47" y1="28.97" x2="33" y2="28.5" width="0.254" layer="1"/>
+<via x="33" y="28.5" extent="1-16" drill="0.6" shape="square"/>
+<wire x1="33" y1="28.5" x2="29.5" y2="28.5" width="0.254" layer="16"/>
+<wire x1="29.5" y1="28.5" x2="28" y2="27" width="0.254" layer="16"/>
+<wire x1="28" y1="27" x2="28" y2="25.19" width="0.254" layer="16"/>
+<wire x1="28" y1="25.19" x2="27.81" y2="25" width="0.254" layer="16"/>
 </signal>
 <signal name="1">
 <contactref element="X7" pad="1"/>
 </signal>
+<signal name="AASA">
+<contactref element="U1" pad="P51"/>
+<contactref element="SV1" pad="8"/>
+<wire x1="33.97" y1="30.3" x2="33.97" y2="27.97" width="0.254" layer="1"/>
+<wire x1="33.97" y1="27.97" x2="33.5" y2="27.5" width="0.254" layer="1"/>
+<wire x1="33.5" y1="27.5" x2="32" y2="27.5" width="0.254" layer="1"/>
+<wire x1="32" y1="27.5" x2="30.5" y2="26" width="0.254" layer="1"/>
+<wire x1="30.5" y1="26" x2="30.5" y2="25" width="0.254" layer="1"/>
+<wire x1="30.35" y1="25" x2="30.5" y2="25" width="0" layer="19" extent="1-1"/>
+</signal>
+<signal name="SAA">
+<contactref element="U1" pad="P52"/>
+<contactref element="SV1" pad="9"/>
+<wire x1="34.47" y1="30.3" x2="34.47" y2="27.47" width="0.254" layer="1"/>
+<wire x1="34.47" y1="27.47" x2="33" y2="26" width="0.254" layer="1"/>
+<wire x1="33" y1="26" x2="33" y2="25" width="0.254" layer="1"/>
+<wire x1="33" y1="25" x2="32.89" y2="25" width="0" layer="19" extent="1-1"/>
+</signal>
 </signals>

Commit message: mah
Parts:
- SV1: device con-lstb:MA10-1 -> con-lstb:MA12-1
- moved SV1 2.50 mm to (26.5, 25.0)
Connections:
- removed net X: U1.P70
- new net XXZXZ: SV1.11, U1.P57
- net B0: now also U1.P68; no longer U1.P63
- net B1: now also U1.P63; no longer U1.P60
- net FPGA_AUDIO_LEFT: now also U1.P69; no longer U1.P68
- net FPGA_AUDIO_RIGHT: now also U1.P70; no longer U1.P69
- net G0: now also U1.P60; no longer U1.P59
- net G1: now also U1.P59; no longer U1.P57
- net GND: now also SV1.12
Routing:
- net GND: track 666.1 -> 694.1 mm
- net FPGA_AUDIO_RIGHT: track 0.00 -> 22.9 mm
- net FPGA_AUDIO_LEFT: track 0.00 -> 21.2 mm
- net B0: track 0.00 -> 18.5 mm
- net B1: track 0.00 -> 15.6 mm
- net G0: track 0.00 -> 14.4 mm
- net G1: track 0.00 -> 10.00 mm
- net VCC: track 398.4 -> 404.4 mm, vias 22 -> 23
- net XXZXZ: track 0.00 -> 5.73 mm
- net R0: track 10.00 -> 10.5 mm
