File: eagle/homeboard/homeboard15.brd (EAGLE design)
At the start: 100 x 80 mm, 122 parts, among them IC1 XCF02S, IC2 25LC080SN, IC3 ATMEGA32U2-TQFP, Q5 BC848SMD, Q6 BC848SMD, Q7 BC848SMD, Q8 BC848SMD, T1 BSS138, T2 BC848, T3 BSS138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

Commit message: mah
Routing:
- net VCCAUX: track 95.8 -> 113.9 mm, vias 6 -> 7
- net VCC: track 404.4 -> 398.6 mm
- net GND: track 694.1 -> 693.5 mm
Changed lines of the file:
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@@
 <wire x1="18.25" y1="29.5" x2="15.25" y2="29.5" width="0.254" layer="16"/>
 <wire x1="15.25" y1="29.5" x2="15.25" y2="25.14" width="0.254" layer="16"/>
-<wire x1="26" y1="29.5" x2="21.5" y2="29.5" width="0.254" layer="16"/>
+<wire x1="25" y1="29.5" x2="21.5" y2="29.5" width="0.254" layer="16"/>
 <wire x1="21.5" y1="29.5" x2="21.25" y2="30" width="0.254" layer="16"/>
-<wire x1="26" y1="29.5" x2="26" y2="30.5" width="0.254" layer="16"/>
-<wire x1="26" y1="30.5" x2="26.5" y2="31" width="0.254" layer="16"/>
+<wire x1="25" y1="29.5" x2="26.5" y2="31" width="0.254" layer="16"/>
 <wire x1="26.75" y1="30.25" x2="26.75" y2="30.75" width="0.254" layer="16"/>
 <wire x1="26.75" y1="30.75" x2="26.5" y2="31" width="0.254" layer="16"/>
@@
 <wire x1="75.393396875" y1="28.437409375" x2="75.393396875" y2="29.087409375" width="0.254" layer="1"/>
 <wire x1="75.393396875" y1="28.437409375" x2="75.393396875" y2="27.787409375" width="0.254" layer="1"/>
-<via x="65" y="22.5" extent="1-16" drill="0.6" shape="square"/>
-<wire x1="65" y1="22.5" x2="51.5" y2="22.5" width="0.254" layer="16"/>
+<via x="65" y="22" extent="1-16" drill="0.6" shape="square"/>
 <wire x1="75.393396875" y1="27.787409375" x2="76.962590625" y2="27.787409375" width="0.254" layer="1"/>
 <wire x1="76.962590625" y1="27.787409375" x2="77" y2="27.75" width="0.254" layer="1"/>
@@
 <wire x1="77" y1="22.75" x2="76.25" y2="22" width="0.254" layer="1"/>
 <wire x1="76.25" y1="22" x2="75.5" y2="22" width="0.254" layer="1"/>
-<wire x1="75.5" y1="22" x2="65.5" y2="22" width="0.254" layer="1"/>
-<wire x1="65.5" y1="22" x2="65" y2="22.5" width="0.254" layer="1"/>
+<wire x1="75.5" y1="22" x2="65" y2="22" width="0.254" layer="1"/>
 <contactref element="JP3" pad="4"/>
 <wire x1="73.77" y1="18.25" x2="75.5" y2="18.25" width="0.254" layer="1"/>
@@
 <contactref element="JP1" pad="2"/>
 <wire x1="26.6" y1="21.6" x2="26.5" y2="21" width="0.254" layer="16"/>
-<wire x1="16" y1="22.5" x2="28.5" y2="22.5" width="0.254" layer="16"/>
-<wire x1="28.5" y1="22.5" x2="36.5" y2="22.5" width="0.254" layer="16"/>
-<wire x1="36.5" y1="22.5" x2="44" y2="22.5" width="0.254" layer="16"/>
-<wire x1="44" y1="22.5" x2="51.5" y2="22.5" width="0.254" layer="16"/>
-<wire x1="26.6" y1="21.6" x2="28.6" y2="22.4" width="0.254" layer="16"/>
-<wire x1="28.6" y1="22.4" x2="28.5" y2="22.5" width="0.254" layer="16"/>
-<wire x1="34.25" y1="21.1" x2="36.25" y2="22.25" width="0.254" layer="16"/>
-<wire x1="36.25" y1="22.25" x2="36.5" y2="22.5" width="0.254" layer="16"/>
-<wire x1="42" y1="21.1" x2="44" y2="22.5" width="0.254" layer="16"/>
-<wire x1="49.5" y1="21.1" x2="51.5" y2="22.5" width="0.254" layer="16"/>
+<wire x1="19.5" y1="22" x2="27" y2="22" width="0.254" layer="16"/>
+<wire x1="27" y1="22" x2="34.5" y2="22" width="0.254" layer="16"/>
+<wire x1="34.5" y1="22" x2="42" y2="22" width="0.254" layer="16"/>
+<wire x1="42" y1="22" x2="49.5" y2="22" width="0.254" layer="16"/>
+<wire x1="49.5" y1="22" x2="65" y2="22" width="0.254" layer="16"/>
 <wire x1="26.5" y1="21" x2="26.65" y2="21" width="0.254" layer="16"/>
 <wire x1="26.65" y1="21" x2="26.75" y2="21.1" width="0.254" layer="16"/>
@@
 <wire x1="12.53" y1="25" x2="12.53" y2="32.47" width="0.254" layer="1"/>
 <wire x1="12.53" y1="32.47" x2="11.5" y2="33.5" width="0.254" layer="1"/>
-<via x="16" y="22.5" extent="1-16" drill="0.6" shape="square"/>
-<wire x1="16" y1="22.5" x2="13.5" y2="22.5" width="0.254" layer="1"/>
-<wire x1="13.5" y1="22.5" x2="12.5" y2="23.5" width="0.254" layer="1"/>
-<wire x1="12.5" y1="23.5" x2="12.5" y2="24.97" width="0.254" layer="1"/>
+<via x="19.5" y="22" extent="1-16" drill="0.6" shape="square"/>
+<wire x1="19.5" y1="22" x2="13.5" y2="22" width="0.254" layer="1"/>
+<wire x1="13.5" y1="22" x2="12.5" y2="23" width="0.254" layer="1"/>
+<wire x1="12.5" y1="23" x2="12.5" y2="24.97" width="0.254" layer="1"/>
 <wire x1="12.5" y1="24.97" x2="12.53" y2="25" width="0.254" layer="1"/>
+<wire x1="26.6" y1="21.6" x2="27" y2="21.6" width="0.254" layer="16"/>
+<wire x1="27" y1="21.6" x2="27" y2="22" width="0.254" layer="16"/>
+<wire x1="34.25" y1="21.1" x2="34.5" y2="21.1" width="0.254" layer="16"/>
+<wire x1="34.5" y1="21.1" x2="34.5" y2="22" width="0.254" layer="16"/>
+<wire x1="42" y1="21.1" x2="42" y2="22" width="0.254" layer="16"/>
+<wire x1="49.5" y1="21.1" x2="49.5" y2="22" width="0.254" layer="16"/>
 <wire x1="88.7" y1="64.0426" x2="89.5" y2="64.0426" width="0" layer="19" extent="1-1"/>
 <wire x1="87.2074" y1="60.15" x2="88.7" y2="64.0426" width="0" layer="19" extent="1-1"/>
@@
 <wire x1="12" y1="49" x2="11.599" y2="49" width="0.6" layer="1"/>
 <wire x1="11.599" y1="49" x2="11.599" y2="49.5" width="0.6" layer="1"/>
-<wire x1="32" y1="31.25" x2="32" y2="31.75" width="0.254" layer="16"/>
-<wire x1="20.3" y1="19.75" x2="20.3" y2="20.7" width="0.254" layer="1"/>
-<wire x1="20.3" y1="20.7" x2="20.5" y2="22.5" width="0.254" layer="1"/>
-<wire x1="20.5" y1="22.5" x2="19.5" y2="22.5" width="0.254" layer="1"/>
+<wire x1="32" y1="29.75" x2="32" y2="31.75" width="0.254" layer="16"/>
 <wire x1="14.25" y1="42.25" x2="14" y2="42.5" width="0.6" layer="16"/>
 <wire x1="14" y1="42.5" x2="14" y2="47.5" width="0.6" layer="16"/>
@@
 <wire x1="13.5" y1="48" x2="13" y2="48" width="0.6" layer="1"/>
 <wire x1="13" y1="48" x2="12" y2="49" width="0.6" layer="1"/>
-<wire x1="20.5" y1="22.5" x2="32.47" y2="30.3" width="0" layer="19" extent="1-1"/>
+<wire x1="32" y1="29.75" x2="27.75" y2="29.75" width="0.254" layer="16"/>
+<wire x1="27.75" y1="29.75" x2="26" y2="28" width="0.254" layer="16"/>
+<wire x1="26" y1="28" x2="21.5" y2="28" width="0.254" layer="16"/>
+<wire x1="21.5" y1="28" x2="21.5" y2="27.5" width="0.254" layer="16"/>
+<via x="21.5" y="27.5" extent="1-16" drill="0.6" shape="square"/>
+<wire x1="21.5" y1="27.5" x2="21.5" y2="22" width="0.254" layer="1"/>
+<wire x1="21.5" y1="22" x2="20" y2="20.5" width="0.254" layer="1"/>
+<wire x1="20" y1="20.5" x2="20" y2="19.5" width="0.254" layer="1"/>
+<wire x1="20" y1="19.5" x2="20.3" y2="19.75" width="0" layer="19" extent="1-1"/>
 </signal>
 <signal name="D_FASTBLANKING">

Commit message: mah
Parts:
- moved X6 40.2 mm to (91.5, 53.0)
- moved X1 20.2 mm to (87.2, 71.5), turned to 90 degrees
- moved X5 13.5 mm to (65.5, 68.5)
- moved C34 3.64 mm to (18.8, 50.0), flipped to the bottom, turned to 270 degrees
- moved X3 1.00 mm to (9.00, 75.2)
Routing:
- net GND: track 693.5 -> 687.1 mm, vias 35 -> 34
- net VCC: track 398.6 -> 399.9 mm, vias 23 -> 24
- net VCC5: track 98.1 -> 98.8 mm

Commit message: mah
Parts:
- removed J1: (no value), con-jack:DCJ0303
- added SV2: (no value), con-lstb:MA12-1
- moved JP2 74.3 mm to (78.0, 3.00)
- moved R7 3.55 mm to (14.2, 69.0), turned to 90 degrees
- moved R47 3.01 mm to (5.25, 65.2)
- moved R4 1.68 mm to (8.00, 62.0)
- moved T1 1.35 mm to (7.75, 65.2)
- moved R51 1.25 mm to (10.8, 65.2)
- moved R6 1.25 mm to (13.5, 62.0)
- moved R5 1.12 mm to (3.00, 65.2), turned to 270 degrees
- moved T3 1.12 mm to (13.5, 65.2)
Connections:
- net GND: no longer J1.3
- net VCC5: no longer J1.1
Routing:
- net GND: track 687.1 -> 774.3 mm, vias 34 -> 33
- net VCC: track 399.9 -> 425.9 mm
- net PS2CLK: track 12.5 -> 5.94 mm, vias 1 -> 0
- net VCC5: track 98.8 -> 99.5 mm
- net CLK_5V: track 8.24 -> 7.70 mm
- net PS2DAT: track 6.26 -> 6.10 mm, vias 1 -> 0
