File: eagle/homeboard/homeboard15.sch (EAGLE design)
At the start: 121 parts, among them IC1 XCF02S, IC2 25LC080SN, IC3 ATMEGA32U2-TQFP, Q5 BC848SMD, Q6 BC848SMD, Q7 BC848SMD, Q8 BC848SMD, T1 BSS138, T2 BC848, T3 BSS138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

Commit message: mah
Parts:
- removed X8: DC21MMX, powersupply:DC21MMX
- added J1: (no value), con-jack:DCJ0303
- added X7: DC21MMX, powersupply:DC21MMX
Connections:
- net GND: now also J1.3, X7.3; no longer X8.1, X8.3
- net VCC5: now also J1.1, X7.2; no longer X8.2
Changed lines of the file:
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@@
 <part name="R54" library="rcl" deviceset="R-EU_" device="R0805" value="22"/>
 <part name="SUPPLY12" library="supply2" deviceset="GND" device=""/>
-<part name="X8" library="powersupply" deviceset="DC21MM" device="X"/>
 <part name="SUPPLY13" library="supply2" deviceset="GND" device=""/>
 <part name="C33" library="rcl" deviceset="CPOL-EU" device="D" value="100u"/>
@@
 <part name="SV1" library="con-lstb" deviceset="MA10-1" device=""/>
 <part name="SUPPLY17" library="supply2" deviceset="GND" device=""/>
+<part name="J1" library="con-jack" deviceset="DCJ0303" device=""/>
+<part name="X7" library="powersupply" deviceset="DC21MM" device="X"/>
+<part name="SUPPLY18" library="supply2" deviceset="GND" device=""/>
 </parts>
 <sheets>
@@
 <instance part="R54" gate="G$1" x="-287.02" y="-35.56" rot="MR180"/>
 <instance part="SUPPLY12" gate="GND" x="-292.1" y="-78.74"/>
-<instance part="X8" gate="G$1" x="-256.54" y="106.68"/>
 <instance part="SUPPLY13" gate="GND" x="-261.62" y="83.82"/>
 <instance part="C33" gate="G$1" x="-226.06" y="68.58" smashed="yes">
@@
 <instance part="SV1" gate="1" x="43.18" y="-58.42" rot="R270"/>
 <instance part="SUPPLY17" gate="GND" x="22.86" y="-68.58" rot="R270"/>
+<instance part="J1" gate="G$1" x="-271.78" y="93.98"/>
+<instance part="X7" gate="G$1" x="-309.88" y="88.9"/>
+<instance part="SUPPLY18" gate="GND" x="-294.64" y="86.36"/>
 </instances>
 <busses>
@@
 </segment>
 <segment>
-<pinref part="X8" gate="G$1" pin="3"/>
-<wire x1="-241.3" y1="106.68" x2="-238.76" y2="106.68" width="0.1524" layer="91"/>
-<wire x1="-238.76" y1="106.68" x2="-238.76" y2="91.44" width="0.1524" layer="91"/>
-<pinref part="X8" gate="G$1" pin="1"/>
-<wire x1="-238.76" y1="91.44" x2="-261.62" y2="91.44" width="0.1524" layer="91"/>
-<wire x1="-261.62" y1="91.44" x2="-261.62" y2="96.52" width="0.1524" layer="91"/>
-<pinref part="SUPPLY13" gate="GND" pin="GND"/>
-<wire x1="-261.62" y1="86.36" x2="-261.62" y2="91.44" width="0.1524" layer="91"/>
-<junction x="-261.62" y="91.44"/>
-</segment>
-<segment>
 <pinref part="SUPPLY14" gate="GND" pin="GND"/>
 <pinref part="C33" gate="G$1" pin="-"/>
@@
 <pinref part="SUPPLY17" gate="GND" pin="GND"/>
 <wire x1="35.56" y1="-68.58" x2="25.4" y2="-68.58" width="0.1524" layer="91"/>
+</segment>
+<segment>
+<pinref part="SUPPLY13" gate="GND" pin="GND"/>
+<wire x1="-261.62" y1="86.36" x2="-261.62" y2="91.44" width="0.1524" layer="91"/>
+<pinref part="J1" gate="G$1" pin="3"/>
+<wire x1="-261.62" y1="91.44" x2="-264.16" y2="91.44" width="0.1524" layer="91"/>
+</segment>
+<segment>
+<pinref part="X7" gate="G$1" pin="3"/>
+<pinref part="SUPPLY18" gate="GND" pin="GND"/>
 </segment>
 </net>
@@
 <wire x1="-208.28" y1="114.3" x2="-208.28" y2="91.44" width="0.1524" layer="91"/>
 <junction x="-208.28" y="91.44"/>
-<pinref part="X8" gate="G$1" pin="2"/>
-<wire x1="-251.46" y1="96.52" x2="-226.06" y2="96.52" width="0.1524" layer="91"/>
 <wire x1="-226.06" y1="96.52" x2="-226.06" y2="73.66" width="0.1524" layer="91"/>
 <wire x1="-226.06" y1="73.66" x2="-208.28" y2="73.66" width="0.1524" layer="91"/>
@@
 <wire x1="-251.46" y1="73.66" x2="-251.46" y2="68.58" width="0.1524" layer="91"/>
 <junction x="-238.76" y="73.66"/>
-</segment>
-</net>
+<pinref part="J1" gate="G$1" pin="1"/>
+<wire x1="-226.06" y1="96.52" x2="-256.54" y2="96.52" width="0.1524" layer="91"/>
+<wire x1="-256.54" y1="96.52" x2="-264.16" y2="96.52" width="0.1524" layer="91"/>
+<wire x1="-279.4" y1="73.66" x2="-279.4" y2="101.6" width="0.1524" layer="91"/>
+<wire x1="-279.4" y1="101.6" x2="-256.54" y2="101.6" width="0.1524" layer="91"/>
+<wire x1="-256.54" y1="101.6" x2="-256.54" y2="96.52" width="0.1524" layer="91"/>
+<junction x="-256.54" y="96.52"/>
+<pinref part="X7" gate="G$1" pin="2"/>
+<wire x1="-304.8" y1="78.74" x2="-304.8" y2="73.66" width="0.1524" layer="91"/>
+<wire x1="-304.8" y1="73.66" x2="-279.4" y2="73.66" width="0.1524" layer="91"/>
+</segment>
+</net>

Commit message: mah
Connections:
- removed net N$1113: SV1.9, U1B5.IO_L32N_5GCLK3
- removed net QQQ: SV1.8, U1B5.IO_L32P_5GCLK2
- new net AASA: SV1.8, U1B5.IO_L31N_5D4
- new net SAA: SV1.9, U1B5.IO_L32P_5GCLK2
- net R0: now also U1B4.IO_L32N_4GCLK1; no longer U1B4.IO_L32P_4GCLK0
- net R1: now also U1B5.IO_L32N_5GCLK3; no longer U1B5.IO_L31N_5D4
- net XXX: now also U1B4.IO_L32P_4GCLK0; no longer U1B4.IO_L32N_4GCLK1
Changed lines of the file:
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@@
 </segment>
 <segment>
-<pinref part="U1" gate="B5" pin="IO_L31N_5D4"/>
-<wire x1="99.06" y1="-73.66" x2="137.16" y2="-73.66" width="0.1524" layer="91"/>
-<wire x1="137.16" y1="-73.66" x2="137.16" y2="-40.64" width="0.1524" layer="91"/>
-<label x="99.06" y="-73.66" size="1.778" layer="95"/>
+<pinref part="U1" gate="B5" pin="IO_L32N_5GCLK3"/>
+<wire x1="129.54" y1="-78.74" x2="129.54" y2="-40.64" width="0.1524" layer="91"/>
+<wire x1="129.54" y1="-78.74" x2="99.06" y2="-78.74" width="0.1524" layer="91"/>
+<label x="99.06" y="-78.74" size="1.778" layer="95"/>
 </segment>
 </net>
@@
 </segment>
 <segment>
-<pinref part="U1" gate="B4" pin="IO_L32P_4GCLK0"/>
-<wire x1="162.56" y1="-40.64" x2="162.56" y2="-81.28" width="0.1524" layer="91"/>
-<wire x1="162.56" y1="-81.28" x2="185.42" y2="-81.28" width="0.1524" layer="91"/>
+<wire x1="160.02" y1="-81.28" x2="185.42" y2="-81.28" width="0.1524" layer="91"/>
 <label x="185.42" y="-81.28" size="1.778" layer="95"/>
+<pinref part="U1" gate="B4" pin="IO_L32N_4GCLK1"/>
+<wire x1="160.02" y1="-81.28" x2="160.02" y2="-40.64" width="0.1524" layer="91"/>
 </segment>
 </net>
@@
 <segment>
 <pinref part="SV1" gate="1" pin="10"/>
-<wire x1="160.02" y1="-83.82" x2="55.88" y2="-83.82" width="0.1524" layer="91"/>
+<wire x1="162.56" y1="-83.82" x2="55.88" y2="-83.82" width="0.1524" layer="91"/>
 <wire x1="55.88" y1="-83.82" x2="55.88" y2="-66.04" width="0.1524" layer="91"/>
-<pinref part="U1" gate="B4" pin="IO_L32N_4GCLK1"/>
-<wire x1="160.02" y1="-40.64" x2="160.02" y2="-83.82" width="0.1524" layer="91"/>
-</segment>
-</net>
-<net name="N$1113" class="0">
-<segment>
-<pinref part="U1" gate="B5" pin="IO_L32N_5GCLK3"/>
-<wire x1="129.54" y1="-78.74" x2="129.54" y2="-40.64" width="0.1524" layer="91"/>
-<pinref part="SV1" gate="1" pin="9"/>
-<wire x1="129.54" y1="-78.74" x2="53.34" y2="-78.74" width="0.1524" layer="91"/>
-<wire x1="53.34" y1="-78.74" x2="53.34" y2="-66.04" width="0.1524" layer="91"/>
-<label x="99.06" y="-78.74" size="1.778" layer="95"/>
+<pinref part="U1" gate="B4" pin="IO_L32P_4GCLK0"/>
+<wire x1="162.56" y1="-40.64" x2="162.56" y2="-83.82" width="0.1524" layer="91"/>
 </segment>
 </net>
@@
 </segment>
 </net>
-<net name="QQQ" class="0">
-<segment>
-<pinref part="U1" gate="B5" pin="IO_L32P_5GCLK2"/>
-<wire x1="132.08" y1="-76.2" x2="132.08" y2="-40.64" width="0.1524" layer="91"/>
-<wire x1="132.08" y1="-76.2" x2="81.28" y2="-76.2" width="0.1524" layer="91"/>
-<label x="99.06" y="-76.2" size="1.778" layer="95"/>
+<net name="AASA" class="0">
+<segment>
+<pinref part="U1" gate="B5" pin="IO_L31N_5D4"/>
+<wire x1="81.28" y1="-73.66" x2="137.16" y2="-73.66" width="0.1524" layer="91"/>
+<wire x1="137.16" y1="-73.66" x2="137.16" y2="-40.64" width="0.1524" layer="91"/>
+<label x="99.06" y="-73.66" size="1.778" layer="95"/>
 <pinref part="SV1" gate="1" pin="8"/>
 <wire x1="81.28" y1="-99.06" x2="50.8" y2="-99.06" width="0.1524" layer="91"/>
 <wire x1="50.8" y1="-99.06" x2="50.8" y2="-66.04" width="0.1524" layer="91"/>
-<wire x1="81.28" y1="-76.2" x2="81.28" y2="-99.06" width="0.1524" layer="91"/>
-</segment>
-</net>
+<wire x1="81.28" y1="-73.66" x2="81.28" y2="-99.06" width="0.1524" layer="91"/>
+</segment>
+</net>
+<net name="SAA" class="0">
+<segment>
+<pinref part="U1" gate="B5" pin="IO_L32P_5GCLK2"/>
+<wire x1="132.08" y1="-76.2" x2="132.08" y2="-40.64" width="0.1524" layer="91"/>
+<label x="99.06" y="-76.2" size="1.778" layer="95"/>
+<pinref part="SV1" gate="1" pin="9"/>
+<wire x1="132.08" y1="-76.2" x2="53.34" y2="-76.2" width="0.1524" layer="91"/>
+<wire x1="53.34" y1="-76.2" x2="53.34" y2="-66.04" width="0.1524" layer="91"/>
+</segment>
+</net>

Commit message: mah
Parts:
- SV1: device con-lstb:MA10-1 -> con-lstb:MA12-1
Connections:
- removed net X: U1B4.IOVREF_4
- new net XXZXZ: SV1.11, U1B4.IO_L31P_4DOUTBUSY
- net B0: now also U1B4.IO_L01P_4VRN_4; no longer U1B4.IO_L27P_4D1
- net B1: now also U1B4.IO_L27P_4D1; no longer U1B4.IO_L30N_4D2
- net FPGA_AUDIO_LEFT: now also U1B4.IO_L01N_4VRP_4; no longer U1B4.IO_L01P_4VRN_4
- net FPGA_AUDIO_RIGHT: now also U1B4.IOVREF_4; no longer U1B4.IO_L01N_4VRP_4
- net G0: now also U1B4.IO_L30N_4D2; no longer U1B4.IO_L30P_4D3
- net G1: now also U1B4.IO_L30P_4D3; no longer U1B4.IO_L31P_4DOUTBUSY
- net GND: now also SV1.12

Commit message: mah
Parts:
- removed J1: (no value), con-jack:DCJ0303
- added SV2: (no value), con-lstb:MA12-1
Connections:
- net GND: no longer J1.3
- net VCC5: no longer J1.1
Changed lines of the file:
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@@
 <part name="U$3" library="adafruit" deviceset="PINHD-1X10" device=""/>
 <part name="SUPPLY17" library="supply2" deviceset="GND" device=""/>
-<part name="J1" library="con-jack" deviceset="DCJ0303" device=""/>
 <part name="X7" library="powersupply" deviceset="DC21MM" device="X"/>
 <part name="SUPPLY18" library="supply2" deviceset="GND" device=""/>
 <part name="SV1" library="con-lstb" deviceset="MA12-1" device=""/>
+<part name="SV2" library="con-lstb" deviceset="MA12-1" device="">
+<attribute name="MF" value=""/>
+<attribute name="MPN" value=""/>
+<attribute name="OC_FARNELL" value="unknown"/>
+<attribute name="OC_NEWARK" value="unknown"/>
+</part>
 </parts>
 <sheets>
@@
 <instance part="U$3" gate="G$1" x="22.86" y="-149.86" rot="R180"/>
 <instance part="SUPPLY17" gate="GND" x="22.86" y="-68.58" rot="R270"/>
-<instance part="J1" gate="G$1" x="-271.78" y="93.98"/>
 <instance part="X7" gate="G$1" x="-309.88" y="88.9"/>
 <instance part="SUPPLY18" gate="GND" x="-294.64" y="86.36"/>
 <instance part="SV1" gate="1" x="45.72" y="-58.42" rot="R270"/>
+<instance part="SV2" gate="1" x="157.48" y="109.22" rot="R270"/>
 </instances>
 <busses>
@@
 <pinref part="SUPPLY13" gate="GND" pin="GND"/>
 <wire x1="-261.62" y1="86.36" x2="-261.62" y2="91.44" width="0.1524" layer="91"/>
-<pinref part="J1" gate="G$1" pin="3"/>
 <wire x1="-261.62" y1="91.44" x2="-264.16" y2="91.44" width="0.1524" layer="91"/>
 </segment>
@@
 <wire x1="-251.46" y1="73.66" x2="-251.46" y2="68.58" width="0.1524" layer="91"/>
 <junction x="-238.76" y="73.66"/>
-<pinref part="J1" gate="G$1" pin="1"/>
 <wire x1="-226.06" y1="96.52" x2="-256.54" y2="96.52" width="0.1524" layer="91"/>
 <wire x1="-256.54" y1="96.52" x2="-264.16" y2="96.52" width="0.1524" layer="91"/>
