File: eagle/homeboard/homeboard18.brd (EAGLE design)
At the start: 100 x 80 mm, 132 parts, among them IC1 XCF02S, IC2 25LC080SN, IC3 ATMEGA32U2-TQFP, Q5 BC848SMD, Q6 BC848SMD, Q7 BC848SMD, Q8 BC848SMD, T1 BSS138, T2 BC848, T3 BSS138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

Commit message: bed
Parts:
- moved C42 1.12 mm to (17.5, 38.5)
- moved C1 1.00 mm to (72.2, 18.5)
- moved C10 1.00 mm to (60.5, 40.5)
- moved C11 1.00 mm to (46.2, 40.8)
- moved C12 1.00 mm to (47.5, 46.8)
- moved C13 1.00 mm to (61.0, 46.8)
- moved C14 1.00 mm to (47.5, 35.2)
- moved C15 1.00 mm to (51.2, 36.8)
- moved C16 1.00 mm to (45.2, 34.2)
- moved C17 1.00 mm to (61.0, 34.8)
- moved C18 1.00 mm to (56.5, 35.2)
- moved C19 1.00 mm to (49.8, 47.5)
- moved C2 1.00 mm to (40.2, 67.0)
- moved C20 1.00 mm to (56.5, 47.0)
- moved C21 1.00 mm to (49.8, 34.0)
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Routing:
- net VCCAUX: track 96.1 -> 122.9 mm, vias 7 -> 8
- net VCC: track 442.3 -> 466.2 mm, vias 26 -> 27
- net VCCINT: track 75.0 -> 97.4 mm, vias 6 -> 7
- net GND: track 756.1 -> 754.3 mm
- net N$84: track 19.6 -> 18.7 mm
- net N$83: track 18.6 -> 17.7 mm
- net N$82: track 17.1 -> 16.5 mm
- net N$81: track 16.1 -> 15.5 mm
- net N$86: track 17.5 -> 16.9 mm
- net N$85: track 18.5 -> 17.9 mm
- net N$80: track 15.1 -> 14.5 mm
- net N$79: track 14.1 -> 13.5 mm
- net N$78: track 13.1 -> 12.5 mm
- net N$77: track 12.1 -> 11.5 mm

Commit message: work time
Parts:
- added H1, H2, H3, H4: MOUNT-HOLE3.0, holes:3,0
- moved U$5 75.5 mm to (84.8, 24.2)
- moved U$2 58.5 mm to (78.9, 27.9)
- moved X8 33.0 mm to (7.50, 71.5)
- moved C2 21.8 mm to (18.8, 63.5)
- moved R17 21.8 mm to (23.8, 61.5)
- moved R18 21.8 mm to (16.5, 63.5)
- moved R19 21.8 mm to (21.2, 61.5)
- moved R21 21.8 mm to (18.8, 59.5)
- moved R22 21.8 mm to (14.2, 63.5)
- moved T2 21.8 mm to (15.2, 59.5)
- moved X5 14.5 mm to (31.0, 68.5)
- moved C33 8.00 mm to (9.25, 28.0)
- moved C39 1.58 mm to (19.0, 30.5)
- moved C40 1.50 mm to (19.0, 46.5)
- moved C42 1.50 mm to (19.0, 38.5)
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Connections:
- removed net AA: SV1.6, U1.P46
- removed net N$100: SV1.4, U1.P41
- removed net N$101: SV1.5, U1.P44
- removed net N$99: SV1.3, U1.P40
- new net N$10: SV1.3
- new net N$11: SV1.4
- new net N$13: SV1.5
- new net N$15: SV1.6
- net PS2CLK: now also U1.P46; no longer U1.P141
- net PS2DAT: now also U1.P44; no longer U1.P140
- net SD_CLK: now also U1.P41
- net SD_CS: now also U1.P140
- net SD_DI: now also U1.P141
- net SD_DO: now also U1.P40
Routing:
- net GND: track 754.3 -> 871.0 mm, vias 26 -> 30
- net SD_DI: track 0.00 -> 34.3 mm, vias 0 -> 1
- net SD_CS: track 0.00 -> 31.6 mm, vias 0 -> 1
- net SD_CLK: track 0.00 -> 24.6 mm, vias 0 -> 1
- net PS2CLK: track 14.1 -> 38.3 mm
- net PS2DAT: track 4.33 -> 28.1 mm
- net SD_DO: track 0.00 -> 18.5 mm, vias 0 -> 1
- net CLK16: track 27.2 -> 10.1 mm
- net N$99: track 16.3 -> 0.00 mm
- net N$100: track 14.3 -> 0.00 mm
- net N$101: track 12.6 -> 0.00 mm
- net AA: track 10.9 -> 0.00 mm
- net CASIN: track 26.3 -> 16.3 mm
- net VCC: track 466.2 -> 474.9 mm
- net VCC5: track 84.5 -> 91.6 mm
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