File: eagle/homeboard/homeboard18.sch (EAGLE design)
At the start: 132 parts, among them IC1 XCF02S, IC2 25LC080SN, IC3 ATMEGA32U2-TQFP, Q5 BC848SMD, Q6 BC848SMD, Q7 BC848SMD, Q8 BC848SMD, T1 BSS138, T2 BC848, T3 BSS138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

Commit message: work time
Parts:
- added H1, H2, H3, H4: MOUNT-HOLE3.0, holes:MOUNT-HOLE3.0
Connections:
- removed net AA: SV1.6, U1B5.IO_L28P_5D7
- removed net N$100: SV1.4, U1B5.IO_L01N_5RDWR_B
- removed net N$101: SV1.5, U1B5.IOVREF_5
- removed net N$99: SV1.3, U1B5.IO_L01P_5CS_B
- new net N$10: SV1.3
- new net N$11: SV1.4
- new net N$13: SV1.5
- new net N$15: SV1.6
- net PS2CLK: now also U1B5.IO_L28P_5D7; no longer U1B0.IO_L01N_0VRP_0
- net PS2DAT: now also U1B5.IOVREF_5; no longer U1B0.IO_L01P_0VRN_0
- net SD_CLK: now also U1B5.IO_L01N_5RDWR_B
- net SD_CS: now also U1B0.IO_L01P_0VRN_0
- net SD_DI: now also U1B0.IO_L01N_0VRP_0
- net SD_DO: now also U1B5.IO_L01P_5CS_B
Changed lines of the file:
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@@
 <part name="C42" library="rcl" deviceset="CPOL-EU" device="D" value="100u"/>
 <part name="SUPPLY23" library="supply2" deviceset="GND" device=""/>
+<part name="H1" library="holes" deviceset="MOUNT-HOLE" device="3.0"/>
+<part name="H2" library="holes" deviceset="MOUNT-HOLE" device="3.0"/>
+<part name="H3" library="holes" deviceset="MOUNT-HOLE" device="3.0"/>
+<part name="H4" library="holes" deviceset="MOUNT-HOLE" device="3.0"/>
 </parts>
 <sheets>
@@
 </instance>
 <instance part="SUPPLY23" gate="GND" x="520.7" y="15.24"/>
+<instance part="H1" gate="G$1" x="-223.52" y="167.64"/>
+<instance part="H2" gate="G$1" x="-213.36" y="167.64"/>
+<instance part="H3" gate="G$1" x="-223.52" y="160.02"/>
+<instance part="H4" gate="G$1" x="-213.36" y="160.02"/>
 </instances>
 <busses>
@@
 </segment>
 <segment>
-<wire x1="86.36" y1="76.2" x2="129.54" y2="76.2" width="0.1524" layer="91"/>
-<label x="86.36" y="76.2" size="1.778" layer="95"/>
-<pinref part="U1" gate="B0" pin="IO_L01N_0VRP_0"/>
-<wire x1="129.54" y1="76.2" x2="129.54" y2="73.66" width="0.1524" layer="91"/>
+<wire x1="190.5" y1="134.62" x2="233.68" y2="134.62" width="0.1524" layer="91"/>
+<label x="190.5" y="134.62" size="1.778" layer="95"/>
+</segment>
+<segment>
+<wire x1="76.2" y1="-66.04" x2="139.7" y2="-66.04" width="0.1524" layer="91"/>
+<wire x1="139.7" y1="-66.04" x2="139.7" y2="-40.64" width="0.1524" layer="91"/>
+<pinref part="U1" gate="B5" pin="IO_L28P_5D7"/>
+<label x="99.06" y="-66.04" size="1.778" layer="95"/>
+<wire x1="76.2" y1="-66.04" x2="76.2" y2="-93.98" width="0.1524" layer="91"/>
+<wire x1="76.2" y1="-93.98" x2="45.72" y2="-93.98" width="0.1524" layer="91"/>
+<label x="53.34" y="-93.98" size="1.778" layer="95"/>
 </segment>
 </net>
@@
 </segment>
 <segment>
-<wire x1="127" y1="78.74" x2="86.36" y2="78.74" width="0.1524" layer="91"/>
-<label x="86.36" y="78.74" size="1.778" layer="95"/>
-<pinref part="U1" gate="B0" pin="IO_L01P_0VRN_0"/>
-<wire x1="127" y1="78.74" x2="127" y2="73.66" width="0.1524" layer="91"/>
+<wire x1="231.14" y1="137.16" x2="190.5" y2="137.16" width="0.1524" layer="91"/>
+<label x="190.5" y="137.16" size="1.778" layer="95"/>
+</segment>
+<segment>
+<pinref part="U1" gate="B5" pin="IOVREF_5"/>
+<wire x1="73.66" y1="-63.5" x2="127" y2="-63.5" width="0.1524" layer="91"/>
+<wire x1="127" y1="-63.5" x2="127" y2="-40.64" width="0.1524" layer="91"/>
+<label x="99.06" y="-63.5" size="1.778" layer="95"/>
+<wire x1="73.66" y1="-63.5" x2="73.66" y2="-91.44" width="0.1524" layer="91"/>
+<wire x1="73.66" y1="-91.44" x2="43.18" y2="-91.44" width="0.1524" layer="91"/>
+<label x="53.34" y="-91.44" size="1.778" layer="95"/>
 </segment>
 </net>
@@
 </segment>
 </net>
-<net name="N$99" class="0">
-<segment>
-<pinref part="U1" gate="B5" pin="IO_L01P_5CS_B"/>
-<wire x1="147.32" y1="-40.64" x2="147.32" y2="-58.42" width="0.1524" layer="91"/>
-<wire x1="147.32" y1="-58.42" x2="68.58" y2="-58.42" width="0.1524" layer="91"/>
-<label x="99.06" y="-58.42" size="1.778" layer="95"/>
-<wire x1="68.58" y1="-58.42" x2="68.58" y2="-86.36" width="0.1524" layer="91"/>
-<wire x1="68.58" y1="-86.36" x2="38.1" y2="-86.36" width="0.1524" layer="91"/>
-<wire x1="38.1" y1="-86.36" x2="38.1" y2="-66.04" width="0.1524" layer="91"/>
-<pinref part="SV1" gate="1" pin="3"/>
-</segment>
-</net>
-<net name="N$100" class="0">
-<segment>
-<pinref part="U1" gate="B5" pin="IO_L01N_5RDWR_B"/>
-<wire x1="71.12" y1="-60.96" x2="144.78" y2="-60.96" width="0.1524" layer="91"/>
-<wire x1="144.78" y1="-60.96" x2="144.78" y2="-40.64" width="0.1524" layer="91"/>
-<label x="99.06" y="-60.96" size="1.778" layer="95"/>
-<wire x1="71.12" y1="-60.96" x2="71.12" y2="-88.9" width="0.1524" layer="91"/>
-<wire x1="71.12" y1="-88.9" x2="40.64" y2="-88.9" width="0.1524" layer="91"/>
-<wire x1="40.64" y1="-88.9" x2="40.64" y2="-66.04" width="0.1524" layer="91"/>
-<pinref part="SV1" gate="1" pin="4"/>
-</segment>
-</net>
-<net name="N$101" class="0">
-<segment>
-<pinref part="U1" gate="B5" pin="IOVREF_5"/>
-<wire x1="73.66" y1="-63.5" x2="127" y2="-63.5" width="0.1524" layer="91"/>
-<wire x1="127" y1="-63.5" x2="127" y2="-40.64" width="0.1524" layer="91"/>
-<label x="99.06" y="-63.5" size="1.778" layer="95"/>
-<wire x1="73.66" y1="-63.5" x2="73.66" y2="-91.44" width="0.1524" layer="91"/>
-<wire x1="73.66" y1="-91.44" x2="43.18" y2="-91.44" width="0.1524" layer="91"/>
-<wire x1="43.18" y1="-91.44" x2="43.18" y2="-66.04" width="0.1524" layer="91"/>
-<pinref part="SV1" gate="1" pin="5"/>
-</segment>
-</net>
 <net name="XXX" class="0">
 <segment>
@@
 </segment>
 </net>
-<net name="AA" class="0">
-<segment>
-<wire x1="76.2" y1="-66.04" x2="139.7" y2="-66.04" width="0.1524" layer="91"/>
-<wire x1="139.7" y1="-66.04" x2="139.7" y2="-40.64" width="0.1524" layer="91"/>
-<pinref part="U1" gate="B5" pin="IO_L28P_5D7"/>
-<label x="99.06" y="-66.04" size="1.778" layer="95"/>
-<wire x1="76.2" y1="-66.04" x2="76.2" y2="-93.98" width="0.1524" layer="91"/>
-<pinref part="SV1" gate="1" pin="6"/>
-<wire x1="76.2" y1="-93.98" x2="45.72" y2="-93.98" width="0.1524" layer="91"/>
-<wire x1="45.72" y1="-93.98" x2="45.72" y2="-66.04" width="0.1524" layer="91"/>
-</segment>
-</net>
 <net name="ABAB" class="0">
 <segment>
@@
 <label x="510.54" y="43.18" size="1.778" layer="95"/>
 </segment>
+<segment>
+<wire x1="127" y1="78.74" x2="86.36" y2="78.74" width="0.1524" layer="91"/>
+<label x="86.36" y="78.74" size="1.778" layer="95"/>
+<pinref part="U1" gate="B0" pin="IO_L01P_0VRN_0"/>
+<wire x1="127" y1="78.74" x2="127" y2="73.66" width="0.1524" layer="91"/>
+</segment>
 </net>
 <net name="SD_CLK" class="0">
@@
 <label x="510.54" y="45.72" size="1.778" layer="95"/>
 </segment>
+<segment>
+<pinref part="U1" gate="B5" pin="IO_L01N_5RDWR_B"/>
+<wire x1="71.12" y1="-60.96" x2="144.78" y2="-60.96" width="0.1524" layer="91"/>
+<wire x1="144.78" y1="-60.96" x2="144.78" y2="-40.64" width="0.1524" layer="91"/>
+<label x="99.06" y="-60.96" size="1.778" layer="95"/>
+<wire x1="71.12" y1="-60.96" x2="71.12" y2="-88.9" width="0.1524" layer="91"/>
+<wire x1="71.12" y1="-88.9" x2="40.64" y2="-88.9" width="0.1524" layer="91"/>
+<label x="53.34" y="-88.9" size="1.778" layer="95"/>
+</segment>
 </net>
 <net name="SD_DI" class="0">
@@
 <label x="510.54" y="48.26" size="1.778" layer="95"/>
 </segment>
+<segment>
+<wire x1="86.36" y1="76.2" x2="129.54" y2="76.2" width="0.1524" layer="91"/>
+<label x="86.36" y="76.2" size="1.778" layer="95"/>
+<pinref part="U1" gate="B0" pin="IO_L01N_0VRP_0"/>
+<wire x1="129.54" y1="76.2" x2="129.54" y2="73.66" width="0.1524" layer="91"/>
+</segment>
 </net>
 <net name="SD_DO" class="0">
@@
 <label x="510.54" y="50.8" size="1.778" layer="95"/>
 </segment>
-</net>
+<segment>
+<pinref part="U1" gate="B5" pin="IO_L01P_5CS_B"/>
+<wire x1="147.32" y1="-40.64" x2="147.32" y2="-58.42" width="0.1524" layer="91"/>
+<wire x1="147.32" y1="-58.42" x2="68.58" y2="-58.42" width="0.1524" layer="91"/>
+<label x="99.06" y="-58.42" size="1.778" layer="95"/>
+<wire x1="68.58" y1="-58.42" x2="68.58" y2="-86.36" width="0.1524" layer="91"/>
+<wire x1="68.58" y1="-86.36" x2="38.1" y2="-86.36" width="0.1524" layer="91"/>
+<label x="53.34" y="-86.36" size="1.778" layer="95"/>
+</segment>
+</net>
+<net name="N$10" class="0">
+<segment>
+<pinref part="SV1" gate="1" pin="3"/>
+<wire x1="38.1" y1="-83.82" x2="38.1" y2="-66.04" width="0.1524" layer="91"/>
+<label x="38.1" y="-83.82" size="1.778" layer="95" rot="R90"/>
+</segment>
+</net>
+<net name="N$11" class="0">
+<segment>
+<pinref part="SV1" gate="1" pin="4"/>
+<wire x1="40.64" y1="-83.82" x2="40.64" y2="-66.04" width="0.1524" layer="91"/>
+<label x="40.64" y="-83.82" size="1.778" layer="95" rot="R90"/>
+</segment>
+</net>
+<net name="N$13" class="0">
+<segment>
+<pinref part="SV1" gate="1" pin="5"/>
+<wire x1="43.18" y1="-83.82" x2="43.18" y2="-66.04" width="0.1524" layer="91"/>
+</segment>
+</net>
+<net name="N$15" class="0">
+<segment>
+<pinref part="SV1" gate="1" pin="6"/>
+<wire x1="45.72" y1="-83.82" x2="45.72" y2="-66.04" width="0.1524" layer="91"/>
+</segment>
+</net>
