File: eagle/homeboard/homeboard19.sch (EAGLE design)
At the start: 136 parts, among them IC1 XCF02S, IC2 25LC080SN, IC3 ATMEGA32U2-TQFP, Q5 BC848SMD, Q6 BC848SMD, Q7 BC848SMD, Q8 BC848SMD, T1 BSS138, T2 BC848, T3 BSS138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

Commit message: mah
Parts:
- removed H1, H2, H3, H4: MOUNT-HOLE3.0, holes:MOUNT-HOLE3.0
- added U$1, U$7, U$8, U$9: GNDHOLE, cpcfpga:GNDHOLE
Connections:
- net GND: now also U$1.GND, U$7.GND, U$8.GND, U$9.GND
Changed lines of the file:
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@@
 <part name="C42" library="rcl" deviceset="CPOL-EU" device="D" value="100u"/>
 <part name="SUPPLY23" library="supply2" deviceset="GND" device=""/>
-<part name="H1" library="holes" deviceset="MOUNT-HOLE" device="3.0"/>
-<part name="H2" library="holes" deviceset="MOUNT-HOLE" device="3.0"/>
-<part name="H3" library="holes" deviceset="MOUNT-HOLE" device="3.0"/>
-<part name="H4" library="holes" deviceset="MOUNT-HOLE" device="3.0"/>
+<part name="U$1" library="cpcfpga" deviceset="GNDHOLE" device=""/>
+<part name="U$7" library="cpcfpga" deviceset="GNDHOLE" device=""/>
+<part name="U$8" library="cpcfpga" deviceset="GNDHOLE" device=""/>
+<part name="U$9" library="cpcfpga" deviceset="GNDHOLE" device=""/>
 </parts>
 <sheets>
@@
 <instance part="R54" gate="G$1" x="370.84" y="119.38" rot="MR180"/>
 <instance part="SUPPLY12" gate="GND" x="365.76" y="76.2"/>
-<instance part="SUPPLY13" gate="GND" x="-261.62" y="83.82"/>
+<instance part="SUPPLY13" gate="GND" x="-254" y="147.32"/>
 <instance part="C33" gate="G$1" x="-226.06" y="68.58" smashed="yes">
 <attribute name="NAME" x="-231.521" y="68.0466" size="1.778" layer="95"/>
@@
 </instance>
 <instance part="SUPPLY23" gate="GND" x="520.7" y="15.24"/>
-<instance part="H1" gate="G$1" x="-223.52" y="167.64"/>
-<instance part="H2" gate="G$1" x="-213.36" y="167.64"/>
-<instance part="H3" gate="G$1" x="-223.52" y="160.02"/>
-<instance part="H4" gate="G$1" x="-213.36" y="160.02"/>
+<instance part="U$1" gate="G$1" x="-246.38" y="180.34"/>
+<instance part="U$7" gate="G$1" x="-246.38" y="172.72"/>
+<instance part="U$8" gate="G$1" x="-246.38" y="165.1"/>
+<instance part="U$9" gate="G$1" x="-246.38" y="157.48"/>
 </instances>
 <busses>
@@
 <segment>
 <pinref part="SUPPLY13" gate="GND" pin="GND"/>
-<wire x1="-261.62" y1="86.36" x2="-261.62" y2="91.44" width="0.1524" layer="91"/>
-<wire x1="-261.62" y1="91.44" x2="-264.16" y2="91.44" width="0.1524" layer="91"/>
-</segment>
-<segment>
+<wire x1="-254" y1="149.86" x2="-254" y2="157.48" width="0.1524" layer="91"/>
+<pinref part="U$9" gate="G$1" pin="GND"/>
+<pinref part="U$8" gate="G$1" pin="GND"/>
+<wire x1="-254" y1="157.48" x2="-254" y2="165.1" width="0.1524" layer="91"/>
+<junction x="-254" y="157.48"/>
+<pinref part="U$7" gate="G$1" pin="GND"/>
+<wire x1="-254" y1="165.1" x2="-254" y2="172.72" width="0.1524" layer="91"/>
+<junction x="-254" y="165.1"/>
+<pinref part="U$1" gate="G$1" pin="GND"/>
+<wire x1="-254" y1="172.72" x2="-254" y2="180.34" width="0.1524" layer="91"/>
+<junction x="-254" y="172.72"/>
+</segment>
+<segment>

Commit message: stuff
Connections:
- removed net N$1: SV3.3, U1B0.IO_L27N_0
- new net X_CAS: U1B1.IO_L31N_1VREF_1
- net CASIN: now also U1B0.IO_L27N_0; no longer U1B1.IO_L31N_1VREF_1
Changed lines of the file:
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@@
 </segment>
 <segment>
-<pinref part="U1" gate="B1" pin="IO_L31N_1VREF_1"/>
-<wire x1="177.8" y1="73.66" x2="177.8" y2="114.3" width="0.1524" layer="91"/>
-<wire x1="177.8" y1="114.3" x2="162.56" y2="114.3" width="0.1524" layer="91"/>
-<label x="162.56" y="114.3" size="1.778" layer="95"/>
+<pinref part="U1" gate="B0" pin="IO_L27N_0"/>
+<wire x1="134.62" y1="93.98" x2="134.62" y2="81.28" width="0.1524" layer="91"/>
+<wire x1="134.62" y1="81.28" x2="134.62" y2="73.66" width="0.1524" layer="91"/>
+<wire x1="86.36" y1="81.28" x2="134.62" y2="81.28" width="0.1524" layer="91"/>
+<junction x="134.62" y="81.28"/>
+<label x="86.36" y="81.28" size="1.778" layer="95"/>
 </segment>
 </net>
@@
 </segment>
 </net>
-<net name="N$1" class="0">
-<segment>
-<pinref part="SV3" gate="1" pin="3"/>
-<pinref part="U1" gate="B0" pin="IO_L27N_0"/>
-<wire x1="106.68" y1="93.98" x2="134.62" y2="93.98" width="0.1524" layer="91"/>
-<wire x1="134.62" y1="93.98" x2="134.62" y2="73.66" width="0.1524" layer="91"/>
-</segment>
-</net>
 <net name="N$2" class="0">
 <segment>
@@
 </segment>
 </net>
+<net name="X_CAS" class="0">
+<segment>
+<pinref part="U1" gate="B1" pin="IO_L31N_1VREF_1"/>
+<wire x1="177.8" y1="73.66" x2="177.8" y2="114.3" width="0.1524" layer="91"/>
+<wire x1="177.8" y1="114.3" x2="162.56" y2="114.3" width="0.1524" layer="91"/>
+<label x="162.56" y="114.3" size="1.778" layer="95"/>
+</segment>
+</net>

Commit message: mah
Connections:
- removed net SAA: SV1.9, U1B5.IO_L32P_5GCLK2
- new net XAACLK16: U1B0.IO_L32P_0GCLK6
- net CLK16: now also U1B4.IO_L32N_4GCLK1; no longer U1B0.IO_L32P_0GCLK6
- net R0: now also U1B5.IO_L32N_5GCLK3; no longer U1B4.IO_L32N_4GCLK1
- net R1: now also SV1.9, U1B5.IO_L32P_5GCLK2; no longer U1B5.IO_L32N_5GCLK3
Changed lines of the file:
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@@
+</segment>
+<segment>
+<pinref part="U1" gate="B5" pin="IO_L32P_5GCLK2"/>
+<wire x1="132.08" y1="-76.2" x2="132.08" y2="-40.64" width="0.1524" layer="91"/>
+<label x="99.06" y="-76.2" size="1.778" layer="95"/>
+<wire x1="132.08" y1="-76.2" x2="53.34" y2="-76.2" width="0.1524" layer="91"/>
+<wire x1="53.34" y1="-76.2" x2="53.34" y2="-66.04" width="0.1524" layer="91"/>
+<pinref part="SV1" gate="1" pin="9"/>
+</segment>
+</net>
+<net name="R0" class="0">
+<segment>
+<pinref part="R10" gate="G$1" pin="1"/>
+<wire x1="111.76" y1="248.92" x2="106.68" y2="248.92" width="0.1524" layer="91"/>
+<label x="106.68" y="248.92" size="1.778" layer="95"/>
 </segment>
 <segment>
@@
 <wire x1="129.54" y1="-78.74" x2="99.06" y2="-78.74" width="0.1524" layer="91"/>
 <label x="99.06" y="-78.74" size="1.778" layer="95"/>
-</segment>
-</net>
-<net name="R0" class="0">
-<segment>
-<pinref part="R10" gate="G$1" pin="1"/>
-<wire x1="111.76" y1="248.92" x2="106.68" y2="248.92" width="0.1524" layer="91"/>
-<label x="106.68" y="248.92" size="1.778" layer="95"/>
-</segment>
-<segment>
-<wire x1="160.02" y1="-81.28" x2="185.42" y2="-81.28" width="0.1524" layer="91"/>
-<label x="185.42" y="-81.28" size="1.778" layer="95"/>
-<pinref part="U1" gate="B4" pin="IO_L32N_4GCLK1"/>
-<wire x1="160.02" y1="-81.28" x2="160.02" y2="-40.64" width="0.1524" layer="91"/>
 </segment>
 </net>
@@
 </segment>
 <segment>
-<wire x1="147.32" y1="119.38" x2="162.56" y2="119.38" width="0.1524" layer="91"/>
-<label x="162.56" y="119.38" size="1.778" layer="95"/>
-<pinref part="U1" gate="B0" pin="IO_L32P_0GCLK6"/>
-<wire x1="147.32" y1="73.66" x2="147.32" y2="119.38" width="0.1524" layer="91"/>
+<wire x1="160.02" y1="-81.28" x2="185.42" y2="-81.28" width="0.1524" layer="91"/>
+<label x="185.42" y="-81.28" size="1.778" layer="95"/>
+<pinref part="U1" gate="B4" pin="IO_L32N_4GCLK1"/>
+<wire x1="160.02" y1="-81.28" x2="160.02" y2="-40.64" width="0.1524" layer="91"/>
 </segment>
 </net>
@@
 </segment>
 </net>
-<net name="SAA" class="0">
-<segment>
-<pinref part="U1" gate="B5" pin="IO_L32P_5GCLK2"/>
-<wire x1="132.08" y1="-76.2" x2="132.08" y2="-40.64" width="0.1524" layer="91"/>
-<label x="99.06" y="-76.2" size="1.778" layer="95"/>
-<wire x1="132.08" y1="-76.2" x2="53.34" y2="-76.2" width="0.1524" layer="91"/>
-<wire x1="53.34" y1="-76.2" x2="53.34" y2="-66.04" width="0.1524" layer="91"/>
-<pinref part="SV1" gate="1" pin="9"/>
-</segment>
-</net>
 <net name="N$2" class="0">
 <segment>
@@
 </segment>
 </net>
+<net name="XAACLK16" class="0">
+<segment>
+<wire x1="147.32" y1="119.38" x2="162.56" y2="119.38" width="0.1524" layer="91"/>
+<label x="162.56" y="119.38" size="1.778" layer="95"/>
+<pinref part="U1" gate="B0" pin="IO_L32P_0GCLK6"/>
+<wire x1="147.32" y1="73.66" x2="147.32" y2="119.38" width="0.1524" layer="91"/>
+</segment>
+</net>

Commit message: going to bed
Parts:
- removed SV1: (no value), con-lstb:MA10-1
- added SV5: (no value), con-lstb:MA05-2
Connections:
- removed net ABAB: SV1.8, U1B5.IO_L31P_5D5
- removed net BB: SV1.7, U1B5.IO_L28N_5D6
- removed net N$10: SV1.3
- removed net N$11: SV1.4
- removed net N$13: SV1.5
- removed net N$15: SV1.6
- new net EXP_A: SV5.5, U1B5.IO_L28N_5D6
- new net EXP_B: SV5.6, U1B5.IO_L31P_5D5
- net GND: now also SV5.7, SV5.8; no longer SV1.2
- net R1: no longer SV1.9
- net VCC: now also SV5.3, SV5.4; no longer SV1.1
- net VCC5: now also SV5.10, SV5.9
- net VCCAUX: now also SV5.2
- net VCCINT: now also SV5.1
- net XXX: no longer SV1.10
Changed lines of the file:
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@@
 <part name="SUPPLY18" library="supply2" deviceset="GND" device=""/>
 <part name="SV3" library="con-lstb" deviceset="MA10-1" device=""/>
-<part name="SV1" library="con-lstb" deviceset="MA10-1" device="">
-<attribute name="MF" value=""/>
-<attribute name="MPN" value=""/>
-<attribute name="OC_FARNELL" value="unknown"/>
-<attribute name="OC_NEWARK" value="unknown"/>
-</part>
 <part name="SUPPLY19" library="supply2" deviceset="GND" device=""/>
 <part name="Q1" library="special" deviceset="XTAL/S" device=""/>
@@
 <part name="U$8" library="cpcfpga" deviceset="GNDHOLE" device=""/>
 <part name="U$9" library="cpcfpga" deviceset="GNDHOLE" device=""/>
+<part name="SV5" library="con-lstb" deviceset="MA05-2" device=""/>
 </parts>
 <sheets>
@@
 <instance part="SUPPLY18" gate="GND" x="-294.64" y="86.36"/>
 <instance part="SV3" gate="1" x="99.06" y="99.06"/>
-<instance part="SV1" gate="1" x="43.18" y="-58.42" rot="R270"/>
 <instance part="SUPPLY19" gate="GND" x="109.22" y="83.82"/>
 <instance part="Q1" gate="G$1" x="353.06" y="101.6" rot="R90"/>
@@
 <instance part="U$8" gate="G$1" x="-246.38" y="165.1"/>
 <instance part="U$9" gate="G$1" x="-246.38" y="157.48"/>
+<instance part="SV5" gate="G$1" x="35.56" y="-124.46" rot="R180"/>
 </instances>
 <busses>
@@
 <pinref part="SUPPLY17" gate="GND" pin="GND"/>
 <wire x1="35.56" y1="-68.58" x2="25.4" y2="-68.58" width="0.1524" layer="91"/>
-<pinref part="SV1" gate="1" pin="2"/>
 </segment>
 <segment>
@@
 <wire x1="520.7" y1="58.42" x2="520.7" y2="30.48" width="0.1524" layer="91"/>
 <junction x="520.7" y="30.48"/>
+</segment>
+<segment>
+<pinref part="SV5" gate="G$1" pin="7"/>
+<wire x1="20.32" y1="-127" x2="27.94" y2="-127" width="0.1524" layer="91"/>
+<label x="20.32" y="-127" size="1.778" layer="95"/>
+</segment>
+<segment>
+<pinref part="SV5" gate="G$1" pin="8"/>
+<wire x1="50.8" y1="-127" x2="43.18" y2="-127" width="0.1524" layer="91"/>
+<label x="50.8" y="-127" size="1.778" layer="95" rot="MR0"/>
 </segment>
 </net>
@@
 <label x="33.02" y="-76.2" size="1.778" layer="95" rot="R270"/>
 <wire x1="33.02" y1="-76.2" x2="33.02" y2="-66.04" width="0.1524" layer="91"/>
-<pinref part="SV1" gate="1" pin="1"/>
 </segment>
 <segment>
@@
 <wire x1="510.54" y1="33.02" x2="528.32" y2="33.02" width="0.1524" layer="91"/>
 <label x="510.54" y="33.02" size="1.778" layer="95"/>
+</segment>
+<segment>
+<pinref part="SV5" gate="G$1" pin="3"/>
+<wire x1="20.32" y1="-121.92" x2="27.94" y2="-121.92" width="0.1524" layer="91"/>
+<label x="20.32" y="-121.92" size="1.778" layer="95"/>
+</segment>
+<segment>
+<pinref part="SV5" gate="G$1" pin="4"/>
+<wire x1="50.8" y1="-121.92" x2="43.18" y2="-121.92" width="0.1524" layer="91"/>
+<label x="50.8" y="-121.92" size="1.778" layer="95" rot="MR0"/>
 </segment>
 </net>
@@
 <wire x1="-152.4" y1="38.1" x2="-172.72" y2="38.1" width="0.1524" layer="91"/>
 <junction x="-152.4" y="38.1"/>
+</segment>
+<segment>
+<pinref part="SV5" gate="G$1" pin="1"/>
+<wire x1="20.32" y1="-119.38" x2="27.94" y2="-119.38" width="0.1524" layer="91"/>
+<label x="20.32" y="-119.38" size="1.778" layer="95"/>
 </segment>
 </net>
@@
 <label x="203.2" y="276.86" size="1.778" layer="95" rot="MR0"/>
 </segment>
+<segment>
+<pinref part="SV5" gate="G$1" pin="2"/>
+<wire x1="50.8" y1="-119.38" x2="43.18" y2="-119.38" width="0.1524" layer="91"/>
+<label x="50.8" y="-119.38" size="1.778" layer="95" rot="MR0"/>
+</segment>
 </net>
 <net name="D_FASTBLANKING" class="0">
@@
 <wire x1="132.08" y1="-76.2" x2="53.34" y2="-76.2" width="0.1524" layer="91"/>
 <wire x1="53.34" y1="-76.2" x2="53.34" y2="-66.04" width="0.1524" layer="91"/>
-<pinref part="SV1" gate="1" pin="9"/>
 </segment>
 </net>
@@
 <junction x="-304.8" y="73.66"/>
 </segment>
+<segment>
+<pinref part="SV5" gate="G$1" pin="9"/>
+<wire x1="20.32" y1="-129.54" x2="27.94" y2="-129.54" width="0.1524" layer="91"/>
+<label x="20.32" y="-129.54" size="1.778" layer="95"/>
+</segment>
+<segment>
+<pinref part="SV5" gate="G$1" pin="10"/>
+<wire x1="50.8" y1="-129.54" x2="43.18" y2="-129.54" width="0.1524" layer="91"/>
+<label x="50.8" y="-129.54" size="1.778" layer="95" rot="MR0"/>
+</segment>
 </net>
 <net name="N$53" class="0">
@@
 <pinref part="U1" gate="B4" pin="IO_L32P_4GCLK0"/>
 <wire x1="162.56" y1="-40.64" x2="162.56" y2="-83.82" width="0.1524" layer="91"/>
-<pinref part="SV1" gate="1" pin="10"/>
-</segment>
-</net>
-<net name="BB" class="0">
+</segment>
+</net>
+<net name="EXP_A" class="0">
 <segment>
 <pinref part="U1" gate="B5" pin="IO_L28N_5D6"/>
@@
 <wire x1="142.24" y1="-68.58" x2="142.24" y2="-40.64" width="0.1524" layer="91"/>
 <label x="99.06" y="-68.58" size="1.778" layer="95"/>
-<pinref part="SV1" gate="1" pin="7"/>
 <wire x1="48.26" y1="-66.04" x2="48.26" y2="-96.52" width="0.1524" layer="91"/>
 <wire x1="48.26" y1="-96.52" x2="78.74" y2="-96.52" width="0.1524" layer="91"/>
 <wire x1="78.74" y1="-96.52" x2="78.74" y2="-68.58" width="0.1524" layer="91"/>
+</segment>
+<segment>
+<pinref part="SV5" gate="G$1" pin="5"/>
+<wire x1="20.32" y1="-124.46" x2="27.94" y2="-124.46" width="0.1524" layer="91"/>
+<label x="20.32" y="-124.46" size="1.778" layer="95"/>
 </segment>
 </net>
@@
 </segment>
 </net>
-<net name="ABAB" class="0">
+<net name="EXP_B" class="0">
 <segment>
 <pinref part="U1" gate="B5" pin="IO_L31P_5D5"/>
@@
 <wire x1="81.28" y1="-99.06" x2="50.8" y2="-99.06" width="0.1524" layer="91"/>
 <wire x1="50.8" y1="-99.06" x2="50.8" y2="-66.04" width="0.1524" layer="91"/>
-<pinref part="SV1" gate="1" pin="8"/>
 <wire x1="81.28" y1="-71.12" x2="81.28" y2="-99.06" width="0.1524" layer="91"/>
+</segment>
+<segment>
+<pinref part="SV5" gate="G$1" pin="6"/>
+<wire x1="50.8" y1="-124.46" x2="43.18" y2="-124.46" width="0.1524" layer="91"/>
+<label x="50.8" y="-124.46" size="1.778" layer="95" rot="MR0"/>
 </segment>
 </net>
@@
 <net name="N$10" class="0">
 <segment>
-<pinref part="SV1" gate="1" pin="3"/>
 <wire x1="38.1" y1="-83.82" x2="38.1" y2="-66.04" width="0.1524" layer="91"/>
 <label x="38.1" y="-83.82" size="1.778" layer="95" rot="R90"/>
@@
 <net name="N$11" class="0">
 <segment>
-<pinref part="SV1" gate="1" pin="4"/>
 <wire x1="40.64" y1="-83.82" x2="40.64" y2="-66.04" width="0.1524" layer="91"/>
 <label x="40.64" y="-83.82" size="1.778" layer="95" rot="R90"/>
@@
 <net name="N$13" class="0">
 <segment>
-<pinref part="SV1" gate="1" pin="5"/>
 <wire x1="43.18" y1="-83.82" x2="43.18" y2="-66.04" width="0.1524" layer="91"/>
 </segment>
@@
 <net name="N$15" class="0">
 <segment>
-<pinref part="SV1" gate="1" pin="6"/>
 <wire x1="45.72" y1="-83.82" x2="45.72" y2="-66.04" width="0.1524" layer="91"/>
 </segment>

Commit message: mah
Connections:
- removed net XAACLK16: U1B0.IO_L32P_0GCLK6
- new net N$3: SV3.3, U1B0.IO_L27N_0
- net CASIN: now also U1B0.IO_L30P_0; no longer U1B0.IO_L27N_0
- net N$4: now also U1B0.IO_L31N_0; no longer U1B0.IO_L30P_0
- net N$5: now also U1B0.IO_L31P_0VREF_0; no longer U1B0.IO_L31N_0
- net N$6: now also U1B0.IO_L32N_0GCLK7; no longer U1B0.IO_L31P_0VREF_0
- net N$7: now also U1B0.IO_L32P_0GCLK6; no longer U1B0.IO_L32N_0GCLK7
Changed lines of the file:
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@@
 </segment>
 <segment>
-<pinref part="U1" gate="B0" pin="IO_L27N_0"/>
-<wire x1="134.62" y1="93.98" x2="134.62" y2="81.28" width="0.1524" layer="91"/>
-<wire x1="134.62" y1="81.28" x2="134.62" y2="73.66" width="0.1524" layer="91"/>
-<wire x1="86.36" y1="81.28" x2="134.62" y2="81.28" width="0.1524" layer="91"/>
-<junction x="134.62" y="81.28"/>
 <label x="86.36" y="81.28" size="1.778" layer="95"/>
+<wire x1="86.36" y1="81.28" x2="121.92" y2="81.28" width="0.1524" layer="91"/>
+<wire x1="121.92" y1="81.28" x2="121.92" y2="83.82" width="0.1524" layer="91"/>
+<pinref part="U1" gate="B0" pin="IO_L30P_0"/>
+<wire x1="121.92" y1="83.82" x2="137.16" y2="83.82" width="0.1524" layer="91"/>
+<wire x1="137.16" y1="83.82" x2="137.16" y2="73.66" width="0.1524" layer="91"/>
 </segment>
 </net>
@@
 </segment>
 </net>
-<net name="N$2" class="0">
-<segment>
-<pinref part="SV3" gate="1" pin="4"/>
-<pinref part="U1" gate="B0" pin="IO_L27P_0"/>
-<wire x1="106.68" y1="96.52" x2="132.08" y2="96.52" width="0.1524" layer="91"/>
-<wire x1="132.08" y1="96.52" x2="132.08" y2="73.66" width="0.1524" layer="91"/>
-</segment>
-</net>
-<net name="N$3" class="0">
-<segment>
-<pinref part="SV3" gate="1" pin="5"/>
-<pinref part="U1" gate="B0" pin="IO_L30N_0"/>
-<wire x1="106.68" y1="99.06" x2="139.7" y2="99.06" width="0.1524" layer="91"/>
-<wire x1="139.7" y1="99.06" x2="139.7" y2="73.66" width="0.1524" layer="91"/>
-</segment>
-</net>
-<net name="N$4" class="0">
-<segment>
-<pinref part="SV3" gate="1" pin="6"/>
-<pinref part="U1" gate="B0" pin="IO_L30P_0"/>
-<wire x1="106.68" y1="101.6" x2="137.16" y2="101.6" width="0.1524" layer="91"/>
-<wire x1="137.16" y1="101.6" x2="137.16" y2="73.66" width="0.1524" layer="91"/>
-</segment>
-</net>
-<net name="N$5" class="0">
-<segment>
-<pinref part="SV3" gate="1" pin="7"/>
-<pinref part="U1" gate="B0" pin="IO_L31N_0"/>
-<wire x1="106.68" y1="104.14" x2="142.24" y2="104.14" width="0.1524" layer="91"/>
-<wire x1="142.24" y1="104.14" x2="142.24" y2="73.66" width="0.1524" layer="91"/>
-</segment>
-</net>
-<net name="N$6" class="0">
-<segment>
-<pinref part="SV3" gate="1" pin="8"/>
-<pinref part="U1" gate="B0" pin="IO_L31P_0VREF_0"/>
-<wire x1="106.68" y1="106.68" x2="144.78" y2="106.68" width="0.1524" layer="91"/>
-<wire x1="144.78" y1="106.68" x2="144.78" y2="73.66" width="0.1524" layer="91"/>
-</segment>
-</net>
-<net name="N$7" class="0">
-<segment>
-<pinref part="SV3" gate="1" pin="9"/>
-<pinref part="U1" gate="B0" pin="IO_L32N_0GCLK7"/>
-<wire x1="106.68" y1="109.22" x2="149.86" y2="109.22" width="0.1524" layer="91"/>
-<wire x1="149.86" y1="109.22" x2="149.86" y2="73.66" width="0.1524" layer="91"/>
-</segment>
-</net>
-<net name="N$8" class="0">
-<segment>
-<pinref part="SV3" gate="1" pin="10"/>
-<wire x1="106.68" y1="111.76" x2="182.88" y2="111.76" width="0.1524" layer="91"/>
-<pinref part="U1" gate="B1" pin="IO_L32N_1GCLK5"/>
-<wire x1="182.88" y1="111.76" x2="182.88" y2="73.66" width="0.1524" layer="91"/>
-</segment>
-</net>
 <net name="FPGA_RESET" class="0">
 <segment>
@@
 <wire x1="147.32" y1="119.38" x2="162.56" y2="119.38" width="0.1524" layer="91"/>
 <label x="162.56" y="119.38" size="1.778" layer="95"/>
+</segment>
+</net>
+<net name="N$3" class="0">
+<segment>
+<pinref part="U1" gate="B0" pin="IO_L27N_0"/>
+<pinref part="SV3" gate="1" pin="3"/>
+<wire x1="134.62" y1="93.98" x2="134.62" y2="73.66" width="0.1524" layer="91"/>
+<wire x1="106.68" y1="93.98" x2="134.62" y2="93.98" width="0.1524" layer="91"/>
+</segment>
+</net>
+<net name="N$1" class="0">
+<segment>
+<pinref part="SV3" gate="1" pin="4"/>
+<pinref part="U1" gate="B0" pin="IO_L27P_0"/>
+<wire x1="106.68" y1="96.52" x2="132.08" y2="96.52" width="0.1524" layer="91"/>
+<wire x1="132.08" y1="96.52" x2="132.08" y2="73.66" width="0.1524" layer="91"/>
+</segment>
+</net>
+<net name="N$2" class="0">
+<segment>
+<pinref part="SV3" gate="1" pin="5"/>
+<pinref part="U1" gate="B0" pin="IO_L30N_0"/>
+<wire x1="106.68" y1="99.06" x2="139.7" y2="99.06" width="0.1524" layer="91"/>
+<wire x1="139.7" y1="99.06" x2="139.7" y2="73.66" width="0.1524" layer="91"/>
+</segment>
+</net>
+<net name="N$4" class="0">
+<segment>
+<pinref part="SV3" gate="1" pin="6"/>
+<wire x1="106.68" y1="101.6" x2="142.24" y2="101.6" width="0.1524" layer="91"/>
+<pinref part="U1" gate="B0" pin="IO_L31N_0"/>
+<wire x1="142.24" y1="101.6" x2="142.24" y2="73.66" width="0.1524" layer="91"/>
+</segment>
+</net>
+<net name="N$5" class="0">
+<segment>
+<pinref part="SV3" gate="1" pin="7"/>
+<pinref part="U1" gate="B0" pin="IO_L31P_0VREF_0"/>
+<wire x1="106.68" y1="104.14" x2="144.78" y2="104.14" width="0.1524" layer="91"/>
+<wire x1="144.78" y1="104.14" x2="144.78" y2="73.66" width="0.1524" layer="91"/>
+</segment>
+</net>
+<net name="N$6" class="0">
+<segment>
+<pinref part="SV3" gate="1" pin="8"/>
+<pinref part="U1" gate="B0" pin="IO_L32N_0GCLK7"/>
+<wire x1="106.68" y1="106.68" x2="149.86" y2="106.68" width="0.1524" layer="91"/>
+<wire x1="149.86" y1="106.68" x2="149.86" y2="73.66" width="0.1524" layer="91"/>
+</segment>
+</net>
+<net name="N$7" class="0">
+<segment>
+<pinref part="SV3" gate="1" pin="9"/>
 <pinref part="U1" gate="B0" pin="IO_L32P_0GCLK6"/>
-<wire x1="147.32" y1="73.66" x2="147.32" y2="119.38" width="0.1524" layer="91"/>
-</segment>
-</net>
+<wire x1="106.68" y1="109.22" x2="147.32" y2="109.22" width="0.1524" layer="91"/>
+<wire x1="147.32" y1="109.22" x2="147.32" y2="73.66" width="0.1524" layer="91"/>
+</segment>
+</net>
+<net name="N$16" class="0">
+<segment>
+<pinref part="SV3" gate="1" pin="10"/>
+<pinref part="U1" gate="B1" pin="IO_L32N_1GCLK5"/>
+<wire x1="106.68" y1="111.76" x2="182.88" y2="111.76" width="0.1524" layer="91"/>
+<wire x1="182.88" y1="111.76" x2="182.88" y2="73.66" width="0.1524" layer="91"/>
+</segment>
+</net>
