File: eagle/homeboard/homeboard19.sch (EAGLE design)
At the start: 136 parts, among them IC1 XCF02S, IC2 25LC080SN, IC3 ATMEGA32U2-TQFP, Q5 BC848SMD, Q6 BC848SMD, Q7 BC848SMD, Q8 BC848SMD, T1 BSS138, T2 BC848, T3 BSS138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

Commit message: mah
Connections:
- net FPGA_RESET renamed AT_CLKO
- removed net X_CAS: U1B1.IO_L31N_1VREF_1
- net B0: now also U1B4.IO_L27P_4D1; no longer U1B4.IO_L01P_4VRN_4
- net B1: now also U1B4.IO_L30N_4D2; no longer U1B4.IO_L27P_4D1
- net FPGA_AUDIO_LEFT: now also U1B4.IO_L01P_4VRN_4; no longer U1B4.IO_L01N_4VRP_4
- net FPGA_AUDIO_RIGHT: now also U1B4.IO_L01N_4VRP_4; no longer U1B4.IOVREF_4
- net G0: now also U1B4.IO_L30P_4D3; no longer U1B4.IO_L30N_4D2
- net G1: now also U1B4.IO_L31P_4DOUTBUSY; no longer U1B4.IO_L30P_4D3
- net N$16: now also U1B1.IO_L31N_1VREF_1; no longer U1B1.IO_L32N_1GCLK5
- net PC5: now also U1B1.IO_L32N_1GCLK5
Changed lines of the file:
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@@
 <pinref part="U1" gate="B4" pin="IO_L31N_4INIT_B"/>
 <wire x1="175.26" y1="-40.64" x2="175.26" y2="-63.5" width="0.1524" layer="91"/>
-<wire x1="175.26" y1="-63.5" x2="185.42" y2="-63.5" width="0.1524" layer="91"/>
-<label x="180.34" y="-63.5" size="1.778" layer="95"/>
+<wire x1="175.26" y1="-63.5" x2="200.66" y2="-63.5" width="0.1524" layer="91"/>
+<label x="200.66" y="-63.5" size="1.778" layer="95"/>
 </segment>
 </net>
@@
 <pinref part="U1" gate="B4" pin="IO_L27N_4DIND0"/>
 <wire x1="172.72" y1="-40.64" x2="172.72" y2="-60.96" width="0.1524" layer="91"/>
-<wire x1="172.72" y1="-60.96" x2="185.42" y2="-60.96" width="0.1524" layer="91"/>
-<label x="180.34" y="-60.96" size="1.778" layer="95"/>
+<wire x1="172.72" y1="-60.96" x2="200.66" y2="-60.96" width="0.1524" layer="91"/>
+<label x="200.66" y="-60.96" size="1.778" layer="95"/>
 </segment>
 </net>
@@
 </segment>
 <segment>
-<pinref part="U1" gate="B4" pin="IO_L30P_4D3"/>
-<wire x1="185.42" y1="-71.12" x2="165.1" y2="-71.12" width="0.1524" layer="91"/>
-<wire x1="165.1" y1="-71.12" x2="165.1" y2="-40.64" width="0.1524" layer="91"/>
-<label x="185.42" y="-71.12" size="1.778" layer="95"/>
+<wire x1="200.66" y1="-71.12" x2="177.8" y2="-71.12" width="0.1524" layer="91"/>
+<label x="200.66" y="-71.12" size="1.778" layer="95"/>
+<pinref part="U1" gate="B4" pin="IO_L31P_4DOUTBUSY"/>
+<wire x1="177.8" y1="-40.64" x2="177.8" y2="-71.12" width="0.1524" layer="91"/>
 </segment>
 </net>
@@
 </segment>
 <segment>
-<pinref part="U1" gate="B4" pin="IO_L30N_4D2"/>
-<wire x1="185.42" y1="-68.58" x2="167.64" y2="-68.58" width="0.1524" layer="91"/>
-<wire x1="167.64" y1="-68.58" x2="167.64" y2="-40.64" width="0.1524" layer="91"/>
-<label x="185.42" y="-68.58" size="1.778" layer="95"/>
+<wire x1="200.66" y1="-68.58" x2="165.1" y2="-68.58" width="0.1524" layer="91"/>
+<label x="200.66" y="-68.58" size="1.778" layer="95"/>
+<pinref part="U1" gate="B4" pin="IO_L30P_4D3"/>
+<wire x1="165.1" y1="-40.64" x2="165.1" y2="-68.58" width="0.1524" layer="91"/>
 </segment>
 </net>
@@
 </segment>
 <segment>
-<pinref part="U1" gate="B4" pin="IO_L27P_4D1"/>
-<wire x1="185.42" y1="-66.04" x2="170.18" y2="-66.04" width="0.1524" layer="91"/>
-<wire x1="170.18" y1="-66.04" x2="170.18" y2="-40.64" width="0.1524" layer="91"/>
-<label x="185.42" y="-66.04" size="1.778" layer="95"/>
+<wire x1="200.66" y1="-66.04" x2="167.64" y2="-66.04" width="0.1524" layer="91"/>
+<label x="200.66" y="-66.04" size="1.778" layer="95"/>
+<pinref part="U1" gate="B4" pin="IO_L30N_4D2"/>
+<wire x1="167.64" y1="-40.64" x2="167.64" y2="-66.04" width="0.1524" layer="91"/>
 </segment>
 </net>
@@
 </segment>
 <segment>
-<pinref part="U1" gate="B4" pin="IO_L01P_4VRN_4"/>
-<wire x1="185.42" y1="-58.42" x2="182.88" y2="-58.42" width="0.1524" layer="91"/>
-<wire x1="182.88" y1="-58.42" x2="182.88" y2="-40.64" width="0.1524" layer="91"/>
-<label x="185.42" y="-58.42" size="1.778" layer="95"/>
+<wire x1="200.66" y1="-58.42" x2="170.18" y2="-58.42" width="0.1524" layer="91"/>
+<label x="200.66" y="-58.42" size="1.778" layer="95"/>
+<pinref part="U1" gate="B4" pin="IO_L27P_4D1"/>
+<wire x1="170.18" y1="-40.64" x2="170.18" y2="-58.42" width="0.1524" layer="91"/>
 </segment>
 </net>
@@
 </segment>
 <segment>
-<pinref part="U1" gate="B4" pin="IO_L01N_4VRP_4"/>
-<wire x1="185.42" y1="-55.88" x2="180.34" y2="-55.88" width="0.1524" layer="91"/>
-<wire x1="180.34" y1="-55.88" x2="180.34" y2="-40.64" width="0.1524" layer="91"/>
-<label x="185.42" y="-55.88" size="1.778" layer="95"/>
+<wire x1="200.66" y1="-55.88" x2="182.88" y2="-55.88" width="0.1524" layer="91"/>
+<label x="200.66" y="-55.88" size="1.778" layer="95"/>
+<pinref part="U1" gate="B4" pin="IO_L01P_4VRN_4"/>
+<wire x1="182.88" y1="-55.88" x2="182.88" y2="-40.64" width="0.1524" layer="91"/>
 </segment>
 </net>
@@
 </segment>
 <segment>
-<pinref part="U1" gate="B4" pin="IOVREF_4"/>
-<wire x1="185.42" y1="-53.34" x2="157.48" y2="-53.34" width="0.1524" layer="91"/>
-<wire x1="157.48" y1="-53.34" x2="157.48" y2="-40.64" width="0.1524" layer="91"/>
-<label x="185.42" y="-53.34" size="1.778" layer="95"/>
+<wire x1="200.66" y1="-53.34" x2="180.34" y2="-53.34" width="0.1524" layer="91"/>
+<label x="200.66" y="-53.34" size="1.778" layer="95"/>
+<pinref part="U1" gate="B4" pin="IO_L01N_4VRP_4"/>
+<wire x1="180.34" y1="-53.34" x2="180.34" y2="-40.64" width="0.1524" layer="91"/>
 </segment>
 </net>
@@
 </segment>
 </net>
-<net name="FPGA_RESET" class="0">
+<net name="AT_CLKO" class="0">
 <segment>
 <wire x1="180.34" y1="116.84" x2="162.56" y2="116.84" width="0.1524" layer="91"/>
@@
 <label x="454.66" y="81.28" size="1.778" layer="95"/>
 </segment>
+<segment>
+<wire x1="182.88" y1="119.38" x2="162.56" y2="119.38" width="0.1524" layer="91"/>
+<label x="162.56" y="119.38" size="1.778" layer="95"/>
+<pinref part="U1" gate="B1" pin="IO_L32N_1GCLK5"/>
+<wire x1="182.88" y1="73.66" x2="182.88" y2="119.38" width="0.1524" layer="91"/>
+</segment>
 </net>
 <net name="SD_CS" class="0">
@@
 <net name="X_CAS" class="0">
 <segment>
-<pinref part="U1" gate="B1" pin="IO_L31N_1VREF_1"/>
-<wire x1="177.8" y1="73.66" x2="177.8" y2="114.3" width="0.1524" layer="91"/>
 <wire x1="177.8" y1="114.3" x2="162.56" y2="114.3" width="0.1524" layer="91"/>
 <label x="162.56" y="114.3" size="1.778" layer="95"/>
-</segment>
-</net>
-<net name="XAACLK16" class="0">
-<segment>
-<wire x1="147.32" y1="119.38" x2="162.56" y2="119.38" width="0.1524" layer="91"/>
-<label x="162.56" y="119.38" size="1.778" layer="95"/>
 </segment>
 </net>
@@
 <segment>
 <pinref part="SV3" gate="1" pin="10"/>
-<pinref part="U1" gate="B1" pin="IO_L32N_1GCLK5"/>
-<wire x1="106.68" y1="111.76" x2="182.88" y2="111.76" width="0.1524" layer="91"/>
-<wire x1="182.88" y1="111.76" x2="182.88" y2="73.66" width="0.1524" layer="91"/>
-</segment>
-</net>
+<wire x1="106.68" y1="111.76" x2="177.8" y2="111.76" width="0.1524" layer="91"/>
+<pinref part="U1" gate="B1" pin="IO_L31N_1VREF_1"/>
+<wire x1="177.8" y1="73.66" x2="177.8" y2="111.76" width="0.1524" layer="91"/>
+</segment>
+</net>

Commit message: mah
Connections:
- net FL_DI: now also U1B3.IO
- net FL_DO: now also U1B3.IO_L01P_3VRN_3
- net FL_HOLD: now also U1B3.IO_L20N_3
- net FL_SCLK: now also U1B3.IO_L20P_3
- net FL_SEL: now also U1B4.IOVREF_4
- net FL_WP: now also U1B3.IO_L01N_3VRP_3
Other:
- moved on the sheet: IC2
Changed lines of the file:
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@@
 <instance part="SUPPLY4" gate="GND" x="-20.32" y="152.4"/>
 <instance part="SUPPLY5" gate="GND" x="-20.32" y="198.12"/>
-<instance part="IC2" gate="G$1" x="254" y="93.98"/>
+<instance part="IC2" gate="G$1" x="259.08" y="-83.82"/>
 <instance part="R48" gate="G$1" x="144.78" y="177.8"/>
 <instance part="C1" gate="G$1" x="132.08" y="172.72" rot="R180"/>
@@
 <segment>
 <pinref part="IC2" gate="G$1" pin="GND"/>
-<wire x1="274.32" y1="83.82" x2="261.62" y2="83.82" width="0.1524" layer="91"/>
-<label x="269.24" y="83.82" size="1.778" layer="95"/>
+<wire x1="279.4" y1="-93.98" x2="266.7" y2="-93.98" width="0.1524" layer="91"/>
+<label x="274.32" y="-93.98" size="1.778" layer="95"/>
 </segment>
 <segment>
@@
 <segment>
 <pinref part="IC2" gate="G$1" pin="VCC"/>
-<label x="269.24" y="106.68" size="1.778" layer="95"/>
-<wire x1="261.62" y1="106.68" x2="274.32" y2="106.68" width="0.1524" layer="91"/>
+<label x="274.32" y="-71.12" size="1.778" layer="95"/>
+<wire x1="266.7" y1="-71.12" x2="279.4" y2="-71.12" width="0.1524" layer="91"/>
 </segment>
 <segment>
@@
 <segment>
 <pinref part="IC2" gate="G$1" pin="!CS"/>
-<wire x1="233.68" y1="96.52" x2="241.3" y2="96.52" width="0.1524" layer="91"/>
-<label x="233.68" y="96.52" size="1.778" layer="95"/>
+<wire x1="238.76" y1="-81.28" x2="246.38" y2="-81.28" width="0.1524" layer="91"/>
+<label x="238.76" y="-81.28" size="1.778" layer="95"/>
 </segment>
 <segment>
@@
 <wire x1="231.14" y1="45.72" x2="210.82" y2="45.72" width="0.1524" layer="91"/>
 <label x="231.14" y="45.72" size="1.778" layer="95"/>
+</segment>
+<segment>
+<pinref part="U1" gate="B4" pin="IOVREF_4"/>
+<wire x1="236.22" y1="-45.72" x2="157.48" y2="-45.72" width="0.1524" layer="91"/>
+<wire x1="157.48" y1="-45.72" x2="157.48" y2="-40.64" width="0.1524" layer="91"/>
+<wire x1="236.22" y1="-58.42" x2="236.22" y2="-45.72" width="0.1524" layer="91"/>
+<label x="236.22" y="-58.42" size="1.778" layer="95" rot="R90"/>
 </segment>
 </net>
@@
 <segment>
 <pinref part="IC2" gate="G$1" pin="!HOLD"/>
-<label x="233.68" y="88.9" size="1.778" layer="95"/>
-<wire x1="233.68" y1="88.9" x2="241.3" y2="88.9" width="0.1524" layer="91"/>
+<label x="238.76" y="-88.9" size="1.778" layer="95"/>
+<wire x1="238.76" y1="-88.9" x2="246.38" y2="-88.9" width="0.1524" layer="91"/>
 </segment>
 <segment>
@@
 <label x="231.14" y="53.34" size="1.778" layer="95"/>
 </segment>
+<segment>
+<pinref part="U1" gate="B3" pin="IO_L20N_3"/>
+<wire x1="210.82" y1="2.54" x2="248.92" y2="2.54" width="0.1524" layer="91"/>
+<wire x1="248.92" y1="2.54" x2="248.92" y2="-58.42" width="0.1524" layer="91"/>
+<label x="248.92" y="-58.42" size="1.778" layer="95" rot="R90"/>
+</segment>
 </net>
 <net name="FL_SCLK" class="0">
 <segment>
 <pinref part="IC2" gate="G$1" pin="SCK"/>
-<wire x1="233.68" y1="91.44" x2="241.3" y2="91.44" width="0.1524" layer="91"/>
-<label x="233.68" y="91.44" size="1.778" layer="95"/>
+<wire x1="238.76" y1="-86.36" x2="246.38" y2="-86.36" width="0.1524" layer="91"/>
+<label x="238.76" y="-86.36" size="1.778" layer="95"/>
 </segment>
 <segment>
@@
 <label x="231.14" y="55.88" size="1.778" layer="95"/>
 </segment>
+<segment>
+<pinref part="U1" gate="B3" pin="IO_L20P_3"/>
+<wire x1="210.82" y1="5.08" x2="246.38" y2="5.08" width="0.1524" layer="91"/>
+<wire x1="246.38" y1="5.08" x2="246.38" y2="-58.42" width="0.1524" layer="91"/>
+<label x="246.38" y="-58.42" size="1.778" layer="95" rot="R90"/>
+</segment>
 </net>
 <net name="FL_DI" class="0">
 <segment>
 <pinref part="IC2" gate="G$1" pin="SI"/>
-<wire x1="233.68" y1="93.98" x2="241.3" y2="93.98" width="0.1524" layer="91"/>
-<label x="233.68" y="93.98" size="1.778" layer="95"/>
+<wire x1="238.76" y1="-83.82" x2="246.38" y2="-83.82" width="0.1524" layer="91"/>
+<label x="238.76" y="-83.82" size="1.778" layer="95"/>
 </segment>
 <segment>
@@
 <label x="231.14" y="48.26" size="1.778" layer="95"/>
 </segment>
+<segment>
+<wire x1="243.84" y1="-58.42" x2="243.84" y2="12.7" width="0.1524" layer="91"/>
+<pinref part="U1" gate="B3" pin="IO"/>
+<wire x1="243.84" y1="12.7" x2="210.82" y2="12.7" width="0.1524" layer="91"/>
+<label x="243.84" y="-58.42" size="1.778" layer="95" rot="R90"/>
+</segment>
 </net>
 <net name="FL_DO" class="0">
 <segment>
 <pinref part="IC2" gate="G$1" pin="SO"/>
-<wire x1="274.32" y1="93.98" x2="269.24" y2="93.98" width="0.1524" layer="91"/>
-<label x="269.24" y="93.98" size="1.778" layer="95"/>
+<wire x1="279.4" y1="-83.82" x2="274.32" y2="-83.82" width="0.1524" layer="91"/>
+<label x="274.32" y="-83.82" size="1.778" layer="95"/>
 </segment>
 <segment>
@@
 <label x="231.14" y="43.18" size="1.778" layer="95"/>
 </segment>
+<segment>
+<wire x1="238.76" y1="-58.42" x2="238.76" y2="10.16" width="0.1524" layer="91"/>
+<pinref part="U1" gate="B3" pin="IO_L01P_3VRN_3"/>
+<wire x1="238.76" y1="10.16" x2="210.82" y2="10.16" width="0.1524" layer="91"/>
+<label x="238.76" y="-58.42" size="1.778" layer="95" rot="R90"/>
+</segment>
 </net>
 <net name="FL_WP" class="0">
 <segment>
 <pinref part="IC2" gate="G$1" pin="!WP"/>
-<wire x1="233.68" y1="101.6" x2="241.3" y2="101.6" width="0.1524" layer="91"/>
-<label x="233.68" y="101.6" size="1.778" layer="95"/>
+<wire x1="238.76" y1="-76.2" x2="246.38" y2="-76.2" width="0.1524" layer="91"/>
+<label x="238.76" y="-76.2" size="1.778" layer="95"/>
 </segment>
 <segment>
@@
 <label x="231.14" y="50.8" size="1.778" layer="95"/>
 </segment>
-</net>
+<segment>
+<pinref part="U1" gate="B3" pin="IO_L01N_3VRP_3"/>
+<wire x1="210.82" y1="7.62" x2="241.3" y2="7.62" width="0.1524" layer="91"/>
+<wire x1="241.3" y1="7.62" x2="241.3" y2="-58.42" width="0.1524" layer="91"/>
+<label x="241.3" y="-58.42" size="1.778" layer="95" rot="R90"/>
+</segment>
+</net>

Commit message: stuff
Connections:
- net FL_DI: no longer U1B2.IO_L20N_2
- net FL_DO: no longer U1B2.IO_L21N_2
- net FL_HOLD: no longer U1B2.IO_L01N_2VRP_2
- net FL_SCLK: no longer U1B2.IO_L01P_2VRN_2
- net FL_SEL: no longer U1B2.IO_L21P_2
- net FL_WP: no longer U1B2.IO_L20P_2
- net JOY1_DOWN: now also U1B2.IO_L20N_2
- net JOY1_FIRE1: now also U1B2.IO_L20P_2
- net JOY1_FIRE2: now also U1B2.IO_L01P_2VRN_2
- net JOY1_LEFT: now also U1B2.IO_L21N_2
- net JOY1_RIGHT: now also U1B2.IO_L21P_2
- net JOY1_UP: now also U1B2.IO_L01N_2VRP_2
Changed lines of the file:
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@@
 <label x="-27.94" y="180.34" size="1.778" layer="95"/>
+</segment>
+<segment>
+<pinref part="U1" gate="B2" pin="IO_L20P_2"/>
+<wire x1="231.14" y1="50.8" x2="210.82" y2="50.8" width="0.1524" layer="91"/>
+<label x="231.14" y="50.8" size="1.778" layer="95"/>
 </segment>
 </net>
@@
 <label x="-27.94" y="177.8" size="1.778" layer="95"/>
 </segment>
+<segment>
+<pinref part="U1" gate="B2" pin="IO_L01P_2VRN_2"/>
+<wire x1="210.82" y1="55.88" x2="231.14" y2="55.88" width="0.1524" layer="91"/>
+<label x="231.14" y="55.88" size="1.778" layer="95"/>
+</segment>
 </net>
 <net name="JOY1_RIGHT" class="0">
@@
 <label x="-27.94" y="172.72" size="1.778" layer="95"/>
 </segment>
+<segment>
+<pinref part="U1" gate="B2" pin="IO_L21P_2"/>
+<wire x1="231.14" y1="45.72" x2="210.82" y2="45.72" width="0.1524" layer="91"/>
+<label x="231.14" y="45.72" size="1.778" layer="95"/>
+</segment>
 </net>
 <net name="JOY1_LEFT" class="0">
@@
 <label x="-27.94" y="170.18" size="1.778" layer="95"/>
 </segment>
+<segment>
+<pinref part="U1" gate="B2" pin="IO_L21N_2"/>
+<wire x1="231.14" y1="43.18" x2="210.82" y2="43.18" width="0.1524" layer="91"/>
+<label x="231.14" y="43.18" size="1.778" layer="95"/>
+</segment>
 </net>
 <net name="JOY1_DOWN" class="0">
@@
 <label x="-27.94" y="167.64" size="1.778" layer="95"/>
 </segment>
+<segment>
+<pinref part="U1" gate="B2" pin="IO_L20N_2"/>
+<wire x1="231.14" y1="48.26" x2="210.82" y2="48.26" width="0.1524" layer="91"/>
+<label x="231.14" y="48.26" size="1.778" layer="95"/>
+</segment>
 </net>
 <net name="JOY1_UP" class="0">
@@
 <label x="-27.94" y="165.1" size="1.778" layer="95"/>
 </segment>
+<segment>
+<pinref part="U1" gate="B2" pin="IO_L01N_2VRP_2"/>
+<wire x1="231.14" y1="53.34" x2="210.82" y2="53.34" width="0.1524" layer="91"/>
+<label x="231.14" y="53.34" size="1.778" layer="95"/>
+</segment>
 </net>
 <net name="JOY0_UP" class="0">
@@
 <wire x1="76.2" y1="-111.76" x2="144.78" y2="-111.76" width="0.1524" layer="91"/>
 <label x="76.2" y="-111.76" size="1.778" layer="95"/>
-</segment>
-<segment>
-<pinref part="U1" gate="B2" pin="IO_L21P_2"/>
-<wire x1="231.14" y1="45.72" x2="210.82" y2="45.72" width="0.1524" layer="91"/>
-<label x="231.14" y="45.72" size="1.778" layer="95"/>
 </segment>
 <segment>
@@
 </segment>
 <segment>
-<pinref part="U1" gate="B2" pin="IO_L01N_2VRP_2"/>
-<wire x1="231.14" y1="53.34" x2="210.82" y2="53.34" width="0.1524" layer="91"/>
-<label x="231.14" y="53.34" size="1.778" layer="95"/>
-</segment>
-<segment>
 <pinref part="U1" gate="B3" pin="IO_L20N_3"/>
 <wire x1="210.82" y1="2.54" x2="248.92" y2="2.54" width="0.1524" layer="91"/>
@@
 </segment>
 <segment>
-<pinref part="U1" gate="B2" pin="IO_L01P_2VRN_2"/>
-<wire x1="210.82" y1="55.88" x2="231.14" y2="55.88" width="0.1524" layer="91"/>
-<label x="231.14" y="55.88" size="1.778" layer="95"/>
-</segment>
-<segment>
 <pinref part="U1" gate="B3" pin="IO_L20P_3"/>
 <wire x1="210.82" y1="5.08" x2="246.38" y2="5.08" width="0.1524" layer="91"/>
@@
 </segment>
 <segment>
-<pinref part="U1" gate="B2" pin="IO_L20N_2"/>
-<wire x1="231.14" y1="48.26" x2="210.82" y2="48.26" width="0.1524" layer="91"/>
-<label x="231.14" y="48.26" size="1.778" layer="95"/>
-</segment>
-<segment>
 <wire x1="243.84" y1="-58.42" x2="243.84" y2="12.7" width="0.1524" layer="91"/>
 <pinref part="U1" gate="B3" pin="IO"/>
@@
 </segment>
 <segment>
-<pinref part="U1" gate="B2" pin="IO_L21N_2"/>
-<wire x1="231.14" y1="43.18" x2="210.82" y2="43.18" width="0.1524" layer="91"/>
-<label x="231.14" y="43.18" size="1.778" layer="95"/>
-</segment>
-<segment>
 <wire x1="238.76" y1="-58.42" x2="238.76" y2="10.16" width="0.1524" layer="91"/>
 <pinref part="U1" gate="B3" pin="IO_L01P_3VRN_3"/>
@@
 </segment>
 <segment>
-<pinref part="U1" gate="B2" pin="IO_L20P_2"/>
-<wire x1="231.14" y1="50.8" x2="210.82" y2="50.8" width="0.1524" layer="91"/>
-<label x="231.14" y="50.8" size="1.778" layer="95"/>
-</segment>
-<segment>
