File: eagle/homeboard/homeboard19.brd (EAGLE design)
At the start: 94.5 x 70.8 mm, 136 parts, among them IC1 XCF02S, IC2 25LC080SN, IC3 ATMEGA32U2-TQFP, Q5 BC848SMD, Q6 BC848SMD, Q7 BC848SMD, Q8 BC848SMD, T1 BSS138, T2 BC848, T3 BSS138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

Commit message: stuff
Parts:
- moved U$8 18.2 mm to (72.0, 66.2)
- moved R3 13.1 mm to (57.8, 49.2)
- moved R2 8.75 mm to (61.5, 49.0)
- moved R48 4.03 mm to (71.2, 15.8), turned to 90 degrees
- moved C3 0.71 mm to (75.5, 13.0), turned to 270 degrees
Routing:
- net PC5: track 19.2 -> 29.2 mm
- net GND: track 778.3 -> 770.3 mm
- net AT_CLKO: track 38.4 -> 43.3 mm
- net JOY1_RIGHT: track 31.1 -> 27.3 mm
- net JOY1_FIRE2: track 33.2 -> 29.7 mm
- net JOY1_LEFT: track 30.4 -> 26.8 mm
- net JOY1_UP: track 28.1 -> 24.6 mm
- net JOY1_DOWN: track 28.6 -> 25.0 mm
- net JOY1_FIRE1: track 34.4 -> 30.9 mm
- net N$43: track 11.7 -> 8.76 mm
- net N$52: track 3.02 -> 5.47 mm
- net PROM_INITB: track 32.2 -> 30.5 mm
- net FPGA_AUDIO_RIGHT: track 24.7 -> 23.2 mm
- net N$38: track 21.8 -> 20.6 mm
- net N$51: track 6.70 -> 5.64 mm
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
Commit message: progress
Parts:
- moved SJ1 32.2 mm to (66.5, 42.0), flipped to the bottom, turned to 270 degrees
- moved C38 10.1 mm to (72.5, 45.8)
- moved C37 6.02 mm to (72.5, 50.2), turned to 90 degrees
- moved Q1 5.93 mm to (70.0, 48.2), turned to 270 degrees
- moved C27 3.80 mm to (73.2, 40.5), turned to 270 degrees
- moved IC3 3.41 mm to (75.5, 38.8), turned to 0 degrees
- moved R10 0.50 mm to (52.8, 17.5)
- moved R9 0.50 mm to (50.5, 17.5)
Connections:
- new net N$8: IC3.1, SJ1.2
- net EXTCLK: now also U1.P100
- net N$14: now also SJ1.1; no longer IC3.1
- net PC2: now also U1.P99; no longer U1.P100
- net PD0: now also U1.P98; no longer U1.P99
- net PD1: now also U1.P97; no longer U1.P98
- net PD2: now also U1.P96; no longer U1.P97
- net PD3: now also U1.P92; no longer U1.P95
- net PD5: now also U1.P95; no longer U1.P92
- net PD6: now also U1.P90; no longer U1.P96
Routing:
- net TDI_FPGA: track 59.2 -> 1.84 mm, vias 1 -> 0
- net AT_CLKO: track 43.3 -> 0.00 mm, vias 2 -> 0
- net TMS: track 42.3 -> 6.17 mm, vias 3 -> 0
- net TCK: track 36.5 -> 4.54 mm, vias 2 -> 0
- net VCC: track 468.2 -> 441.4 mm, vias 23 -> 21
- net TDO_PROM: track 21.0 -> 2.04 mm, vias 2 -> 0
- net EMER_BOOT: track 26.3 -> 11.6 mm, vias 2 -> 1
- net AT_RESET: track 15.2 -> 2.07 mm, vias 1 -> 0
- net N$69: track 32.1 -> 19.1 mm
- net N$49: track 16.3 -> 4.65 mm
- net N$9: track 13.3 -> 2.52 mm
- net N$68: track 14.9 -> 5.96 mm
- net PC5: track 29.2 -> 21.6 mm
- net GND: track 770.3 -> 762.9 mm
- net PC4: track 6.96 -> 0.00 mm
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
Commit message: progress
Parts:
- moved C41 2.50 mm to (88.0, 46.8)
- moved R53 2.50 mm to (85.2, 52.2)
- moved R54 2.50 mm to (87.8, 52.2)
- moved U$5 2.50 mm to (83.8, 65.5)
- moved X6 2.50 mm to (84.2, 60.5)
- moved SV2 0.59 mm to (97.2, 28.0), turned to 270 degrees
Routing:
- net GND: track 762.9 -> 762.1 mm

Commit message: progress
Parts:
- moved R3 1.58 mm to (59.2, 49.8), flipped to the top, turned to 90 degrees
- moved R2 1.00 mm to (61.5, 48.0), flipped to the top, turned to 90 degrees
- moved R56 0.50 mm to (90.0, 43.2)
Routing:
- net JOY0_RIGHT: track 41.8 -> 3.05 mm
- net TMS: track 6.17 -> 15.0 mm, vias 0 -> 1
- net AT_CLKO: track 0.00 -> 4.56 mm, vias 0 -> 1
- net N$39: track 7.12 -> 2.61 mm, vias 1 -> 0
- net TCK: track 4.54 -> 8.72 mm, vias 0 -> 1
- net N$43: track 8.76 -> 5.06 mm, vias 1 -> 0
Changed lines of the file:
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@@
 <element name="IC1" library="smd-special" package="VO20" value="XCF02S" x="83.093396875" y="15.237409375" rot="R90"/>
 <element name="R1" library="rcl" package="R0805" value="100" x="41.4986" y="43.2594" rot="MR270"/>
-<element name="R2" library="rcl" package="R0805" value="100" x="61.5" y="49" rot="MR270"/>
-<element name="R3" library="rcl" package="R0805" value="100" x="57.75" y="49.25" rot="MR270"/>
+<element name="R2" library="rcl" package="R0805" value="100" x="61.5" y="48" rot="R90"/>
+<element name="R3" library="rcl" package="R0805" value="100" x="59.25" y="49.75" rot="R90"/>
 <element name="T1" library="zetex" package="SOT-23" value="BSS138" x="30" y="14.75" rot="MR0">
 <attribute name="OC_NEWARK" value="unknown" x="30" y="40.75" size="1.778" layer="28" rot="MR0" display="off"/>
@@
 <attribute name="OC_FARNELL" value="unknown" x="97.207109375" y="27.957109375" size="1.778" layer="27" rot="R270" display="off"/>
 </element>
-<element name="R56" library="rcl" package="R0805" value="4700" x="90" y="43.75"/>
+<element name="R56" library="rcl" package="R0805" value="4700" x="90" y="43.25"/>
 <element name="U$3" library="cpcfpga" package="SDCARD-NOHOLE" value="SDMMCNOHOLE" x="28.75" y="49.75" rot="R270"/>
 <element name="C39" library="rcl" package="PANASONIC_D" value="100u" x="18.5" y="25.75" rot="R270"/>
@@
 <wire x1="86.35" y1="66.135" x2="98.27" y2="78.43" width="0" layer="19" extent="1-1"/>
 <wire x1="96" y1="46.95" x2="86.35" y2="64.865" width="0" layer="19" extent="1-1"/>
-<wire x1="89.05" y1="43.75" x2="96" y2="46.95" width="0" layer="19" extent="1-1"/>
-<wire x1="88.75" y1="39.25" x2="89.05" y2="43.75" width="0" layer="19" extent="1-16"/>
+<wire x1="89.05" y1="43.25" x2="96" y2="46.95" width="0" layer="19" extent="1-1"/>
+<wire x1="88.75" y1="39.25" x2="89.05" y2="43.25" width="0" layer="19" extent="1-16"/>
 <wire x1="91.52" y1="27.44" x2="91.5" y2="27.5" width="0" layer="19" extent="1-1"/>
 <wire x1="97.15" y1="38" x2="93.25" y2="38.25" width="0" layer="19" extent="1-1"/>
@@
 <wire x1="79.76226875" y1="37.623221875" x2="88.98" y2="29.98" width="0" layer="19" extent="1-1"/>
 <wire x1="81" y1="19" x2="88.98" y2="29.98" width="0" layer="19" extent="1-1"/>
-<wire x1="61.5" y1="48.05" x2="79.76226875" y2="37.623221875" width="0" layer="19" extent="1-16"/>
+<wire x1="61.5" y1="48.95" x2="62.55" y2="48.95" width="0.254" layer="1"/>
+<wire x1="62.55" y1="48.95" x2="63" y2="48.5" width="0.254" layer="1"/>
+<wire x1="63" y1="48.5" x2="63" y2="48" width="0.254" layer="1"/>
+<via x="63" y="48" extent="1-16" drill="0.7" shape="square"/>
+<wire x1="63" y1="48" x2="63" y2="46" width="0.254" layer="16"/>
+<wire x1="63" y1="46" x2="79.76226875" y2="37.623221875" width="0" layer="19" extent="1-16"/>
 </signal>
 <signal name="TMS">
@@
 <wire x1="85.58" y1="27.42" x2="79.76226875" y2="36.823221875" width="0" layer="19" extent="1-1"/>
 <wire x1="79.5" y1="19" x2="85.58" y2="27.42" width="0" layer="19" extent="1-1"/>
-<wire x1="57.75" y1="48.3" x2="79.76226875" y2="36.823221875" width="0" layer="19" extent="1-16"/>
+<wire x1="59.25" y1="50.7" x2="61.8" y2="50.7" width="0.254" layer="1"/>
+<wire x1="64.5" y1="45.5" x2="79.76226875" y2="36.823221875" width="0" layer="19" extent="1-16"/>
+<wire x1="65" y1="47.5" x2="65" y2="45.5" width="0" layer="19" extent="1-16"/>
+<wire x1="65" y1="45.5" x2="79.76226875" y2="36.823221875" width="0" layer="19" extent="1-16"/>
+<wire x1="61.8" y1="50.7" x2="64.5" y2="48" width="0.254" layer="1"/>
+<wire x1="64.5" y1="48" x2="64.5" y2="47" width="0.254" layer="1"/>
+<via x="64.5" y="47" extent="1-16" drill="0.7" shape="square"/>
+<wire x1="64.5" y1="47" x2="64.5" y2="45.5" width="0.254" layer="16"/>
 </signal>
 <signal name="TDI_FPGA">
@@
 <contactref element="R2" pad="1"/>
 <contactref element="U1" pad="P110"/>
-<wire x1="61.47" y1="44.45" x2="61.47" y2="47.03" width="0.254" layer="1"/>
-<wire x1="61.47" y1="47.03" x2="60" y2="48.5" width="0.254" layer="1"/>
-<wire x1="60" y1="48.5" x2="60" y2="49" width="0.254" layer="1"/>
-<via x="60" y="49" extent="1-16" drill="0.7" shape="square"/>
-<wire x1="60" y1="49" x2="61" y2="50" width="0.254" layer="16"/>
-<wire x1="61" y1="50" x2="61.5" y2="50" width="0.254" layer="16"/>
-<wire x1="61.5" y1="50" x2="61.5" y2="49.95" width="0.254" layer="16"/>
+<wire x1="61.47" y1="44.45" x2="61.47" y2="47.02" width="0.254" layer="1"/>
+<wire x1="61.47" y1="47.02" x2="61.5" y2="47.05" width="0.254" layer="1"/>
 </signal>
 <signal name="N$42">
@@
 <contactref element="R3" pad="1"/>
 <contactref element="U1" pad="P111"/>
-<wire x1="60.97" y1="44.45" x2="60.97" y2="46.53" width="0.254" layer="1"/>
-<wire x1="60.97" y1="46.53" x2="59" y2="48.5" width="0.254" layer="1"/>
-<wire x1="59" y1="48.5" x2="59" y2="49.75" width="0.254" layer="1"/>
-<wire x1="59" y1="49.75" x2="59.5" y2="50.25" width="0.254" layer="1"/>
-<via x="59.5" y="50.25" extent="1-16" drill="0.7" shape="square"/>
-<wire x1="59.5" y1="50.25" x2="58.25" y2="50.25" width="0.254" layer="16"/>
-<wire x1="58.25" y1="50.25" x2="58" y2="50" width="0.254" layer="16"/>
-<wire x1="57.75" y1="50.2" x2="57.8" y2="50.2" width="0.254" layer="16"/>
-<wire x1="57.8" y1="50.2" x2="58" y2="50" width="0.254" layer="16"/>
+<wire x1="60.97" y1="44.45" x2="60.97" y2="45.53" width="0.254" layer="1"/>
+<wire x1="60.97" y1="45.53" x2="59.25" y2="47.25" width="0.254" layer="1"/>
+<wire x1="59.25" y1="48.8" x2="59.25" y2="47.25" width="0.254" layer="1"/>
 </signal>
 <signal name="N$35">
@@
 <wire x1="21.75" y1="55.45" x2="21.75" y2="56.25" width="0.254" layer="16"/>
 <wire x1="21.75" y1="56.25" x2="23.5" y2="58" width="0.254" layer="16"/>
-<wire x1="55.47" y1="44.45" x2="55.47" y2="45.97" width="0.254" layer="1"/>
-<wire x1="55.47" y1="45.97" x2="56" y2="46.5" width="0.254" layer="1"/>
-<wire x1="56" y1="46.5" x2="56" y2="51.5" width="0.254" layer="1"/>
+<wire x1="55.47" y1="44.45" x2="55.47" y2="45.47" width="0.254" layer="1"/>
+<wire x1="55.47" y1="45.47" x2="56" y2="46" width="0.254" layer="1"/>
+<wire x1="56" y1="46" x2="56" y2="51.5" width="0.254" layer="1"/>
 <wire x1="56" y1="51.5" x2="55" y2="52.5" width="0.254" layer="1"/>
 <wire x1="55" y1="52.5" x2="36" y2="52.5" width="0.254" layer="1"/>
@@
 <wire x1="33" y1="55.45" x2="33" y2="56.7232" width="0.254" layer="16"/>
 <wire x1="33" y1="56.7232" x2="31.7432" y2="57.98" width="0.254" layer="16"/>
-<wire x1="57.5" y1="55" x2="38.5" y2="55" width="0.254" layer="1"/>
-<wire x1="38.5" y1="55" x2="37" y2="56.5" width="0.254" layer="1"/>
-<wire x1="37" y1="56.5" x2="33.2232" y2="56.5" width="0.254" layer="1"/>
-<wire x1="33.2232" y1="56.5" x2="31.7432" y2="57.98" width="0.254" layer="1"/>
-<wire x1="60.47" y1="44.45" x2="60.47" y2="46.03" width="0.254" layer="1"/>
-<wire x1="60.47" y1="46.03" x2="58.5" y2="48" width="0.254" layer="1"/>
-<wire x1="58.5" y1="48" x2="58.5" y2="54" width="0.254" layer="1"/>
-<wire x1="58.5" y1="54" x2="57.5" y2="55" width="0.254" layer="1"/>
+<wire x1="33" y1="55.45" x2="60.47" y2="44.45" width="0" layer="19" extent="1-16"/>
 </signal>
 <signal name="JOY0_FIRE2">
@@
 <contactref element="IC3" pad="22"/>
 <contactref element="U1" pad="P124"/>
-<wire x1="54.47" y1="44.45" x2="79.76226875" y2="40.023221875" width="0" layer="19" extent="1-1"/>
+<wire x1="54.47" y1="44.45" x2="54.47" y2="46.97" width="0.254" layer="1"/>
+<wire x1="54.47" y1="46.97" x2="54.5" y2="47" width="0.254" layer="1"/>
+<via x="54.5" y="47" extent="1-16" drill="0.7" shape="square"/>
+<wire x1="54.5" y1="47" x2="56.5" y2="47" width="0.254" layer="16"/>
+<wire x1="56.5" y1="47" x2="79.76226875" y2="40.023221875" width="0" layer="19" extent="1-16"/>
 </signal>
 <signal name="N$12">
@@
 <wire x1="91.52" y1="33.23" x2="91.5" y2="33.25" width="0.254" layer="16"/>
 <contactref element="R56" pad="2"/>
-<wire x1="91.25" y1="33.75" x2="90.95" y2="43.75" width="0" layer="19" extent="1-16"/>
-<wire x1="79.76226875" y1="41.623221875" x2="90.95" y2="43.75" width="0" layer="19" extent="1-1"/>
+<wire x1="91.25" y1="33.75" x2="90.95" y2="43.25" width="0" layer="19" extent="1-16"/>
+<wire x1="79.76226875" y1="41.623221875" x2="90.95" y2="43.25" width="0" layer="19" extent="1-1"/>
 </signal>
 <signal name="PC4">
@@
 <contactref element="SV3" pad="10"/>
 <contactref element="U1" pad="P123"/>
-<wire x1="54.97" y1="44.45" x2="54.97" y2="46.22" width="0.254" layer="1"/>
-<wire x1="54.97" y1="46.22" x2="55.5" y2="46.75" width="0.254" layer="1"/>
-<wire x1="55.5" y1="46.75" x2="55.5" y2="49" width="0.254" layer="1"/>
+<wire x1="54.97" y1="44.45" x2="54.97" y2="45.72" width="0.254" layer="1"/>
+<wire x1="54.97" y1="45.72" x2="55.5" y2="46.25" width="0.254" layer="1"/>
+<wire x1="55.5" y1="46.25" x2="55.5" y2="49" width="0.254" layer="1"/>
 <wire x1="55.5" y1="49" x2="55" y2="49.5" width="0.254" layer="1"/>
 <wire x1="55" y1="49.5" x2="54.5" y2="49.5" width="0.254" layer="1"/>

Commit message: progress
Parts:
- moved C32 2.50 mm to (89.0, 18.5)
- moved R55 1.50 mm to (90.0, 22.5)
- moved R56 1.50 mm to (88.5, 43.2)
- moved SV4 1.50 mm to (88.8, 31.2)
- moved R9 1.41 mm to (49.5, 16.5), turned to 0 degrees
- moved U$9 0.90 mm to (89.0, 11.0)
- moved C41 0.50 mm to (88.5, 46.8)
- moved R53 0.50 mm to (85.8, 52.2)
- moved R54 0.50 mm to (88.2, 52.2)
- moved U$5 0.50 mm to (84.2, 65.5)
- moved X6 0.50 mm to (84.8, 60.5)
Connections:
- removed net XXX: U1.P55
- new net EXP_C: SV5.8, U1.P51
- net CSYNC: now also U1.P52; no longer U1.P51
- net GND: no longer SV5.8
- net R0: now also U1.P55; no longer U1.P53
- net R1: now also U1.P53; no longer U1.P52
Routing:
- net VCC: track 441.4 -> 417.4 mm, vias 21 -> 20
- net EXP_C: track 0.00 -> 22.5 mm
- net GND: track 762.1 -> 750.5 mm, vias 28 -> 27
- net EMER_BOOT: track 11.6 -> 0.00 mm, vias 1 -> 0
- net R1: track 5.21 -> 8.80 mm
- net TMS: track 15.0 -> 11.6 mm
- net N$9: track 2.52 -> 0.00 mm, vias 1 -> 0
- net AT_RESET: track 2.07 -> 0.00 mm
- net PC5: track 21.6 -> 19.8 mm
- net TDI_FPGA: track 1.84 -> 0.00 mm
- net CSYNC: track 12.3 -> 13.1 mm
Other:
- board size 94.5 x 70.8 mm -> 93.5 x 70.8 mm

Commit message: progress
Parts:
- moved U$5 78.7 mm to (9.25, 41.5), flipped to the bottom, turned to 90 degrees
- moved R53 16.1 mm to (71.2, 45.2), flipped to the top, turned to 0 degrees
- moved R54 16.0 mm to (73.0, 47.5), flipped to the top, turned to 0 degrees
- moved C38 9.86 mm to (77.5, 54.2)
- moved C37 6.02 mm to (68.0, 54.2), turned to 270 degrees
- moved C41 6.02 mm to (84.0, 50.8), flipped to the top
- moved Q1 5.49 mm to (72.8, 53.0), turned to 0 degrees
Routing:
- net N$36: track 3.25 -> 23.4 mm, vias 0 -> 1
- net N$66: track 6.08 -> 25.6 mm, vias 0 -> 1
- net N$14: track 7.30 -> 21.3 mm, vias 0 -> 2
- net N$9: track 0.00 -> 11.8 mm
- net GND: track 750.5 -> 761.0 mm, vias 27 -> 28
- net VCC5: track 92.7 -> 99.2 mm, vias 3 -> 4
- net N$68: track 5.96 -> 3.54 mm, vias 1 -> 0
- net N$12: track 16.0 -> 17.9 mm, vias 0 -> 1
- net VCC: track 417.4 -> 418.7 mm, vias 20 -> 21
- net N$49: track 4.65 -> 4.83 mm, vias 1 -> 0

Commit message: progress
Parts:
- removed SJ2: (no value), jumper:SJ
- removed T4: BC848, transistor:SOT23
- moved U$8 26.2 mm to (89.0, 46.2)
- moved R52 14.5 mm to (81.5, 46.0), turned to 180 degrees
- moved R56 7.02 mm to (81.5, 43.8), turned to 180 degrees
Routing:
- net GND: track 761.0 -> 748.6 mm
- net PD5: track 15.0 -> 14.4 mm

Commit message: basic jtag conns
Parts:
- moved C29 7.02 mm to (72.5, 26.2), flipped to the bottom
- moved IC2 1.00 mm to (74.3, 26.1)
Routing:
- net TDI_FPGA: track 0.00 -> 47.1 mm, vias 0 -> 1
- net GND: track 748.6 -> 794.7 mm
- net TCK: track 8.72 -> 52.6 mm, vias 1 -> 3
- net TMS: track 11.6 -> 54.6 mm, vias 1 -> 3
- net AT_CLKO: track 4.56 -> 32.9 mm, vias 1 -> 2
- net TDO_PROM: track 2.04 -> 25.8 mm, vias 0 -> 2
- net EMER_BOOT: track 0.00 -> 5.54 mm, vias 0 -> 1
- net FL_WP: track 13.8 -> 12.8 mm
- net FL_SEL: track 14.2 -> 13.2 mm
- net FL_SCLK: track 14.1 -> 13.1 mm
- net FL_HOLD: track 12.5 -> 11.5 mm
- net FL_DO: track 12.2 -> 11.2 mm
- net FL_DI: track 15.5 -> 14.5 mm
Other:
- board text added: "CPCFPGA.COM"
- board text added: "CPCFPGA.COM rev 1 (c) 2012 Ranulf Doswell"
