File: eagle/homeboard/homeboard20.brd (EAGLE design)
At the start: 93.5 x 71.8 mm, 134 parts, among them IC1 XCF02S, IC2 25LC080SN, IC3 ATMEGA32U2-TQFP, Q5 BC848SMD, Q6 BC848SMD, Q7 BC848SMD, Q8 BC848SMD, T1 BSS138, T2 BC848, T3 BSS138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

Commit message: more work
Parts:
- moved SJ1 1.80 mm to (68.0, 42.0)
Routing:
- net A1: track 14.0 -> 0.00 mm
- net A2: track 12.5 -> 0.00 mm
- net A3: track 11.1 -> 0.00 mm
- net A4: track 9.75 -> 0.00 mm
- net A5: track 8.17 -> 0.00 mm
- net A6: track 6.79 -> 0.00 mm
- net VCC: track 461.0 -> 454.4 mm, vias 26 -> 24
- net N$8: track 5.83 -> 1.83 mm
- net N$14: track 21.8 -> 18.3 mm
- net EXTCLK: track 6.96 -> 4.73 mm
Changed lines of the file:
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@@
 <attribute name="OC_FARNELL" value="unknown" x="36.25" y="13.25" size="1.016" layer="27" rot="R270" display="off"/>
 </element>
-<element name="SJ1" library="jumper" package="SJ_2" value="" x="66.5" y="41" rot="MR270"/>
+<element name="SJ1" library="jumper" package="SJ_2" value="" x="68" y="42" rot="MR270"/>
 <element name="SV4" library="con-lstb" package="MA10-2" value="" x="89.55" y="30.5" rot="R270">
 <attribute name="OC_NEWARK" value="unknown" x="89.55" y="30.5" size="1.778" layer="27" rot="R270" display="off"/>
@@
 <wire x1="72.75" y1="42.75" x2="71.5" y2="42.75" width="0.6" layer="1"/>
 <wire x1="70.75" y1="42.75" x2="70.25" y2="43.25" width="0.6" layer="1"/>
-<wire x1="70.25" y1="43.25" x2="70.25" y2="45" width="0.6" layer="1"/>
-<wire x1="70.25" y1="45" x2="70.25" y2="50.25" width="0.6" layer="1"/>
+<wire x1="70.25" y1="43.25" x2="70.25" y2="50.25" width="0.6" layer="1"/>
 <wire x1="70.25" y1="50.25" x2="69" y2="50.25" width="0.6" layer="1"/>
 <wire x1="70.75" y1="42.75" x2="71.5" y2="42.75" width="0.6" layer="1"/>
 <wire x1="63.25" y1="43.75" x2="64.25" y2="43.75" width="0.6" layer="1"/>
-<wire x1="64.25" y1="43.75" x2="64.5" y2="44" width="0.6" layer="1"/>
-<via x="64.5" y="44" extent="1-16" drill="0.6" shape="square"/>
-<wire x1="64.5" y1="44" x2="68.5" y2="44" width="0.6" layer="16"/>
-<wire x1="68.5" y1="44" x2="69.5" y2="45" width="0.6" layer="16"/>
-<via x="69.5" y="45" extent="1-16" drill="0.6" shape="square"/>
-<wire x1="69.5" y1="45" x2="70.25" y2="45" width="0.6" layer="1"/>
 <wire x1="67.5" y1="12.4" x2="69.6" y2="12.4" width="0.8" layer="1"/>
 <wire x1="69.6" y1="12.4" x2="70" y2="12" width="0.8" layer="1"/>
@@
 <wire x1="12.5" y1="27.75" x2="12.599" y2="27.75" width="0" layer="19" extent="1-1"/>
 <wire x1="84.5" y1="18.85" x2="84.5" y2="19" width="0" layer="19" extent="16-16"/>
+<wire x1="70.25" y1="43.25" x2="64.25" y2="43.75" width="0" layer="19" extent="1-1"/>
 <wire x1="64.75" y1="53.55" x2="69" y2="50.25" width="0" layer="19" extent="1-1"/>
 <wire x1="62.5" y1="53.55" x2="64.75" y2="53.55" width="0" layer="19" extent="1-1"/>
@@
 <contactref element="C38" pad="2"/>
 <contactref element="SJ1" pad="1"/>
-<wire x1="66.5" y1="42.524" x2="68.5" y2="42.5" width="0.254" layer="16"/>
-<wire x1="68.5" y1="42.5" x2="69.524" y2="43.524" width="0.254" layer="16"/>
 <wire x1="69.524" y1="43.524" x2="70.524" y2="43.524" width="0.254" layer="16"/>
 <via x="71.5" y="44" extent="1-16" drill="0.7" shape="square"/>
@@
 <wire x1="70.524" y1="43.524" x2="71" y2="44" width="0.254" layer="16"/>
 <wire x1="71" y1="44" x2="71.5" y2="44" width="0.254" layer="16"/>
+<wire x1="68" y1="43.524" x2="69.524" y2="43.524" width="0" layer="19" extent="16-16"/>
 </signal>
 <signal name="EXP_B">
@@
 <contactref element="IC3" pad="1"/>
 <contactref element="SJ1" pad="2"/>
-<wire x1="66.5" y1="41" x2="69.5" y2="41" width="0.254" layer="16"/>
-<wire x1="69.5" y1="41" x2="69.5" y2="42" width="0.254" layer="16"/>
+<wire x1="69.5" y1="41" x2="69.5" y2="42" width="0" layer="19" extent="1-16"/>
 <via x="69.5" y="42" extent="1-16" drill="0.7" shape="square"/>
 <wire x1="71.17706875" y1="41.623221875" x2="69.876778125" y2="41.623221875" width="0.254" layer="1"/>
 <wire x1="69.876778125" y1="41.623221875" x2="69.5" y2="42" width="0.254" layer="1"/>
+<wire x1="68" y1="42" x2="69.5" y2="42" width="0" layer="19" extent="16-16"/>
 </signal>
 <signal name="EXTCLK">
@@
 <wire x1="67.75" y1="38.5" x2="68.5" y2="39" width="0.254" layer="1"/>
 <via x="68.5" y="39" extent="1-16" drill="0.7" shape="square"/>
-<wire x1="68.5" y1="39" x2="67" y2="39" width="0.254" layer="16"/>
-<wire x1="67" y1="39" x2="66.5" y2="39.5" width="0.254" layer="16"/>
-<wire x1="66.5" y1="39.476" x2="66.5" y2="39.5" width="0.254" layer="16"/>
+<wire x1="68.5" y1="39" x2="68" y2="40.476" width="0" layer="19" extent="16-16"/>
 </signal>
 <signal name="EXP_C">
@@
 <signal name="A1">
 <contactref element="U1" pad="P102"/>
-<wire x1="63.92" y1="39.5" x2="67" y2="39.5" width="0.254" layer="1"/>
-<wire x1="67" y1="39.5" x2="68" y2="40.5" width="0.254" layer="1"/>
-<wire x1="68" y1="40.5" x2="68" y2="50" width="0.254" layer="1"/>
 </signal>
 <signal name="A2">
 <contactref element="U1" pad="P103"/>
-<wire x1="63.92" y1="40" x2="66.5" y2="40" width="0.254" layer="1"/>
-<wire x1="66.5" y1="40" x2="67.5" y2="41" width="0.254" layer="1"/>
-<wire x1="67.5" y1="41" x2="67.5" y2="49.5" width="0.254" layer="1"/>
 </signal>
 <signal name="A3">
 <contactref element="U1" pad="P104"/>
-<wire x1="63.92" y1="40.5" x2="66" y2="40.5" width="0.254" layer="1"/>
-<wire x1="66" y1="40.5" x2="67" y2="41.5" width="0.254" layer="1"/>
-<wire x1="67" y1="41.5" x2="67" y2="49.1284" width="0.254" layer="1"/>
 </signal>
 <signal name="A4">
 <contactref element="U1" pad="P105"/>
-<wire x1="63.92" y1="41" x2="65.5" y2="41" width="0.254" layer="1"/>
-<wire x1="65.5" y1="41" x2="66.5" y2="42" width="0.254" layer="1"/>
-<wire x1="66.5" y1="42" x2="66.5" y2="48.7568" width="0.254" layer="1"/>
 </signal>
 <signal name="A5">
 <contactref element="U1" pad="P107"/>
-<wire x1="63.92" y1="42" x2="65.5" y2="42" width="0.254" layer="1"/>
-<wire x1="65.5" y1="42" x2="66" y2="42.5" width="0.254" layer="1"/>
-<wire x1="66" y1="42.5" x2="66" y2="48.3852" width="0.254" layer="1"/>
 </signal>
 <signal name="A6">
 <contactref element="U1" pad="P108"/>
-<wire x1="63.92" y1="42.5" x2="65" y2="42.5" width="0.254" layer="1"/>
-<wire x1="65" y1="42.5" x2="65.5" y2="43" width="0.254" layer="1"/>
-<wire x1="65.5" y1="43" x2="65.5" y2="48" width="0.254" layer="1"/>
 </signal>
 </signals>

Commit message: more work
Parts:
- moved C27 2.00 mm to (75.2, 40.5)
- moved C41 2.00 mm to (79.8, 46.0)
- moved IC3 2.00 mm to (77.5, 38.8)
- moved R53 2.00 mm to (74.2, 47.0)
- moved R54 2.00 mm to (76.5, 47.0)
- moved SJ1 2.00 mm to (70.0, 42.0)
Routing:
- net JOY1_FIRE1: track 19.5 -> 59.3 mm
- net JOY1_FIRE2: track 17.1 -> 56.6 mm
- net JOY1_LEFT: track 18.2 -> 55.9 mm
- net JOY1_DOWN: track 14.5 -> 52.1 mm
- net JOY1_UP: track 13.1 -> 50.1 mm
- net TDI_FPGA: track 57.7 -> 38.7 mm
- net TCK: track 58.4 -> 42.8 mm
- net TDO_PROM: track 38.2 -> 24.2 mm
- net AT_CLKO: track 37.7 -> 27.2 mm
- net TMS: track 60.7 -> 53.4 mm
- net EXTCLK: track 4.73 -> 8.71 mm
- net SPI_SCLK: track 6.46 -> 3.60 mm
- net SPI_MISO: track 6.08 -> 3.25 mm
- net PC4: track 19.4 -> 21.7 mm
- net N$14: track 18.3 -> 20.5 mm
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
Commit message: more work
Parts:
- moved R55 4.85 mm to (89.8, 41.2), turned to 180 degrees
- moved R56 4.51 mm to (89.2, 41.2), turned to 0 degrees
- moved U$8 4.00 mm to (89.0, 48.0)
- moved SV4 3.50 mm to (89.5, 27.0)
- moved R2 0.90 mm to (63.0, 49.2)
Routing:
- net JOY1_RIGHT: track 18.7 -> 56.6 mm
- net GND: track 770.7 -> 756.8 mm
- net AT_RESET: track 12.9 -> 0.00 mm
- net TMS: track 53.4 -> 41.4 mm
- net EMER_BOOT: track 23.6 -> 11.9 mm
- net TDO_EXP: track 10.7 -> 0.00 mm
- net VCC: track 454.7 -> 462.2 mm
- net N$39: track 0.00 -> 4.68 mm
- net N$43: track 0.00 -> 4.44 mm

Commit message: tidy up of top of board
Parts:
- removed U$5: MC33269D, cpcfpga:SO8
Connections:
- net GND: no longer U$5.1
- net VCC: no longer U$5.2, U$5.3, U$5.6, U$5.7
- net VCC5: no longer U$5.4
Routing:
- net VCC: track 462.2 -> 473.8 mm, vias 24 -> 23
- net CASIN: track 36.7 -> 47.3 mm
- net GND: track 756.8 -> 753.7 mm
- net VCC5: track 99.2 -> 96.5 mm
- net SD_CS: track 31.9 -> 33.4 mm
- net SD_DI: track 34.7 -> 35.7 mm
- net PC5: track 37.3 -> 36.3 mm
- net AT_CLKO: track 27.2 -> 26.2 mm
- net N$1: track 16.0 -> 16.7 mm

Commit message: work
Routing:
- net GND: track 753.7 -> 786.2 mm
- net VCC: track 473.8 -> 481.4 mm
Changed lines of the file:
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@@
 <wire x1="10" y1="66" x2="16" y2="66" width="0.8" layer="16"/>
 <wire x1="16" y1="66" x2="17.5" y2="64.5" width="0.8" layer="16"/>
-<wire x1="30" y1="65.25" x2="48.5" y2="65.25" width="0.8" layer="16"/>
+<wire x1="30" y1="65.25" x2="31" y2="65.25" width="0.8" layer="16"/>
+<wire x1="31" y1="65.25" x2="48.5" y2="65.25" width="0.8" layer="16"/>
 <wire x1="48.5" y1="65.25" x2="62.5" y2="65.25" width="0.8" layer="16"/>
 <wire x1="62.5" y1="65.25" x2="67.75" y2="65.25" width="0.8" layer="16"/>
@@
 <wire x1="26.5" y1="49" x2="27.5" y2="47.5" width="0.254" layer="16"/>
 <wire x1="27.5" y1="47.5" x2="28" y2="47" width="0.254" layer="16"/>
-<wire x1="28" y1="47" x2="29.61" y2="47" width="0.254" layer="16"/>
-<wire x1="29.61" y1="47" x2="33.11" y2="50.5" width="0.254" layer="16"/>
 <wire x1="18.25" y1="54.75" x2="9.75" y2="54.75" width="1.27" layer="16"/>
 <wire x1="9.75" y1="54.75" x2="9" y2="54" width="1.27" layer="16"/>
+<wire x1="28" y1="47" x2="31.5" y2="47" width="0.254" layer="16"/>
+<wire x1="31.5" y1="47" x2="33" y2="48.5" width="0.254" layer="16"/>
+<wire x1="33" y1="48.5" x2="33" y2="50.61" width="0.254" layer="16"/>
+<wire x1="33" y1="50.61" x2="33.11" y2="50.5" width="0.254" layer="16"/>
+<wire x1="33" y1="50.61" x2="33" y2="52.5" width="0.254" layer="16"/>
+<wire x1="33" y1="52.5" x2="19" y2="52.5" width="0.254" layer="16"/>
+<wire x1="19" y1="52.5" x2="18" y2="53.5" width="0.254" layer="16"/>
+<wire x1="18" y1="53.5" x2="18" y2="54.5" width="0.254" layer="16"/>
+<wire x1="18" y1="54.5" x2="18.25" y2="54.75" width="0.254" layer="16"/>
+<wire x1="48.4778" y1="60.25" x2="48.4778" y2="65.2278" width="0.254" layer="16"/>
+<wire x1="30.3716" y1="61.52" x2="30.3716" y2="64.6216" width="0.254" layer="16"/>
+<wire x1="30.3716" y1="64.6216" x2="31" y2="65.25" width="0.254" layer="16"/>
 <wire x1="81" y1="65.5" x2="95.73" y2="78.43" width="0" layer="19" extent="16-16"/>
 <wire x1="17.5" y1="64.5" x2="17.5" y2="64.25" width="0" layer="19" extent="16-16"/>
@@
 <wire x1="9" y1="21" x2="9" y2="21.25" width="0" layer="19" extent="16-16"/>
 <wire x1="6.9" y1="19.5" x2="7" y2="19.5" width="0" layer="19" extent="1-1"/>
-<wire x1="8" y1="49.5" x2="8.25" y2="49.75" width="0" layer="19" extent="16-16"/>
 <wire x1="57.225" y1="17.145" x2="57.5" y2="17.5" width="0" layer="19" extent="1-1"/>
 <wire x1="71.68" y1="9.08" x2="71.65" y2="6.65" width="0" layer="19" extent="16-16"/>
-<wire x1="30.3716" y1="61.52" x2="30.3716" y2="64.8784" width="0" layer="19" extent="16-16"/>
-<wire x1="62.3716" y1="61.52" x2="62.3716" y2="65.1216" width="0" layer="19" extent="16-16"/>
-<wire x1="48.4778" y1="60.25" x2="48.4778" y2="65.2278" width="0" layer="19" extent="16-16"/>
 <wire x1="82" y1="50" x2="79.5" y2="55" width="0" layer="19" extent="16-16"/>
 <wire x1="89" y1="48" x2="84" y2="48" width="0" layer="19" extent="16-16"/>
@@
 <wire x1="88.28" y1="35.89" x2="90.82" y2="35.89" width="0" layer="19" extent="1-1"/>
 <wire x1="96.5" y1="1.4" x2="89" y2="10" width="0" layer="19" extent="1-1"/>
+<wire x1="62.3716" y1="61.52" x2="62.3716" y2="65.1216" width="0.254" layer="16"/>
 </signal>
 <signal name="VCC">
@@
 <wire x1="88.28" y1="15.57" x2="85.5" y2="13.5" width="0" layer="19" extent="1-1"/>
 <wire x1="90.82" y1="15.57" x2="88.28" y2="15.57" width="0" layer="19" extent="1-1"/>
-<wire x1="71" y1="50.25" x2="64.75" y2="53.55" width="0" layer="19" extent="1-1"/>
 <wire x1="96.5" y1="3.1" x2="90.82" y2="15.57" width="0" layer="19" extent="1-1"/>
+<wire x1="71" y1="50.25" x2="68.05" y2="50.25" width="0.254" layer="1"/>
+<wire x1="68.05" y1="50.25" x2="64.75" y2="53.55" width="0.254" layer="1"/>
 </signal>
 <signal name="TCK">
@@
 <wire x1="30.5" y1="47" x2="29" y2="48.5" width="0.254" layer="1"/>
 <via x="29" y="48.5" extent="1-16" drill="0.6" shape="square"/>
-<wire x1="29" y1="48.5" x2="25.5" y2="52" width="0.254" layer="16"/>
-<wire x1="25.5" y1="52" x2="18.25" y2="52" width="0.254" layer="16"/>
-<wire x1="18.25" y1="52" x2="18" y2="52.25" width="0.254" layer="16"/>
+<wire x1="29" y1="48.5" x2="27.5" y2="50" width="0.254" layer="16"/>
+<wire x1="27.5" y1="50" x2="20.25" y2="50" width="0.254" layer="16"/>
+<wire x1="20.25" y1="50" x2="18" y2="52.25" width="0.254" layer="16"/>
 </signal>
 <signal name="PS2CLK">
@@
 <wire x1="16.25" y1="50.2" x2="16.25" y2="52.25" width="0.254" layer="1"/>
 <wire x1="16.25" y1="52.25" x2="16.5" y2="52.5" width="0.254" layer="1"/>
-<wire x1="16.25" y1="52.25" x2="16.2" y2="52.5" width="0" layer="19" extent="1-1"/>
+<wire x1="16.2" y1="52.5" x2="16.2" y2="52.3" width="0.254" layer="1"/>
+<wire x1="16.2" y1="52.3" x2="16.25" y2="52.25" width="0.254" layer="1"/>
 </signal>
 <signal name="N$63">

Commit message: work
Routing:
- net PC5: track 36.3 -> 13.7 mm, vias 3 -> 1
- net TDI_FPGA: track 38.7 -> 25.2 mm, vias 1 -> 0
- net AT_CLKO: track 26.2 -> 13.6 mm, vias 2 -> 1

Commit message: work
Routing:
- net TMS: track 41.4 -> 53.4 mm
- net TCK: track 42.8 -> 50.6 mm
- net PC5: track 13.7 -> 19.7 mm, vias 1 -> 2
- net TDI_FPGA: track 25.2 -> 22.7 mm
- net AT_CLKO: track 13.6 -> 11.1 mm
Changed lines of the file:
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@@
 <wire x1="30.3716" y1="61.52" x2="30.3716" y2="64.6216" width="0.254" layer="16"/>
 <wire x1="30.3716" y1="64.6216" x2="31" y2="65.25" width="0.254" layer="16"/>
+<wire x1="62.3716" y1="61.52" x2="62.3716" y2="65.1216" width="0.254" layer="16"/>
 <wire x1="81" y1="65.5" x2="95.73" y2="78.43" width="0" layer="19" extent="16-16"/>
 <wire x1="17.5" y1="64.5" x2="17.5" y2="64.25" width="0" layer="19" extent="16-16"/>
@@
 <wire x1="88.28" y1="35.89" x2="90.82" y2="35.89" width="0" layer="19" extent="1-1"/>
 <wire x1="96.5" y1="1.4" x2="89" y2="10" width="0" layer="19" extent="1-1"/>
-<wire x1="62.3716" y1="61.52" x2="62.3716" y2="65.1216" width="0.254" layer="16"/>
 </signal>
 <signal name="VCC">
@@
 <wire x1="30.5" y1="50.5" x2="30.5" y2="53.55" width="0.7" layer="1"/>
 <wire x1="30.75" y1="53.55" x2="30.5" y2="53.55" width="0.254" layer="1"/>
+<wire x1="72.25" y1="50.25" x2="68.05" y2="50.25" width="0.7" layer="1"/>
+<wire x1="68.05" y1="50.25" x2="64.75" y2="53.55" width="0.7" layer="1"/>
 <wire x1="97.45" y1="42.5" x2="98.27" y2="78.43" width="0" layer="19" extent="1-1"/>
 <wire x1="97.15" y1="38" x2="97.45" y2="42.5" width="0" layer="19" extent="1-1"/>
@@
 <wire x1="90.82" y1="15.57" x2="88.28" y2="15.57" width="0" layer="19" extent="1-1"/>
 <wire x1="96.5" y1="3.1" x2="90.82" y2="15.57" width="0" layer="19" extent="1-1"/>
-<wire x1="72.25" y1="50.25" x2="68.05" y2="50.25" width="0.7" layer="1"/>
-<wire x1="68.05" y1="50.25" x2="64.75" y2="53.55" width="0.7" layer="1"/>
 </signal>
 <signal name="TCK">
@@
 <via x="78" y="38.5" extent="1-16" drill="0.7" shape="square"/>
 <wire x1="78" y1="38.5" x2="77.5" y2="38.5" width="0.254" layer="16"/>
-<wire x1="77.5" y1="38.5" x2="77.5" y2="43" width="0.254" layer="16"/>
-<wire x1="77.5" y1="43" x2="74" y2="46.5" width="0.254" layer="16"/>
-<wire x1="74" y1="46.5" x2="69.5" y2="46.5" width="0.254" layer="16"/>
-<via x="69.5" y="46.5" extent="1-16" drill="0.7" shape="square"/>
-<wire x1="69.5" y1="46.5" x2="69.5" y2="47" width="0.254" layer="1"/>
+<wire x1="77.5" y1="38.5" x2="77.5" y2="43.5" width="0.254" layer="16"/>
+<wire x1="77.5" y1="43.5" x2="73" y2="48" width="0.254" layer="16"/>
 <wire x1="76.943396875" y1="17.837409375" x2="79.337409375" y2="17.837409375" width="0.254" layer="1"/>
 <wire x1="79.337409375" y1="17.837409375" x2="79.75" y2="18.25" width="0.254" layer="1"/>
@@
 <wire x1="78" y1="33.5" x2="78" y2="38.5" width="0.254" layer="16"/>
 <contactref element="SV4" pad="7"/>
+<wire x1="73" y1="48" x2="68.75" y2="48" width="0.254" layer="16"/>
+<via x="68.75" y="48" extent="1-16" drill="0.6" shape="square"/>
+<wire x1="68.75" y1="48" x2="66" y2="48" width="0.254" layer="1"/>
+<wire x1="66" y1="48" x2="64" y2="50" width="0.254" layer="1"/>
+<wire x1="64" y1="50" x2="63.2" y2="50" width="0.254" layer="1"/>
+<wire x1="63.2" y1="50" x2="63" y2="50.2" width="0.254" layer="1"/>
 <wire x1="79.75" y1="29.75" x2="88.28" y2="30.81" width="0" layer="19" extent="16-16"/>
-<wire x1="63" y1="50.2" x2="69.5" y2="47" width="0" layer="19" extent="1-1"/>
 </signal>
 <signal name="TMS">
@@
 <via x="77" y="36.5" extent="1-16" drill="0.7" shape="square"/>
 <wire x1="77" y1="36.5" x2="77" y2="42.5" width="0.254" layer="16"/>
-<wire x1="77" y1="42.5" x2="73.75" y2="46" width="0.254" layer="16"/>
-<wire x1="73.75" y1="46" x2="70.75" y2="46" width="0.254" layer="16"/>
-<wire x1="70.75" y1="46" x2="70.5" y2="45.75" width="0.254" layer="16"/>
-<wire x1="70.5" y1="45.75" x2="70.5" y2="45.25" width="0.254" layer="16"/>
-<via x="70.5" y="45.25" extent="1-16" drill="0.7" shape="square"/>
-<wire x1="70.5" y1="45.25" x2="70.5" y2="47" width="0.254" layer="1"/>
+<wire x1="77" y1="42.5" x2="72.5" y2="47" width="0.254" layer="16"/>
+<wire x1="72.5" y1="47" x2="70" y2="47" width="0.254" layer="16"/>
 <wire x1="76.943396875" y1="18.487409375" x2="78.487409375" y2="18.487409375" width="0.254" layer="1"/>
 <wire x1="78.487409375" y1="18.487409375" x2="78.75" y2="18.75" width="0.254" layer="1"/>
@@
 <wire x1="77" y1="33" x2="77" y2="36.5" width="0.254" layer="16"/>
 <contactref element="SV4" pad="10"/>
+<via x="70" y="47" extent="1-16" drill="0.6" shape="square"/>
+<wire x1="70" y1="47" x2="70" y2="49.25" width="0.254" layer="1"/>
+<wire x1="70" y1="49.25" x2="67.25" y2="49.25" width="0.254" layer="1"/>
+<wire x1="67.25" y1="49.25" x2="64.5" y2="52" width="0.254" layer="1"/>
+<wire x1="64.5" y1="52" x2="61.5" y2="52" width="0.254" layer="1"/>
+<wire x1="61.5" y1="52" x2="61" y2="51.5" width="0.254" layer="1"/>
+<wire x1="61" y1="51.5" x2="61" y2="50.95" width="0.254" layer="1"/>
+<wire x1="61" y1="50.95" x2="60.75" y2="50.7" width="0.254" layer="1"/>
 <wire x1="78.75" y1="29.25" x2="90.82" y2="28.27" width="0" layer="19" extent="16-16"/>
-<wire x1="60.75" y1="50.7" x2="70.5" y2="47" width="0" layer="19" extent="1-1"/>
 </signal>
 <signal name="TDI_FPGA">
@@
 <wire x1="44.5" y1="44" x2="44.5" y2="45" width="0.254" layer="16"/>
 <wire x1="44.5" y1="45" x2="62.5" y2="45" width="0.254" layer="16"/>
-<wire x1="62.5" y1="45" x2="62.5" y2="47.5" width="0.254" layer="16"/>
 <contactref element="SV4" pad="5"/>
 <wire x1="88.28" y1="33.35" x2="81.76226875" y2="39.223221875" width="0" layer="19" extent="1-1"/>
@@
 <wire x1="55" y1="46.75" x2="55" y2="45.5" width="0.254" layer="16"/>
 <wire x1="55" y1="45.5" x2="62" y2="45.5" width="0.254" layer="16"/>
-<wire x1="62" y1="45.5" x2="62" y2="48" width="0.254" layer="16"/>
 <wire x1="62" y1="45.5" x2="81.76226875" y2="40.023221875" width="0" layer="19" extent="1-16"/>
 </signal>
@@
 <wire x1="54.5" y1="48" x2="55.5" y2="48" width="0.254" layer="16"/>
 <wire x1="55.5" y1="48" x2="55.5" y2="46" width="0.254" layer="16"/>
-<wire x1="55.5" y1="46" x2="61.5" y2="46" width="0.254" layer="16"/>
+<wire x1="55.5" y1="46" x2="62" y2="46" width="0.254" layer="16"/>
 <contactref element="U1" pad="P93"/>
-<wire x1="63.92" y1="35" x2="80.26966875" y2="43.115821875" width="0" layer="19" extent="1-1"/>
-<wire x1="61.5" y1="46" x2="63.92" y2="35" width="0" layer="19" extent="1-16"/>
+<wire x1="62" y1="46" x2="62.5" y2="46.5" width="0.254" layer="16"/>
+<via x="62.5" y="46.5" extent="1-16" drill="0.6" shape="square"/>
+<wire x1="62.5" y1="46.5" x2="67.25" y2="46.5" width="0.254" layer="1"/>
+<wire x1="67.25" y1="46.5" x2="80.26966875" y2="43.115821875" width="0" layer="19" extent="1-1"/>
+<wire x1="63.92" y1="35" x2="62" y2="46" width="0" layer="19" extent="1-16"/>
 </signal>
 <signal name="SD_CS">

Commit message: work
Parts:
- moved SJ1 9.18 mm to (74.5, 50.0), turned to 0 degrees
- moved C20 0.50 mm to (56.5, 40.2)
- moved C29 0.50 mm to (75.8, 26.2)
- moved IC2 0.50 mm to (79.8, 26.1)
- moved R34 0.25 mm to (75.8, 13.8)
Routing:
- net TMS: track 53.4 -> 12.9 mm, vias 3 -> 1
- net TCK: track 50.6 -> 15.0 mm, vias 3 -> 1
- net PC4: track 21.7 -> 0.00 mm, vias 2 -> 0
- net N$14: track 20.5 -> 0.00 mm, vias 2 -> 0
- net GND: track 786.2 -> 766.6 mm, vias 30 -> 28
- net N$66: track 21.9 -> 3.43 mm, vias 1 -> 0
- net N$12: track 21.8 -> 4.22 mm, vias 1 -> 0
- net VCC: track 481.7 -> 465.3 mm, vias 23 -> 22
- net PD6: track 15.1 -> 0.00 mm
- net PD5: track 14.0 -> 0.23 mm
- net PD4: track 12.5 -> 0.00 mm
- net N$36: track 18.0 -> 5.86 mm, vias 1 -> 0
- net N$69: track 19.0 -> 7.15 mm, vias 1 -> 0
- net PD3: track 11.2 -> 0.00 mm
- net TDO_PROM: track 24.2 -> 14.2 mm, vias 2 -> 1
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