File: eagle/homeboard/homeboard20.sch (EAGLE design)
At the start: 134 parts, among them IC1 XCF02S, IC2 25LC080SN, IC3 ATMEGA32U2-TQFP, Q5 BC848SMD, Q6 BC848SMD, Q7 BC848SMD, Q8 BC848SMD, T1 BSS138, T2 BC848, T3 BSS138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

Commit message: tidy up of top of board
Parts:
- removed U$5: MC33269D, cpcfpga:MC33269D
Connections:
- net GND: no longer U$5.GND
- net VCC: no longer U$5.VOUT1, U$5.VOUT2, U$5.VOUT3, U$5.VOUT4
- net VCC5: no longer U$5.VCC
Other:
- note removed: "Choose one of these 3.3v regs"
Changed lines of the file:
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@@
 <part name="C33" library="rcl" deviceset="CPOL-EU" device="D" value="100u"/>
 <part name="SUPPLY14" library="supply2" deviceset="GND" device=""/>
-<part name="U$5" library="cpcfpga" deviceset="MC33269D" device=""/>
 <part name="SUPPLY15" library="supply2" deviceset="GND" device=""/>
 <part name="U$6" library="cpcfpga" deviceset="AS6C4008" device=""/>
@@
 <sheet>
 <plain>
-<text x="-167.64" y="86.36" size="1.778" layer="91">Choose one of these 3.3v regs</text>
 <text x="271.78" y="-254" size="1.778" layer="91">Possible alternative:</text>
 </plain>
@@
 </instance>
 <instance part="SUPPLY14" gate="GND" x="-226.06" y="58.42"/>
-<instance part="U$5" gate="G$1" x="-187.96" y="86.36"/>
 <instance part="SUPPLY15" gate="GND" x="48.26" y="-43.18"/>
 <instance part="U$6" gate="G$1" x="45.72" y="20.32" rot="MR270"/>
@@
 <pinref part="REG1.2" gate="G$1" pin="GND"/>
 <pinref part="SUPPLY3" gate="GND" pin="GND"/>
-<wire x1="-203.2" y1="83.82" x2="-205.74" y2="83.82" width="0.1524" layer="91"/>
-<wire x1="-205.74" y1="83.82" x2="-205.74" y2="53.34" width="0.1524" layer="91"/>
+<wire x1="-205.74" y1="106.68" x2="-205.74" y2="53.34" width="0.1524" layer="91"/>
 <pinref part="REG2.5" gate="G$1" pin="GND"/>
 <wire x1="-205.74" y1="53.34" x2="-203.2" y2="53.34" width="0.1524" layer="91"/>
@@
 <pinref part="U$4" gate="G$1" pin="GND"/>
 <wire x1="-203.2" y1="106.68" x2="-205.74" y2="106.68" width="0.1524" layer="91"/>
-<wire x1="-205.74" y1="106.68" x2="-205.74" y2="83.82" width="0.1524" layer="91"/>
-<junction x="-205.74" y="83.82"/>
-<pinref part="U$5" gate="G$1" pin="GND"/>
 </segment>
 <segment>
@@
 <wire x1="-109.22" y1="129.54" x2="-101.6" y2="129.54" width="0.1524" layer="91"/>
 <junction x="-109.22" y="129.54"/>
-<wire x1="-167.64" y1="91.44" x2="-170.18" y2="91.44" width="0.1524" layer="91"/>
-<label x="-167.64" y="91.44" size="1.778" layer="95"/>
 <pinref part="U$4" gate="G$1" pin="VOUT1"/>
 <wire x1="-172.72" y1="114.3" x2="-170.18" y2="114.3" width="0.1524" layer="91"/>
 <wire x1="-170.18" y1="114.3" x2="-170.18" y2="111.76" width="0.1524" layer="91"/>
-<wire x1="-170.18" y1="111.76" x2="-170.18" y2="91.44" width="0.1524" layer="91"/>
-<wire x1="-172.72" y1="86.36" x2="-170.18" y2="86.36" width="0.1524" layer="91"/>
-<wire x1="-170.18" y1="86.36" x2="-170.18" y2="88.9" width="0.1524" layer="91"/>
-<junction x="-170.18" y="91.44"/>
-<wire x1="-170.18" y1="88.9" x2="-170.18" y2="91.44" width="0.1524" layer="91"/>
-<wire x1="-172.72" y1="83.82" x2="-170.18" y2="83.82" width="0.1524" layer="91"/>
-<wire x1="-170.18" y1="83.82" x2="-170.18" y2="86.36" width="0.1524" layer="91"/>
-<junction x="-170.18" y="86.36"/>
-<wire x1="-172.72" y1="88.9" x2="-170.18" y2="88.9" width="0.1524" layer="91"/>
-<junction x="-170.18" y="88.9"/>
-<wire x1="-172.72" y1="91.44" x2="-170.18" y2="91.44" width="0.1524" layer="91"/>
 <pinref part="C6" gate="G$1" pin="1"/>
 <wire x1="-170.18" y1="111.76" x2="-165.1" y2="111.76" width="0.1524" layer="91"/>
-<junction x="-170.18" y="111.76"/>
 <pinref part="C7" gate="G$1" pin="1"/>
 <wire x1="-165.1" y1="111.76" x2="-160.02" y2="111.76" width="0.1524" layer="91"/>
@@
 <wire x1="-93.98" y1="129.54" x2="-101.6" y2="129.54" width="0.1524" layer="91"/>
 <junction x="-101.6" y="129.54"/>
-<pinref part="U$5" gate="G$1" pin="VOUT1"/>
-<pinref part="U$5" gate="G$1" pin="VOUT4"/>
-<pinref part="U$5" gate="G$1" pin="VOUT2"/>
-<pinref part="U$5" gate="G$1" pin="VOUT3"/>
 <pinref part="C39" gate="G$1" pin="+"/>
 <junction x="-160.02" y="111.76"/>
@@
 <wire x1="-208.28" y1="73.66" x2="-198.12" y2="73.66" width="0.1524" layer="91"/>
 <label x="-198.12" y="73.66" size="1.778" layer="95"/>
-<wire x1="-203.2" y1="91.44" x2="-208.28" y2="91.44" width="0.1524" layer="91"/>
-<wire x1="-208.28" y1="91.44" x2="-208.28" y2="73.66" width="0.1524" layer="91"/>
 <junction x="-208.28" y="73.66"/>
 <pinref part="U$4" gate="G$1" pin="VCC"/>
 <wire x1="-203.2" y1="114.3" x2="-208.28" y2="114.3" width="0.1524" layer="91"/>
-<wire x1="-208.28" y1="114.3" x2="-208.28" y2="91.44" width="0.1524" layer="91"/>
-<junction x="-208.28" y="91.44"/>
+<wire x1="-208.28" y1="114.3" x2="-208.28" y2="73.66" width="0.1524" layer="91"/>
 <wire x1="-226.06" y1="96.52" x2="-226.06" y2="73.66" width="0.1524" layer="91"/>
 <wire x1="-226.06" y1="73.66" x2="-208.28" y2="73.66" width="0.1524" layer="91"/>
@@
 <wire x1="-226.06" y1="71.12" x2="-226.06" y2="73.66" width="0.1524" layer="91"/>
 <junction x="-226.06" y="73.66"/>
-<pinref part="U$5" gate="G$1" pin="VCC"/>
 <wire x1="-226.06" y1="96.52" x2="-256.54" y2="96.52" width="0.1524" layer="91"/>
 <wire x1="-256.54" y1="96.52" x2="-264.16" y2="96.52" width="0.1524" layer="91"/>

Commit message: work
Connections:
- removed net A5: U1B2.IO_L01P_2VRN_2
- removed net A6: U1B2.IO_L01N_2VRP_2
- new net Q1: U1B2.IO_L24P_2
- new net Q2: U1B2.IO_L22N_2
- net EXTCLK: now also U1B2.IO_L01P_2VRN_2; no longer U1B2.IO_L22N_2
- net PC4: now also U1B2.IO_L01N_2VRP_2; no longer U1B2.IO_L24P_2
Changed lines of the file:
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@@
 </segment>
 <segment>
-<pinref part="U1" gate="B2" pin="IO_L22N_2"/>
-<wire x1="231.14" y1="38.1" x2="210.82" y2="38.1" width="0.1524" layer="91"/>
-<label x="231.14" y="38.1" size="1.778" layer="95"/>
+<pinref part="U1" gate="B2" pin="IO_L01P_2VRN_2"/>
+<wire x1="210.82" y1="55.88" x2="231.14" y2="55.88" width="0.1524" layer="91"/>
+<label x="231.14" y="55.88" size="1.778" layer="95"/>
 </segment>
 </net>
@@
 </segment>
 <segment>
-<pinref part="U1" gate="B2" pin="IO_L24P_2"/>
-<wire x1="231.14" y1="33.02" x2="210.82" y2="33.02" width="0.1524" layer="91"/>
-<label x="231.14" y="33.02" size="1.778" layer="95"/>
+<pinref part="U1" gate="B2" pin="IO_L01N_2VRP_2"/>
+<wire x1="231.14" y1="53.34" x2="210.82" y2="53.34" width="0.1524" layer="91"/>
+<label x="231.14" y="53.34" size="1.778" layer="95"/>
 </segment>
 </net>
@@
 </segment>
 </net>
-<net name="A5" class="0">
-<segment>
-<pinref part="U1" gate="B2" pin="IO_L01P_2VRN_2"/>
-<wire x1="210.82" y1="55.88" x2="231.14" y2="55.88" width="0.1524" layer="91"/>
-<label x="231.14" y="55.88" size="1.778" layer="95"/>
-</segment>
-</net>
-<net name="A6" class="0">
-<segment>
-<pinref part="U1" gate="B2" pin="IO_L01N_2VRP_2"/>
-<wire x1="231.14" y1="53.34" x2="210.82" y2="53.34" width="0.1524" layer="91"/>
-<label x="231.14" y="53.34" size="1.778" layer="95"/>
-</segment>
-</net>
+<net name="Q1" class="0">
+<segment>
+<pinref part="U1" gate="B2" pin="IO_L24P_2"/>
+<wire x1="231.14" y1="33.02" x2="210.82" y2="33.02" width="0.1524" layer="91"/>
+<label x="231.14" y="33.02" size="1.778" layer="95"/>
+</segment>
+</net>
+<net name="Q2" class="0">
+<segment>
+<pinref part="U1" gate="B2" pin="IO_L22N_2"/>
+<wire x1="231.14" y1="38.1" x2="210.82" y2="38.1" width="0.1524" layer="91"/>
+<label x="231.14" y="38.1" size="1.778" layer="95"/>
+</segment>
+</net>

Commit message: work
Connections:
- removed net A1: U1B2.IO_L21P_2
- removed net A2: U1B2.IO_L21N_2
- removed net A3: U1B2.IO_L20P_2
- removed net A4: U1B2.IO_L20N_2
- new net Q3: U1B2.IO_L40N_2
- new net Q4: U1B2.IO_L22P_2
- new net Q5: U1B2.IO_L23N_2VREF_2
- new net Q6: U1B2.IO_L24N_2
- new net Q7: U1B2.IO_L23P_2
- net PC2: now also U1B2.IO_L20N_2; no longer U1B2.IO_L22P_2
- net PC5: no longer U1B2.IO_L40N_2
- net PD0: now also U1B2.IO_L20P_2; no longer U1B2.IO_L23N_2VREF_2
- net PD1: now also U1B2.IO_L21N_2; no longer U1B2.IO_L23P_2
- net PD2: now also U1B2.IO_L21P_2; no longer U1B2.IO_L24N_2
Changed lines of the file:
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@@
 </segment>
 <segment>
-<pinref part="U1" gate="B2" pin="IO_L24N_2"/>
-<wire x1="231.14" y1="30.48" x2="210.82" y2="30.48" width="0.1524" layer="91"/>
-<label x="231.14" y="30.48" size="1.778" layer="95"/>
+<pinref part="U1" gate="B2" pin="IO_L21P_2"/>
+<wire x1="231.14" y1="45.72" x2="210.82" y2="45.72" width="0.1524" layer="91"/>
+<label x="231.14" y="45.72" size="1.778" layer="95"/>
 </segment>
 </net>
@@
 </segment>
 <segment>
-<pinref part="U1" gate="B2" pin="IO_L22P_2"/>
-<wire x1="231.14" y1="40.64" x2="210.82" y2="40.64" width="0.1524" layer="91"/>
-<label x="231.14" y="40.64" size="1.778" layer="95"/>
+<pinref part="U1" gate="B2" pin="IO_L20N_2"/>
+<wire x1="231.14" y1="48.26" x2="210.82" y2="48.26" width="0.1524" layer="91"/>
+<label x="231.14" y="48.26" size="1.778" layer="95"/>
 </segment>
 </net>
@@
 </segment>
 <segment>
-<pinref part="U1" gate="B2" pin="IO_L23N_2VREF_2"/>
-<wire x1="231.14" y1="25.4" x2="210.82" y2="25.4" width="0.1524" layer="91"/>
-<label x="231.14" y="25.4" size="1.778" layer="95"/>
+<pinref part="U1" gate="B2" pin="IO_L20P_2"/>
+<wire x1="231.14" y1="50.8" x2="210.82" y2="50.8" width="0.1524" layer="91"/>
+<label x="231.14" y="50.8" size="1.778" layer="95"/>
 </segment>
 </net>
@@
 </segment>
 <segment>
-<pinref part="U1" gate="B2" pin="IO_L23P_2"/>
-<wire x1="231.14" y1="35.56" x2="210.82" y2="35.56" width="0.1524" layer="91"/>
-<label x="231.14" y="35.56" size="1.778" layer="95"/>
+<pinref part="U1" gate="B2" pin="IO_L21N_2"/>
+<wire x1="231.14" y1="43.18" x2="210.82" y2="43.18" width="0.1524" layer="91"/>
+<label x="231.14" y="43.18" size="1.778" layer="95"/>
 </segment>
 </net>
@@
 <pinref part="U1" gate="B1" pin="IO_L32N_1GCLK5"/>
 <wire x1="182.88" y1="73.66" x2="182.88" y2="119.38" width="0.1524" layer="91"/>
-</segment>
-<segment>
-<pinref part="U1" gate="B2" pin="IO_L40N_2"/>
-<wire x1="231.14" y1="27.94" x2="210.82" y2="27.94" width="0.1524" layer="91"/>
-<label x="231.14" y="27.94" size="1.778" layer="95"/>
 </segment>
 </net>
@@
 </segment>
 </net>
-<net name="A1" class="0">
-<segment>
-<pinref part="U1" gate="B2" pin="IO_L21P_2"/>
-<wire x1="231.14" y1="45.72" x2="210.82" y2="45.72" width="0.1524" layer="91"/>
-<label x="231.14" y="45.72" size="1.778" layer="95"/>
-</segment>
-</net>
-<net name="A2" class="0">
-<segment>
-<pinref part="U1" gate="B2" pin="IO_L21N_2"/>
-<wire x1="231.14" y1="43.18" x2="210.82" y2="43.18" width="0.1524" layer="91"/>
-<label x="231.14" y="43.18" size="1.778" layer="95"/>
-</segment>
-</net>
-<net name="A3" class="0">
-<segment>
-<pinref part="U1" gate="B2" pin="IO_L20P_2"/>
-<wire x1="231.14" y1="50.8" x2="210.82" y2="50.8" width="0.1524" layer="91"/>
-<label x="231.14" y="50.8" size="1.778" layer="95"/>
-</segment>
-</net>
-<net name="A4" class="0">
-<segment>
-<pinref part="U1" gate="B2" pin="IO_L20N_2"/>
-<wire x1="231.14" y1="48.26" x2="210.82" y2="48.26" width="0.1524" layer="91"/>
-<label x="231.14" y="48.26" size="1.778" layer="95"/>
-</segment>
-</net>
 <net name="Q1" class="0">
 <segment>
@@
 </segment>
 </net>
+<net name="Q3" class="0">
+<segment>
+<pinref part="U1" gate="B2" pin="IO_L40N_2"/>
+<wire x1="231.14" y1="27.94" x2="210.82" y2="27.94" width="0.1524" layer="91"/>
+<label x="231.14" y="27.94" size="1.778" layer="95"/>
+</segment>
+</net>
+<net name="Q4" class="0">
+<segment>
+<pinref part="U1" gate="B2" pin="IO_L22P_2"/>
+<wire x1="231.14" y1="40.64" x2="210.82" y2="40.64" width="0.1524" layer="91"/>
+<label x="231.14" y="40.64" size="1.778" layer="95"/>
+</segment>
+</net>
+<net name="Q5" class="0">
+<segment>
+<pinref part="U1" gate="B2" pin="IO_L23N_2VREF_2"/>
+<wire x1="231.14" y1="25.4" x2="210.82" y2="25.4" width="0.1524" layer="91"/>
+<label x="231.14" y="25.4" size="1.778" layer="95"/>
+</segment>
+</net>
+<net name="Q6" class="0">
+<segment>
+<pinref part="U1" gate="B2" pin="IO_L24N_2"/>
+<wire x1="231.14" y1="30.48" x2="210.82" y2="30.48" width="0.1524" layer="91"/>
+<label x="231.14" y="30.48" size="1.778" layer="95"/>
+</segment>
+</net>
+<net name="Q7" class="0">
+<segment>
+<pinref part="U1" gate="B2" pin="IO_L23P_2"/>
+<wire x1="231.14" y1="35.56" x2="210.82" y2="35.56" width="0.1524" layer="91"/>
+<label x="231.14" y="35.56" size="1.778" layer="95"/>
+</segment>
+</net>

Commit message: bedtime
Connections:
- removed net Q2: U1B2.IO_L22N_2
- new net W1: U1B3.IO_L23P_3VREF_3
- new net W2: U1B3.IO_L23N_3
- new net W3: U1B3.IO_L22N_3
- new net W4: U1B3.IO_L22P_3
- new net W5: U1B3.IO_L21N_3
- new net W6: U1B3.IO_L21P_3
- net EXTCLK: now also U1B2.IO_L22N_2; no longer U1B2.IO_L01P_2VRN_2
- net JOY1_DOWN: now also U1B2.IO_L20N_2; no longer U1B3.IO_L22N_3
- net JOY1_FIRE1: now also U1B2.IO_L20P_2; no longer U1B3.IO_L22P_3
- net JOY1_FIRE2: now also U1B2.IO_L01P_2VRN_2; no longer U1B3.IO_L23N_3
- net JOY1_LEFT: now also U1B2.IO_L21N_2; no longer U1B3.IO_L21N_3
- net JOY1_RIGHT: now also U1B2.IO_L21P_2; no longer U1B3.IO_L21P_3
- net JOY1_UP: now also U1B2.IO_L01N_2VRP_2; no longer U1B3.IO_L23P_3VREF_3
- net PC2: no longer U1B2.IO_L20N_2
- net PC4: no longer U1B2.IO_L01N_2VRP_2
- net PD0: no longer U1B2.IO_L20P_2
- net PD1: no longer U1B2.IO_L21N_2
- net PD2: no longer U1B2.IO_L21P_2
Changed lines of the file:
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@@
 </segment>
 <segment>
-<pinref part="U1" gate="B3" pin="IO_L22P_3"/>
-<wire x1="210.82" y1="-5.08" x2="279.4" y2="-5.08" width="0.1524" layer="91"/>
-<label x="279.4" y="-5.08" size="1.778" layer="95" rot="MR0"/>
+<pinref part="U1" gate="B2" pin="IO_L20P_2"/>
+<wire x1="231.14" y1="50.8" x2="210.82" y2="50.8" width="0.1524" layer="91"/>
+<label x="231.14" y="50.8" size="1.778" layer="95"/>
 </segment>
 </net>
@@
 </segment>
 <segment>
-<pinref part="U1" gate="B3" pin="IO_L23N_3"/>
-<wire x1="210.82" y1="-10.16" x2="279.4" y2="-10.16" width="0.1524" layer="91"/>
-<label x="279.4" y="-10.16" size="1.778" layer="95" rot="MR0"/>
+<pinref part="U1" gate="B2" pin="IO_L01P_2VRN_2"/>
+<wire x1="210.82" y1="55.88" x2="231.14" y2="55.88" width="0.1524" layer="91"/>
+<label x="231.14" y="55.88" size="1.778" layer="95"/>
 </segment>
 </net>
@@
 </segment>
 <segment>
-<pinref part="U1" gate="B3" pin="IO_L21P_3"/>
-<wire x1="210.82" y1="0" x2="279.4" y2="0" width="0.1524" layer="91"/>
-<label x="279.4" y="0" size="1.778" layer="95" rot="MR0"/>
+<pinref part="U1" gate="B2" pin="IO_L21P_2"/>
+<wire x1="231.14" y1="45.72" x2="210.82" y2="45.72" width="0.1524" layer="91"/>
+<label x="231.14" y="45.72" size="1.778" layer="95"/>
 </segment>
 </net>
@@
 </segment>
 <segment>
-<pinref part="U1" gate="B3" pin="IO_L21N_3"/>
-<wire x1="210.82" y1="-2.54" x2="279.4" y2="-2.54" width="0.1524" layer="91"/>
-<label x="279.4" y="-2.54" size="1.778" layer="95" rot="MR0"/>
+<pinref part="U1" gate="B2" pin="IO_L21N_2"/>
+<wire x1="231.14" y1="43.18" x2="210.82" y2="43.18" width="0.1524" layer="91"/>
+<label x="231.14" y="43.18" size="1.778" layer="95"/>
 </segment>
 </net>
@@
 </segment>
 <segment>
-<pinref part="U1" gate="B3" pin="IO_L22N_3"/>
-<wire x1="210.82" y1="-7.62" x2="279.4" y2="-7.62" width="0.1524" layer="91"/>
-<label x="279.4" y="-7.62" size="1.778" layer="95" rot="MR0"/>
+<pinref part="U1" gate="B2" pin="IO_L20N_2"/>
+<wire x1="231.14" y1="48.26" x2="210.82" y2="48.26" width="0.1524" layer="91"/>
+<label x="231.14" y="48.26" size="1.778" layer="95"/>
 </segment>
 </net>
@@
 </segment>
 <segment>
-<pinref part="U1" gate="B3" pin="IO_L23P_3VREF_3"/>
-<wire x1="210.82" y1="-20.32" x2="279.4" y2="-20.32" width="0.1524" layer="91"/>
-<label x="279.4" y="-20.32" size="1.778" layer="95" rot="MR0"/>
+<pinref part="U1" gate="B2" pin="IO_L01N_2VRP_2"/>
+<wire x1="231.14" y1="53.34" x2="210.82" y2="53.34" width="0.1524" layer="91"/>
+<label x="231.14" y="53.34" size="1.778" layer="95"/>
 </segment>
 </net>
@@
 <label x="454.66" y="129.54" size="1.778" layer="95"/>
 </segment>
-<segment>
-<pinref part="U1" gate="B2" pin="IO_L21P_2"/>
-<wire x1="231.14" y1="45.72" x2="210.82" y2="45.72" width="0.1524" layer="91"/>
-<label x="231.14" y="45.72" size="1.778" layer="95"/>
-</segment>
 </net>
 <net name="PD3" class="0">
@@
 </segment>
 <segment>
-<pinref part="U1" gate="B2" pin="IO_L01P_2VRN_2"/>
-<wire x1="210.82" y1="55.88" x2="231.14" y2="55.88" width="0.1524" layer="91"/>
-<label x="231.14" y="55.88" size="1.778" layer="95"/>
+<pinref part="U1" gate="B2" pin="IO_L22N_2"/>
+<wire x1="231.14" y1="38.1" x2="210.82" y2="38.1" width="0.1524" layer="91"/>
+<label x="231.14" y="38.1" size="1.778" layer="95"/>
 </segment>
 </net>
@@
 <label x="454.66" y="86.36" size="1.778" layer="95"/>
 </segment>
-<segment>
-<pinref part="U1" gate="B2" pin="IO_L20N_2"/>
-<wire x1="231.14" y1="48.26" x2="210.82" y2="48.26" width="0.1524" layer="91"/>
-<label x="231.14" y="48.26" size="1.778" layer="95"/>
-</segment>
 </net>
 <net name="PD0" class="0">
@@
 <label x="454.66" y="134.62" size="1.778" layer="95"/>
 </segment>
-<segment>
-<pinref part="U1" gate="B2" pin="IO_L20P_2"/>
-<wire x1="231.14" y1="50.8" x2="210.82" y2="50.8" width="0.1524" layer="91"/>
-<label x="231.14" y="50.8" size="1.778" layer="95"/>
-</segment>
 </net>
 <net name="PD1" class="0">
@@
 <wire x1="454.66" y1="132.08" x2="441.96" y2="132.08" width="0.1524" layer="91"/>
 <label x="454.66" y="132.08" size="1.778" layer="95"/>
-</segment>
-<segment>
-<pinref part="U1" gate="B2" pin="IO_L21N_2"/>
-<wire x1="231.14" y1="43.18" x2="210.82" y2="43.18" width="0.1524" layer="91"/>
-<label x="231.14" y="43.18" size="1.778" layer="95"/>
 </segment>
 </net>
@@
 <wire x1="441.96" y1="83.82" x2="454.66" y2="83.82" width="0.1524" layer="91"/>
 <label x="454.66" y="83.82" size="1.778" layer="95"/>
-</segment>
-<segment>
-<pinref part="U1" gate="B2" pin="IO_L01N_2VRP_2"/>
-<wire x1="231.14" y1="53.34" x2="210.82" y2="53.34" width="0.1524" layer="91"/>
-<label x="231.14" y="53.34" size="1.778" layer="95"/>
 </segment>
 </net>
@@
 </segment>
 </net>
-<net name="Q2" class="0">
-<segment>
-<pinref part="U1" gate="B2" pin="IO_L22N_2"/>
-<wire x1="231.14" y1="38.1" x2="210.82" y2="38.1" width="0.1524" layer="91"/>
-<label x="231.14" y="38.1" size="1.778" layer="95"/>
-</segment>
-</net>
 <net name="Q3" class="0">
 <segment>
@@
 </segment>
 </net>
+<net name="W1" class="0">
+<segment>
+<pinref part="U1" gate="B3" pin="IO_L23P_3VREF_3"/>
+<wire x1="210.82" y1="-20.32" x2="279.4" y2="-20.32" width="0.1524" layer="91"/>
+<label x="279.4" y="-20.32" size="1.778" layer="95" rot="MR0"/>
+</segment>
+</net>
+<net name="W2" class="0">
+<segment>
+<pinref part="U1" gate="B3" pin="IO_L23N_3"/>
+<wire x1="210.82" y1="-10.16" x2="279.4" y2="-10.16" width="0.1524" layer="91"/>
+<label x="279.4" y="-10.16" size="1.778" layer="95" rot="MR0"/>
+</segment>
+</net>
+<net name="W3" class="0">
+<segment>
+<pinref part="U1" gate="B3" pin="IO_L22N_3"/>
+<wire x1="210.82" y1="-7.62" x2="279.4" y2="-7.62" width="0.1524" layer="91"/>
+<label x="279.4" y="-7.62" size="1.778" layer="95" rot="MR0"/>
+</segment>
+</net>
+<net name="W4" class="0">
+<segment>
+<pinref part="U1" gate="B3" pin="IO_L22P_3"/>
+<wire x1="210.82" y1="-5.08" x2="279.4" y2="-5.08" width="0.1524" layer="91"/>
+<label x="279.4" y="-5.08" size="1.778" layer="95" rot="MR0"/>
+</segment>
+</net>
+<net name="W5" class="0">
+<segment>
+<pinref part="U1" gate="B3" pin="IO_L21N_3"/>
+<wire x1="210.82" y1="-2.54" x2="279.4" y2="-2.54" width="0.1524" layer="91"/>
+<label x="279.4" y="-2.54" size="1.778" layer="95" rot="MR0"/>
+</segment>
+</net>
+<net name="W6" class="0">
+<segment>
+<pinref part="U1" gate="B3" pin="IO_L21P_3"/>
+<wire x1="210.82" y1="0" x2="279.4" y2="0" width="0.1524" layer="91"/>
+<label x="279.4" y="0" size="1.778" layer="95" rot="MR0"/>
+</segment>
+</net>
