File: eagle/homeboard/homeboard22.brd (EAGLE design)
At the start: 93.5 x 71.8 mm, 133 parts, among them IC1 XCF02S, IC2 25LC080SN, IC3 ATMEGA32U2-TQFP, Q5 BC848SMD, Q6 BC848SMD, Q7 BC848SMD, Q8 BC848SMD, T1 BSS138, T2 BC848, T3 BSS138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

Commit message: mah
Parts:
- moved C32 1.80 mm to (83.0, 19.0)
- moved R23 1.50 mm to (71.0, 15.5)
- moved R55 1.41 mm to (90.8, 42.2), turned to 270 degrees
- moved R56 1.41 mm to (88.2, 42.2), flipped to the top, turned to 270 degrees
- moved SV4 1.12 mm to (90.5, 27.5)
Routing:
- net TDO_PROM: track 14.7 -> 30.5 mm, vias 1 -> 2
- net TMS: track 56.2 -> 65.7 mm
- net TCK: track 54.6 -> 63.2 mm
- net GND: track 800.1 -> 806.1 mm
- net AT_RESET: track 4.29 -> 0.00 mm
- net SPI_SEL: track 0.00 -> 4.17 mm
- net TDI_FPGA: track 46.2 -> 49.6 mm
- net SPI_MISO: track 3.25 -> 0.00 mm, vias 1 -> 0
- net SPI_MOSI: track 4.42 -> 1.95 mm, vias 1 -> 0
- net VCC: track 509.7 -> 507.3 mm, vias 24 -> 23
- net FPGA_AUDIO_LEFT: track 14.6 -> 16.1 mm
- net EMER_BOOT: track 14.6 -> 15.7 mm
- net N$38: track 20.8 -> 20.0 mm
- net FPGA_AUDIO_RIGHT: track 21.4 -> 20.7 mm
- net SPI_SCLK: track 3.60 -> 4.31 mm, vias 1 -> 0
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
Commit message: more
Parts:
- removed SJ1: (no value), jumper:SJ_2
- added JP2: (no value), adafruit:1X03
- moved R53 7.83 mm to (81.2, 50.5)
- moved R54 7.83 mm to (83.5, 50.5)
- moved C37 5.48 mm to (71.5, 50.5), flipped to the top
- moved C27 4.46 mm to (71.5, 42.3), turned to 0 degrees
- moved R56 4.03 mm to (92.2, 42.8)
- moved C38 2.30 mm to (77.0, 50.5), flipped to the top
- moved R55 1.82 mm to (89.0, 42.8)
- moved Q1 1.12 mm to (72.8, 54.2)
- moved C41 0.79 mm to (80.5, 45.8), turned to 0 degrees
Connections:
- removed net Q1: U1.P95
- removed net Q7: U1.P97
- removed net W3: U1.P83
- removed net W4: U1.P82
- removed net W5: U1.P80
- removed net W6: U1.P79
- new net Q3A: U1.P92
- net AT_RESET: now also R56.2, SV4.1; no longer R55.2, SV4.2
- net EMER_BOOT: now also R55.2, SV4.2; no longer R56.2, SV4.1
- net EXTCLK: now also JP2.3; no longer SJ1.3
- net N$14: now also JP2.1; no longer SJ1.1
- net N$8: now also JP2.2; no longer SJ1.2
- net PC2: now also U1.P98
- net PC4: now also U1.P99
- net PD0: now also U1.P97
- net PD1: now also U1.P96
- net PD2: now also U1.P95
- net PD3: now also U1.P83; no longer U1.P92
- net PD4: now also U1.P82; no longer U1.P90
- net PD5: now also U1.P80; no longer U1.P89
- net PD6: now also U1.P79; no longer U1.P87
- net Q4: now also U1.P90; no longer U1.P99
- net Q5: now also U1.P89; no longer U1.P98
- net Q6: now also U1.P87; no longer U1.P96
Routing:
- net GND: track 806.1 -> 842.8 mm
- net PD5: track 0.23 -> 26.8 mm, vias 0 -> 2
- net PD6: track 0.00 -> 25.7 mm, vias 0 -> 2
- net W6: track 24.1 -> 0.00 mm, vias 1 -> 0
- net W5: track 22.6 -> 0.00 mm, vias 1 -> 0
- net PD4: track 0.00 -> 22.1 mm, vias 0 -> 2
- net W4: track 20.2 -> 0.00 mm, vias 1 -> 0
- net VCC: track 507.3 -> 526.3 mm, vias 23 -> 22
- net PD3: track 0.00 -> 18.3 mm, vias 0 -> 2
- net N$69: track 7.15 -> 24.9 mm, vias 0 -> 1
- net W3: track 16.4 -> 0.00 mm, vias 1 -> 0
- net AT_RESET: track 0.00 -> 15.3 mm, vias 0 -> 1
- net PC4: track 7.29 -> 20.9 mm, vias 0 -> 2
- net TDO_EXP: track 3.31 -> 14.2 mm
- net TDO_PROM: track 30.5 -> 40.8 mm
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
Commit message: more
Parts:
- moved SV2 17.5 mm to (96.7, 45.5)
- moved R52 2.26 mm to (96.8, 40.2)
Connections:
- new net N_C: SV4.9
- net VCC: no longer SV4.9
Routing:
- net TMS: track 68.4 -> 86.7 mm
- net TCK: track 65.9 -> 77.6 mm
- net TDO_PROM: track 40.8 -> 44.0 mm

Commit message: bit more
Connections:
- removed net N$26: SV4.18
- removed net N$27: SV4.16
- removed net N$28: SV4.14
- removed net N_C: SV4.9
- removed net XAXAXA: SV4.12
- new net A: SV4.11
- net GND: now also SV4.9; no longer SV4.11
- net SPI_MISO: now also SV4.14
- net SPI_MOSI: now also SV4.18
- net SPI_SCLK: now also SV4.16
- net SPI_SEL: now also SV4.12
Routing:
- net GND: track 842.8 -> 874.5 mm, vias 31 -> 30
- net SPI_MOSI: track 1.95 -> 23.4 mm
- net SPI_SCLK: track 4.10 -> 23.7 mm
- net SPI_MISO: track 1.12 -> 19.0 mm
- net SPI_SEL: track 7.36 -> 22.1 mm
- net VCC: track 526.3 -> 532.7 mm
- net TDO_PROM: track 44.0 -> 45.4 mm
- net TCK: track 77.6 -> 78.6 mm
- net PD3: track 18.3 -> 17.6 mm
- net TMS: track 86.7 -> 86.2 mm
Other:
- board size 93.5 x 71.8 mm -> 94 x 71.8 mm

Commit message: bit more
Parts:
- removed JP1: (no value), pinhead:2X10
- removed R52: 4K7, resistor:M0805
- removed RESET_SW: (no value), jumper:JP1
- removed SV2: (no value), con-lstb:MA03-2
- moved C41 3.00 mm to (83.5, 45.8)
- moved C29 1.50 mm to (75.8, 26.8)
- moved IC2 1.50 mm to (78.3, 26.6)
- moved C38 0.50 mm to (76.5, 50.5)
Connections:
- removed net A: SV4.11
- removed net N$21: SV4.17
- removed net N$24: SV4.15
- removed net N$25: SV4.13
- removed net N$29: U1.P86
- removed net Q5: U1.P89
- removed net Q6: U1.P87
- removed net RESET: R52.2, RESET_SW.1
- removed net W2: U1.P85
- new net HDR_MISO: SV4.13, U1.P87
- new net HDR_MOSI: SV4.17, U1.P85
- new net HDR_SCLK: SV4.15, U1.P86
- new net HDR_SEL: SV4.11, U1.P89
- net GND: no longer JP1.1, RESET_SW.2, SV2.6
- net SPI_MISO: no longer SV2.4
- net SPI_MOSI: no longer SV2.2
- net SPI_SCLK: no longer SV2.3
- net SPI_SEL: no longer SV2.1
- net VCC: no longer JP1.2, R52.1, SV2.5
Routing:
- net HDR_MOSI: track 0.00 -> 35.8 mm
- net HDR_SCLK: track 0.00 -> 33.9 mm, vias 0 -> 1
- net HDR_MISO: track 0.00 -> 32.7 mm, vias 0 -> 1
- net HDR_SEL: track 0.00 -> 31.1 mm, vias 0 -> 1
- net W2: track 13.3 -> 0.00 mm, vias 1 -> 0
- net GND: track 874.5 -> 885.2 mm
- net W1: track 10.2 -> 0.00 mm, vias 1 -> 0
- net VCC: track 532.7 -> 527.9 mm, vias 22 -> 23
- net N$9: track 3.00 -> 5.50 mm
- net PD4: track 22.1 -> 23.7 mm
- net FL_SEL: track 21.5 -> 20.0 mm
- net FL_SCLK: track 18.4 -> 16.9 mm
- net FL_HOLD: track 16.8 -> 15.3 mm
- net FL_DI: track 19.8 -> 18.3 mm
- net FL_DO: track 16.9 -> 15.4 mm
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
Commit message: wired up, got spare pins tho
Parts:
- removed R11: 75, rcl:R0805
- removed R12: 750, rcl:R0805
- moved C30 26.3 mm to (97.8, 28.5), turned to 0 degrees
- moved C29 3.61 mm to (73.8, 29.8), flipped to the top, turned to 180 degrees
- moved C28 3.16 mm to (98.0, 32.5)
Connections:
- removed net D_FASTBLANKING: R11.1, R12.2
- removed net VCC_B3: R11.2
- removed net W1: U1.P84
- new net HDR_SPARE: SV4.9, U1.P89
- net GND: no longer R12.1, SV4.9
- net HDR_MISO: now also U1.P86; no longer U1.P87
- net HDR_MOSI: now also U1.P84; no longer U1.P85
- net HDR_SCLK: now also U1.P85; no longer U1.P86
- net HDR_SEL: now also U1.P87; no longer U1.P89
Routing:
- net HDR_SPARE: track 0.00 -> 30.5 mm, vias 0 -> 1
- net VCC: track 527.9 -> 555.1 mm, vias 23 -> 22
- net GND: track 885.2 -> 892.0 mm, vias 30 -> 31
- net HDR_MOSI: track 35.8 -> 37.1 mm
- net PD3: track 18.6 -> 19.2 mm

Commit message: wired up, got spare pins tho
Routing:
- net PC4: track 20.5 -> 19.1 mm
- net PD3: track 19.2 -> 18.5 mm
- net PD5: track 28.4 -> 27.9 mm
Changed lines of the file:
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@@
 <wire x1="83.5" y1="20.75" x2="83.5" y2="20.5440125" width="0.254" layer="1"/>
 <wire x1="83.5" y1="20.5440125" x2="83.393396875" y2="20.437409375" width="0.254" layer="1"/>
-<wire x1="76.75" y1="30.75" x2="80.75" y2="30.75" width="0.254" layer="1"/>
-<wire x1="80.75" y1="30.75" x2="81.5" y2="30" width="0.254" layer="1"/>
+<wire x1="77" y1="31" x2="80.5" y2="31" width="0.254" layer="1"/>
+<wire x1="80.5" y1="31" x2="81.5" y2="30" width="0.254" layer="1"/>
 <wire x1="81.5" y1="30" x2="81.5" y2="22" width="0.254" layer="1"/>
 <wire x1="81.5" y1="22" x2="82.5" y2="21" width="0.254" layer="1"/>
 <wire x1="82.5" y1="21" x2="83.3059875" y2="21" width="0.254" layer="1"/>
 <wire x1="83.3059875" y1="21" x2="83.393396875" y2="21.087409375" width="0.254" layer="1"/>
-<wire x1="76.75" y1="30.75" x2="76.5" y2="30.5" width="0.254" layer="1"/>
+<wire x1="77" y1="31" x2="76.5" y2="30.5" width="0.254" layer="1"/>
 <wire x1="76.5" y1="30.5" x2="76.5" y2="29" width="0.254" layer="1"/>
 <wire x1="76.375325" y1="29.18058125" x2="76.375325" y2="29.124675" width="0.254" layer="1"/>
@@
 <wire x1="59.75" y1="25.75" x2="61.25" y2="25.75" width="0.6" layer="1"/>
 <wire x1="61.25" y1="25.75" x2="64" y2="23" width="0.6" layer="1"/>
-<wire x1="64" y1="23" x2="75" y2="23" width="0.6" layer="1"/>
-<wire x1="75" y1="23" x2="76" y2="22" width="0.6" layer="1"/>
-<wire x1="76" y1="22" x2="81.5" y2="22" width="0.6" layer="1"/>
+<wire x1="64" y1="23" x2="74" y2="23" width="0.6" layer="1"/>
+<wire x1="74" y1="23" x2="75" y2="22" width="0.6" layer="1"/>
+<wire x1="75" y1="22" x2="81.5" y2="22" width="0.6" layer="1"/>
 <wire x1="81.5" y1="22" x2="83" y2="20.5" width="0.6" layer="1"/>
 <wire x1="83" y1="20.5" x2="83.5" y2="21" width="0.6" layer="1"/>
@@
 <contactref element="IC3" pad="9"/>
 <contactref element="U1" pad="P83"/>
-<wire x1="63.92" y1="30" x2="65.5" y2="30" width="0.254" layer="1"/>
-<wire x1="65.5" y1="30" x2="66" y2="29.5" width="0.254" layer="1"/>
-<wire x1="66" y1="29.5" x2="67.5" y2="29.5" width="0.254" layer="1"/>
-<wire x1="67.5" y1="29.5" x2="67.5" y2="30" width="0.254" layer="1"/>
+<wire x1="63.92" y1="30" x2="67.5" y2="30" width="0.254" layer="1"/>
 <via x="67.5" y="30" extent="1-16" drill="0.6" shape="square"/>
 <wire x1="67.5" y1="30" x2="67.5" y2="32.25" width="0.254" layer="16"/>
@@
 <wire x1="70" y1="28.5" x2="70" y2="29" width="0.254" layer="1"/>
 <via x="70" y="29" extent="1-16" drill="0.6" shape="square"/>
-<wire x1="70" y1="29" x2="69.75" y2="29" width="0.254" layer="16"/>
-<wire x1="69.75" y1="29" x2="69.75" y2="31.25" width="0.254" layer="16"/>
-<wire x1="69.75" y1="31.25" x2="76.25" y2="31.25" width="0.254" layer="16"/>
+<wire x1="70" y1="29" x2="70" y2="31.25" width="0.254" layer="16"/>
+<wire x1="70" y1="31.25" x2="76.25" y2="31.25" width="0.254" layer="16"/>
 <wire x1="76.25" y1="31.25" x2="76.25" y2="38.25" width="0.254" layer="16"/>
 <wire x1="76.25" y1="38.25" x2="75.5" y2="38.75" width="0.254" layer="16"/>
@@
 <wire x1="63.92" y1="38" x2="68" y2="38" width="0.254" layer="1"/>
 <wire x1="68" y1="38" x2="69" y2="39" width="0.254" layer="1"/>
-<wire x1="69" y1="39" x2="69" y2="40.5" width="0.254" layer="1"/>
-<via x="69" y="40.5" extent="1-16" drill="0.6" shape="square"/>
-<wire x1="69" y1="40.5" x2="70" y2="40.5" width="0.254" layer="16"/>
-<wire x1="70" y1="40.5" x2="71" y2="39.5" width="0.254" layer="16"/>
+<wire x1="69" y1="39" x2="69" y2="39.5" width="0.254" layer="1"/>
+<via x="69" y="39.5" extent="1-16" drill="0.6" shape="square"/>
 <wire x1="76" y1="41" x2="76" y2="41.75" width="0.254" layer="16"/>
 <wire x1="79.25" y1="41.75" x2="76" y2="41.75" width="0.254" layer="1"/>
 <wire x1="76" y1="41" x2="73.5" y2="41" width="0.254" layer="16"/>
 <wire x1="73.5" y1="41" x2="72" y2="39.5" width="0.254" layer="16"/>
-<wire x1="72" y1="39.5" x2="71" y2="39.5" width="0.254" layer="16"/>
+<wire x1="72" y1="39.5" x2="69" y2="39.5" width="0.254" layer="16"/>
 </signal>
 <signal name="PC5">
@@
 <wire x1="63.92" y1="38.5" x2="67.5" y2="38.5" width="0.254" layer="1"/>
 <wire x1="67.5" y1="38.5" x2="68" y2="39" width="0.254" layer="1"/>
-<wire x1="68" y1="39" x2="68" y2="41" width="0.254" layer="1"/>
-<wire x1="68" y1="41" x2="68.5" y2="41.5" width="0.254" layer="1"/>
-<wire x1="68.5" y1="41.5" x2="69" y2="41.5" width="0.254" layer="1"/>
-<wire x1="69" y1="41.5" x2="69.5" y2="42" width="0.254" layer="1"/>
+<wire x1="68" y1="39" x2="68" y2="40.5" width="0.254" layer="1"/>
+<wire x1="68" y1="40.5" x2="69.5" y2="42" width="0.254" layer="1"/>
 <wire x1="69.5" y1="42" x2="69.5" y2="44" width="0.254" layer="1"/>
 </signal>

Commit message: moving down
Connections:
- removed net Q3: U1.P93
- removed net Q3A: U1.P92
- removed net Q4: U1.P90
- new net A: U1.P84
- new net C: U1.P86
- new net D: U1.P85
- net HDR_MISO: now also U1.P90; no longer U1.P86
- net HDR_MOSI: now also U1.P87; no longer U1.P84
- net HDR_SCLK: now also U1.P89; no longer U1.P85
- net HDR_SEL: now also U1.P92; no longer U1.P87
- net HDR_SPARE: now also U1.P93; no longer U1.P89
Changed lines of the file:
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@@
 <signal name="HDR_MOSI">
 <contactref element="SV4" pad="17"/>
-<contactref element="U1" pad="P84"/>
-<wire x1="63.92" y1="30.5" x2="66.5" y2="30.5" width="0.254" layer="1"/>
-<wire x1="66.5" y1="30.5" x2="67" y2="31" width="0.254" layer="1"/>
-<wire x1="67" y1="31" x2="71" y2="31" width="0.254" layer="1"/>
-<wire x1="71" y1="31" x2="71.5" y2="31.5" width="0.254" layer="1"/>
-<wire x1="71.5" y1="31.5" x2="81" y2="31.5" width="0.254" layer="1"/>
+<contactref element="U1" pad="P87"/>
+<wire x1="63.92" y1="32" x2="65.5" y2="32" width="0.254" layer="1"/>
+<wire x1="65.5" y1="32" x2="66.5" y2="33" width="0.254" layer="1"/>
+<wire x1="66.5" y1="33" x2="70.5" y2="33" width="0.254" layer="1"/>
+<wire x1="70.5" y1="33" x2="72" y2="31.5" width="0.254" layer="1"/>
+<wire x1="72" y1="31.5" x2="81" y2="31.5" width="0.254" layer="1"/>
 <wire x1="81" y1="31.5" x2="82" y2="30.5" width="0.254" layer="1"/>
-<wire x1="82" y1="30.5" x2="82" y2="23" width="0.254" layer="1"/>
-<wire x1="82" y1="23" x2="82.5" y2="22.5" width="0.254" layer="1"/>
-<wire x1="82.5" y1="22.5" x2="85.5" y2="22.5" width="0.254" layer="1"/>
-<wire x1="85.5" y1="22.5" x2="86.5" y2="21.5" width="0.254" layer="1"/>
-<wire x1="86.5" y1="21.5" x2="86.5" y2="19" width="0.254" layer="1"/>
-<wire x1="86.5" y1="19" x2="87" y2="18.5" width="0.254" layer="1"/>
-<wire x1="87" y1="18.5" x2="89" y2="18.5" width="0.254" layer="1"/>
+<wire x1="82" y1="30.5" x2="82" y2="23.5" width="0.254" layer="1"/>
+<wire x1="82" y1="23.5" x2="83" y2="22.5" width="0.254" layer="1"/>
+<wire x1="83" y1="22.5" x2="86" y2="22.5" width="0.254" layer="1"/>
+<wire x1="86" y1="22.5" x2="87" y2="21.5" width="0.254" layer="1"/>
+<wire x1="87" y1="21.5" x2="87" y2="19" width="0.254" layer="1"/>
+<wire x1="87" y1="19" x2="87.5" y2="18.5" width="0.254" layer="1"/>
+<wire x1="87.5" y1="18.5" x2="89" y2="18.5" width="0.254" layer="1"/>
 <wire x1="89" y1="18.5" x2="89.25" y2="18.75" width="0.254" layer="1"/>
-<wire x1="89.25" y1="18.75" x2="89.28" y2="18.61" width="0" layer="19" extent="1-1"/>
+<wire x1="89.25" y1="18.75" x2="89.28" y2="18.61" width="0" layer="19" extent="1-16"/>
 </signal>
 <signal name="HDR_SCLK">
 <contactref element="SV4" pad="15"/>
-<wire x1="70.5" y1="31.5" x2="71" y2="32" width="0.254" layer="1"/>
-<wire x1="71" y1="32" x2="81.5" y2="32" width="0.254" layer="1"/>
 <wire x1="81.5" y1="32" x2="82.5" y2="31" width="0.254" layer="1"/>
 <wire x1="82.5" y1="31" x2="82.5" y2="24.5" width="0.254" layer="1"/>
@@
 <wire x1="86.5" y1="23.5" x2="86.93" y2="23.5" width="0.254" layer="16"/>
 <wire x1="86.93" y1="23.5" x2="89.28" y2="21.15" width="0.254" layer="16"/>
-<contactref element="U1" pad="P85"/>
-<wire x1="63.92" y1="31" x2="66" y2="31" width="0.254" layer="1"/>
-<wire x1="66" y1="31" x2="66.5" y2="31.5" width="0.254" layer="1"/>
-<wire x1="66.5" y1="31.5" x2="70.5" y2="31.5" width="0.254" layer="1"/>
+<contactref element="U1" pad="P89"/>
+<wire x1="63.92" y1="33" x2="65.5" y2="33" width="0.254" layer="1"/>
+<wire x1="65.5" y1="33" x2="66" y2="33.5" width="0.254" layer="1"/>
+<wire x1="66" y1="33.5" x2="71" y2="33.5" width="0.254" layer="1"/>
+<wire x1="71" y1="33.5" x2="72.5" y2="32" width="0.254" layer="1"/>
+<wire x1="72.5" y1="32" x2="81.5" y2="32" width="0.254" layer="1"/>
 </signal>
 <signal name="HDR_MISO">
 <contactref element="SV4" pad="13"/>
-<wire x1="70" y1="32" x2="70.5" y2="32.5" width="0.254" layer="1"/>
-<wire x1="70.5" y1="32.5" x2="82" y2="32.5" width="0.254" layer="1"/>
 <wire x1="82" y1="32.5" x2="83" y2="31.5" width="0.254" layer="1"/>
 <wire x1="83" y1="31.5" x2="83" y2="25.5" width="0.254" layer="1"/>
@@
 <wire x1="88.5" y1="24" x2="88.97" y2="24" width="0.254" layer="16"/>
 <wire x1="88.97" y1="24" x2="89.28" y2="23.69" width="0.254" layer="16"/>
-<contactref element="U1" pad="P86"/>
-<wire x1="63.92" y1="31.5" x2="65.5" y2="31.5" width="0.254" layer="1"/>
-<wire x1="65.5" y1="31.5" x2="66" y2="32" width="0.254" layer="1"/>
-<wire x1="66" y1="32" x2="70" y2="32" width="0.254" layer="1"/>
-</signal>
-<signal name="Q3">
-<contactref element="U1" pad="P93"/>
-</signal>
-<signal name="Q4">
 <contactref element="U1" pad="P90"/>
-</signal>
-<signal name="Q3A">
-<contactref element="U1" pad="P92"/>
+<wire x1="63.92" y1="33.5" x2="65" y2="33.5" width="0.254" layer="1"/>
+<wire x1="65" y1="33.5" x2="65.5" y2="34" width="0.254" layer="1"/>
+<wire x1="65.5" y1="34" x2="71.5" y2="34" width="0.254" layer="1"/>
+<wire x1="71.5" y1="34" x2="73" y2="32.5" width="0.254" layer="1"/>
+<wire x1="73" y1="32.5" x2="82" y2="32.5" width="0.254" layer="1"/>
 </signal>
 <signal name="HDR_SEL">
@@
 <wire x1="85.5" y1="26.5" x2="89.01" y2="26.5" width="0.254" layer="16"/>
 <wire x1="89.01" y1="26.5" x2="89.28" y2="26.23" width="0.254" layer="16"/>
-<contactref element="U1" pad="P87"/>
-<wire x1="63.92" y1="32" x2="65" y2="32" width="0.254" layer="1"/>
-<wire x1="65" y1="32" x2="65.5" y2="32.5" width="0.254" layer="1"/>
-<wire x1="65.5" y1="32.5" x2="69.5" y2="32.5" width="0.254" layer="1"/>
-<wire x1="69.5" y1="32.5" x2="70" y2="33" width="0.254" layer="1"/>
-<wire x1="70" y1="33" x2="82.5" y2="33" width="0.254" layer="1"/>
+<contactref element="U1" pad="P92"/>
+<wire x1="63.92" y1="34.5" x2="72" y2="34.5" width="0.254" layer="1"/>
+<wire x1="72" y1="34.5" x2="73.5" y2="33" width="0.254" layer="1"/>
+<wire x1="73.5" y1="33" x2="82.5" y2="33" width="0.254" layer="1"/>
 </signal>
 <signal name="HDR_SPARE">
 <contactref element="SV4" pad="9"/>
-<contactref element="U1" pad="P89"/>
-<wire x1="63.92" y1="33" x2="69" y2="33" width="0.254" layer="1"/>
-<wire x1="69" y1="33" x2="69.5" y2="33.5" width="0.254" layer="1"/>
-<wire x1="69.5" y1="33.5" x2="83" y2="33.5" width="0.254" layer="1"/>
+<contactref element="U1" pad="P93"/>
+<wire x1="63.92" y1="35" x2="72.5" y2="35" width="0.254" layer="1"/>
+<wire x1="72.5" y1="35" x2="74" y2="33.5" width="0.254" layer="1"/>
+<wire x1="74" y1="33.5" x2="83" y2="33.5" width="0.254" layer="1"/>
 <wire x1="83" y1="33.5" x2="84" y2="32.5" width="0.254" layer="1"/>
-<wire x1="84" y1="32.5" x2="84" y2="28.5" width="0.254" layer="1"/>
-<wire x1="84" y1="28.5" x2="84.5" y2="28" width="0.254" layer="1"/>
-<wire x1="84.5" y1="28" x2="85" y2="28" width="0.254" layer="1"/>
+<wire x1="84" y1="32.5" x2="84" y2="29" width="0.254" layer="1"/>
+<wire x1="84" y1="29" x2="85" y2="28" width="0.254" layer="1"/>
 <via x="85" y="28" extent="1-16" drill="0.6" shape="square"/>
-<wire x1="85" y1="28" x2="87.25" y2="28" width="0.254" layer="16"/>
-<wire x1="87.25" y1="28" x2="88" y2="28.75" width="0.254" layer="16"/>
-<wire x1="88" y1="28.75" x2="89.25" y2="28.75" width="0.254" layer="16"/>
-<wire x1="89.25" y1="28.75" x2="89.28" y2="28.77" width="0" layer="19" extent="16-16"/>
+<wire x1="85" y1="28" x2="88.51" y2="28" width="0.254" layer="16"/>
+<wire x1="88.51" y1="28" x2="89.28" y2="28.77" width="0.254" layer="16"/>
+</signal>
+<signal name="C">
+<contactref element="U1" pad="P86"/>
+</signal>
+<signal name="D">
+<contactref element="U1" pad="P85"/>
+</signal>
+<signal name="A">
+<contactref element="U1" pad="P84"/>
 </signal>
 </signals>
