File: eagle/homeboard/homeboard22.sch (EAGLE design)
At the start: 133 parts, among them IC1 XCF02S, IC2 25LC080SN, IC3 ATMEGA32U2-TQFP, Q5 BC848SMD, Q6 BC848SMD, Q7 BC848SMD, Q8 BC848SMD, T1 BSS138, T2 BC848, T3 BSS138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

Commit message: more
Parts:
- removed SJ1: (no value), jumper:SJ2W
- added JP2: (no value), adafruit:PINHD-1X3
Connections:
- removed net Q1: U1B2.IO_L24P_2
- removed net Q7: U1B2.IO_L23P_2
- removed net W3: U1B3.IO_L22N_3
- removed net W4: U1B3.IO_L22P_3
- removed net W5: U1B3.IO_L21N_3
- removed net W6: U1B3.IO_L21P_3
- new net Q3A: U1B2.IO_L40P_2VREF_2
- net AT_RESET: now also R56.2, SV4.1; no longer R55.2, SV4.2
- net EMER_BOOT: now also R55.2, SV4.2; no longer R56.2, SV4.1
- net EXTCLK: now also JP2.3; no longer SJ1.3
- net N$14: now also JP2.1; no longer SJ1.1
- net N$8: now also JP2.2; no longer SJ1.2
- net PC2: now also U1B2.IO_L23N_2VREF_2
- net PC4: now also U1B2.IO_L22P_2
- net PD0: now also U1B2.IO_L23P_2
- net PD1: now also U1B2.IO_L24N_2
- net PD2: now also U1B2.IO_L24P_2
- net PD3: now also U1B3.IO_L22N_3; no longer U1B2.IO_L40P_2VREF_2
- net PD4: now also U1B3.IO_L22P_3; no longer U1B3.IO_L40N_3VREF_3
- net PD5: now also U1B3.IO_L21N_3; no longer U1B3.IO_L40P_3
- net PD6: now also U1B3.IO_L21P_3; no longer U1B3.IO_L24N_3
- net Q4: now also U1B3.IO_L40N_3VREF_3; no longer U1B2.IO_L22P_2
- net Q5: now also U1B3.IO_L40P_3; no longer U1B2.IO_L23N_2VREF_2
- net Q6: now also U1B3.IO_L24N_3; no longer U1B2.IO_L24N_2
Changed lines of the file:
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@@
 <part name="U$9" library="cpcfpga" deviceset="GNDHOLE" device=""/>
 <part name="SV5" library="con-lstb" deviceset="MA05-2" device=""/>
-<part name="SJ1" library="jumper" deviceset="SJ2W" device=""/>
 <part name="SV4" library="con-lstb" deviceset="MA10-2" device=""/>
+<part name="JP2" library="adafruit" deviceset="PINHD-1X3" device=""/>
 </parts>
 <sheets>
@@
 <instance part="U$9" gate="G$1" x="-246.38" y="157.48"/>
 <instance part="SV5" gate="G$1" x="35.56" y="-124.46" rot="R180"/>
-<instance part="SJ1" gate="G$1" x="330.2" y="109.22" rot="R90"/>
 <instance part="SV4" gate="G$1" x="302.26" y="30.48" rot="R180"/>
+<instance part="JP2" gate="A" x="330.2" y="119.38" rot="R90"/>
 </instances>
 <busses>
@@
 </segment>
 <segment>
-<wire x1="281.94" y1="40.64" x2="289.56" y2="40.64" width="0.1524" layer="91"/>
-<label x="281.94" y="40.64" size="1.778" layer="95"/>
-<pinref part="R56" gate="G$1" pin="2"/>
-<wire x1="289.56" y1="40.64" x2="294.64" y2="40.64" width="0.1524" layer="91"/>
-<junction x="289.56" y="40.64"/>
-<pinref part="SV4" gate="G$1" pin="1"/>
+<wire x1="322.58" y1="40.64" x2="312.42" y2="40.64" width="0.1524" layer="91"/>
+<label x="322.58" y="40.64" size="1.778" layer="95" rot="MR0"/>
+<pinref part="R55" gate="G$1" pin="2"/>
+<wire x1="312.42" y1="40.64" x2="309.88" y2="40.64" width="0.1524" layer="91"/>
+<junction x="312.42" y="40.64"/>
+<pinref part="SV4" gate="G$1" pin="2"/>
 </segment>
 </net>
@@
 <label x="454.66" y="129.54" size="1.778" layer="95"/>
 </segment>
+<segment>
+<pinref part="U1" gate="B2" pin="IO_L24P_2"/>
+<wire x1="231.14" y1="33.02" x2="210.82" y2="33.02" width="0.1524" layer="91"/>
+<label x="231.14" y="33.02" size="1.778" layer="95"/>
+</segment>
 </net>
 <net name="PD3" class="0">
@@
 </segment>
 <segment>
-<pinref part="U1" gate="B2" pin="IO_L40P_2VREF_2"/>
-<wire x1="231.14" y1="22.86" x2="210.82" y2="22.86" width="0.1524" layer="91"/>
-<label x="231.14" y="22.86" size="1.778" layer="95"/>
+<pinref part="U1" gate="B3" pin="IO_L22N_3"/>
+<wire x1="210.82" y1="-7.62" x2="279.4" y2="-7.62" width="0.1524" layer="91"/>
+<label x="279.4" y="-7.62" size="1.778" layer="95" rot="MR0"/>
 </segment>
 </net>
@@
 <net name="EXTCLK" class="0">
 <segment>
-<wire x1="335.28" y1="109.22" x2="340.36" y2="109.22" width="0.1524" layer="91"/>
+<wire x1="332.74" y1="109.22" x2="340.36" y2="109.22" width="0.1524" layer="91"/>
 <label x="340.36" y="109.22" size="1.778" layer="95"/>
-<pinref part="SJ1" gate="G$1" pin="3"/>
+<pinref part="JP2" gate="A" pin="3"/>
+<wire x1="332.74" y1="109.22" x2="332.74" y2="116.84" width="0.1524" layer="91"/>
 </segment>
 <segment>
@@
 <wire x1="320.04" y1="109.22" x2="320.04" y2="106.68" width="0.1524" layer="91"/>
 <junction x="320.04" y="106.68"/>
-<pinref part="SJ1" gate="G$1" pin="1"/>
-<wire x1="325.12" y1="109.22" x2="320.04" y2="109.22" width="0.1524" layer="91"/>
+<wire x1="327.66" y1="109.22" x2="320.04" y2="109.22" width="0.1524" layer="91"/>
+<pinref part="JP2" gate="A" pin="1"/>
+<wire x1="327.66" y1="109.22" x2="327.66" y2="116.84" width="0.1524" layer="91"/>
 </segment>
 </net>
@@
 <label x="454.66" y="86.36" size="1.778" layer="95"/>
 </segment>
+<segment>
+<pinref part="U1" gate="B2" pin="IO_L23N_2VREF_2"/>
+<wire x1="231.14" y1="25.4" x2="210.82" y2="25.4" width="0.1524" layer="91"/>
+<label x="231.14" y="25.4" size="1.778" layer="95"/>
+</segment>
 </net>
 <net name="PD0" class="0">
@@
 <label x="454.66" y="134.62" size="1.778" layer="95"/>
 </segment>
+<segment>
+<pinref part="U1" gate="B2" pin="IO_L23P_2"/>
+<wire x1="231.14" y1="35.56" x2="210.82" y2="35.56" width="0.1524" layer="91"/>
+<label x="231.14" y="35.56" size="1.778" layer="95"/>
+</segment>
 </net>
 <net name="PD1" class="0">
@@
 <label x="454.66" y="132.08" size="1.778" layer="95"/>
 </segment>
+<segment>
+<pinref part="U1" gate="B2" pin="IO_L24N_2"/>
+<wire x1="231.14" y1="30.48" x2="210.82" y2="30.48" width="0.1524" layer="91"/>
+<label x="231.14" y="30.48" size="1.778" layer="95"/>
+</segment>
 </net>
 <net name="PD4" class="0">
@@
 </segment>
 <segment>
-<pinref part="U1" gate="B3" pin="IO_L40N_3VREF_3"/>
-<wire x1="231.14" y1="-22.86" x2="210.82" y2="-22.86" width="0.1524" layer="91"/>
-<label x="231.14" y="-22.86" size="1.778" layer="95"/>
+<pinref part="U1" gate="B3" pin="IO_L22P_3"/>
+<wire x1="210.82" y1="-5.08" x2="279.4" y2="-5.08" width="0.1524" layer="91"/>
+<label x="279.4" y="-5.08" size="1.778" layer="95" rot="MR0"/>
 </segment>
 </net>
@@
 </segment>
 <segment>
-<pinref part="U1" gate="B3" pin="IO_L40P_3"/>
-<wire x1="231.14" y1="-17.78" x2="210.82" y2="-17.78" width="0.1524" layer="91"/>
-<label x="231.14" y="-17.78" size="1.778" layer="95"/>
+<pinref part="U1" gate="B3" pin="IO_L21N_3"/>
+<wire x1="210.82" y1="-2.54" x2="279.4" y2="-2.54" width="0.1524" layer="91"/>
+<label x="279.4" y="-2.54" size="1.778" layer="95" rot="MR0"/>
 </segment>
 </net>
@@
 </segment>
 <segment>
-<pinref part="U1" gate="B3" pin="IO_L24N_3"/>
-<wire x1="231.14" y1="-15.24" x2="210.82" y2="-15.24" width="0.1524" layer="91"/>
-<label x="231.14" y="-15.24" size="1.778" layer="95"/>
+<pinref part="U1" gate="B3" pin="IO_L21P_3"/>
+<wire x1="210.82" y1="0" x2="279.4" y2="0" width="0.1524" layer="91"/>
+<label x="279.4" y="0" size="1.778" layer="95" rot="MR0"/>
 </segment>
 </net>
@@
 </segment>
 <segment>
-<wire x1="322.58" y1="40.64" x2="312.42" y2="40.64" width="0.1524" layer="91"/>
-<label x="322.58" y="40.64" size="1.778" layer="95" rot="MR0"/>
-<pinref part="R55" gate="G$1" pin="2"/>
-<wire x1="312.42" y1="40.64" x2="309.88" y2="40.64" width="0.1524" layer="91"/>
-<junction x="312.42" y="40.64"/>
-<pinref part="SV4" gate="G$1" pin="2"/>
+<wire x1="281.94" y1="40.64" x2="289.56" y2="40.64" width="0.1524" layer="91"/>
+<label x="281.94" y="40.64" size="1.778" layer="95"/>
+<pinref part="R56" gate="G$1" pin="2"/>
+<wire x1="289.56" y1="40.64" x2="294.64" y2="40.64" width="0.1524" layer="91"/>
+<junction x="289.56" y="40.64"/>
+<pinref part="SV4" gate="G$1" pin="1"/>
 </segment>
 </net>
@@
 <label x="454.66" y="83.82" size="1.778" layer="95"/>
 </segment>
+<segment>
+<pinref part="U1" gate="B2" pin="IO_L22P_2"/>
+<wire x1="231.14" y1="40.64" x2="210.82" y2="40.64" width="0.1524" layer="91"/>
+<label x="231.14" y="40.64" size="1.778" layer="95"/>
+</segment>
 </net>
 <net name="PC5" class="0">
@@
 <pinref part="IC3" gate="G$1" pin="XTAL1"/>
 <wire x1="330.2" y1="104.14" x2="383.54" y2="104.14" width="0.1524" layer="91"/>
-<pinref part="SJ1" gate="G$1" pin="2"/>
+<pinref part="JP2" gate="A" pin="2"/>
+<wire x1="330.2" y1="104.14" x2="330.2" y2="116.84" width="0.1524" layer="91"/>
 </segment>
 </net>
@@
 </segment>
 </net>
-<net name="Q1" class="0">
-<segment>
-<pinref part="U1" gate="B2" pin="IO_L24P_2"/>
-<wire x1="231.14" y1="33.02" x2="210.82" y2="33.02" width="0.1524" layer="91"/>
-<label x="231.14" y="33.02" size="1.778" layer="95"/>
-</segment>
-</net>
 <net name="Q3" class="0">
 <segment>
@@
 </segment>
 </net>
-<net name="Q4" class="0">
-<segment>
-<pinref part="U1" gate="B2" pin="IO_L22P_2"/>
-<wire x1="231.14" y1="40.64" x2="210.82" y2="40.64" width="0.1524" layer="91"/>
-<label x="231.14" y="40.64" size="1.778" layer="95"/>
-</segment>
-</net>
-<net name="Q5" class="0">
-<segment>
-<pinref part="U1" gate="B2" pin="IO_L23N_2VREF_2"/>
-<wire x1="231.14" y1="25.4" x2="210.82" y2="25.4" width="0.1524" layer="91"/>
-<label x="231.14" y="25.4" size="1.778" layer="95"/>
-</segment>
-</net>
-<net name="Q6" class="0">
-<segment>
-<pinref part="U1" gate="B2" pin="IO_L24N_2"/>
-<wire x1="231.14" y1="30.48" x2="210.82" y2="30.48" width="0.1524" layer="91"/>
-<label x="231.14" y="30.48" size="1.778" layer="95"/>
-</segment>
-</net>
-<net name="Q7" class="0">
-<segment>
-<pinref part="U1" gate="B2" pin="IO_L23P_2"/>
-<wire x1="231.14" y1="35.56" x2="210.82" y2="35.56" width="0.1524" layer="91"/>
-<label x="231.14" y="35.56" size="1.778" layer="95"/>
-</segment>
-</net>
 <net name="W1" class="0">
 <segment>
@@
 </segment>
 </net>
-<net name="W3" class="0">
+<net name="Q6" class="0">
 <segment>
-<pinref part="U1" gate="B3" pin="IO_L22N_3"/>
-<wire x1="210.82" y1="-7.62" x2="279.4" y2="-7.62" width="0.1524" layer="91"/>
-<label x="279.4" y="-7.62" size="1.778" layer="95" rot="MR0"/>
+<pinref part="U1" gate="B3" pin="IO_L24N_3"/>
+<wire x1="231.14" y1="-15.24" x2="210.82" y2="-15.24" width="0.1524" layer="91"/>
+<label x="231.14" y="-15.24" size="1.778" layer="95"/>
 </segment>
 </net>
-<net name="W4" class="0">
+<net name="Q5" class="0">
 <segment>
-<pinref part="U1" gate="B3" pin="IO_L22P_3"/>
-<wire x1="210.82" y1="-5.08" x2="279.4" y2="-5.08" width="0.1524" layer="91"/>
-<label x="279.4" y="-5.08" size="1.778" layer="95" rot="MR0"/>
+<pinref part="U1" gate="B3" pin="IO_L40P_3"/>
+<wire x1="231.14" y1="-17.78" x2="210.82" y2="-17.78" width="0.1524" layer="91"/>
+<label x="231.14" y="-17.78" size="1.778" layer="95"/>
 </segment>
 </net>
-<net name="W5" class="0">
+<net name="Q4" class="0">
 <segment>
-<pinref part="U1" gate="B3" pin="IO_L21N_3"/>
-<wire x1="210.82" y1="-2.54" x2="279.4" y2="-2.54" width="0.1524" layer="91"/>
-<label x="279.4" y="-2.54" size="1.778" layer="95" rot="MR0"/>
+<pinref part="U1" gate="B3" pin="IO_L40N_3VREF_3"/>
+<wire x1="231.14" y1="-22.86" x2="210.82" y2="-22.86" width="0.1524" layer="91"/>
+<label x="231.14" y="-22.86" size="1.778" layer="95"/>
 </segment>
 </net>
-<net name="W6" class="0">
+<net name="Q3A" class="0">
 <segment>
-<pinref part="U1" gate="B3" pin="IO_L21P_3"/>
-<wire x1="210.82" y1="0" x2="279.4" y2="0" width="0.1524" layer="91"/>
-<label x="279.4" y="0" size="1.778" layer="95" rot="MR0"/>
+<pinref part="U1" gate="B2" pin="IO_L40P_2VREF_2"/>
+<wire x1="231.14" y1="22.86" x2="210.82" y2="22.86" width="0.1524" layer="91"/>
+<label x="231.14" y="22.86" size="1.778" layer="95"/>
 </segment>
 </net>

Commit message: more
Connections:
- new net N_C: SV4.9
- net VCC: no longer SV4.9
Changed lines of the file:
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@@
-</segment>
-<segment>
-<wire x1="281.94" y1="30.48" x2="294.64" y2="30.48" width="0.1524" layer="91"/>
-<label x="281.94" y="30.48" size="1.778" layer="95"/>
-<pinref part="SV4" gate="G$1" pin="9"/>
 </segment>
 <segment>
@@
 </segment>
 </net>
+<net name="N_C" class="0">
+<segment>
+<wire x1="281.94" y1="30.48" x2="294.64" y2="30.48" width="0.1524" layer="91"/>
+<label x="281.94" y="30.48" size="1.778" layer="95"/>
+<pinref part="SV4" gate="G$1" pin="9"/>
+</segment>
+</net>

Commit message: bit more
Connections:
- removed net N$26: SV4.18
- removed net N$27: SV4.16
- removed net N$28: SV4.14
- removed net N_C: SV4.9
- removed net XAXAXA: SV4.12
- new net A: SV4.11
- net GND: now also SV4.9; no longer SV4.11
- net SPI_MISO: now also SV4.14
- net SPI_MOSI: now also SV4.18
- net SPI_SCLK: now also SV4.16
- net SPI_SEL: now also SV4.12
Changed lines of the file:
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@@
-</segment>
-<segment>
-<wire x1="281.94" y1="27.94" x2="294.64" y2="27.94" width="0.1524" layer="91"/>
-<label x="281.94" y="27.94" size="1.778" layer="95"/>
-<pinref part="SV4" gate="G$1" pin="11"/>
 </segment>
 <segment>
@@
 <label x="281.94" y="38.1" size="1.778" layer="95"/>
 <pinref part="SV4" gate="G$1" pin="3"/>
+</segment>
+<segment>
+<wire x1="281.94" y1="30.48" x2="294.64" y2="30.48" width="0.1524" layer="91"/>
+<label x="281.94" y="30.48" size="1.778" layer="95"/>
+<pinref part="SV4" gate="G$1" pin="9"/>
 </segment>
 </net>
@@
 <label x="281.94" y="68.58" size="1.778" layer="95"/>
 </segment>
+<segment>
+<wire x1="322.58" y1="22.86" x2="309.88" y2="22.86" width="0.1524" layer="91"/>
+<pinref part="SV4" gate="G$1" pin="16"/>
+<label x="322.58" y="22.86" size="1.778" layer="95" rot="MR0"/>
+</segment>
 </net>
 <net name="SPI_MOSI" class="0">
@@
 <label x="322.58" y="71.12" size="1.778" layer="95" rot="MR0"/>
 </segment>
+<segment>
+<pinref part="SV4" gate="G$1" pin="18"/>
+<wire x1="322.58" y1="20.32" x2="309.88" y2="20.32" width="0.1524" layer="91"/>
+<label x="322.58" y="20.32" size="1.778" layer="95" rot="MR0"/>
+</segment>
 </net>
 <net name="SPI_MISO" class="0">
@@
 <wire x1="322.58" y1="68.58" x2="309.88" y2="68.58" width="0.1524" layer="91"/>
 <label x="322.58" y="68.58" size="1.778" layer="95" rot="MR0"/>
+</segment>
+<segment>
+<pinref part="SV4" gate="G$1" pin="14"/>
+<wire x1="322.58" y1="25.4" x2="309.88" y2="25.4" width="0.1524" layer="91"/>
+<label x="322.58" y="25.4" size="1.778" layer="95" rot="MR0"/>
 </segment>
 </net>
@@
 <wire x1="281.94" y1="71.12" x2="294.64" y2="71.12" width="0.1524" layer="91"/>
 <label x="281.94" y="71.12" size="1.778" layer="95"/>
+</segment>
+<segment>
+<wire x1="322.58" y1="27.94" x2="309.88" y2="27.94" width="0.1524" layer="91"/>
+<label x="322.58" y="27.94" size="1.778" layer="95" rot="MR0"/>
+<pinref part="SV4" gate="G$1" pin="12"/>
 </segment>
 </net>
@@
 </segment>
 </net>
-<net name="XAXAXA" class="0">
-<segment>
-<wire x1="322.58" y1="27.94" x2="309.88" y2="27.94" width="0.1524" layer="91"/>
-<label x="322.58" y="27.94" size="1.778" layer="95" rot="MR0"/>
-<pinref part="SV4" gate="G$1" pin="12"/>
-</segment>
-</net>
 <net name="N$21" class="0">
 <segment>
@@
 </segment>
 </net>
-<net name="N$26" class="0">
-<segment>
-<pinref part="SV4" gate="G$1" pin="18"/>
-<wire x1="322.58" y1="20.32" x2="309.88" y2="20.32" width="0.1524" layer="91"/>
-<label x="322.58" y="20.32" size="1.778" layer="95" rot="MR0"/>
-</segment>
-</net>
-<net name="N$27" class="0">
-<segment>
-<wire x1="322.58" y1="22.86" x2="309.88" y2="22.86" width="0.1524" layer="91"/>
-<pinref part="SV4" gate="G$1" pin="16"/>
-<label x="322.58" y="22.86" size="1.778" layer="95" rot="MR0"/>
-</segment>
-</net>
-<net name="N$28" class="0">
-<segment>
-<pinref part="SV4" gate="G$1" pin="14"/>
-<wire x1="322.58" y1="25.4" x2="309.88" y2="25.4" width="0.1524" layer="91"/>
-<label x="322.58" y="25.4" size="1.778" layer="95" rot="MR0"/>
-</segment>
-</net>
 <net name="N$29" class="0">
 <segment>
@@
 </segment>
 </net>
-<net name="N_C" class="0">
-<segment>
-<wire x1="281.94" y1="30.48" x2="294.64" y2="30.48" width="0.1524" layer="91"/>
-<label x="281.94" y="30.48" size="1.778" layer="95"/>
-<pinref part="SV4" gate="G$1" pin="9"/>
-</segment>
-</net>
+<net name="A" class="0">
+<segment>
+<wire x1="281.94" y1="27.94" x2="294.64" y2="27.94" width="0.1524" layer="91"/>
+<label x="281.94" y="27.94" size="1.778" layer="95"/>
+<pinref part="SV4" gate="G$1" pin="11"/>
+</segment>
+</net>
