File: eagle/homeboard/homeboard22.sch (EAGLE design)
At the start: 133 parts, among them IC1 XCF02S, IC2 25LC080SN, IC3 ATMEGA32U2-TQFP, Q5 BC848SMD, Q6 BC848SMD, Q7 BC848SMD, Q8 BC848SMD, T1 BSS138, T2 BC848, T3 BSS138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

Commit message: bit more
Parts:
- removed JP1: (no value), pinhead:PINHD-2X10
- removed R52: 4K7, resistor:R-EU_M0805
- removed RESET_SW: (no value), jumper:JP1Q
- removed SV2: (no value), con-lstb:MA03-2
Connections:
- removed net A: SV4.11
- removed net N$21: SV4.17
- removed net N$24: SV4.15
- removed net N$25: SV4.13
- removed net N$29: U1B3.IO_L24P_3
- removed net Q5: U1B3.IO_L40P_3
- removed net Q6: U1B3.IO_L24N_3
- removed net RESET: R52.2, RESET_SW.1
- removed net W2: U1B3.IO_L23N_3
- new net HDR_MISO: SV4.13, U1B3.IO_L24N_3
- new net HDR_MOSI: SV4.17, U1B3.IO_L23N_3
- new net HDR_SCLK: SV4.15, U1B3.IO_L24P_3
- new net HDR_SEL: SV4.11, U1B3.IO_L40P_3
- net GND: no longer JP1.1, RESET_SW.2, SV2.6
- net SPI_MISO: no longer SV2.4
- net SPI_MOSI: no longer SV2.2
- net SPI_SCLK: no longer SV2.3
- net SPI_SEL: no longer SV2.1
- net VCC: no longer JP1.2, R52.1, SV2.5
Changed lines of the file:
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@@
 <part name="SUPPLY7" library="supply2" deviceset="GND" device=""/>
 <part name="R50" library="resistor" deviceset="R-EU_" device="M0805" value="2k2"/>
-<part name="RESET_SW" library="jumper" deviceset="JP1Q" device=""/>
-<part name="R52" library="resistor" deviceset="R-EU_" device="M0805" value="4K7"/>
 <part name="IC3" library="adafruit" deviceset="ATMEGA32U2" device="-TQFP"/>
 <part name="U$4" library="cpcfpga" deviceset="NX1117" device="" value="3.3V"/>
@@
 <part name="U$6" library="cpcfpga" deviceset="AS6C4008" device=""/>
 <part name="C34" library="rcl" deviceset="C-EU" device="C0603" value="100nF"/>
-<part name="JP1" library="pinhead" deviceset="PINHD-2X10" device=""/>
-<part name="SUPPLY16" library="supply2" deviceset="GND" device=""/>
 <part name="SUPPLY17" library="supply2" deviceset="GND" device=""/>
 <part name="X7" library="powersupply" deviceset="DC21MM" device="X"/>
@@
 <part name="SUPPLY22" library="supply2" deviceset="GND" device=""/>
 <part name="R55" library="rcl" deviceset="R-EU_" device="R0805" value="4700"/>
-<part name="SV2" library="con-lstb" deviceset="MA03-2" device=""/>
 <part name="R56" library="rcl" deviceset="R-EU_" device="R0805" value="4700"/>
 <part name="U$3" library="cpcfpga" deviceset="SDMMC" device="NOHOLE"/>
@@
 <instance part="SUPPLY7" gate="GND" x="132.08" y="147.32"/>
 <instance part="R50" gate="G$1" x="210.82" y="276.86" rot="MR0"/>
-<instance part="RESET_SW" gate="A" x="238.76" y="-121.92" rot="R90"/>
-<instance part="R52" gate="G$1" x="238.76" y="-129.54"/>
 <instance part="IC3" gate="G$1" x="406.4" y="106.68"/>
 <instance part="U$4" gate="G$1" x="-195.58" y="111.76"/>
@@
 <instance part="U$6" gate="G$1" x="45.72" y="20.32" rot="MR270"/>
 <instance part="C34" gate="G$1" x="-93.98" y="127"/>
-<instance part="JP1" gate="A" x="-5.08" y="-96.52" rot="R90"/>
-<instance part="SUPPLY16" gate="GND" x="-15.24" y="-114.3"/>
 <instance part="SUPPLY17" gate="GND" x="22.86" y="-68.58" rot="R270"/>
 <instance part="X7" gate="G$1" x="-309.88" y="88.9"/>
@@
 <instance part="SUPPLY22" gate="GND" x="373.38" y="109.22"/>
 <instance part="R55" gate="G$1" x="312.42" y="45.72" rot="MR270"/>
-<instance part="SV2" gate="1" x="302.26" y="68.58" rot="R180"/>
 <instance part="R56" gate="G$1" x="289.56" y="45.72" rot="MR270"/>
 <instance part="U$3" gate="G$1" x="541.02" y="40.64"/>
@@
 </segment>
 <segment>
-<pinref part="RESET_SW" gate="A" pin="2"/>
-<wire x1="231.14" y1="-121.92" x2="223.52" y2="-121.92" width="0.1524" layer="91"/>
-<label x="223.52" y="-121.92" size="1.778" layer="95"/>
-</segment>
-<segment>
 <pinref part="SUPPLY9" gate="GND" pin="GND"/>
 <wire x1="-157.48" y1="101.6" x2="-157.48" y2="104.14" width="0.1524" layer="91"/>
@@
 </segment>
 <segment>
-<pinref part="SUPPLY16" gate="GND" pin="GND"/>
-<pinref part="JP1" gate="A" pin="1"/>
-<wire x1="-15.24" y1="-111.76" x2="-15.24" y2="-99.06" width="0.1524" layer="91"/>
-</segment>
-<segment>
 <wire x1="35.56" y1="-66.04" x2="35.56" y2="-68.58" width="0.1524" layer="91"/>
 <pinref part="SUPPLY17" gate="GND" pin="GND"/>
@@
 </segment>
 <segment>
-<pinref part="SV2" gate="1" pin="6"/>
-<wire x1="322.58" y1="66.04" x2="309.88" y2="66.04" width="0.1524" layer="91"/>
-<label x="322.58" y="66.04" size="1.778" layer="95" rot="MR0"/>
-</segment>
-<segment>
 <pinref part="U$3" gate="G$1" pin="VSS2"/>
 <wire x1="528.32" y1="27.94" x2="520.7" y2="27.94" width="0.1524" layer="91"/>
@@
 </segment>
 <segment>
-<pinref part="R52" gate="G$1" pin="1"/>
-<wire x1="223.52" y1="-129.54" x2="233.68" y2="-129.54" width="0.1524" layer="91"/>
-<label x="223.52" y="-129.54" size="1.778" layer="95"/>
-</segment>
-<segment>
 <pinref part="C26" gate="G$1" pin="1"/>
 <pinref part="C27" gate="G$1" pin="1"/>
@@
 </segment>
 <segment>
-<pinref part="JP1" gate="A" pin="2"/>
-<wire x1="-15.24" y1="-91.44" x2="-15.24" y2="-83.82" width="0.1524" layer="91"/>
-<wire x1="-15.24" y1="-83.82" x2="-27.94" y2="-83.82" width="0.1524" layer="91"/>
-<label x="-27.94" y="-83.82" size="1.778" layer="95"/>
-</segment>
-<segment>
 <label x="33.02" y="-76.2" size="1.778" layer="95" rot="R270"/>
 <wire x1="33.02" y1="-76.2" x2="33.02" y2="-66.04" width="0.1524" layer="91"/>
@@
 </segment>
 <segment>
-<pinref part="SV2" gate="1" pin="5"/>
-<wire x1="281.94" y1="66.04" x2="294.64" y2="66.04" width="0.1524" layer="91"/>
-<label x="281.94" y="66.04" size="1.778" layer="95"/>
-</segment>
-<segment>
 <pinref part="U$3" gate="G$1" pin="VDD"/>
 <wire x1="510.54" y1="33.02" x2="528.32" y2="33.02" width="0.1524" layer="91"/>
@@
 </segment>
 <segment>
-<pinref part="SV2" gate="1" pin="3"/>
-<wire x1="281.94" y1="68.58" x2="294.64" y2="68.58" width="0.1524" layer="91"/>
-<label x="281.94" y="68.58" size="1.778" layer="95"/>
-</segment>
-<segment>
 <wire x1="322.58" y1="22.86" x2="309.88" y2="22.86" width="0.1524" layer="91"/>
 <pinref part="SV4" gate="G$1" pin="16"/>
@@
 </segment>
 <segment>
-<pinref part="SV2" gate="1" pin="2"/>
-<wire x1="322.58" y1="71.12" x2="309.88" y2="71.12" width="0.1524" layer="91"/>
-<label x="322.58" y="71.12" size="1.778" layer="95" rot="MR0"/>
-</segment>
-<segment>
 <pinref part="SV4" gate="G$1" pin="18"/>
 <wire x1="322.58" y1="20.32" x2="309.88" y2="20.32" width="0.1524" layer="91"/>
@@
 </segment>
 <segment>
-<pinref part="SV2" gate="1" pin="4"/>
-<wire x1="322.58" y1="68.58" x2="309.88" y2="68.58" width="0.1524" layer="91"/>
-<label x="322.58" y="68.58" size="1.778" layer="95" rot="MR0"/>
-</segment>
-<segment>
 <pinref part="SV4" gate="G$1" pin="14"/>
 <wire x1="322.58" y1="25.4" x2="309.88" y2="25.4" width="0.1524" layer="91"/>
@@
 <net name="RESET" class="0">
 <segment>
-<pinref part="RESET_SW" gate="A" pin="1"/>
-<pinref part="R52" gate="G$1" pin="2"/>
-<wire x1="243.84" y1="-129.54" x2="246.38" y2="-129.54" width="0.1524" layer="91"/>
-<wire x1="246.38" y1="-129.54" x2="246.38" y2="-121.92" width="0.1524" layer="91"/>
-<junction x="246.38" y="-121.92"/>
-<wire x1="246.38" y1="-121.92" x2="264.16" y2="-121.92" width="0.1524" layer="91"/>
-<label x="251.46" y="-121.92" size="1.778" layer="95"/>
-</segment>
-<segment>
 <wire x1="76.2" y1="-121.92" x2="137.16" y2="-121.92" width="0.1524" layer="91"/>
 <label x="76.2" y="-121.92" size="1.778" layer="95"/>
@@
 </segment>
 <segment>
-<pinref part="SV2" gate="1" pin="1"/>
-<wire x1="281.94" y1="71.12" x2="294.64" y2="71.12" width="0.1524" layer="91"/>
-<label x="281.94" y="71.12" size="1.778" layer="95"/>
-</segment>
-<segment>
 <wire x1="322.58" y1="27.94" x2="309.88" y2="27.94" width="0.1524" layer="91"/>
 <label x="322.58" y="27.94" size="1.778" layer="95" rot="MR0"/>
@@
 </segment>
 </net>
-<net name="N$21" class="0">
+<net name="HDR_MOSI" class="0">
 <segment>
 <pinref part="SV4" gate="G$1" pin="17"/>
@@
 <label x="281.94" y="20.32" size="1.778" layer="95"/>
 </segment>
+<segment>
+<pinref part="U1" gate="B3" pin="IO_L23N_3"/>
+<wire x1="210.82" y1="-10.16" x2="279.4" y2="-10.16" width="0.1524" layer="91"/>
+<label x="279.4" y="-10.16" size="1.778" layer="95" rot="MR0"/>
+</segment>
 </net>
-<net name="N$24" class="0">
+<net name="HDR_SCLK" class="0">
 <segment>
 <pinref part="SV4" gate="G$1" pin="15"/>
@@
 <label x="281.94" y="22.86" size="1.778" layer="95"/>
 </segment>
+<segment>
+<pinref part="U1" gate="B3" pin="IO_L24P_3"/>
+<wire x1="210.82" y1="-12.7" x2="279.4" y2="-12.7" width="0.1524" layer="91"/>
+<label x="279.4" y="-12.7" size="1.778" layer="95" rot="MR0"/>
+</segment>
 </net>
-<net name="N$25" class="0">
+<net name="HDR_MISO" class="0">
 <segment>
 <pinref part="SV4" gate="G$1" pin="13"/>
@@
 <label x="281.94" y="25.4" size="1.778" layer="95"/>
 </segment>
-</net>
-<net name="N$29" class="0">
 <segment>
-<pinref part="U1" gate="B3" pin="IO_L24P_3"/>
-<wire x1="210.82" y1="-12.7" x2="279.4" y2="-12.7" width="0.1524" layer="91"/>
-<label x="279.4" y="-12.7" size="1.778" layer="95" rot="MR0"/>
+<pinref part="U1" gate="B3" pin="IO_L24N_3"/>
+<wire x1="279.4" y1="-15.24" x2="210.82" y2="-15.24" width="0.1524" layer="91"/>
+<label x="279.4" y="-15.24" size="1.778" layer="95" rot="MR0"/>
 </segment>
 </net>
@@
 </segment>
 </net>
-<net name="W2" class="0">
-<segment>
-<pinref part="U1" gate="B3" pin="IO_L23N_3"/>
-<wire x1="210.82" y1="-10.16" x2="279.4" y2="-10.16" width="0.1524" layer="91"/>
-<label x="279.4" y="-10.16" size="1.778" layer="95" rot="MR0"/>
-</segment>
-</net>
-<net name="Q6" class="0">
-<segment>
-<pinref part="U1" gate="B3" pin="IO_L24N_3"/>
-<wire x1="231.14" y1="-15.24" x2="210.82" y2="-15.24" width="0.1524" layer="91"/>
-<label x="231.14" y="-15.24" size="1.778" layer="95"/>
-</segment>
-</net>
-<net name="Q5" class="0">
-<segment>
-<pinref part="U1" gate="B3" pin="IO_L40P_3"/>
-<wire x1="231.14" y1="-17.78" x2="210.82" y2="-17.78" width="0.1524" layer="91"/>
-<label x="231.14" y="-17.78" size="1.778" layer="95"/>
-</segment>
-</net>
 <net name="Q4" class="0">
 <segment>
@@
 </segment>
 </net>
-<net name="A" class="0">
+<net name="HDR_SEL" class="0">
 <segment>
 <wire x1="281.94" y1="27.94" x2="294.64" y2="27.94" width="0.1524" layer="91"/>
@@
 <pinref part="SV4" gate="G$1" pin="11"/>
 </segment>
+<segment>
+<pinref part="U1" gate="B3" pin="IO_L40P_3"/>
+<wire x1="279.4" y1="-17.78" x2="210.82" y2="-17.78" width="0.1524" layer="91"/>
+<label x="279.4" y="-17.78" size="1.778" layer="95" rot="MR0"/>
+</segment>
 </net>

Commit message: wired up, got spare pins tho
Parts:
- removed R11: 75, rcl:R-EU_R0805
- removed R12: 750, rcl:R-EU_R0805
Connections:
- removed net D_FASTBLANKING: R11.1, R12.2
- removed net VCC_B3: R11.2
- removed net W1: U1B3.IO_L23P_3VREF_3
- new net HDR_SPARE: SV4.9, U1B3.IO_L40P_3
- net GND: no longer R12.1, SV4.9
- net HDR_MISO: now also U1B3.IO_L24P_3; no longer U1B3.IO_L24N_3
- net HDR_MOSI: now also U1B3.IO_L23P_3VREF_3; no longer U1B3.IO_L23N_3
- net HDR_SCLK: now also U1B3.IO_L23N_3; no longer U1B3.IO_L24P_3
- net HDR_SEL: now also U1B3.IO_L24N_3; no longer U1B3.IO_L40P_3
Other:
- moved on the sheet: R50
Changed lines of the file:
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@@
 <part name="R32" library="rcl" deviceset="R-EU_" device="R0805" value="680"/>
 <part name="R33" library="rcl" deviceset="R-EU_" device="R0805" value="4700"/>
-<part name="R11" library="rcl" deviceset="R-EU_" device="R0805" value="75"/>
-<part name="R12" library="rcl" deviceset="R-EU_" device="R0805" value="750"/>
 <part name="R17" library="rcl" deviceset="R-EU_" device="R0805" value="10000"/>
 <part name="R18" library="rcl" deviceset="R-EU_" device="R0805" value="4700"/>
@@
 <instance part="R32" gate="G$1" x="127" y="193.04" rot="R90"/>
 <instance part="R33" gate="G$1" x="134.62" y="193.04" rot="R90"/>
-<instance part="R11" gate="G$1" x="137.16" y="307.34"/>
-<instance part="R12" gate="G$1" x="124.46" y="307.34"/>
 <instance part="R17" gate="G$1" x="487.68" y="-60.96" rot="R90"/>
 <instance part="R18" gate="G$1" x="500.38" y="-40.64" rot="R90"/>
@@
 <instance part="SUPPLY6" gate="GND" x="132.08" y="167.64"/>
 <instance part="SUPPLY7" gate="GND" x="132.08" y="147.32"/>
-<instance part="R50" gate="G$1" x="210.82" y="276.86" rot="MR0"/>
+<instance part="R50" gate="G$1" x="124.46" y="304.8" rot="R180"/>
 <instance part="IC3" gate="G$1" x="406.4" y="106.68"/>
 <instance part="U$4" gate="G$1" x="-195.58" y="111.76"/>
@@
 </segment>
 <segment>
-<pinref part="R12" gate="G$1" pin="1"/>
-<wire x1="119.38" y1="307.34" x2="114.3" y2="307.34" width="0.1524" layer="91"/>
-<label x="111.76" y="307.34" size="1.778" layer="95"/>
-</segment>
-<segment>
 <pinref part="R21" gate="G$1" pin="1"/>
 <pinref part="R19" gate="G$1" pin="1"/>
@@
 <pinref part="SV4" gate="G$1" pin="3"/>
 </segment>
-<segment>
-<wire x1="281.94" y1="30.48" x2="294.64" y2="30.48" width="0.1524" layer="91"/>
-<label x="281.94" y="30.48" size="1.778" layer="95"/>
-<pinref part="SV4" gate="G$1" pin="9"/>
-</segment>
 </net>
 <net name="VCC" class="0">
@@
 </segment>
 <segment>
-<wire x1="198.12" y1="256.54" x2="193.04" y2="256.54" width="0.1524" layer="91"/>
-<label x="193.04" y="256.54" size="1.778" layer="95"/>
-</segment>
-<segment>
 <pinref part="C26" gate="G$1" pin="1"/>
 <pinref part="C27" gate="G$1" pin="1"/>
@@
 <segment>
 <pinref part="R50" gate="G$1" pin="2"/>
-<wire x1="205.74" y1="276.86" x2="193.04" y2="276.86" width="0.1524" layer="91"/>
-<label x="203.2" y="276.86" size="1.778" layer="95" rot="MR0"/>
+<wire x1="119.38" y1="304.8" x2="106.68" y2="304.8" width="0.1524" layer="91"/>
+<label x="116.84" y="304.8" size="1.778" layer="95" rot="R180"/>
 </segment>
 <segment>
@@
 </segment>
 </net>
-<net name="D_FASTBLANKING" class="0">
-<segment>
-<pinref part="R12" gate="G$1" pin="2"/>
-<pinref part="R11" gate="G$1" pin="1"/>
-<wire x1="129.54" y1="307.34" x2="132.08" y2="307.34" width="0.1524" layer="91"/>
-<wire x1="129.54" y1="307.34" x2="132.08" y2="309.88" width="0.1524" layer="91"/>
-<wire x1="132.08" y1="309.88" x2="132.08" y2="312.42" width="0.1524" layer="91"/>
-<junction x="129.54" y="307.34"/>
-<label x="132.08" y="312.42" size="1.778" layer="95"/>
-</segment>
-</net>
 <net name="AINLEFT" class="0">
 <segment>
@@
 <pinref part="X1" gate="G$1" pin="8"/>
 </segment>
-<segment>
-<wire x1="251.46" y1="266.7" x2="215.9" y2="266.7" width="0.1524" layer="91"/>
-<label x="251.46" y="266.7" size="1.778" layer="95" rot="MR0"/>
-</segment>
 </net>
 <net name="SCART_GREEN" class="0">
@@
 <wire x1="241.3" y1="187.96" x2="241.3" y2="182.88" width="0.1524" layer="91"/>
 <wire x1="241.3" y1="182.88" x2="266.7" y2="182.88" width="0.1524" layer="91"/>
-<wire x1="251.46" y1="276.86" x2="215.9" y2="276.86" width="0.1524" layer="91"/>
-<label x="251.46" y="276.86" size="1.778" layer="95" rot="MR0"/>
+<wire x1="165.1" y1="304.8" x2="129.54" y2="304.8" width="0.1524" layer="91"/>
+<label x="165.1" y="304.8" size="1.778" layer="95" rot="R180"/>
 <pinref part="R50" gate="G$1" pin="1"/>
 <pinref part="X1" gate="G$1" pin="16"/>
@@
 </segment>
 </net>
-<net name="VCC_B3" class="0">
-<segment>
-<pinref part="R11" gate="G$1" pin="2"/>
-<wire x1="147.32" y1="307.34" x2="142.24" y2="307.34" width="0.1524" layer="91"/>
-<label x="144.78" y="307.34" size="1.778" layer="95"/>
-</segment>
-</net>
 <net name="R1" class="0">
 <segment>
@@
 </segment>
 <segment>
-<wire x1="190.5" y1="134.62" x2="233.68" y2="134.62" width="0.1524" layer="91"/>
-<label x="190.5" y="134.62" size="1.778" layer="95"/>
-</segment>
-<segment>
 <wire x1="76.2" y1="-66.04" x2="139.7" y2="-66.04" width="0.1524" layer="91"/>
 <wire x1="139.7" y1="-66.04" x2="139.7" y2="-40.64" width="0.1524" layer="91"/>
@@
 </segment>
 <segment>
-<wire x1="231.14" y1="137.16" x2="190.5" y2="137.16" width="0.1524" layer="91"/>
-<label x="190.5" y="137.16" size="1.778" layer="95"/>
-</segment>
-<segment>
 <pinref part="U1" gate="B5" pin="IOVREF_5"/>
 <wire x1="73.66" y1="-63.5" x2="127" y2="-63.5" width="0.1524" layer="91"/>
@@
 </segment>
 <segment>
-<pinref part="U1" gate="B3" pin="IO_L23N_3"/>
-<wire x1="210.82" y1="-10.16" x2="279.4" y2="-10.16" width="0.1524" layer="91"/>
-<label x="279.4" y="-10.16" size="1.778" layer="95" rot="MR0"/>
+<pinref part="U1" gate="B3" pin="IO_L23P_3VREF_3"/>
+<wire x1="210.82" y1="-20.32" x2="279.4" y2="-20.32" width="0.1524" layer="91"/>
+<label x="279.4" y="-20.32" size="1.778" layer="95" rot="MR0"/>
 </segment>
 </net>
@@
 </segment>
 <segment>
-<pinref part="U1" gate="B3" pin="IO_L24P_3"/>
-<wire x1="210.82" y1="-12.7" x2="279.4" y2="-12.7" width="0.1524" layer="91"/>
-<label x="279.4" y="-12.7" size="1.778" layer="95" rot="MR0"/>
+<pinref part="U1" gate="B3" pin="IO_L23N_3"/>
+<wire x1="210.82" y1="-10.16" x2="279.4" y2="-10.16" width="0.1524" layer="91"/>
+<label x="279.4" y="-10.16" size="1.778" layer="95" rot="MR0"/>
 </segment>
 </net>
@@
 </segment>
 <segment>
-<pinref part="U1" gate="B3" pin="IO_L24N_3"/>
-<wire x1="279.4" y1="-15.24" x2="210.82" y2="-15.24" width="0.1524" layer="91"/>
-<label x="279.4" y="-15.24" size="1.778" layer="95" rot="MR0"/>
+<pinref part="U1" gate="B3" pin="IO_L24P_3"/>
+<wire x1="210.82" y1="-12.7" x2="279.4" y2="-12.7" width="0.1524" layer="91"/>
+<label x="279.4" y="-12.7" size="1.778" layer="95" rot="MR0"/>
 </segment>
 </net>
@@
 </segment>
 </net>
-<net name="W1" class="0">
-<segment>
-<pinref part="U1" gate="B3" pin="IO_L23P_3VREF_3"/>
-<wire x1="210.82" y1="-20.32" x2="279.4" y2="-20.32" width="0.1524" layer="91"/>
-<label x="279.4" y="-20.32" size="1.778" layer="95" rot="MR0"/>
-</segment>
-</net>
 <net name="Q4" class="0">
 <segment>
@@
 </segment>
 <segment>
+<pinref part="U1" gate="B3" pin="IO_L24N_3"/>
+<wire x1="279.4" y1="-15.24" x2="210.82" y2="-15.24" width="0.1524" layer="91"/>
+<label x="279.4" y="-15.24" size="1.778" layer="95" rot="MR0"/>
+</segment>
+</net>
+<net name="HDR_SPARE" class="0">
+<segment>
+<wire x1="281.94" y1="30.48" x2="294.64" y2="30.48" width="0.1524" layer="91"/>
+<label x="281.94" y="30.48" size="1.778" layer="95"/>
+<pinref part="SV4" gate="G$1" pin="9"/>
+</segment>
+<segment>
