File: eagle/homeboard/homeboard22.sch (EAGLE design)
At the start: 127 parts, among them IC1 XCF02S, IC2 25LC080SN, IC3 ATMEGA32U2-TQFP, Q5 BC848SMD, Q6 BC848SMD, Q7 BC848SMD, Q8 BC848SMD, T1 BSS138, T2 BC848, T3 BSS138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

Commit message: moving down
Connections:
- removed net Q3: U1B2.IO_L40N_2
- removed net Q3A: U1B2.IO_L40P_2VREF_2
- removed net Q4: U1B3.IO_L40N_3VREF_3
- new net A: U1B3.IO_L23P_3VREF_3
- new net C: U1B3.IO_L24P_3
- new net D: U1B3.IO_L23N_3
- net HDR_MISO: now also U1B3.IO_L40N_3VREF_3; no longer U1B3.IO_L24P_3
- net HDR_MOSI: now also U1B3.IO_L24N_3; no longer U1B3.IO_L23P_3VREF_3
- net HDR_SCLK: now also U1B3.IO_L40P_3; no longer U1B3.IO_L23N_3
- net HDR_SEL: now also U1B2.IO_L40P_2VREF_2; no longer U1B3.IO_L24N_3
- net HDR_SPARE: now also U1B2.IO_L40N_2; no longer U1B3.IO_L40P_3
Changed lines of the file:
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@@
 <segment>
 <pinref part="U1" gate="B3" pin="IO_L20N_3"/>
-<wire x1="210.82" y1="2.54" x2="248.92" y2="2.54" width="0.1524" layer="91"/>
-<wire x1="248.92" y1="2.54" x2="248.92" y2="-58.42" width="0.1524" layer="91"/>
-<label x="248.92" y="-58.42" size="1.778" layer="95" rot="R90"/>
+<wire x1="210.82" y1="2.54" x2="231.14" y2="2.54" width="0.1524" layer="91"/>
+<label x="231.14" y="2.54" size="1.778" layer="95"/>
 </segment>
 </net>
@@
 <segment>
 <pinref part="U1" gate="B3" pin="IO_L20P_3"/>
-<wire x1="210.82" y1="5.08" x2="246.38" y2="5.08" width="0.1524" layer="91"/>
-<wire x1="246.38" y1="5.08" x2="246.38" y2="-58.42" width="0.1524" layer="91"/>
-<label x="246.38" y="-58.42" size="1.778" layer="95" rot="R90"/>
+<wire x1="210.82" y1="5.08" x2="231.14" y2="5.08" width="0.1524" layer="91"/>
+<label x="231.14" y="5.08" size="1.778" layer="95"/>
 </segment>
 </net>
@@
 </segment>
 <segment>
-<wire x1="243.84" y1="-58.42" x2="243.84" y2="12.7" width="0.1524" layer="91"/>
+<wire x1="231.14" y1="12.7" x2="210.82" y2="12.7" width="0.1524" layer="91"/>
 <pinref part="U1" gate="B3" pin="IO"/>
-<wire x1="243.84" y1="12.7" x2="210.82" y2="12.7" width="0.1524" layer="91"/>
-<label x="243.84" y="-58.42" size="1.778" layer="95" rot="R90"/>
+<label x="231.14" y="12.7" size="1.778" layer="95"/>
 </segment>
 </net>
@@
 </segment>
 <segment>
-<wire x1="238.76" y1="-58.42" x2="238.76" y2="10.16" width="0.1524" layer="91"/>
+<wire x1="231.14" y1="10.16" x2="210.82" y2="10.16" width="0.1524" layer="91"/>
 <pinref part="U1" gate="B3" pin="IO_L01P_3VRN_3"/>
-<wire x1="238.76" y1="10.16" x2="210.82" y2="10.16" width="0.1524" layer="91"/>
-<label x="238.76" y="-58.42" size="1.778" layer="95" rot="R90"/>
+<label x="231.14" y="10.16" size="1.778" layer="95"/>
 </segment>
 </net>
@@
 <segment>
 <pinref part="U1" gate="B3" pin="IO_L01N_3VRP_3"/>
-<wire x1="210.82" y1="7.62" x2="241.3" y2="7.62" width="0.1524" layer="91"/>
-<wire x1="241.3" y1="7.62" x2="241.3" y2="-58.42" width="0.1524" layer="91"/>
-<label x="241.3" y="-58.42" size="1.778" layer="95" rot="R90"/>
+<wire x1="210.82" y1="7.62" x2="231.14" y2="7.62" width="0.1524" layer="91"/>
+<label x="231.14" y="7.62" size="1.778" layer="95"/>
 </segment>
 </net>
@@
 <segment>
 <pinref part="U1" gate="B3" pin="IO_L22N_3"/>
-<wire x1="210.82" y1="-7.62" x2="279.4" y2="-7.62" width="0.1524" layer="91"/>
-<label x="279.4" y="-7.62" size="1.778" layer="95" rot="MR0"/>
+<wire x1="210.82" y1="-7.62" x2="231.14" y2="-7.62" width="0.1524" layer="91"/>
+<label x="231.14" y="-7.62" size="1.778" layer="95"/>
 </segment>
 </net>
@@
 <segment>
 <pinref part="U1" gate="B3" pin="IO_L22P_3"/>
-<wire x1="210.82" y1="-5.08" x2="279.4" y2="-5.08" width="0.1524" layer="91"/>
-<label x="279.4" y="-5.08" size="1.778" layer="95" rot="MR0"/>
+<wire x1="210.82" y1="-5.08" x2="231.14" y2="-5.08" width="0.1524" layer="91"/>
+<label x="231.14" y="-5.08" size="1.778" layer="95"/>
 </segment>
 </net>
@@
 <segment>
 <pinref part="U1" gate="B3" pin="IO_L21N_3"/>
-<wire x1="210.82" y1="-2.54" x2="279.4" y2="-2.54" width="0.1524" layer="91"/>
-<label x="279.4" y="-2.54" size="1.778" layer="95" rot="MR0"/>
+<wire x1="210.82" y1="-2.54" x2="231.14" y2="-2.54" width="0.1524" layer="91"/>
+<label x="231.14" y="-2.54" size="1.778" layer="95"/>
 </segment>
 </net>
@@
 <segment>
 <pinref part="U1" gate="B3" pin="IO_L21P_3"/>
-<wire x1="210.82" y1="0" x2="279.4" y2="0" width="0.1524" layer="91"/>
-<label x="279.4" y="0" size="1.778" layer="95" rot="MR0"/>
+<wire x1="210.82" y1="0" x2="231.14" y2="0" width="0.1524" layer="91"/>
+<label x="231.14" y="0" size="1.778" layer="95"/>
 </segment>
 </net>
@@
 </segment>
 <segment>
-<pinref part="U1" gate="B3" pin="IO_L23P_3VREF_3"/>
-<wire x1="210.82" y1="-20.32" x2="279.4" y2="-20.32" width="0.1524" layer="91"/>
-<label x="279.4" y="-20.32" size="1.778" layer="95" rot="MR0"/>
+<pinref part="U1" gate="B3" pin="IO_L24N_3"/>
+<wire x1="231.14" y1="-15.24" x2="210.82" y2="-15.24" width="0.1524" layer="91"/>
+<label x="231.14" y="-15.24" size="1.778" layer="95"/>
 </segment>
 </net>
@@
 </segment>
 <segment>
-<pinref part="U1" gate="B3" pin="IO_L23N_3"/>
-<wire x1="210.82" y1="-10.16" x2="279.4" y2="-10.16" width="0.1524" layer="91"/>
-<label x="279.4" y="-10.16" size="1.778" layer="95" rot="MR0"/>
+<pinref part="U1" gate="B3" pin="IO_L40P_3"/>
+<wire x1="231.14" y1="-17.78" x2="210.82" y2="-17.78" width="0.1524" layer="91"/>
+<label x="231.14" y="-17.78" size="1.778" layer="95"/>
 </segment>
 </net>
@@
 </segment>
 <segment>
-<pinref part="U1" gate="B3" pin="IO_L24P_3"/>
-<wire x1="210.82" y1="-12.7" x2="279.4" y2="-12.7" width="0.1524" layer="91"/>
-<label x="279.4" y="-12.7" size="1.778" layer="95" rot="MR0"/>
-</segment>
-</net>
-<net name="Q3" class="0">
+<pinref part="U1" gate="B3" pin="IO_L40N_3VREF_3"/>
+<wire x1="231.14" y1="-22.86" x2="210.82" y2="-22.86" width="0.1524" layer="91"/>
+<label x="231.14" y="-22.86" size="1.778" layer="95"/>
+</segment>
+</net>
+<net name="HDR_SEL" class="0">
+<segment>
+<wire x1="281.94" y1="27.94" x2="294.64" y2="27.94" width="0.1524" layer="91"/>
+<label x="281.94" y="27.94" size="1.778" layer="95"/>
+<pinref part="SV4" gate="G$1" pin="11"/>
+</segment>
+<segment>
+<pinref part="U1" gate="B2" pin="IO_L40P_2VREF_2"/>
+<wire x1="231.14" y1="22.86" x2="210.82" y2="22.86" width="0.1524" layer="91"/>
+<label x="231.14" y="22.86" size="1.778" layer="95"/>
+</segment>
+</net>
+<net name="HDR_SPARE" class="0">
+<segment>
+<wire x1="281.94" y1="30.48" x2="294.64" y2="30.48" width="0.1524" layer="91"/>
+<label x="281.94" y="30.48" size="1.778" layer="95"/>
+<pinref part="SV4" gate="G$1" pin="9"/>
+</segment>
 <segment>
 <pinref part="U1" gate="B2" pin="IO_L40N_2"/>
@@
 </segment>
 </net>
-<net name="Q4" class="0">
-<segment>
-<pinref part="U1" gate="B3" pin="IO_L40N_3VREF_3"/>
-<wire x1="231.14" y1="-22.86" x2="210.82" y2="-22.86" width="0.1524" layer="91"/>
-<label x="231.14" y="-22.86" size="1.778" layer="95"/>
-</segment>
-</net>
-<net name="Q3A" class="0">
-<segment>
-<pinref part="U1" gate="B2" pin="IO_L40P_2VREF_2"/>
-<wire x1="231.14" y1="22.86" x2="210.82" y2="22.86" width="0.1524" layer="91"/>
-<label x="231.14" y="22.86" size="1.778" layer="95"/>
-</segment>
-</net>
-<net name="HDR_SEL" class="0">
-<segment>
-<wire x1="281.94" y1="27.94" x2="294.64" y2="27.94" width="0.1524" layer="91"/>
-<label x="281.94" y="27.94" size="1.778" layer="95"/>
-<pinref part="SV4" gate="G$1" pin="11"/>
-</segment>
-<segment>
-<pinref part="U1" gate="B3" pin="IO_L24N_3"/>
-<wire x1="279.4" y1="-15.24" x2="210.82" y2="-15.24" width="0.1524" layer="91"/>
-<label x="279.4" y="-15.24" size="1.778" layer="95" rot="MR0"/>
-</segment>
-</net>
-<net name="HDR_SPARE" class="0">
-<segment>
-<wire x1="281.94" y1="30.48" x2="294.64" y2="30.48" width="0.1524" layer="91"/>
-<label x="281.94" y="30.48" size="1.778" layer="95"/>
-<pinref part="SV4" gate="G$1" pin="9"/>
-</segment>
-<segment>
-<pinref part="U1" gate="B3" pin="IO_L40P_3"/>
-<wire x1="279.4" y1="-17.78" x2="210.82" y2="-17.78" width="0.1524" layer="91"/>
-<label x="279.4" y="-17.78" size="1.778" layer="95" rot="MR0"/>
-</segment>
-</net>
+<net name="C" class="0">
+<segment>
+<pinref part="U1" gate="B3" pin="IO_L24P_3"/>
+<wire x1="210.82" y1="-12.7" x2="231.14" y2="-12.7" width="0.1524" layer="91"/>
+<label x="231.14" y="-12.7" size="1.778" layer="95"/>
+</segment>
+</net>
+<net name="D" class="0">
+<segment>
+<pinref part="U1" gate="B3" pin="IO_L23N_3"/>
+<wire x1="210.82" y1="-10.16" x2="231.14" y2="-10.16" width="0.1524" layer="91"/>
+<label x="231.14" y="-10.16" size="1.778" layer="95"/>
+</segment>
+</net>
+<net name="A" class="0">
+<segment>
+<pinref part="U1" gate="B3" pin="IO_L23P_3VREF_3"/>
+<wire x1="210.82" y1="-20.32" x2="231.14" y2="-20.32" width="0.1524" layer="91"/>
+<label x="231.14" y="-20.32" size="1.778" layer="95"/>
+</segment>
+</net>

Commit message: moving down
Connections:
- removed net A: U1B3.IO_L23P_3VREF_3
- removed net C: U1B3.IO_L24P_3
- removed net D: U1B3.IO_L23N_3
- new net F: U1B3.IO_L22P_3
- new net G: U1B3.IO_L21N_3
- new net H: U1B3.IO_L21P_3
- net PD3: now also U1B3.IO_L24P_3; no longer U1B3.IO_L22N_3
- net PD4: now also U1B3.IO_L23N_3; no longer U1B3.IO_L22P_3
- net PD5: now also U1B3.IO_L23P_3VREF_3; no longer U1B3.IO_L21N_3
- net PD6: now also U1B3.IO_L22N_3; no longer U1B3.IO_L21P_3
Changed lines of the file:
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@@
 </segment>
 <segment>
-<pinref part="U1" gate="B3" pin="IO_L22N_3"/>
-<wire x1="210.82" y1="-7.62" x2="231.14" y2="-7.62" width="0.1524" layer="91"/>
-<label x="231.14" y="-7.62" size="1.778" layer="95"/>
+<pinref part="U1" gate="B3" pin="IO_L24P_3"/>
+<wire x1="210.82" y1="-12.7" x2="231.14" y2="-12.7" width="0.1524" layer="91"/>
+<label x="231.14" y="-12.7" size="1.778" layer="95"/>
 </segment>
 </net>
@@
 </segment>
 <segment>
-<pinref part="U1" gate="B3" pin="IO_L22P_3"/>
-<wire x1="210.82" y1="-5.08" x2="231.14" y2="-5.08" width="0.1524" layer="91"/>
-<label x="231.14" y="-5.08" size="1.778" layer="95"/>
+<pinref part="U1" gate="B3" pin="IO_L23N_3"/>
+<wire x1="210.82" y1="-10.16" x2="231.14" y2="-10.16" width="0.1524" layer="91"/>
+<label x="231.14" y="-10.16" size="1.778" layer="95"/>
 </segment>
 </net>
@@
 </segment>
 <segment>
-<pinref part="U1" gate="B3" pin="IO_L21N_3"/>
-<wire x1="210.82" y1="-2.54" x2="231.14" y2="-2.54" width="0.1524" layer="91"/>
-<label x="231.14" y="-2.54" size="1.778" layer="95"/>
+<pinref part="U1" gate="B3" pin="IO_L23P_3VREF_3"/>
+<wire x1="210.82" y1="-20.32" x2="231.14" y2="-20.32" width="0.1524" layer="91"/>
+<label x="231.14" y="-20.32" size="1.778" layer="95"/>
 </segment>
 </net>
@@
 </segment>
 <segment>
-<pinref part="U1" gate="B3" pin="IO_L21P_3"/>
-<wire x1="210.82" y1="0" x2="231.14" y2="0" width="0.1524" layer="91"/>
-<label x="231.14" y="0" size="1.778" layer="95"/>
+<pinref part="U1" gate="B3" pin="IO_L22N_3"/>
+<wire x1="210.82" y1="-7.62" x2="231.14" y2="-7.62" width="0.1524" layer="91"/>
+<label x="231.14" y="-7.62" size="1.778" layer="95"/>
 </segment>
 </net>
@@
 </segment>
 </net>
-<net name="C" class="0">
-<segment>
-<pinref part="U1" gate="B3" pin="IO_L24P_3"/>
-<wire x1="210.82" y1="-12.7" x2="231.14" y2="-12.7" width="0.1524" layer="91"/>
-<label x="231.14" y="-12.7" size="1.778" layer="95"/>
-</segment>
-</net>
-<net name="D" class="0">
-<segment>
-<pinref part="U1" gate="B3" pin="IO_L23N_3"/>
-<wire x1="210.82" y1="-10.16" x2="231.14" y2="-10.16" width="0.1524" layer="91"/>
-<label x="231.14" y="-10.16" size="1.778" layer="95"/>
-</segment>
-</net>
-<net name="A" class="0">
-<segment>
-<pinref part="U1" gate="B3" pin="IO_L23P_3VREF_3"/>
-<wire x1="210.82" y1="-20.32" x2="231.14" y2="-20.32" width="0.1524" layer="91"/>
-<label x="231.14" y="-20.32" size="1.778" layer="95"/>
-</segment>
-</net>
+<net name="F" class="0">
+<segment>
+<pinref part="U1" gate="B3" pin="IO_L22P_3"/>
+<wire x1="210.82" y1="-5.08" x2="231.14" y2="-5.08" width="0.1524" layer="91"/>
+<label x="231.14" y="-5.08" size="1.778" layer="95"/>
+</segment>
+</net>
+<net name="G" class="0">
+<segment>
+<pinref part="U1" gate="B3" pin="IO_L21N_3"/>
+<wire x1="210.82" y1="-2.54" x2="231.14" y2="-2.54" width="0.1524" layer="91"/>
+<label x="231.14" y="-2.54" size="1.778" layer="95"/>
+</segment>
+</net>
+<net name="H" class="0">
+<segment>
+<pinref part="U1" gate="B3" pin="IO_L21P_3"/>
+<wire x1="210.82" y1="0" x2="231.14" y2="0" width="0.1524" layer="91"/>
+<label x="231.14" y="0" size="1.778" layer="95"/>
+</segment>
+</net>

Commit message: moving down
Connections:
- removed net F: U1B3.IO_L22P_3
- removed net G: U1B3.IO_L21N_3
- removed net H: U1B3.IO_L21P_3
- new net L: U1B3.IO_L01N_3VRP_3
- new net M: U1B3.IO_L01P_3VRN_3
- new net N: U1B4.IOVREF_4
- net FL_DI: now also U1B3.IO_L21P_3; no longer U1B3.IO
- net FL_DO: now also U1B3.IO_L20P_3; no longer U1B3.IO_L01P_3VRN_3
- net FL_HOLD: now also U1B3.IO_L22P_3; no longer U1B3.IO_L20N_3
- net FL_SCLK: now also U1B3.IO_L21N_3; no longer U1B3.IO_L20P_3
- net FL_SEL: now also U1B3.IO; no longer U1B4.IOVREF_4
- net FL_WP: now also U1B3.IO_L20N_3; no longer U1B3.IO_L01N_3VRP_3
Changed lines of the file:
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@@
 </segment>
 <segment>
-<pinref part="U1" gate="B4" pin="IOVREF_4"/>
-<wire x1="236.22" y1="-45.72" x2="157.48" y2="-45.72" width="0.1524" layer="91"/>
-<wire x1="157.48" y1="-45.72" x2="157.48" y2="-40.64" width="0.1524" layer="91"/>
-<wire x1="236.22" y1="-58.42" x2="236.22" y2="-45.72" width="0.1524" layer="91"/>
-<label x="236.22" y="-58.42" size="1.778" layer="95" rot="R90"/>
+<wire x1="231.14" y1="12.7" x2="210.82" y2="12.7" width="0.1524" layer="91"/>
+<pinref part="U1" gate="B3" pin="IO"/>
+<label x="231.14" y="12.7" size="1.778" layer="95"/>
 </segment>
 </net>
@@
 </segment>
 <segment>
+<pinref part="U1" gate="B3" pin="IO_L22P_3"/>
+<wire x1="210.82" y1="-5.08" x2="231.14" y2="-5.08" width="0.1524" layer="91"/>
+<label x="231.14" y="-5.08" size="1.778" layer="95"/>
+</segment>
+</net>
+<net name="FL_SCLK" class="0">
+<segment>
+<pinref part="IC2" gate="G$1" pin="SCK"/>
+<wire x1="238.76" y1="-86.36" x2="246.38" y2="-86.36" width="0.1524" layer="91"/>
+<label x="238.76" y="-86.36" size="1.778" layer="95"/>
+</segment>
+<segment>
+<wire x1="76.2" y1="-106.68" x2="149.86" y2="-106.68" width="0.1524" layer="91"/>
+<label x="76.2" y="-106.68" size="1.778" layer="95"/>
+</segment>
+<segment>
+<pinref part="U1" gate="B3" pin="IO_L21N_3"/>
+<wire x1="210.82" y1="-2.54" x2="231.14" y2="-2.54" width="0.1524" layer="91"/>
+<label x="231.14" y="-2.54" size="1.778" layer="95"/>
+</segment>
+</net>
+<net name="FL_DI" class="0">
+<segment>
+<pinref part="IC2" gate="G$1" pin="SI"/>
+<wire x1="238.76" y1="-83.82" x2="246.38" y2="-83.82" width="0.1524" layer="91"/>
+<label x="238.76" y="-83.82" size="1.778" layer="95"/>
+</segment>
+<segment>
+<wire x1="76.2" y1="-104.14" x2="152.4" y2="-104.14" width="0.1524" layer="91"/>
+<label x="76.2" y="-104.14" size="1.778" layer="95"/>
+</segment>
+<segment>
+<pinref part="U1" gate="B3" pin="IO_L21P_3"/>
+<wire x1="210.82" y1="0" x2="231.14" y2="0" width="0.1524" layer="91"/>
+<label x="231.14" y="0" size="1.778" layer="95"/>
+</segment>
+</net>
+<net name="FL_DO" class="0">
+<segment>
+<pinref part="IC2" gate="G$1" pin="SO"/>
+<wire x1="279.4" y1="-83.82" x2="274.32" y2="-83.82" width="0.1524" layer="91"/>
+<label x="274.32" y="-83.82" size="1.778" layer="95"/>
+</segment>
+<segment>
+<wire x1="147.32" y1="-114.3" x2="76.2" y2="-114.3" width="0.1524" layer="91"/>
+<label x="76.2" y="-114.3" size="1.778" layer="95"/>
+</segment>
+<segment>
+<pinref part="U1" gate="B3" pin="IO_L20P_3"/>
+<wire x1="210.82" y1="5.08" x2="231.14" y2="5.08" width="0.1524" layer="91"/>
+<label x="231.14" y="5.08" size="1.778" layer="95"/>
+</segment>
+</net>
+<net name="FL_WP" class="0">
+<segment>
+<pinref part="IC2" gate="G$1" pin="!WP"/>
+<wire x1="238.76" y1="-76.2" x2="246.38" y2="-76.2" width="0.1524" layer="91"/>
+<label x="238.76" y="-76.2" size="1.778" layer="95"/>
+</segment>
+<segment>
+<wire x1="76.2" y1="-116.84" x2="139.7" y2="-116.84" width="0.1524" layer="91"/>
+<label x="76.2" y="-116.84" size="1.778" layer="95"/>
+</segment>
+<segment>
 <pinref part="U1" gate="B3" pin="IO_L20N_3"/>
 <wire x1="210.82" y1="2.54" x2="231.14" y2="2.54" width="0.1524" layer="91"/>
 <label x="231.14" y="2.54" size="1.778" layer="95"/>
-</segment>
-</net>
-<net name="FL_SCLK" class="0">
-<segment>
-<pinref part="IC2" gate="G$1" pin="SCK"/>
-<wire x1="238.76" y1="-86.36" x2="246.38" y2="-86.36" width="0.1524" layer="91"/>
-<label x="238.76" y="-86.36" size="1.778" layer="95"/>
-</segment>
-<segment>
-<wire x1="76.2" y1="-106.68" x2="149.86" y2="-106.68" width="0.1524" layer="91"/>
-<label x="76.2" y="-106.68" size="1.778" layer="95"/>
-</segment>
-<segment>
-<pinref part="U1" gate="B3" pin="IO_L20P_3"/>
-<wire x1="210.82" y1="5.08" x2="231.14" y2="5.08" width="0.1524" layer="91"/>
-<label x="231.14" y="5.08" size="1.778" layer="95"/>
-</segment>
-</net>
-<net name="FL_DI" class="0">
-<segment>
-<pinref part="IC2" gate="G$1" pin="SI"/>
-<wire x1="238.76" y1="-83.82" x2="246.38" y2="-83.82" width="0.1524" layer="91"/>
-<label x="238.76" y="-83.82" size="1.778" layer="95"/>
-</segment>
-<segment>
-<wire x1="76.2" y1="-104.14" x2="152.4" y2="-104.14" width="0.1524" layer="91"/>
-<label x="76.2" y="-104.14" size="1.778" layer="95"/>
-</segment>
-<segment>
-<wire x1="231.14" y1="12.7" x2="210.82" y2="12.7" width="0.1524" layer="91"/>
-<pinref part="U1" gate="B3" pin="IO"/>
-<label x="231.14" y="12.7" size="1.778" layer="95"/>
-</segment>
-</net>
-<net name="FL_DO" class="0">
-<segment>
-<pinref part="IC2" gate="G$1" pin="SO"/>
-<wire x1="279.4" y1="-83.82" x2="274.32" y2="-83.82" width="0.1524" layer="91"/>
-<label x="274.32" y="-83.82" size="1.778" layer="95"/>
-</segment>
-<segment>
-<wire x1="147.32" y1="-114.3" x2="76.2" y2="-114.3" width="0.1524" layer="91"/>
-<label x="76.2" y="-114.3" size="1.778" layer="95"/>
-</segment>
-<segment>
-<wire x1="231.14" y1="10.16" x2="210.82" y2="10.16" width="0.1524" layer="91"/>
-<pinref part="U1" gate="B3" pin="IO_L01P_3VRN_3"/>
-<label x="231.14" y="10.16" size="1.778" layer="95"/>
-</segment>
-</net>
-<net name="FL_WP" class="0">
-<segment>
-<pinref part="IC2" gate="G$1" pin="!WP"/>
-<wire x1="238.76" y1="-76.2" x2="246.38" y2="-76.2" width="0.1524" layer="91"/>
-<label x="238.76" y="-76.2" size="1.778" layer="95"/>
-</segment>
-<segment>
-<wire x1="76.2" y1="-116.84" x2="139.7" y2="-116.84" width="0.1524" layer="91"/>
-<label x="76.2" y="-116.84" size="1.778" layer="95"/>
-</segment>
-<segment>
-<pinref part="U1" gate="B3" pin="IO_L01N_3VRP_3"/>
-<wire x1="210.82" y1="7.62" x2="231.14" y2="7.62" width="0.1524" layer="91"/>
-<label x="231.14" y="7.62" size="1.778" layer="95"/>
 </segment>
 </net>
@@
 </segment>
 </net>
-<net name="F" class="0">
-<segment>
-<pinref part="U1" gate="B3" pin="IO_L22P_3"/>
-<wire x1="210.82" y1="-5.08" x2="231.14" y2="-5.08" width="0.1524" layer="91"/>
-<label x="231.14" y="-5.08" size="1.778" layer="95"/>
-</segment>
-</net>
-<net name="G" class="0">
-<segment>
-<pinref part="U1" gate="B3" pin="IO_L21N_3"/>
-<wire x1="210.82" y1="-2.54" x2="231.14" y2="-2.54" width="0.1524" layer="91"/>
-<label x="231.14" y="-2.54" size="1.778" layer="95"/>
-</segment>
-</net>
-<net name="H" class="0">
-<segment>
-<pinref part="U1" gate="B3" pin="IO_L21P_3"/>
-<wire x1="210.82" y1="0" x2="231.14" y2="0" width="0.1524" layer="91"/>
-<label x="231.14" y="0" size="1.778" layer="95"/>
-</segment>
-</net>
+<net name="L" class="0">
+<segment>
+<pinref part="U1" gate="B3" pin="IO_L01N_3VRP_3"/>
+<wire x1="210.82" y1="7.62" x2="231.14" y2="7.62" width="0.1524" layer="91"/>
+<label x="231.14" y="7.62" size="1.778" layer="95"/>
+</segment>
+</net>
+<net name="M" class="0">
+<segment>
+<wire x1="231.14" y1="10.16" x2="210.82" y2="10.16" width="0.1524" layer="91"/>
+<pinref part="U1" gate="B3" pin="IO_L01P_3VRN_3"/>
+<label x="231.14" y="10.16" size="1.778" layer="95"/>
+</segment>
+</net>
+<net name="N" class="0">
+<segment>
+<pinref part="U1" gate="B4" pin="IOVREF_4"/>
+<wire x1="236.22" y1="-45.72" x2="157.48" y2="-45.72" width="0.1524" layer="91"/>
+<wire x1="157.48" y1="-45.72" x2="157.48" y2="-40.64" width="0.1524" layer="91"/>
+<wire x1="236.22" y1="-58.42" x2="236.22" y2="-45.72" width="0.1524" layer="91"/>
+<label x="236.22" y="-58.42" size="1.778" layer="95" rot="R90"/>
+</segment>
+</net>
