File: eagle/homeboard/homeboard23.brd (EAGLE design)
At the start: 94 x 71.8 mm, 128 parts, among them IC1 XCF02S, IC2 25LC080SN, IC3 ATMEGA32U2-TQFP, Q5 BC848SMD, Q6 BC848SMD, Q7 BC848SMD, Q8 BC848SMD, T1 BSS138, T2 BC848, T3 BSS138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

Commit message: more
Parts:
- moved C30 35.5 mm to (64.8, 41.5), flipped to the bottom, turned to 180 degrees
- moved C18 6.01 mm to (58.2, 22.2), turned to 270 degrees
- moved C25 4.83 mm to (56.0, 22.2), turned to 270 degrees
- moved C21 4.51 mm to (49.5, 22.2), turned to 270 degrees
- moved C24 4.51 mm to (51.8, 22.2), turned to 270 degrees
- moved C11 4.50 mm to (41.8, 33.5), turned to 0 degrees
- moved C10 4.32 mm to (64.8, 34.0), turned to 180 degrees
- moved C9 3.81 mm to (41.8, 41.5), turned to 0 degrees
- moved C16 3.72 mm to (41.8, 26.8), turned to 0 degrees
- moved C17 3.54 mm to (64.5, 27.0), turned to 180 degrees
- moved C12 1.00 mm to (46.5, 39.5)
Routing:
- net GND: track 950.0 -> 1000.7 mm
- net VCC: track 548.3 -> 557.5 mm, vias 22 -> 23
- net VCCINT: track 119.8 -> 115.3 mm
- net SD_CLK: track 24.9 -> 21.8 mm
- net TDO_FPGA: track 39.6 -> 41.6 mm
- net N$40: track 57.9 -> 59.6 mm
- net N$12: track 20.5 -> 19.4 mm
- net FL_SEL: track 20.4 -> 19.3 mm
- net EXTCLK: track 14.1 -> 15.0 mm

Commit message: more
Routing:
- net VCCAUX: track 141.7 -> 132.9 mm
- net VCC: track 557.5 -> 558.5 mm

Commit message: more
Parts:
- moved C14 6.52 mm to (47.0, 21.5), turned to 270 degrees
Routing:
- net GND: track 1000.7 -> 1009.7 mm
- net VCC: track 558.5 -> 560.4 mm
- net SD_CLK: track 21.9 -> 23.2 mm

Commit message: more
Parts:
- moved C15 3.54 mm to (51.8, 26.0)
Routing:
- net GND: track 1009.7 -> 1012.8 mm
- net VCCAUX: track 132.8 -> 131.2 mm
- net VCC: track 560.4 -> 559.0 mm
- net VCCINT: track 115.0 -> 114.0 mm

Commit message: more
Routing:
- net VCC: track 559.0 -> 561.6 mm
Changed lines of the file:
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@@
 <wire x1="63.92" y1="26" x2="62.25" y2="26" width="0.254" layer="1"/>
 <via x="62.25" y="26" extent="1-16" drill="0.6" shape="square"/>
-<wire x1="62.25" y1="26" x2="61" y2="26" width="0.254" layer="16"/>
-<wire x1="59.75" y1="26" x2="60" y2="26" width="0.254" layer="1"/>
 <via x="52.75" y="24.5" extent="1-16" drill="0.6" shape="square"/>
-<wire x1="60" y1="26" x2="62.25" y2="26" width="0.254" layer="1"/>
 <wire x1="47.5" y1="41.75" x2="47.5" y2="40.5" width="0.254" layer="16"/>
 <wire x1="47.5" y1="40.5" x2="45.6" y2="40.5" width="0.254" layer="16"/>
@@
 <wire x1="58.75" y1="41.75" x2="58.25" y2="41.75" width="0.6" layer="1"/>
 <via x="58.75" y="33.5" extent="1-16" drill="0.6" shape="square"/>
-<wire x1="60.25" y1="30.5" x2="60.25" y2="25.75" width="0.6" layer="1"/>
 <wire x1="62.25" y1="41.5" x2="62.25" y2="42.75" width="0.6" layer="1"/>
 <wire x1="62.25" y1="42.75" x2="63" y2="43.5" width="0.6" layer="1"/>
-<wire x1="62.25" y1="41.5" x2="59" y2="41.5" width="0.6" layer="1"/>
 <wire x1="63.92" y1="41.5" x2="62.25" y2="41.5" width="0.254" layer="1"/>
 <contactref element="C26" pad="1"/>
@@
 <wire x1="65.275" y1="12.425" x2="65" y2="12.4" width="0.8" layer="1"/>
 <wire x1="55.025" y1="12.4" x2="55.025" y2="14.605" width="0.254" layer="1"/>
-<wire x1="58.75" y1="32.25" x2="60.25" y2="30.5" width="0.6" layer="1"/>
 <wire x1="52" y1="12.5" x2="51.85" y2="12.5" width="0.254" layer="1"/>
 <wire x1="51.85" y1="12.5" x2="51.75" y2="12.4" width="0.254" layer="1"/>
@@
 <wire x1="63" y1="45.5" x2="64.5" y2="47" width="0.7" layer="1"/>
 <wire x1="64.5" y1="47" x2="64.5" y2="53.5" width="0.7" layer="1"/>
-<wire x1="60.25" y1="25.75" x2="60" y2="26" width="0.254" layer="1"/>
 <wire x1="85.25" y1="20.25" x2="85.5" y2="20.5" width="0.254" layer="1"/>
 <wire x1="83" y1="19.85" x2="81.9" y2="19.85" width="0.254" layer="16"/>
@@
 <wire x1="76.375325" y1="29.18058125" x2="76.375325" y2="29.124675" width="0.254" layer="1"/>
 <wire x1="76.375325" y1="29.124675" x2="76.5" y2="29" width="0.254" layer="1"/>
-<wire x1="60.25" y1="25.75" x2="62.5" y2="25.75" width="0.6" layer="1"/>
-<wire x1="62.5" y1="25.75" x2="62.5" y2="24.5" width="0.6" layer="1"/>
 <wire x1="62.5" y1="24.5" x2="64" y2="23" width="0.6" layer="1"/>
 <wire x1="64" y1="23" x2="67.5" y2="23" width="0.6" layer="1"/>
@@
 <wire x1="58.97" y1="23.05" x2="58.97" y2="24.22" width="0.254" layer="1"/>
 <wire x1="58.97" y1="24.22" x2="60" y2="24.25" width="0.254" layer="1"/>
-<wire x1="60" y1="24.25" x2="60" y2="25.5" width="0.254" layer="1"/>
-<wire x1="60" y1="25.5" x2="60.25" y2="25.75" width="0.254" layer="1"/>
 <wire x1="76.375325" y1="29.18058125" x2="76.31941875" y2="29.18058125" width="0.254" layer="1"/>
 <via x="75.25" y="30.5" extent="1-16" drill="0.6" shape="square"/>
@@
 <wire x1="62.25" y1="34" x2="63.92" y2="34" width="0.254" layer="1"/>
 <wire x1="62.25" y1="34" x2="58.75" y2="34" width="0.254" layer="1"/>
+<wire x1="62.25" y1="41.5" x2="61.5" y2="41.5" width="0.6" layer="1"/>
+<wire x1="61.5" y1="41.5" x2="61.25" y2="41.25" width="0.6" layer="1"/>
+<wire x1="61.25" y1="41.25" x2="61.25" y2="25.5" width="0.6" layer="1"/>
+<wire x1="62.5" y1="24.5" x2="62.5" y2="25.5" width="0.6" layer="1"/>
+<wire x1="62.5" y1="25.5" x2="62" y2="25.5" width="0.6" layer="1"/>
+<wire x1="62" y1="25.5" x2="61.25" y2="25.5" width="0.6" layer="1"/>
+<wire x1="62.25" y1="26" x2="62.25" y2="25.75" width="0.6" layer="1"/>
+<wire x1="62.25" y1="25.75" x2="62" y2="25.5" width="0.6" layer="1"/>
+<wire x1="60.25" y1="25.5" x2="61.25" y2="25.5" width="0.6" layer="1"/>
+<wire x1="60" y1="24.25" x2="60" y2="25.25" width="0.254" layer="1"/>
+<wire x1="60" y1="25.25" x2="60.25" y2="25.5" width="0.254" layer="1"/>
 <wire x1="97.15" y1="32.5" x2="97.15" y2="38" width="0" layer="19" extent="1-1"/>
 <wire x1="92.25" y1="43.7" x2="97.15" y2="38" width="0" layer="19" extent="1-1"/>
 <wire x1="51.95" y1="53.55" x2="52" y2="53.55" width="0" layer="19" extent="1-1"/>
 <wire x1="64.5" y1="53.5" x2="64.75" y2="53.55" width="0" layer="19" extent="1-1"/>
+<wire x1="37.5" y1="15.75" x2="37.52" y2="15.79" width="0" layer="19" extent="1-1"/>
 <wire x1="23.516" y1="17.9906" x2="23.5" y2="18" width="0" layer="19" extent="16-16"/>
 <wire x1="12.5" y1="27.75" x2="12.599" y2="27.75" width="0" layer="19" extent="1-1"/>

Commit message: more
Routing:
- net VCC: track 561.6 -> 557.5 mm
- net SD_CLK: track 23.2 -> 21.5 mm
- net GND: track 1012.8 -> 1013.5 mm

Commit message: more
Parts:
- moved C12 1.35 mm to (46.0, 40.8)
- moved C19 0.25 mm to (49.8, 40.0)
- moved C6 0.25 mm to (51.8, 37.2)
Routing:
- net VCC: track 557.5 -> 544.5 mm
- net GND: track 1013.5 -> 1003.3 mm
- net VCCINT: track 113.8 -> 114.4 mm

Commit message: more
Parts:
- moved C8 1.35 mm to (60.0, 28.2)
- moved C19 1.00 mm to (48.8, 40.0), turned to 0 degrees
- moved C22 0.50 mm to (51.5, 40.8)
- moved C12 0.25 mm to (45.8, 40.8)
Routing:
- net GND: track 1003.3 -> 996.0 mm
- net VCC: track 544.5 -> 541.6 mm, vias 23 -> 24
