File: eagle/homeboard/homeboard24.brd (EAGLE design)
At the start: 94 x 71.8 mm, 124 parts, among them IC1 XCF02S, IC2 25LC080SN, IC3 ATMEGA32U2-TQFP, Q5 BC848SMD, Q6 BC848SMD, Q7 BC848SMD, Q8 BC848SMD, T1 BSS138, T2 BC848, T3 BSS138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

Commit message: moving around
Parts:
- moved C19 0.56 mm to (49.2, 39.8), turned to 270 degrees
Routing:
- net GND: track 983.6 -> 984.1 mm
Changed lines of the file:
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@@
 <element name="C17" library="rcl" package="C0603" value="100nF" x="64.5" y="27" rot="MR180"/>
 <element name="C18" library="rcl" package="C0603" value="100nF" x="58.25" y="22.25" rot="MR270"/>
-<element name="C19" library="rcl" package="C0603" value="100nF" x="48.75" y="40" rot="MR0"/>
+<element name="C19" library="rcl" package="C0603" value="100nF" x="49.25" y="39.75" rot="MR270"/>
 <element name="C20" library="rcl" package="C0603" value="100nF" x="58.25" y="39.5" rot="MR270"/>
 <element name="C21" library="rcl" package="C0603" value="100nF" x="49.5" y="22.25" rot="MR270"/>
@@
 <wire x1="48.47" y1="44.45" x2="48.47" y2="43.03" width="0.254" layer="1"/>
 <wire x1="48.47" y1="43.03" x2="48.5" y2="43" width="0.254" layer="1"/>
-<wire x1="48.5" y1="43" x2="48.5" y2="41" width="0.254" layer="16"/>
-<wire x1="48.5" y1="41" x2="48" y2="40.5" width="0.254" layer="16"/>
-<wire x1="48" y1="40.5" x2="48" y2="40.1" width="0.254" layer="16"/>
-<wire x1="48" y1="40.1" x2="47.9" y2="40" width="0.254" layer="16"/>
-<wire x1="47.9" y1="40" x2="46.1" y2="40" width="0.254" layer="16"/>
+<wire x1="48.5" y1="43" x2="48.5" y2="41.5" width="0.254" layer="16"/>
+<wire x1="48" y1="41" x2="48" y2="40.1" width="0.254" layer="16"/>
 <wire x1="46.1" y1="40" x2="45.75" y2="39.9" width="0.254" layer="16"/>
 <wire x1="58.25" y1="27" x2="56.5" y2="27" width="0.254" layer="16"/>
@@
 <wire x1="51" y1="37.4" x2="51" y2="38" width="0.254" layer="16"/>
 <wire x1="51" y1="38" x2="50" y2="39" width="0.254" layer="16"/>
-<wire x1="50" y1="39" x2="48.5" y2="39" width="0.254" layer="16"/>
-<wire x1="48.5" y1="39" x2="48" y2="39.5" width="0.254" layer="16"/>
-<wire x1="48" y1="39.5" x2="48" y2="40" width="0.254" layer="16"/>
+<wire x1="48" y1="39.5" x2="48" y2="40.1" width="0.254" layer="16"/>
 <wire x1="51" y1="35.5" x2="51" y2="37.4" width="0.254" layer="16"/>
 <contactref element="C13" pad="2"/>
@@
 <wire x1="91.81" y1="36.39" x2="91.77" y2="36.35" width="0.254" layer="16"/>
 <wire x1="91.77" y1="36.35" x2="89.23" y2="36.35" width="0.254" layer="16"/>
+<wire x1="48.5" y1="41.5" x2="48" y2="41" width="0.254" layer="16"/>
+<wire x1="46.1" y1="40" x2="47.9" y2="40" width="0.254" layer="16"/>
+<wire x1="47.9" y1="40" x2="48" y2="40.1" width="0.254" layer="16"/>
+<wire x1="50" y1="39" x2="49.5" y2="39" width="0.254" layer="16"/>
+<wire x1="49.5" y1="39" x2="48.5" y2="39" width="0.254" layer="16"/>
+<wire x1="48.5" y1="39" x2="48" y2="39.5" width="0.254" layer="16"/>
+<wire x1="49.25" y1="38.9" x2="49.4" y2="38.9" width="0.254" layer="16"/>
+<wire x1="49.4" y1="38.9" x2="49.5" y2="39" width="0.254" layer="16"/>
+<wire x1="46.97" y1="44.45" x2="46.97" y2="44.47" width="0.254" layer="1"/>
+<wire x1="46.97" y1="44.47" x2="47" y2="44.5" width="0.254" layer="1"/>
+<wire x1="59.47" y1="44.45" x2="59.47" y2="44.47" width="0.254" layer="1"/>
+<wire x1="59.47" y1="44.47" x2="59.5" y2="44.5" width="0.254" layer="1"/>
 <wire x1="73.17706875" y1="40.023221875" x2="73.25" y2="40" width="0" layer="19" extent="1-1"/>
-<wire x1="59.47" y1="44.45" x2="59.5" y2="44.5" width="0" layer="19" extent="1-1"/>
-<wire x1="46.97" y1="44.45" x2="47" y2="44.5" width="0" layer="19" extent="1-1"/>
 <wire x1="89.23" y1="36.35" x2="89.11" y2="36.39" width="0" layer="19" extent="16-16"/>
 <wire x1="79.65" y1="5" x2="81.5" y2="6.5" width="0" layer="19" extent="1-16"/>
@@
 <via x="44" y="41.5" extent="1-16" drill="0.6" shape="square"/>
 <wire x1="47.47" y1="44.45" x2="47.47" y2="41.78" width="0.254" layer="1"/>
-<wire x1="47.47" y1="41.78" x2="47.5" y2="41.75" width="0.254" layer="1"/>
-<via x="47.5" y="41.75" extent="1-16" drill="0.6" shape="square"/>
+<wire x1="47.47" y1="41.78" x2="47.25" y2="41.75" width="0.254" layer="1"/>
+<via x="47.25" y="41.75" extent="1-16" drill="0.6" shape="square"/>
 <wire x1="63.92" y1="26" x2="62.25" y2="26" width="0.254" layer="1"/>
 <via x="62.25" y="26" extent="1-16" drill="0.6" shape="square"/>
@@
 <wire x1="44.25" y1="41.75" x2="44" y2="41.5" width="0.254" layer="1"/>
 <wire x1="44" y1="41.5" x2="47.25" y2="41.5" width="0.254" layer="1"/>
-<wire x1="47.25" y1="41.5" x2="47.5" y2="41.75" width="0.254" layer="1"/>
+<wire x1="47.25" y1="41.5" x2="47.25" y2="41.75" width="0.254" layer="1"/>
 <wire x1="51" y1="33.5" x2="52.5" y2="35" width="0.7" layer="1"/>
 <via x="52.5" y="35" extent="1-16" drill="0.6" shape="square"/>
@@
 <wire x1="44" y1="41.5" x2="44" y2="43" width="0.7" layer="1"/>
 <wire x1="44" y1="43" x2="42.25" y2="44.75" width="0.7" layer="1"/>
-<wire x1="45.75" y1="41.6" x2="47.35" y2="41.6" width="0.254" layer="16"/>
-<wire x1="47.35" y1="41.6" x2="47.5" y2="41.75" width="0.254" layer="16"/>
+<wire x1="45.75" y1="41.6" x2="47.1" y2="41.6" width="0.254" layer="16"/>
+<wire x1="47.1" y1="41.6" x2="47.25" y2="41.75" width="0.254" layer="16"/>
 <wire x1="52.5" y1="26" x2="52.5" y2="27" width="0.254" layer="16"/>
 <wire x1="52.5" y1="27" x2="49" y2="27" width="0.254" layer="16"/>
@@
 <wire x1="55.5" y1="25.5" x2="55.5" y2="28.25" width="0.7" layer="1"/>
 <wire x1="50.5" y1="25.5" x2="55.5" y2="25.5" width="0.254" layer="1"/>
-<wire x1="56" y1="44.5" x2="55.97" y2="44.45" width="0" layer="19" extent="1-1"/>
+<wire x1="55.97" y1="44.45" x2="55.97" y2="44.47" width="0.254" layer="1"/>
+<wire x1="55.97" y1="44.47" x2="56" y2="44.5" width="0.254" layer="1"/>
 </signal>
 <signal name="VCCAUX">
@@
 <wire x1="58.1" y1="23.1" x2="58" y2="23" width="0.254" layer="16"/>
 <wire x1="48" y1="22" x2="48" y2="18" width="0.254" layer="16"/>
-<wire x1="49.75" y1="42.25" x2="49.75" y2="40.25" width="0.254" layer="16"/>
-<wire x1="49.75" y1="40.25" x2="49.5" y2="40" width="0.254" layer="16"/>
-<wire x1="49.5" y1="40" x2="49.6" y2="40" width="0.254" layer="16"/>
 <wire x1="49.47" y1="41.47" x2="48.5" y2="40.5" width="0.254" layer="1"/>
 <wire x1="48.5" y1="40.5" x2="47.5" y2="40.5" width="0.254" layer="1"/>
@@
 <wire x1="58" y1="40.5" x2="58.25" y2="40.25" width="0.254" layer="16"/>
 <wire x1="58.25" y1="40.25" x2="58.25" y2="40.35" width="0.254" layer="16"/>
+<wire x1="49.75" y1="42.25" x2="49.75" y2="40.75" width="0.254" layer="16"/>
+<wire x1="49.75" y1="40.75" x2="49.5" y2="40.5" width="0.254" layer="16"/>
+<wire x1="49.25" y1="40.6" x2="49.4" y2="40.6" width="0.254" layer="16"/>
+<wire x1="49.4" y1="40.6" x2="49.5" y2="40.5" width="0.254" layer="16"/>
 </signal>
 <signal name="SCART_RIGHT">
@@
 <wire x1="67" y1="42.5" x2="67" y2="40" width="0.254" layer="1"/>
 <wire x1="67" y1="40" x2="66.5" y2="39.5" width="0.254" layer="1"/>
-<wire x1="66.5" y1="39.5" x2="64" y2="39.5" width="0.254" layer="1"/>
+<wire x1="66.5" y1="39.5" x2="63.92" y2="39.5" width="0.254" layer="1"/>
 <via x="68.5" y="50.5" extent="1-16" drill="0.6" shape="square"/>
 <wire x1="68.5" y1="50.5" x2="68.5" y2="52" width="0.254" layer="16"/>
 <wire x1="68.5" y1="52" x2="67.5" y2="53" width="0.254" layer="16"/>
 <wire x1="67.5" y1="53" x2="67" y2="53" width="0.254" layer="16"/>
-<wire x1="64" y1="39.5" x2="63.92" y2="39.5" width="0" layer="19" extent="1-1"/>
 </signal>
 <signal name="JOY1_LEFT">
@@
 <wire x1="65.5" y1="44" x2="65.5" y2="41.5" width="0.254" layer="1"/>
 <wire x1="65.5" y1="41.5" x2="65" y2="41" width="0.254" layer="1"/>
-<wire x1="65" y1="41" x2="64" y2="41" width="0.254" layer="1"/>
-<wire x1="64" y1="41" x2="63.92" y2="41" width="0" layer="19" extent="1-1"/>
+<wire x1="65" y1="41" x2="63.92" y2="41" width="0.254" layer="1"/>
 </signal>
 <signal name="JOY1_UP">
@@
 <wire x1="36.75" y1="47" x2="35.75" y2="48" width="0.254" layer="16"/>
 <wire x1="35.75" y1="48" x2="35.75" y2="50.5" width="0.254" layer="16"/>
-<wire x1="35.75" y1="50.5" x2="35.65" y2="50.5" width="0" layer="19" extent="16-16"/>
+<wire x1="35.75" y1="50.5" x2="35.65" y2="50.5" width="0.254" layer="16"/>
+<wire x1="35.65" y1="50.5" x2="35.5" y2="50.5" width="0.254" layer="16"/>
 </signal>
 <signal name="N$1">
@@
 <wire x1="48.75" y1="47" x2="38.25" y2="47" width="0.254" layer="16"/>
 <wire x1="38.25" y1="47" x2="38.25" y2="50.5" width="0.254" layer="16"/>
-<wire x1="38.25" y1="50.5" x2="38.19" y2="50.5" width="0" layer="19" extent="16-16"/>
+<wire x1="38.25" y1="50.5" x2="38.19" y2="50.5" width="0.254" layer="16"/>
 </signal>
 <signal name="N$2">
@@
 <wire x1="49" y1="48.5" x2="48.5" y2="49" width="0.254" layer="1"/>
 <wire x1="48.5" y1="49" x2="48.5" y2="50.5" width="0.254" layer="1"/>
-<wire x1="48.5" y1="50.5" x2="48.35" y2="50.5" width="0" layer="19" extent="1-1"/>
+<wire x1="48.35" y1="50.5" x2="48.5" y2="50.5" width="0.254" layer="1"/>
 </signal>
 <signal name="N$7">
@@
 <wire x1="52.5" y1="49" x2="52" y2="49" width="0.254" layer="1"/>
 <wire x1="52" y1="49" x2="50.5" y2="50.5" width="0.254" layer="1"/>
-<wire x1="50.5" y1="50.5" x2="51" y2="50.5" width="0.254" layer="1"/>
-<wire x1="51" y1="50.5" x2="50.89" y2="50.5" width="0" layer="19" extent="1-1"/>
+<wire x1="50.5" y1="50.5" x2="50.89" y2="50.5" width="0.254" layer="1"/>
+<wire x1="51" y1="50.5" x2="50.89" y2="50.5" width="0.254" layer="1"/>
 </signal>
 <signal name="N$16">
@@
 <wire x1="55" y1="49.5" x2="54.5" y2="49.5" width="0.254" layer="1"/>
 <wire x1="54.5" y1="49.5" x2="53.5" y2="50.5" width="0.254" layer="1"/>
-<wire x1="53.5" y1="50.5" x2="53.43" y2="50.5" width="0" layer="19" extent="1-1"/>
+<wire x1="53.5" y1="50.5" x2="53.43" y2="50.5" width="0.254" layer="1"/>
 </signal>
 <signal name="N$8">
