File: eagle/homeboard/homeboard27.sch (EAGLE design)
At the start: 124 parts, among them IC1 XCF02S, IC2 25LC080SN, IC3 ATMEGA32U2-TQFP, Q5 BC848SMD, Q6 BC848SMD, Q7 BC848SMD, Q8 BC848SMD, T1 BSS138, T2 BC848, T3 BSS138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

Commit message: added led
Parts:
- added LED1: (no value), adafruit:LEDCHIPLED_0805
- added R11: (no value), resistor:R-EU_M0805
Connections:
- new net N$10: LED1.A, R11.2
- net GND: now also LED1.C
- net VCC: now also R11.1
Changed lines of the file:
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@@
 <attribute name="OC_NEWARK" value="unknown"/>
 </part>
+<part name="R11" library="resistor" deviceset="R-EU_" device="M0805"/>
+<part name="SUPPLY17" library="supply2" deviceset="GND" device=""/>
+<part name="LED1" library="adafruit" deviceset="LED" device="CHIPLED_0805"/>
 </parts>
 <sheets>
@@
 <instance part="C13" gate="G$1" x="-93.98" y="109.22"/>
 <instance part="SV1" gate="G$1" x="302.26" y="33.02" rot="R180"/>
+<instance part="R11" gate="G$1" x="-294.64" y="12.7"/>
+<instance part="SUPPLY17" gate="GND" x="-269.24" y="10.16"/>
+<instance part="LED1" gate="G$1" x="-281.94" y="12.7" rot="R90"/>
 </instances>
 <busses>
@@
 <wire x1="60.96" y1="-68.58" x2="68.58" y2="-68.58" width="0.1524" layer="91"/>
 <label x="60.96" y="-68.58" size="1.778" layer="95"/>
+</segment>
+<segment>
+<pinref part="LED1" gate="G$1" pin="C"/>
+<pinref part="SUPPLY17" gate="GND" pin="GND"/>
+<wire x1="-276.86" y1="12.7" x2="-269.24" y2="12.7" width="0.1524" layer="91"/>
 </segment>
 </net>
@@
 <label x="91.44" y="-73.66" size="1.778" layer="95" rot="MR0"/>
 </segment>
+<segment>
+<pinref part="R11" gate="G$1" pin="1"/>
+<wire x1="-299.72" y1="12.7" x2="-309.88" y2="12.7" width="0.1524" layer="91"/>
+<label x="-309.88" y="12.7" size="1.778" layer="95"/>
+</segment>
 </net>
 <net name="TCK" class="0">
@@
 </segment>
 </net>
+<net name="N$10" class="0">
+<segment>
+<pinref part="LED1" gate="G$1" pin="A"/>
+<pinref part="R11" gate="G$1" pin="2"/>
+<wire x1="-284.48" y1="12.7" x2="-289.56" y2="12.7" width="0.1524" layer="91"/>
+</segment>
+</net>
