File: eagle/homeboard/homeboard28.brd (EAGLE design)
At the start: 94 x 71.8 mm, 126 parts, among them IC1 XCF02S, IC2 25LC080SN, IC3 ATMEGA32U2-TQFP, Q5 BC848SMD, Q6 BC848SMD, Q7 BC848SMD, Q8 BC848SMD, T1 BSS138, T2 BC848, T3 BSS138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

Commit message: reworked ground planes
Routing:
- net VCC: track 545.1 -> 545.7 mm
- net GND: track 1024.2 -> 1024.6 mm, vias 82 -> 83
- added copper zone on layer 1, net GND
- added copper zone on layer 16, net GND
Changed lines of the file:
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@@
 <wire x1="58.5" y1="38.5" x2="58" y2="38.5" width="0.254" layer="16"/>
 <wire x1="48.5" y1="32" x2="49" y2="32.5" width="0.254" layer="16"/>
-<wire x1="49" y1="32.5" x2="53" y2="37" width="0.254" layer="16"/>
-<wire x1="53" y1="37" x2="53.5" y2="38.4" width="0.254" layer="16"/>
+<wire x1="49" y1="32.5" x2="53.25" y2="36.25" width="0.254" layer="16"/>
+<wire x1="53.25" y1="36.25" x2="53.5" y2="38.4" width="0.254" layer="16"/>
 <wire x1="53.5" y1="38.4" x2="53.75" y2="38.65" width="0.254" layer="16"/>
 <wire x1="51.5" y1="29" x2="46.5" y2="29.25" width="0.254" layer="16"/>
@@
 <via x="26.5" y="30.25" extent="1-16" drill="0.6" shape="square"/>
 <via x="2.5" y="1.5" extent="1-16" drill="0.6" shape="square"/>
-<via x="53" y="37" extent="1-16" drill="0.6" shape="square"/>
+<via x="53.25" y="36.25" extent="1-16" drill="0.6" shape="square"/>
 <via x="59.5" y="35.25" extent="1-16" drill="0.6" shape="square"/>
 <via x="59.5" y="31" extent="1-16" drill="0.6" shape="square"/>
@@
 <via x="69" y="51.25" extent="1-16" drill="0.6" shape="square"/>
 <wire x1="69" y1="51.25" x2="69" y2="43.75" width="0.254" layer="1"/>
-<via x="74.25" y="46.5" extent="1-16" drill="0.6" shape="square"/>
-<wire x1="88.5" y1="63" x2="90" y2="65" width="0" layer="19" extent="16-16"/>
-<wire x1="89.23" y1="36.35" x2="89.25" y2="36.25" width="0" layer="19" extent="16-16"/>
-<wire x1="60" y1="29.1" x2="60" y2="29" width="0" layer="19" extent="16-16"/>
-<wire x1="48.5" y1="65" x2="48.4778" y2="65.2278" width="0" layer="19" extent="16-16"/>
-<wire x1="80" y1="57" x2="80" y2="56.75" width="0" layer="19" extent="16-16"/>
-<wire x1="89" y1="36.5" x2="89.25" y2="36.5" width="0" layer="19" extent="16-16"/>
-<wire x1="32.25" y1="6.5" x2="32.5" y2="6.5" width="0" layer="19" extent="16-16"/>
-<wire x1="16.5" y1="65" x2="16.5" y2="64.5" width="0" layer="19" extent="16-16"/>
-<wire x1="50.75" y1="29.25" x2="51.5" y2="29" width="0" layer="19" extent="16-16"/>
-<wire x1="59.5" y1="35.25" x2="60.5" y2="35.5" width="0" layer="19" extent="16-16"/>
-<wire x1="85" y1="65" x2="86" y2="65.5" width="0" layer="19" extent="16-16"/>
-<wire x1="26.5" y1="30.25" x2="27" y2="29.25" width="0" layer="19" extent="16-16"/>
-<wire x1="59.75" y1="38.5" x2="58.5" y2="38.5" width="0" layer="19" extent="16-16"/>
-<wire x1="84.75" y1="52.25" x2="85.05" y2="53.5" width="0" layer="19" extent="1-1"/>
-<wire x1="59.5" y1="31" x2="60.5" y2="30" width="0" layer="19" extent="16-16"/>
-<wire x1="71.25" y1="27.5" x2="71.5" y2="29" width="0" layer="19" extent="16-16"/>
-<wire x1="46.5" y1="38.5" x2="46.1" y2="40" width="0" layer="19" extent="16-16"/>
-<wire x1="79.5" y1="65" x2="81" y2="65.5" width="0" layer="19" extent="16-16"/>
-<wire x1="23.25" y1="48.5" x2="21.75" y2="49" width="0" layer="19" extent="16-16"/>
-<wire x1="41.2" y1="9.08" x2="41.2" y2="10.8" width="0" layer="19" extent="16-16"/>
-<wire x1="34.25" y1="33.25" x2="32.5" y2="33.5" width="0" layer="19" extent="16-16"/>
-<wire x1="20.5" y1="64.5" x2="18.5" y2="65.25" width="0" layer="19" extent="16-16"/>
-<wire x1="49.25" y1="34.75" x2="49" y2="32.5" width="0" layer="19" extent="16-16"/>
-<wire x1="87.75" y1="55.75" x2="87" y2="53.5" width="0" layer="19" extent="1-1"/>
-<wire x1="81" y1="15.5" x2="83.393396875" y2="15.237409375" width="0" layer="19" extent="1-1"/>
-<wire x1="17" y1="45" x2="19.5" y2="45.15" width="0" layer="19" extent="1-1"/>
-<wire x1="23" y1="51.5" x2="21.75" y2="49" width="0" layer="19" extent="16-16"/>
-<wire x1="56.5" y1="31.5" x2="59.5" y2="31" width="0" layer="19" extent="1-1"/>
-<wire x1="53.5" y1="32.25" x2="56.5" y2="31.5" width="0" layer="19" extent="1-1"/>
-<wire x1="24.5" y1="37" x2="21" y2="36.65" width="0" layer="19" extent="1-1"/>
-<wire x1="12.5" y1="24" x2="9" y2="23.75" width="0" layer="19" extent="16-16"/>
-<wire x1="74.25" y1="46.5" x2="73.0874375" y2="43.1625625" width="0" layer="19" extent="1-1"/>
-<wire x1="36.25" y1="6.25" x2="32.5" y2="6.5" width="0" layer="19" extent="16-16"/>
-<wire x1="16" y1="30" x2="19.5" y2="28.15" width="0" layer="19" extent="1-1"/>
-<wire x1="52.5" y1="65" x2="48.5" y2="65.25" width="0" layer="19" extent="16-16"/>
-<wire x1="82.5" y1="2" x2="83.5" y2="6.5" width="0" layer="19" extent="16-16"/>
-<wire x1="92.5" y1="55.5" x2="87.75" y2="55.75" width="0" layer="19" extent="1-1"/>
-<wire x1="25.5" y1="22.5" x2="20.75" y2="23.75" width="0" layer="19" extent="16-16"/>
-<wire x1="93" y1="47.5" x2="89.5" y2="51" width="0" layer="19" extent="1-1"/>
-<wire x1="1.5" y1="12.5" x2="2" y2="7.5" width="0" layer="19" extent="16-16"/>
-<wire x1="15" y1="39" x2="19.5" y2="36.65" width="0" layer="19" extent="1-1"/>
-<wire x1="1.25" y1="59" x2="4.5" y2="55" width="0" layer="19" extent="1-1"/>
-<wire x1="36" y1="57" x2="33" y2="52.5" width="0" layer="19" extent="16-16"/>
-<wire x1="74" y1="65" x2="79.5" y2="65" width="0" layer="19" extent="1-1"/>
-<wire x1="2.5" y1="1.5" x2="6.4318" y2="6" width="0" layer="19" extent="16-16"/>
-<wire x1="69.5" y1="58.5" x2="68.5" y2="64.5" width="0" layer="19" extent="16-16"/>
-<wire x1="41.5" y1="64.5" x2="48.4778" y2="65.2278" width="0" layer="19" extent="16-16"/>
+<via x="82.5" y="6.5" extent="1-16" drill="0.6" shape="square"/>
+<polygon width="0.254" layer="16" isolate="0.6">
+<vertex x="0" y="72"/>
+<vertex x="12.5" y="72"/>
+<vertex x="12.5" y="66"/>
+<vertex x="94" y="66"/>
+<vertex x="94" y="15.5"/>
+<vertex x="93" y="15.5"/>
+<vertex x="93" y="43"/>
+<vertex x="79" y="43"/>
+<vertex x="79" y="56.5"/>
+<vertex x="66" y="56.5"/>
+<vertex x="66" y="50.5"/>
+<vertex x="68.5" y="50.5"/>
+<vertex x="68.5" y="41"/>
+<vertex x="70" y="41"/>
+<vertex x="71" y="40"/>
+<vertex x="76" y="40"/>
+<vertex x="76" y="42.5"/>
+<vertex x="88" y="42.5"/>
+<vertex x="88" y="10"/>
+<vertex x="56" y="10"/>
+<vertex x="56" y="19"/>
+<vertex x="54.5" y="19"/>
+<vertex x="54.5" y="25.5"/>
+<vertex x="53.5" y="25.5"/>
+<vertex x="53.5" y="19"/>
+<vertex x="51.5" y="19"/>
+<vertex x="51.5" y="11.5"/>
+<vertex x="39" y="11.5"/>
+<vertex x="39" y="19.5"/>
+<vertex x="0" y="19.5"/>
+</polygon>
+<polygon width="0.254" layer="16" isolate="0.6">
+<vertex x="-0.5" y="-0.5"/>
+<vertex x="-0.5" y="22.5"/>
+<vertex x="33.5" y="22.5"/>
+<vertex x="33.5" y="6.5"/>
+<vertex x="39" y="6.5"/>
+<vertex x="39" y="0"/>
+<vertex x="82" y="0"/>
+<vertex x="81.5" y="17.5"/>
+<vertex x="94.5" y="17.5"/>
+<vertex x="94.5" y="0"/>
+</polygon>
+<polygon width="0.4064" layer="1">
+<vertex x="0" y="72"/>
+<vertex x="94.5" y="72"/>
+<vertex x="94.5" y="43"/>
+<vertex x="79.5" y="43"/>
+<vertex x="79.5" y="57"/>
+<vertex x="66.5" y="57"/>
+<vertex x="66.5" y="45.5"/>
+<vertex x="70" y="45.5"/>
+<vertex x="70" y="41"/>
+<vertex x="55.5" y="41"/>
+<vertex x="55.5" y="52.5"/>
+<vertex x="28.5" y="52.5"/>
+<vertex x="28.5" y="48"/>
+<vertex x="53.5" y="48"/>
+<vertex x="53.5" y="44"/>
+<vertex x="-0.5" y="44"/>
+<vertex x="-0.5" y="72"/>
+</polygon>
+<polygon width="0.4064" layer="1">
+<vertex x="-0.5" y="0.5"/>
+<vertex x="-0.5" y="48.5"/>
+<vertex x="69" y="48.5"/>
+<vertex x="69" y="39.5"/>
+<vertex x="74.5" y="39.5"/>
+<vertex x="74.5" y="45"/>
+<vertex x="88" y="45"/>
+<vertex x="88" y="17.5"/>
+<vertex x="88" y="14.5"/>
+<vertex x="67.5" y="14.5"/>
+<vertex x="67.5" y="22"/>
+<vertex x="74" y="22"/>
+<vertex x="74" y="27.5"/>
+<vertex x="66" y="27.5"/>
+<vertex x="66" y="12"/>
+<vertex x="56.5" y="12"/>
+<vertex x="56.5" y="18.5"/>
+<vertex x="54.5" y="18.5"/>
+<vertex x="54.5" y="24.5"/>
+<vertex x="51" y="24.5"/>
+<vertex x="51" y="12"/>
+<vertex x="39" y="12"/>
+<vertex x="39" y="19.5"/>
+<vertex x="33.5" y="19.5"/>
+<vertex x="33.5" y="6.5"/>
+<vertex x="39" y="6.5"/>
+<vertex x="39" y="0.5"/>
+</polygon>
+<polygon width="0.4064" layer="1">
+<vertex x="94.5" y="0"/>
+<vertex x="94.5" y="17"/>
+<vertex x="82" y="17"/>
+<vertex x="82" y="0"/>
+</polygon>
+<via x="50.75" y="38.5" extent="1-16" drill="0.6" shape="square"/>
+<wire x1="41.2" y1="10.8" x2="41.2" y2="9.08" width="0" layer="19" extent="16-16"/>
 </signal>
 <signal name="VCC">
@@
 <wire x1="75.5" y1="43.085490625" x2="75.46966875" y2="43.115821875" width="0.254" layer="1"/>
 <wire x1="75.46966875" y1="43.115821875" x2="74.66966875" y2="43.115821875" width="0.254" layer="1"/>
-<wire x1="53" y1="39.5" x2="51" y2="37.5" width="0.254" layer="1"/>
-<via x="51" y="37.5" extent="1-16" drill="0.6" shape="square"/>
-<wire x1="51" y1="37.5" x2="48" y2="37.5" width="0.254" layer="16"/>
+<wire x1="53" y1="38.5" x2="52" y2="37.5" width="0.254" layer="1"/>
+<via x="52" y="37.5" extent="1-16" drill="0.6" shape="square"/>
+<wire x1="52" y1="37.5" x2="48" y2="37.5" width="0.254" layer="16"/>
 <via x="48" y="37.5" extent="1-16" drill="0.6" shape="square"/>
 <wire x1="48" y1="37.5" x2="45" y2="37.5" width="0.254" layer="1"/>
 <wire x1="53.25" y1="41.5" x2="53.5" y2="41.75" width="0.254" layer="1"/>
-<wire x1="53" y1="39.5" x2="53" y2="41.25" width="0.254" layer="1"/>
+<wire x1="53" y1="38.5" x2="53" y2="41.25" width="0.254" layer="1"/>
 <wire x1="53" y1="41.25" x2="53.5" y2="41.75" width="0.254" layer="1"/>
 <wire x1="45" y1="37.5" x2="45" y2="39" width="0.254" layer="1"/>

Commit message: maybe final
Routing:
- net GND: track 1024.6 -> 1037.5 mm, vias 83 -> 88
- net TDO_PROM: track 38.2 -> 41.0 mm
- net TCK: track 72.1 -> 74.1 mm
Other:
- board text added: "2012-04-02"
- board text added: "MOSI SCLK MISO SEL TMS TDO TDO2 GND VCC RST"
- board text added: "P83 P84 P85 P86 P87 TCK TDI GND VCC HWB"
- board text added: "VCC GND P137 P135 P132 P130 P129 P128 P127 P123"
- board text removed: "123"
- board text removed: "127"
- board text removed: "128"
- board text removed: "129"
- board text removed: "130"
- board text removed: "132"
- board text removed: "135"
- board text removed: "137"

Commit message: maybe final
Parts:
- moved R1 6.00 mm to (39.8, 46.2)
Routing:
- net N$42: track 10.6 -> 5.45 mm
- net TDI_FPGA: track 67.1 -> 62.0 mm
- net N$4: track 13.9 -> 13.0 mm
- net N$3: track 16.8 -> 16.2 mm
- net SD_CS: track 29.5 -> 29.0 mm
- net GND: vias 88 -> 89
Changed lines of the file:
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@@
 <element name="U1" library="xilinx_spartan3_virtex4_and_5" package="TQ144" value="XC3S400TQ144" x="53.22" y="33.75"/>
 <element name="IC1" library="smd-special" package="VO20" value="XCF02S" x="83.093396875" y="15.237409375" rot="R90"/>
-<element name="R1" library="rcl" package="R0805" value="100" x="33.7594" y="46.2486" rot="R180"/>
+<element name="R1" library="rcl" package="R0805" value="100" x="39.7594" y="46.2486" rot="R180"/>
 <element name="R2" library="rcl" package="R0805" value="100" x="62.75" y="49" rot="R90"/>
 <element name="R3" library="rcl" package="R0805" value="100" x="60.5" y="49.75" rot="R90"/>
@@
 <via x="40" y="22.75" extent="1-16" drill="0.6" shape="square"/>
 <via x="3.75" y="23.75" extent="1-16" drill="0.6" shape="square"/>
+<via x="32" y="47.5" extent="1-16" drill="0.6" shape="square"/>
 </signal>
 <signal name="VCC">
@@
 <contactref element="R1" pad="2"/>
 <contactref element="IC3" pad="21"/>
-<wire x1="44.5" y1="45" x2="62" y2="45" width="0.254" layer="16"/>
+<wire x1="44" y1="45" x2="62" y2="45" width="0.254" layer="16"/>
 <wire x1="62" y1="45" x2="63" y2="44" width="0.254" layer="16"/>
 <wire x1="88" y1="37.5" x2="88" y2="35" width="0.254" layer="1"/>
 <wire x1="88" y1="35" x2="89.25" y2="33.75" width="0.254" layer="1"/>
-<wire x1="37.5" y1="45.5" x2="44" y2="45.5" width="0.254" layer="16"/>
-<wire x1="44" y1="45.5" x2="44.5" y2="45" width="0.254" layer="16"/>
-<wire x1="32.8094" y1="46.2486" x2="31.5014" y2="46.2486" width="0.254" layer="1"/>
-<wire x1="31.5014" y1="46.2486" x2="31.5" y2="46.25" width="0.254" layer="1"/>
-<via x="31.5" y="46.25" extent="1-16" drill="0.6" shape="square"/>
-<wire x1="31.5" y1="46.25" x2="36.75" y2="46.25" width="0.254" layer="16"/>
-<wire x1="36.75" y1="46.25" x2="37.5" y2="45.5" width="0.254" layer="16"/>
+<wire x1="38.25" y1="45.5" x2="43.5" y2="45.5" width="0.254" layer="16"/>
+<wire x1="43.5" y1="45.5" x2="44" y2="45" width="0.254" layer="16"/>
+<wire x1="38.8094" y1="46.2486" x2="39.0014" y2="46.2486" width="0.254" layer="1"/>
+<via x="37.25" y="46.5" extent="1-16" drill="0.6" shape="square"/>
+<wire x1="37.25" y1="46.5" x2="38.25" y2="45.5" width="0.254" layer="16"/>
 <contactref element="SV1" pad="7"/>
 <wire x1="89.25" y1="33.75" x2="89.25" y2="33.79" width="0.254" layer="1"/>
@@
 <wire x1="79" y1="39.25" x2="81.735490625" y2="39.25" width="0.254" layer="1"/>
 <wire x1="81.735490625" y1="39.25" x2="81.76226875" y2="39.223221875" width="0.254" layer="1"/>
+<wire x1="37.25" y1="46.5" x2="37.5" y2="46.25" width="0.254" layer="1"/>
+<wire x1="37.5" y1="46.25" x2="38.808" y2="46.25" width="0.254" layer="1"/>
+<wire x1="38.808" y1="46.25" x2="38.8094" y2="46.2486" width="0.254" layer="1"/>
 </signal>
 <signal name="PROM_INITB">
@@
 <contactref element="R1" pad="1"/>
 <contactref element="U1" pad="P144"/>
-<wire x1="44.47" y1="44.45" x2="44.47" y2="44.53" width="0.254" layer="1"/>
-<wire x1="44.47" y1="44.53" x2="43.5" y2="45.5" width="0.254" layer="1"/>
-<wire x1="34.708" y1="46.25" x2="34.7094" y2="46.2486" width="0.254" layer="1"/>
-<wire x1="34.708" y1="46.25" x2="36.75" y2="46.25" width="0.254" layer="1"/>
-<wire x1="36.75" y1="46.25" x2="37.5" y2="45.5" width="0.254" layer="1"/>
-<wire x1="37.5" y1="45.5" x2="43.5" y2="45.5" width="0.254" layer="1"/>
+<wire x1="44.47" y1="44.45" x2="44.47" y2="44.03" width="0.254" layer="1"/>
+<wire x1="42.25" y1="46.25" x2="44.47" y2="44.03" width="0.254" layer="1"/>
+<wire x1="42.25" y1="46.25" x2="40.75" y2="46.25" width="0.254" layer="1"/>
+<wire x1="40.75" y1="46.25" x2="40.7094" y2="46.2094" width="0.254" layer="1"/>
+<wire x1="40.7094" y1="46.2486" x2="40.7094" y2="46.2094" width="0.254" layer="1"/>
+<wire x1="40.7094" y1="46.2094" x2="40.5" y2="46" width="0.254" layer="1"/>
 </signal>
 <signal name="N$43">
@@
 <wire x1="27.5" y1="50" x2="20.25" y2="50" width="0.254" layer="16"/>
 <wire x1="20.25" y1="50" x2="18" y2="52.25" width="0.254" layer="16"/>
-<wire x1="50.5" y1="47" x2="43" y2="47" width="0.254" layer="1"/>
-<wire x1="43" y1="47" x2="41.5" y2="48.5" width="0.254" layer="1"/>
-<wire x1="41.5" y1="48.5" x2="29" y2="48.5" width="0.254" layer="1"/>
+<wire x1="50.5" y1="47" x2="44.5" y2="47" width="0.254" layer="1"/>
+<wire x1="44.5" y1="47" x2="43" y2="48.5" width="0.254" layer="1"/>
+<wire x1="43" y1="48.5" x2="29" y2="48.5" width="0.254" layer="1"/>
 </signal>
 <signal name="PS2CLK">
@@
 <wire x1="45.97" y1="44.45" x2="45.97" y2="45.53" width="0.254" layer="1"/>
 <wire x1="45.97" y1="45.53" x2="45.5" y2="46" width="0.254" layer="1"/>
-<wire x1="45.5" y1="46" x2="42" y2="46" width="0.254" layer="1"/>
-<wire x1="42" y1="46" x2="40.5" y2="47.5" width="0.254" layer="1"/>
-<wire x1="40.5" y1="47.5" x2="27" y2="47.5" width="0.254" layer="1"/>
-<wire x1="27" y1="47.5" x2="26.5" y2="47" width="0.254" layer="1"/>
-<via x="26.5" y="47" extent="1-16" drill="0.6" shape="square"/>
-<wire x1="26.5" y1="47" x2="26.5" y2="42.5" width="0.254" layer="16"/>
+<wire x1="45.5" y1="46" x2="43.5" y2="46" width="0.254" layer="1"/>
+<wire x1="43.5" y1="46" x2="42" y2="47.5" width="0.254" layer="1"/>
+<via x="26.5" y="46" extent="1-16" drill="0.6" shape="square"/>
 <wire x1="26.5" y1="42.5" x2="27" y2="42" width="0.254" layer="16"/>
 <wire x1="27" y1="42" x2="29.69" y2="42" width="0.254" layer="16"/>
 <wire x1="29.69" y1="42" x2="29.74" y2="41.95" width="0.254" layer="16"/>
+<wire x1="26.5" y1="42.5" x2="26.5" y2="46" width="0.254" layer="16"/>
+<wire x1="42" y1="47.5" x2="34.5" y2="47.5" width="0.254" layer="1"/>
+<wire x1="34.5" y1="47.5" x2="33" y2="46" width="0.254" layer="1"/>
+<wire x1="33" y1="46" x2="26.5" y2="46" width="0.254" layer="1"/>
 </signal>
 <signal name="SD_CLK">
@@
 <wire x1="46.47" y1="44.45" x2="46.47" y2="46.03" width="0.254" layer="1"/>
 <wire x1="46.47" y1="46.03" x2="46" y2="46.5" width="0.254" layer="1"/>
-<wire x1="46" y1="46.5" x2="42.5" y2="46.5" width="0.254" layer="1"/>
-<wire x1="42.5" y1="46.5" x2="41" y2="48" width="0.254" layer="1"/>
-<wire x1="41" y1="48" x2="25.5" y2="48" width="0.254" layer="1"/>
-<wire x1="25.5" y1="48" x2="25" y2="47.5" width="0.254" layer="1"/>
-<via x="25" y="47.5" extent="1-16" drill="0.6" shape="square"/>
-<wire x1="25" y1="47.5" x2="25" y2="40" width="0.254" layer="16"/>
+<wire x1="46" y1="46.5" x2="44" y2="46.5" width="0.254" layer="1"/>
+<wire x1="44" y1="46.5" x2="42.5" y2="48" width="0.254" layer="1"/>
+<via x="25" y="47" extent="1-16" drill="0.6" shape="square"/>
 <wire x1="25" y1="40" x2="25.5" y2="39.5" width="0.254" layer="16"/>
 <wire x1="25.5" y1="39.5" x2="29.69" y2="39.5" width="0.254" layer="16"/>
 <wire x1="29.69" y1="39.5" x2="29.74" y2="39.45" width="0.254" layer="16"/>
+<wire x1="25" y1="40" x2="25" y2="47" width="0.254" layer="16"/>
+<wire x1="42.5" y1="48" x2="34" y2="48" width="0.254" layer="1"/>
+<wire x1="34" y1="48" x2="32.5" y2="46.5" width="0.254" layer="1"/>
+<wire x1="32.5" y1="46.5" x2="27.5" y2="46.5" width="0.254" layer="1"/>
+<wire x1="27.5" y1="46.5" x2="27" y2="47" width="0.254" layer="1"/>
+<wire x1="27" y1="47" x2="25" y2="47" width="0.254" layer="1"/>
 </signal>
 <signal name="SD_DO">
@@
 <via x="47.5" y="46" extent="1-16" drill="0.6" shape="square"/>
 <contactref element="SV3" pad="3"/>
-<wire x1="47.5" y1="46" x2="38.25" y2="46" width="0.254" layer="16"/>
-<wire x1="38.25" y1="46" x2="35.75" y2="48.5" width="0.254" layer="16"/>
-<wire x1="35.75" y1="48.5" x2="35.75" y2="50.25" width="0.254" layer="16"/>
+<wire x1="47.5" y1="46" x2="47" y2="46.5" width="0.254" layer="16"/>
+<wire x1="47" y1="46.5" x2="38.75" y2="46.5" width="0.254" layer="16"/>
+<wire x1="38.75" y1="46.5" x2="35.75" y2="49.5" width="0.254" layer="16"/>
+<wire x1="35.75" y1="49.5" x2="35.75" y2="50.25" width="0.254" layer="16"/>
 <wire x1="35.75" y1="50.25" x2="35.5" y2="50.5" width="0.254" layer="16"/>
 <wire x1="35.65" y1="50.5" x2="35.5" y2="50.5" width="0.254" layer="16"/>
@@
 <wire x1="51.47" y1="44.45" x2="51.47" y2="47.03" width="0.254" layer="1"/>
 <wire x1="51.47" y1="47.03" x2="51" y2="47.5" width="0.254" layer="1"/>
-<wire x1="51" y1="47.5" x2="43.5" y2="47.5" width="0.254" layer="1"/>
-<wire x1="43.5" y1="47.5" x2="43.25" y2="47.75" width="0.254" layer="1"/>
-<wire x1="43.25" y1="47.75" x2="43.25" y2="50.48" width="0.254" layer="1"/>
 <wire x1="43.25" y1="50.48" x2="43.27" y2="50.5" width="0.254" layer="1"/>
+<wire x1="51" y1="47.5" x2="45" y2="47.5" width="0.254" layer="1"/>
+<wire x1="45" y1="47.5" x2="43.25" y2="49.25" width="0.254" layer="1"/>
+<wire x1="43.25" y1="50.48" x2="43.25" y2="49.25" width="0.254" layer="1"/>
 </signal>
 <signal name="N$5">
