File: eagle/homeboard/homeboard29.brd (EAGLE design)
At the start: 94 x 71.8 mm, 126 parts, among them IC1 XCF02S, IC2 25LC080SN, IC3 ATMEGA32U2-TQFP, Q5 BC848SMD, Q6 BC848SMD, Q7 BC848SMD, Q8 BC848SMD, T1 BSS138, T2 BC848, T3 BSS138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

Commit message: tidied up a bit, ready to send to laenpcb.org
Parts:
- renumbered U$4 to REG3.3
Other:
- board text added: "2012-04-03 #29"
- board text added: "CAS IN"
- board text added: "Joystick 0"
- board text added: "Joystick 1"
- board text added: "PS/2 keyboard"
- board text added: "SCART"
- board text added: "SDCARD"
- board text added: "USB"
Changed lines of the file:
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@@
 <layer number="17" name="Pads" color="2" fill="1" visible="yes" active="yes"/>
 <layer number="18" name="Vias" color="2" fill="1" visible="yes" active="yes"/>
-<layer number="19" name="Unrouted" color="6" fill="1" visible="yes" active="yes"/>
+<layer number="19" name="Unrouted" color="14" fill="1" visible="yes" active="yes"/>
 <layer number="20" name="Dimension" color="15" fill="1" visible="yes" active="yes"/>
 <layer number="21" name="tPlace" color="7" fill="1" visible="yes" active="yes"/>
@@
 <layer number="24" name="bOrigins" color="15" fill="1" visible="yes" active="yes"/>
 <layer number="25" name="tNames" color="7" fill="1" visible="yes" active="yes"/>
-<layer number="26" name="bNames" color="7" fill="1" visible="no" active="yes"/>
+<layer number="26" name="bNames" color="7" fill="1" visible="yes" active="yes"/>
 <layer number="27" name="tValues" color="7" fill="1" visible="no" active="yes"/>
 <layer number="28" name="bValues" color="7" fill="1" visible="no" active="yes"/>
@@
 <layer number="31" name="tCream" color="7" fill="4" visible="no" active="yes"/>
 <layer number="32" name="bCream" color="7" fill="5" visible="no" active="yes"/>
-<layer number="33" name="tFinish" color="6" fill="3" visible="no" active="yes"/>
-<layer number="34" name="bFinish" color="6" fill="6" visible="no" active="yes"/>
+<layer number="33" name="tFinish" color="6" fill="3" visible="yes" active="yes"/>
+<layer number="34" name="bFinish" color="6" fill="6" visible="yes" active="yes"/>
 <layer number="35" name="tGlue" color="7" fill="4" visible="no" active="yes"/>
 <layer number="36" name="bGlue" color="7" fill="5" visible="no" active="yes"/>
@@
 <layer number="39" name="tKeepout" color="4" fill="11" visible="yes" active="yes"/>
 <layer number="40" name="bKeepout" color="1" fill="11" visible="yes" active="yes"/>
-<layer number="41" name="tRestrict" color="4" fill="10" visible="no" active="yes"/>
-<layer number="42" name="bRestrict" color="1" fill="10" visible="no" active="yes"/>
+<layer number="41" name="tRestrict" color="4" fill="10" visible="yes" active="yes"/>
+<layer number="42" name="bRestrict" color="1" fill="10" visible="yes" active="yes"/>
 <layer number="43" name="vRestrict" color="2" fill="10" visible="no" active="yes"/>
-<layer number="44" name="Drills" color="7" fill="1" visible="no" active="yes"/>
-<layer number="45" name="Holes" color="7" fill="1" visible="no" active="yes"/>
+<layer number="44" name="Drills" color="7" fill="1" visible="yes" active="yes"/>
+<layer number="45" name="Holes" color="7" fill="1" visible="yes" active="yes"/>
 <layer number="46" name="Milling" color="3" fill="1" visible="no" active="yes"/>
 <layer number="47" name="Measures" color="7" fill="1" visible="no" active="yes"/>
@@
 <layer number="112" name="tSilk" color="7" fill="1" visible="yes" active="yes"/>
 <layer number="116" name="Patch_BOT" color="9" fill="4" visible="no" active="yes"/>
-<layer number="121" name="_tsilk" color="7" fill="1" visible="no" active="yes"/>
-<layer number="122" name="_bsilk" color="7" fill="1" visible="no" active="yes"/>
+<layer number="121" name="_tsilk" color="7" fill="1" visible="yes" active="yes"/>
+<layer number="122" name="_bsilk" color="15" fill="1" visible="yes" active="yes"/>
 <layer number="123" name="tTestmark" color="7" fill="1" visible="no" active="yes"/>
 <layer number="124" name="bTestmark" color="7" fill="1" visible="no" active="yes"/>
@@
 <text x="87.5" y="42.25" size="0.7" layer="112" rot="R180">HWB</text>
 <text x="52.25" y="54" size="1.2" layer="112" rot="R180">CPC2012 prototype</text>
+<text x="65.25" y="54.75" size="1.3" layer="122" ratio="13" rot="MR0">CPC2012 prototype rev 1</text>
+<text x="65.25" y="52.75" size="1.27" layer="122" ratio="13" rot="MR0">(c) 2012 Ranulf Doswell</text>
+<text x="87" y="17.5" size="0.7" layer="122" rot="MR90">P83 P84 P85 P86 P87 TCK TDI GND VCC</text>
+<text x="93.25" y="15.75" size="0.56" layer="122" rot="MR90">MOSI     SCLK MISO SEL  TMS  TDO  TDO2 GND  VCC  RST</text>
+<text x="28.75" y="48.75" size="0.56" layer="122" rot="SMR180">VCC    GND P137 P135 P132 P130 P129 P128 P127 P123</text>
+<text x="64.5" y="44" size="1.27" layer="122" ratio="10" rot="SMR0">laborare est aemulari</text>
+<text x="39" y="14.75" size="0.8128" layer="122" rot="MR90">P47</text>
+<text x="32.75" y="12.25" size="0.8128" layer="122" rot="MR90">P50</text>
+<text x="39" y="12.25" size="0.8128" layer="122" rot="MR90">P51</text>
+<text x="32.75" y="14.75" size="0.8128" layer="122" rot="MR90">GND</text>
+<text x="33.5" y="9" size="0.8128" layer="122" rot="MR270">5V</text>
+<text x="39" y="7.5" size="0.8128" layer="122" rot="MR90">5V</text>
+<text x="39" y="9.75" size="0.8128" layer="122" rot="MR90">VCC</text>
+<text x="32.5" y="17.5" size="0.8128" layer="122" rot="MR90">VCCINT</text>
+<text x="39" y="17.75" size="0.8128" layer="122" rot="MR90">VCCAUX</text>
+<text x="33.5" y="12.25" size="0.8128" layer="122" rot="MR270">VCC</text>
+<text x="73.5" y="21" size="0.8128" layer="122" rot="MR0">GND</text>
+<text x="71" y="21" size="0.8128" layer="122" rot="MR0">VCC</text>
+<text x="68.5" y="21" size="0.8128" layer="122" rot="MR0">VCC</text>
+<text x="66.5" y="28" size="0.8128" layer="112">P76</text>
+<text x="68.5" y="29.25" size="0.8128" layer="122" rot="MR0">P76</text>
+<text x="69" y="28" size="0.8128" layer="112">P77</text>
+<text x="68.749721875" y="29.999884375" size="0.8128" layer="122" rot="MR180">P77</text>
+<text x="73.64644375" y="28.14644375" size="0.8128" layer="122" rot="MR0">P74</text>
+<text x="77" y="45.5" size="0.8128" layer="122" rot="MR0">-FPGA-XTAL-</text>
+<text x="36.75" y="53.25" size="1.27" layer="122" rot="MR0">2012-04-03  #29</text>
+<text x="36.5" y="64.5" size="1.778" layer="122" rot="SMR0">Joystick 0</text>
+<text x="68.5" y="64.5" size="1.778" layer="122" rot="SMR0">Joystick 1</text>
+<text x="11.25" y="65" size="1.778" layer="122" rot="SMR0">CAS IN</text>
+<text x="87" y="62.5" size="1.778" layer="122" rot="SMR0">USB</text>
+<text x="6.5" y="1" size="1.778" layer="122" rot="SMR0">5V</text>
+<text x="25.5" y="1" size="1.27" layer="122" rot="SMR0">PS/2 keyboard</text>
+<text x="76.5" y="0.5" size="1.27" layer="122" rot="SMR0">SCART</text>
+<text x="1.5" y="37.5" size="1.27" layer="122" rot="MR270">SDCARD</text>
+<text x="86.999915625" y="40.499825" size="0.7" layer="122" rot="MR90">HWB</text>
+<text x="28.49998125" y="7.250065625" size="0.8128" layer="122" rot="MR180">5V</text>
+<text x="29.99996875" y="12.000065625" size="0.8128" layer="122" rot="MR0">GND</text>
+<text x="90.75" y="67.75" size="2.2" layer="122" font="vector" ratio="12" rot="MR0">CPCFPGA.COM rev 1 (c) 2012 Ranulf Doswell</text>
 </plain>
 <attributes>
@@
 <element name="R50" library="resistor" package="M0805" value="2k2" x="40.75" y="18.25" rot="MR90"/>
 <element name="IC3" library="adafruit" package="TQFP32-08" value="ATMEGA32U2-TQFP" x="77.46966875" y="38.823221875"/>
-<element name="U$4" library="cpcfpga" package="SOT223" value="3.3V" x="9.5" y="27.75" rot="R270"/>
+<element name="REG3.3" library="cpcfpga" package="SOT223" value="3.3V" x="9.5" y="27.75" rot="R270"/>
 <element name="C6" library="rcl" package="C0603" value="100nF" x="53.75" y="39.5" rot="MR270"/>
 <element name="C7" library="rcl" package="C0603" value="100nF" x="60.5" y="40.5" rot="MR270"/>
@@
 <contactref element="C5" pad="1"/>
 <contactref element="REG2.5" pad="1"/>
-<contactref element="U$4" pad="1"/>
+<contactref element="REG3.3" pad="1"/>
 <wire x1="2" y1="30" x2="2" y2="36" width="0.8" layer="16"/>
 <wire x1="2" y1="36" x2="2" y2="36.25" width="0.6096" layer="16"/>
@@
 <contactref element="C27" pad="1"/>
 <contactref element="C29" pad="1"/>
-<contactref element="U$4" pad="4"/>
+<contactref element="REG3.3" pad="4"/>
 <contactref element="C6" pad="1"/>
 <contactref element="C7" pad="1"/>
@@
 <contactref element="REG1.2" pad="3"/>
 <contactref element="REG2.5" pad="3"/>
-<contactref element="U$4" pad="3"/>
+<contactref element="REG3.3" pad="3"/>
 <contactref element="C33" pad="+"/>
 <contactref element="X7" pad="2"/>
@@
 <wire x1="41" y1="49.5" x2="41" y2="50.25" width="0.254" layer="16"/>
 <wire x1="41" y1="50.25" x2="40.75" y2="50.5" width="0.254" layer="16"/>
-<wire x1="40.75" y1="50.5" x2="40.73" y2="50.5" width="0" layer="19" extent="16-16"/>
+<wire x1="40.73" y1="50.5" x2="40.75" y2="50.5" width="0.254" layer="16"/>
 </signal>
 <signal name="N$4">
@@
 <wire x1="46" y1="50" x2="46" y2="50.25" width="0.254" layer="1"/>
 <wire x1="46" y1="50.25" x2="45.75" y2="50.5" width="0.254" layer="1"/>
-<wire x1="45.75" y1="50.5" x2="45.81" y2="50.5" width="0" layer="19" extent="1-1"/>
+<wire x1="45.75" y1="50.5" x2="45.81" y2="50.5" width="0.254" layer="1"/>
 </signal>
 <signal name="N$6">
@@
 <wire x1="51.5" y1="48.5" x2="51" y2="49" width="0.254" layer="1"/>
 <wire x1="51" y1="49" x2="51" y2="50.5" width="0.254" layer="1"/>
-<wire x1="51" y1="50.5" x2="50.89" y2="50.5" width="0" layer="19" extent="1-1"/>
+<wire x1="51" y1="50.5" x2="50.89" y2="50.5" width="0.254" layer="1"/>
 </signal>
 <signal name="N$7">
