File: eagle/homeboard/homeboard29.sch (EAGLE design)
At the start: 126 parts, among them IC1 XCF02S, IC2 25LC080SN, IC3 ATMEGA32U2-TQFP, Q5 BC848SMD, Q6 BC848SMD, Q7 BC848SMD, Q8 BC848SMD, T1 BSS138, T2 BC848, T3 BSS138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

Commit message: tidied up a bit, ready to send to laenpcb.org
Parts:
- renumbered U$4 to REG3.3
Changed lines of the file:
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@@
 <part name="R50" library="resistor" deviceset="R-EU_" device="M0805" value="2k2"/>
 <part name="IC3" library="adafruit" deviceset="ATMEGA32U2" device="-TQFP"/>
-<part name="U$4" library="cpcfpga" deviceset="NX1117" device="" value="3.3V"/>
+<part name="REG3.3" library="cpcfpga" deviceset="NX1117" device="" value="3.3V"/>
 <part name="C6" library="rcl" deviceset="C-EU" device="C0603" value="100nF"/>
 <part name="C7" library="rcl" deviceset="C-EU" device="C0603" value="100nF"/>
@@
 <instance part="R50" gate="G$1" x="124.46" y="304.8" rot="R180"/>
 <instance part="IC3" gate="G$1" x="406.4" y="106.68"/>
-<instance part="U$4" gate="G$1" x="-195.58" y="111.76"/>
+<instance part="REG3.3" gate="G$1" x="-195.58" y="111.76"/>
 <instance part="C6" gate="G$1" x="-147.32" y="109.22"/>
 <instance part="C7" gate="G$1" x="-139.7" y="109.22"/>
@@
 <wire x1="-205.74" y1="30.48" x2="-205.74" y2="22.86" width="0.1524" layer="91"/>
 <junction x="-205.74" y="30.48"/>
-<pinref part="U$4" gate="G$1" pin="GND"/>
+<pinref part="REG3.3" gate="G$1" pin="GND"/>
 <wire x1="-203.2" y1="106.68" x2="-205.74" y2="106.68" width="0.1524" layer="91"/>
 </segment>
@@
 <pinref part="C29" gate="G$1" pin="1"/>
 <wire x1="-139.7" y1="129.54" x2="-124.46" y2="129.54" width="0.1524" layer="91"/>
-<pinref part="U$4" gate="G$1" pin="VOUT1"/>
+<pinref part="REG3.3" gate="G$1" pin="VOUT1"/>
 <wire x1="-172.72" y1="114.3" x2="-170.18" y2="114.3" width="0.1524" layer="91"/>
 <wire x1="-170.18" y1="114.3" x2="-170.18" y2="111.76" width="0.1524" layer="91"/>
@@
 <label x="-198.12" y="73.66" size="1.778" layer="95"/>
 <junction x="-208.28" y="73.66"/>
-<pinref part="U$4" gate="G$1" pin="VCC"/>
+<pinref part="REG3.3" gate="G$1" pin="VCC"/>
 <wire x1="-203.2" y1="114.3" x2="-208.28" y2="114.3" width="0.1524" layer="91"/>
 <wire x1="-208.28" y1="114.3" x2="-208.28" y2="73.66" width="0.1524" layer="91"/>
