File: eagle/homeboard/submitted/homeboard29.sch (EAGLE design)
At the start: 126 parts, among them IC1 XCF02S, IC2 25LC080SN, IC3 ATMEGA32U2-TQFP, Q5 BC848SMD, Q6 BC848SMD, Q7 BC848SMD, Q8 BC848SMD, T1 BSS138, T2 BC848, T3 BSS138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

Commit message: added some more notes to homeboard
Parts:
- C1, C3, C4, C5: value (none) -> 100nF
- R23, R34: value (none) -> 75
- R48, R49: value (none) -> 2200
Changed lines of the file:
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@@
 <part name="Q7" library="bc548" deviceset="BC848*" device="SMD"/>
 <part name="Q8" library="bc548" deviceset="BC848*" device="SMD"/>
-<part name="R23" library="resistor" deviceset="R-EU_" device="M0805"/>
-<part name="R34" library="resistor" deviceset="R-EU_" device="M0805"/>
-<part name="C3" library="resistor" deviceset="C-EU" device="C0603"/>
-<part name="C4" library="resistor" deviceset="C-EU" device="C0603"/>
+<part name="R23" library="resistor" deviceset="R-EU_" device="M0805" value="75"/>
+<part name="R34" library="resistor" deviceset="R-EU_" device="M0805" value="75"/>
+<part name="C3" library="resistor" deviceset="C-EU" device="C0603" value="100nF"/>
+<part name="C4" library="resistor" deviceset="C-EU" device="C0603" value="100nF"/>
 <part name="U$2" library="cpcfpga" deviceset="TXO_7C" device=""/>
 <part name="REG2.5" library="cpcfpga" deviceset="NX1117" device="" value="2.5V"/>
@@
 <part name="SUPPLY5" library="supply2" deviceset="GND" device=""/>
 <part name="IC2" library="microchip" deviceset="25*" device="SN" technology="LC080"/>
-<part name="R48" library="resistor" deviceset="R-EU_" device="M0805"/>
-<part name="C1" library="resistor" deviceset="C-EU" device="C0603"/>
-<part name="C5" library="resistor" deviceset="C-EU" device="C0603"/>
-<part name="R49" library="resistor" deviceset="R-EU_" device="M0805"/>
+<part name="R48" library="resistor" deviceset="R-EU_" device="M0805" value="2200"/>
+<part name="C1" library="resistor" deviceset="C-EU" device="C0603" value="100nF"/>
+<part name="C5" library="resistor" deviceset="C-EU" device="C0603" value="100nF"/>
+<part name="R49" library="resistor" deviceset="R-EU_" device="M0805" value="2200"/>
 <part name="SUPPLY6" library="supply2" deviceset="GND" device=""/>
 <part name="SUPPLY7" library="supply2" deviceset="GND" device=""/>

Commit message: added more values
Parts:
- C37, C38: value (none) -> 20pF
- LED1: value (none) -> 20mA
- R11: value (none) -> 75
Changed lines of the file:
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@@
 <part name="SUPPLY19" library="supply2" deviceset="GND" device=""/>
 <part name="Q1" library="special" deviceset="XTAL/S" device=""/>
-<part name="C37" library="rcl" deviceset="C-EU" device="C0805"/>
-<part name="C38" library="rcl" deviceset="C-EU" device="C0805"/>
+<part name="C37" library="rcl" deviceset="C-EU" device="C0805" value="20pF"/>
+<part name="C38" library="rcl" deviceset="C-EU" device="C0805" value="20pF"/>
 <part name="SUPPLY20" library="supply2" deviceset="GND" device=""/>
 <part name="PWR_HDR" library="jumper" deviceset="JP1Q" device=""/>
@@
 <attribute name="OC_NEWARK" value="unknown"/>
 </part>
-<part name="R11" library="resistor" deviceset="R-EU_" device="M0805"/>
+<part name="R11" library="resistor" deviceset="R-EU_" device="M0805" value="75"/>
 <part name="SUPPLY17" library="supply2" deviceset="GND" device=""/>
-<part name="LED1" library="adafruit" deviceset="LED" device="CHIPLED_0805"/>
+<part name="LED1" library="adafruit" deviceset="LED" device="CHIPLED_0805" value="20mA"/>
 </parts>
 <sheets>
